File: KiCad PCB Files/5V_to_3V3_MP2322GQH.kicad_sch (KiCad schematic)
At the start: 14 parts, among them IC4 MP2322GQH-Z

Commit message: Restored Samacsys parts footprints
PCB components are not placed, just dropped in place
Parts:
- removed L2: MAKK2016T3R3M, INDPM2016X100N, symbol SamacSys_Parts:MAKK2016T3R3M
- added L3: MAKK2016T3R3M, SamacSys_Parts:INDPM2016X100N, symbol SamacSys_Parts:MAKK2016T3R3M
- IC4: footprint MP2322GQHZ -> SamacSys_Parts:MP2322GQHZ
Connections:
- net at C22.2, C23.1, C24.1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: now also L3.2
- net at C21.2, IC4.8 (SW): now also L3.1
Changed lines of the file:
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@@
+    )
+  )
+  (symbol (lib_id "SamacSys_Parts:MAKK2016T3R3M") (at 162.56 64.77 0) (unit 1)
+    (in_bom yes) (on_board yes) (dnp no) (fields_autoplaced)
+    (property "Reference" "L3" (at 172.72 59.69 0)
+      (effects (font (size 1.27 1.27)))
+    )
+    (property "Value" "MAKK2016T3R3M" (at 172.72 62.23 0)
+      (effects (font (size 1.27 1.27)))
+    )
+    (property "Footprint" "SamacSys_Parts:INDPM2016X100N" (at 179.07 63.5 0)
+      (effects (font (size 1.27 1.27)) (justify left) hide)
+    )
+    (property "Datasheet" "https://mouser.componentsearchengine.com/Datasheets/1/MAKK2016T3R3M.pdf" (at 179.07 66.04 0)
+      (effects (font (size 1.27 1.27)) (justify left) hide)
+    )
+    (property "Description" "Fixed Inductors 0806 3.3uH 255mOhms +/-20% 1150A HiCur" (at 179.07 68.58 0)
+      (effects (font (size 1.27 1.27)) (justify left) hide)
+    )
+    (property "Height" "1" (at 179.07 71.12 0)
+      (effects (font (size 1.27 1.27)) (justify left) hide)
+    )
+    (property "Manufacturer_Name" "TAIYO YUDEN" (at 179.07 73.66 0)
+      (effects (font (size 1.27 1.27)) (justify left) hide)
+    )
+    (property "Manufacturer_Part_Number" "MAKK2016T3R3M" (at 179.07 76.2 0)
+      (effects (font (size 1.27 1.27)) (justify left) hide)
+    )
+    (property "Mouser Part Number" "963-MAKK2016T3R3M" (at 179.07 78.74 0)
+      (effects (font (size 1.27 1.27)) (justify left) hide)
+    )
+    (property "Mouser Price/Stock" "https://www.mouser.co.uk/ProductDetail/TAIYO-YUDEN/MAKK2016T3R3M?qs=Z6svWd%2FY2UTQY1%2FASu%252BfUw%3D%3D" (at 179.07 81.28 0)
+      (effects (font (size 1.27 1.27)) (justify left) hide)
+    )
+    (property "Arrow Part Number" "" (at 179.07 83.82 0)
+      (effects (font (size 1.27 1.27)) (justify left) hide)
+    )
+    (property "Arrow Price/Stock" "" (at 179.07 86.36 0)
+      (effects (font (size 1.27 1.27)) (justify left) hide)
+    )
+    (pin "1")
+    (pin "2")
+    (instances
+      (project "VXDash"
+        (path "/f2858fc4-50de-4ff0-a01c-5b985ee14aef/21f2fd69-aa93-4550-8877-dde4aa3e5582"
+          (reference "L3") (unit 1)
+        )
+      )
     )
   )
@@
       (effects (font (size 1.27 1.27)))
     )
-    (property "Footprint" "MP2322GQHZ" (at 135.89 52.07 0)
+    (property "Footprint" "SamacSys_Parts:MP2322GQHZ" (at 135.89 52.07 0)
       (effects (font (size 1.27 1.27)) (justify left) hide)
     )
@@
         )
       )
-    )
-  )
-  (symbol (lib_id "SamacSys_Parts:MAKK2016T3R3M") (at 162.56 64.77 0) (unit 1)
-    (in_bom yes) (on_board yes) (dnp no) (fields_autoplaced)
-    (property "Reference" "L2" (at 172.72 59.69 0)
-      (effects (font (size 1.27 1.27)))
-    )
-    (property "Value" "MAKK2016T3R3M" (at 172.72 62.23 0)
-      (effects (font (size 1.27 1.27)))
-    )
-    (property "Footprint" "INDPM2016X100N" (at 179.07 63.5 0)
-      (effects (font (size 1.27 1.27)) (justify left) hide)
-    )
-    (property "Datasheet" "https://mouser.componentsearchengine.com/Datasheets/1/MAKK2016T3R3M.pdf" (at 179.07 66.04 0)
-      (effects (font (size 1.27 1.27)) (justify left) hide)
-    )
-    (property "Description" "Fixed Inductors 0806 3.3uH 255mOhms +/-20% 1150A HiCur" (at 179.07 68.58 0)
-      (effects (font (size 1.27 1.27)) (justify left) hide)
-    )
-    (property "Height" "1" (at 179.07 71.12 0)
-      (effects (font (size 1.27 1.27)) (justify left) hide)
-    )
-    (property "Manufacturer_Name" "TAIYO YUDEN" (at 179.07 73.66 0)
-      (effects (font (size 1.27 1.27)) (justify left) hide)
-    )
-    (property "Manufacturer_Part_Number" "MAKK2016T3R3M" (at 179.07 76.2 0)
-      (effects (font (size 1.27 1.27)) (justify left) hide)
-    )
-    (property "Mouser Part Number" "963-MAKK2016T3R3M" (at 179.07 78.74 0)
-      (effects (font (size 1.27 1.27)) (justify left) hide)
-    )
-    (property "Mouser Price/Stock" "https://www.mouser.co.uk/ProductDetail/TAIYO-YUDEN/MAKK2016T3R3M?qs=Z6svWd%2FY2UTQY1%2FASu%252BfUw%3D%3D" (at 179.07 81.28 0)
-      (effects (font (size 1.27 1.27)) (justify left) hide)
-    )
-    (property "Arrow Part Number" "" (at 179.07 83.82 0)
-      (effects (font (size 1.27 1.27)) (justify left) hide)
-    )
-    (property "Arrow Price/Stock" "" (at 179.07 86.36 0)
-      (effects (font (size 1.27 1.27)) (justify left) hide)
-    )
-    (pin "1")
-    (pin "2")
-    (instances
-      (project "VXDash"
-        (path "/f2858fc4-50de-4ff0-a01c-5b985ee14aef/21f2fd69-aa93-4550-8877-dde4aa3e5582"
-          (reference "L2") (unit 1)
-        )
-      )

Commit message: WIP commit
Parts:
- renumbered L3 to L2
Other:
- note added: "Acting as a fuse of sorts ?"
Changed lines of the file:
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@@
     (stroke (width 0) (type default))
+  )
+  (text "Acting as a fuse of sorts ?" (at 227.33 55.88 0)
+    (effects (font (size 1.27 1.27)) (justify left bottom))
   )
   (hierarchical_label "3V3_OUT" (shape output) (at 240.03 64.77 0) (fields_autoplaced)
@@
   (symbol (lib_id "SamacSys_Parts:MAKK2016T3R3M") (at 162.56 64.77 0) (unit 1)
     (in_bom yes) (on_board yes) (dnp no) (fields_autoplaced)
-    (property "Reference" "L3" (at 172.72 59.69 0)
+    (property "Reference" "L2" (at 172.72 59.69 0)
       (effects (font (size 1.27 1.27)))
     )
@@
       (project "VXDash"
         (path "/f2858fc4-50de-4ff0-a01c-5b985ee14aef/21f2fd69-aa93-4550-8877-dde4aa3e5582"
-          (reference "L3") (unit 1)
-        )
-      )
+          (reference "L2") (unit 1)
+        )
+      )

Commit message: v1.0
- First PCB layout publication
- Titled schematics
- Added Revisions to Schematics and PCB
- iBOM release
- PDF export of PCB design
Other:
- title: (none) -> 5 to 3V3 stage
Changed lines of the file:
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@@
 (kicad_sch (version 20230121) (generator eeschema)
   (paper "A4")
+  (title_block
+    (title "5 to 3V3 stage")
+    (date "2023-04-10")
+    (rev "1.0")
+    (comment 1 "https://github.com/martinroger/VXDash")
+    (comment 2 "https://cadlab.io/projects/vxdash")
+  )
   (junction (at 38.1 57.15) (diameter 0) (color 0 0 0 0)
   )
