File: KiCad PCB Files/VXDash.kicad_sch (KiCad schematic)
At the start: 15 parts, among them IC1 CD74HC4050M96, IC2 SP721ABG, IC5 74HC4067BQ-Q100J, J1 Conn_01x04_Socket, J2 MX34036UF2, K1 G6L-1P-DC12, K2 G6L-1P-DC12

Commit message: Restored Samacsys parts footprints
PCB components are not placed, just dropped in place
Parts:
- removed IC2: SP721ABG, SOIC127P600X175-8N, symbol SamacSys_Parts:SP721ABG
- added IC5: SP721ABG, SamacSys_Parts:SOIC127P600X175-8N, symbol SamacSys_Parts:SP721ABG
- F1: footprint (none) -> Fuse:Fuse_1210_3225Metric
- IC1: footprint SOIC127P600X175-16N -> SamacSys_Parts:SOIC127P600X175-16N
- J2: footprint MX34036UF2 -> SamacSys_Parts:MX34036UF2
Connections:
- net AnalogV_Divider1/ESD_protection: now also IC5.1 (IN_1)
- net AnalogV_Divider2/ESD_protection: now also IC5.2 (IN_2)
- net AnalogV_Divider3/ESD_protection: now also IC5.3 (IN_3)
- net AnalogV_Divider4/ESD_protection: now also IC5.5 (IN_4)
- net CONV_5V+: now also IC5.8 (V+)
- net GND: now also IC5.4 (V-)

Commit message: WIP commit
Parts:
- renumbered IC5 to IC2, J2 to J1, J1 to J2
Connections:
- net 5V_SENSOR: now also J1.36; no longer J1.MH2
- net AnalogKR_1: now also J1.25; no longer J1.27
- net AnalogR_1: now also J1.29; no longer J1.31
- net AnalogR_2: now also J1.28; no longer J1.30
- net AnalogR_3: now also J1.27; no longer J1.29
- net AnalogR_4: now also J1.26; no longer J1.28
- net AnalogV_1: now also J1.33; no longer J1.35
- net AnalogV_2: now also J1.32; no longer J1.34
- net AnalogV_3: now also J1.31; no longer J1.33
- net AnalogV_4: now also J1.30; no longer J1.32
- net FUEL_LVL_Rsense: now also J1.34; no longer J1.36
- net GND: now also J1.24; no longer J1.26
- net WATER_T_Rsense: now also J1.35; no longer J1.MH1

Commit message: V0 PCB Layout
Connections:
- net B06_ActHI: now also J1.4; no longer J1.19
- net GND: now also J1.19; no longer J1.4
Changed lines of the file:
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@@
+    (stroke (width 0) (type default))
+  )
+  (wire (pts (xy 238.76 195.58) (xy 243.84 195.58))
     (stroke (width 0) (type default))
   )
@@
     (stroke (width 0) (type default))
   )
+  (wire (pts (xy 124.46 110.49) (xy 130.81 110.49))
+    (stroke (width 0) (type default))
+  )
+  (wire (pts (xy 336.55 176.53) (xy 344.17 176.53))
+    (stroke (width 0) (type default))
+  )
+  (wire (pts (xy 116.84 63.5) (xy 116.84 66.04))
+    (stroke (width 0) (type default))
+  )
+  (wire (pts (xy 138.43 163.83) (xy 142.24 163.83))
+    (stroke (width 0) (type default))
+  )
+  (wire (pts (xy 246.38 88.9) (xy 252.73 88.9))
+    (stroke (width 0) (type default))
+  )
+  (wire (pts (xy 118.11 41.91) (xy 119.38 41.91))
+    (stroke (width 0) (type default))
+  )
+  (wire (pts (xy 285.75 111.76) (xy 290.83 111.76))
+    (stroke (width 0) (type default))
+  )
+  (wire (pts (xy 336.55 153.67) (xy 344.17 153.67))
+    (stroke (width 0) (type default))
+  )
   (wire (pts (xy 238.76 233.68) (xy 243.84 233.68))
     (stroke (width 0) (type default))
   )
-  (wire (pts (xy 124.46 110.49) (xy 130.81 110.49))
-    (stroke (width 0) (type default))
-  )
-  (wire (pts (xy 336.55 176.53) (xy 344.17 176.53))
-    (stroke (width 0) (type default))
-  )
-  (wire (pts (xy 116.84 63.5) (xy 116.84 66.04))
-    (stroke (width 0) (type default))
-  )
-  (wire (pts (xy 138.43 163.83) (xy 142.24 163.83))
-    (stroke (width 0) (type default))
-  )
-  (wire (pts (xy 246.38 88.9) (xy 252.73 88.9))
-    (stroke (width 0) (type default))
-  )
-  (wire (pts (xy 118.11 41.91) (xy 119.38 41.91))
-    (stroke (width 0) (type default))
-  )
-  (wire (pts (xy 285.75 111.76) (xy 290.83 111.76))
-    (stroke (width 0) (type default))
-  )
-  (wire (pts (xy 336.55 153.67) (xy 344.17 153.67))
-    (stroke (width 0) (type default))
-  )
   (wire (pts (xy 238.76 228.6) (xy 243.84 228.6))
     (stroke (width 0) (type default))
@@
   )
   (wire (pts (xy 238.76 231.14) (xy 243.84 231.14))
-    (stroke (width 0) (type default))
-  )
-  (wire (pts (xy 238.76 195.58) (xy 243.84 195.58))
     (stroke (width 0) (type default))
   )
@@
     )
   )
-  (global_label "GND" (shape input) (at 238.76 195.58 180) (fields_autoplaced)
-    (effects (font (size 1.27 1.27)) (justify right))
-    (property "Intersheetrefs" "${INTERSHEET_REFS}" (at 232.4764 195.5006 0)
+  (global_label "GND" (shape input) (at 238.76 233.68 180) (fields_autoplaced)
+    (effects (font (size 1.27 1.27)) (justify right))
+    (property "Intersheetrefs" "${INTERSHEET_REFS}" (at 232.4764 233.6006 0)
       (effects (font (size 1.27 1.27)) (justify right) hide)
     )
@@
     )
   )
-  (global_label "B06_ActHI" (shape input) (at 238.76 233.68 180) (fields_autoplaced)
-    (effects (font (size 1.27 1.27)) (justify right))
-    (property "Intersheetrefs" "${INTERSHEET_REFS}" (at 226.8521 233.6006 0)
-      (effects (font (size 1.27 1.27)) (justify right) hide)
-    )
+  (global_label "B06_ActHI" (shape input) (at 238.76 195.58 180) (fields_autoplaced)
+    (effects (font (size 1.27 1.27)) (justify right))
+    (property "Intersheetrefs" "${INTERSHEET_REFS}" (at 226.8521 195.5006 0)
+      (effects (font (size 1.27 1.27)) (justify right) hide)
+    )

Commit message: Major update
Connections:
- net ABS_ActLO: now also J1.16; no longer J1.14
- net AIRBAG_ActLO: now also J1.11; no longer J1.9
- net ALTERN_ActLO: now also J1.7; no longer J1.5
- net AnalogV_1: now also J1.35; no longer J1.33
- net AnalogV_2: now also J1.34; no longer J1.32
- net AnalogV_3: now also J1.33; no longer J1.31
- net AnalogV_4: now also J1.32; no longer J1.30
- net B06_ActHI: now also J1.3; no longer J1.4
- net BRAKE_ActLO: now also J1.8; no longer J1.6
- net BTN_ActLO: now also J1.13; no longer J1.11
- net COOLANT_ActLO: now also J1.14; no longer J1.12
- net DOOR_ActLO: now also J1.15; no longer J1.13
- net FBEAMS_ActHI: now also J1.4; no longer J1.16
- net FUEL_LVL_Rsense: now also J1.30; no longer J1.34
- net GND: now also IC5.15 (~{E})
- net IGNITION_ActHI: now also J1.2; no longer J1.15
- net IMMO_ActLO: now also J1.12; no longer J1.10
- net L_TURN_ActHI: now also J1.5; no longer J1.17
- net OIL_ALRM_ActLO: now also J1.10; no longer J1.8
- net PARK_ActLO: now also J1.9; no longer J1.7
- net RPM_HALL: now also J1.17; no longer J1.2
- net R_TURN_ActHI: now also J1.6; no longer J1.18
- net S3: no longer IC5.15 (~{E}), IC5.19 (Y12)
- net SPEED_HALL: now also J1.18; no longer J1.3
- net WATER_T_Rsense: now also J1.31; no longer J1.35
- net abs: now also IC5.8 (Y1); no longer IC5.4 (Y5)
- net alternator: now also IC5.21 (Y10); no longer IC5.23 (Y8)
- net b06: now also IC5.17 (Y14); no longer IC5.6 (Y3)
- net brakes: now also IC5.22 (Y9); no longer IC5.9 (Y0)
- net button: now also IC5.5 (Y4); no longer IC5.16 (Y15)
- net coolant: now also IC5.6 (Y3); no longer IC5.8 (Y1)
- net door: now also IC5.7 (Y2); no longer IC5.20 (Y11)
- net full_beams: now also IC5.18 (Y13); no longer IC5.7 (Y2)
- net ignition: now also IC5.16 (Y15); no longer IC5.5 (Y4)
- net immobilizer: now also IC5.4 (Y5); no longer IC5.21 (Y10)
- net left_turn: now also IC5.19 (Y12); no longer IC5.17 (Y14)
- net parking: now also IC5.23 (Y8); no longer IC5.22 (Y9)
- net right_turn: now also IC5.20 (Y11); no longer IC5.18 (Y13)
- no-connect marks 16 -> 17
Other:
- moved on the sheet: IC5

Commit message: v1.0
- First PCB layout publication
- Titled schematics
- Added Revisions to Schematics and PCB
- iBOM release
- PDF export of PCB design
Other:
- title: (none) -> Main architecture
Changed lines of the file:
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@@
 (kicad_sch (version 20230121) (generator eeschema)
   (paper "A3")
+  (title_block
+    (title "Main architecture")
+    (date "2023-04-10")
+    (rev "1.0")
+    (comment 1 "https://github.com/martinroger/VXDash")
+    (comment 2 "https://cadlab.io/projects/vxdash")
+  )
   (junction (at 124.46 95.25) (diameter 0) (color 0 0 0 0)
   )
@@
     (stroke (width 0) (type default))
   )
-  (text_box "TODO : \n- Selection of connector for outside world\n- MUX connections\n- Nextion connector\n- Check Water T sense\n- Fuse fuse fuse"
+  (text_box "TODO and TOCHECK: \n- Check Water T sense, supposedly 100Hz PWM ?\n- Fuse fuse fuse ?\n- Position of RV1, use of it ?\n- K1 replaced by NPN ?\n- Position of D1 and D2 before K2 ?\n- Change Analog V circuits for constant current circuits ? Sketch it\n- Automated text placement on silkscreen\n- Current allocation table\n- Direct 12V -> 3V3"
     (at 321.31 74.93 0) (size 81.28 57.15)
     (stroke (width 0) (type default))

Commit message: Power conversion split, work prep
-3V3 supply now in parallel with 5V stage
- Reorganisation of hierarchical sheets
- WaterT sense is indeed a PWM so is singled out in the hierarchical sheet
Other:
- sheet 5V_to_3V3_MP2322GQH renamed 12V_to_3V3_MP2322GQH
- sheet AnalogR_Divider6 renamed WaterTsense
- sheet 12V_to_3V3_MP2322GQH: file 5V_to_3V3_MP2322GQH.kicad_sch -> 12V_to_3V3_MP2322GQH.kicad_sch
- sheet 12V_to_3V3_MP2322GQH ports: added 12V_IN; removed 5V_IN
- sheet WaterTsense: file AnalogR_Divider.kicad_sch -> WaterTsense.kicad_sch
Changed lines of the file:
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@@
-    )
-  )
-  (global_label "CONV_5V+" (shape bidirectional) (at 275.59 45.72 180) (fields_autoplaced)
-    (effects (font (size 1.27 1.27)) (justify right))
-    (property "Intersheetrefs" "${INTERSHEET_REFS}" (at 263.3193 45.6406 0)
-      (effects (font (size 1.27 1.27)) (justify right) hide)
     )
   )
@@
     (effects (font (size 1.27 1.27)) (justify right))
     (property "Intersheetrefs" "${INTERSHEET_REFS}" (at 108.2583 95.1706 0)
+      (effects (font (size 1.27 1.27)) (justify right) hide)
+    )
+  )
+  (global_label "PROTECTED_12V+" (shape bidirectional) (at 275.59 45.72 180) (fields_autoplaced)
+    (effects (font (size 1.27 1.27)) (justify right))
+    (property "Intersheetrefs" "${INTERSHEET_REFS}" (at 256.4855 45.6406 0)
       (effects (font (size 1.27 1.27)) (justify right) hide)
     )
@@
     (stroke (width 0.1524) (type solid))
     (fill (color 0 0 0 0.0000))
-    (property "Sheetname" "5V_to_3V3_MP2322GQH" (at 279.4 42.4684 0)
+    (property "Sheetname" "12V_to_3V3_MP2322GQH" (at 279.4 42.4684 0)
       (effects (font (size 1.27 1.27)) (justify left bottom))
     )
-    (property "Sheetfile" "5V_to_3V3_MP2322GQH.kicad_sch" (at 279.4 48.8446 0)
+    (property "Sheetfile" "12V_to_3V3_MP2322GQH.kicad_sch" (at 279.4 48.8446 0)
       (effects (font (size 1.27 1.27)) (justify left top) hide)
     )
@@
       (effects (font (size 1.27 1.27)) (justify right))
     )
-    (pin "5V_IN" input (at 279.4 45.72 180)
+    (pin "12V_IN" input (at 279.4 45.72 180)
       (effects (font (size 1.27 1.27)) (justify left))
     )
@@
   (sheet (at 109.22 232.41) (size 29.21 5.08) (fields_autoplaced)
     (stroke (width 0.1524) (type solid))
-    (fill (color 69 255 155 1.0000))
-    (property "Sheetname" "AnalogR_Divider6" (at 109.22 231.6984 0)
+    (fill (color 102 251 255 1.0000))
+    (property "Sheetname" "WaterTsense" (at 109.22 231.6984 0)
       (effects (font (size 1.27 1.27)) (justify left bottom))
     )
-    (property "Sheetfile" "AnalogR_Divider.kicad_sch" (at 109.22 238.0746 0)
+    (property "Sheetfile" "WaterTsense.kicad_sch" (at 109.22 238.0746 0)
       (effects (font (size 1.27 1.27)) (justify left top) hide)
     )

Commit message: Added power input sch
Added power input sheet.
Relays removed.
MOSFETs added for switching power.
Parts:
- removed D1: S5GC-13-F, Diode_SMD:D_SMC, symbol SamacSys_Parts:S5GC-13-F
- removed D2: SMCJ17A, Diode_SMD:D_SMC, symbol SamacSys_Parts:SMCJ17A
- removed K1, K2: G6L-1P-DC12, SamacSys_Parts:G6L-1P_2, symbol SamacSys_Parts:G6L-1P-DC12
- removed RV1: ERZV10D220, SamacSys_Parts:ERZV10D220, symbol SamacSys_Parts:ERZV10D220
Other:
- added sheet Power_Input (Power_Input.kicad_sch)
