File: KiCad PCB Files/12V_to_5V_AP63200WU-7.kicad_sch (KiCad schematic)
At the start: 19 parts

Commit message: Restored Samacsys parts footprints
PCB components are not placed, just dropped in place
Parts:
- removed PS1: AP63200WU-7, SOT95P280X100-6N, symbol SamacSys_Parts:AP63200WU-7
- added PS2: AP63200WU-7, SamacSys_Parts:SOT95P280X100-6N, symbol SamacSys_Parts:AP63200WU-7
- L1: footprint INDPM4441X200N -> SamacSys_Parts:INDPM4441X200N
Connections:
- net 12V_IN: now also PS2.3 (VIN)
- net GND: now also PS2.4 (GND)
- net at C11.1, R3.2, R4.1: now also PS2.1 (FB)
- net at R1.2, R2.1: now also PS2.2 (EN)
- net at C10.2, C11.2, L1.1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: now also PS2.5 (SW)
- net at C10.1: now also PS2.6 (BST)
Changed lines of the file:
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@@
   (junction (at 191.77 71.12) (diameter 0) (color 0 0 0 0)
   )
+  (junction (at 154.94 71.12) (diameter 0) (color 0 0 0 0)
+  )
   (junction (at 87.63 73.66) (diameter 0) (color 0 0 0 0)
   )
-  (junction (at 154.94 71.12) (diameter 0) (color 0 0 0 0)
+  (junction (at 175.26 71.12) (diameter 0) (color 0 0 0 0)
   )
   (junction (at 154.94 55.88) (diameter 0) (color 0 0 0 0)
-  )
-  (junction (at 175.26 71.12) (diameter 0) (color 0 0 0 0)
   )
   (junction (at 36.83 52.07) (diameter 0) (color 0 0 0 0)
@@
     )
   )
-  (symbol (lib_id "SamacSys_Parts:SRP4020TA-100M") (at 154.94 71.12 0) (unit 1)
-    (in_bom yes) (on_board yes) (dnp no) (fields_autoplaced)
-    (property "Reference" "L1" (at 165.1 66.04 0)
-      (effects (font (size 1.27 1.27)))
-    )
-    (property "Value" "SRP4020TA-100M" (at 165.1 68.58 0)
-      (effects (font (size 1.27 1.27)))
-    )
-    (property "Footprint" "INDPM4441X200N" (at 171.45 69.85 0)
-      (effects (font (size 1.27 1.27)) (justify left) hide)
-    )
-    (property "Datasheet" "http://www.bourns.com/docs/Product-Datasheets/SRP4020TA.pdf" (at 171.45 72.39 0)
-      (effects (font (size 1.27 1.27)) (justify left) hide)
-    )
-    (property "Description" "Bourns SRP4020TA Series Shielded Wire-wound SMD Inductor with a Carbonyl Powder Core, 10 uH +/-20% 1.8A Idc" (at 171.45 74.93 0)
-      (effects (font (size 1.27 1.27)) (justify left) hide)
-    )
-    (property "Height" "2" (at 171.45 77.47 0)
-      (effects (font (size 1.27 1.27)) (justify left) hide)
-    )
-    (property "Manufacturer_Name" "Bourns" (at 171.45 80.01 0)
-      (effects (font (size 1.27 1.27)) (justify left) hide)
-    )
-    (property "Manufacturer_Part_Number" "SRP4020TA-100M" (at 171.45 82.55 0)
-      (effects (font (size 1.27 1.27)) (justify left) hide)
-    )
-    (property "Mouser Part Number" "652-SRP4020TA-100M" (at 171.45 85.09 0)
-      (effects (font (size 1.27 1.27)) (justify left) hide)
-    )
-    (property "Mouser Price/Stock" "https://www.mouser.co.uk/ProductDetail/Bourns/SRP4020TA-100M?qs=Ph8%2FHnX6CQx3wposaLflWQ%3D%3D" (at 171.45 87.63 0)
-      (effects (font (size 1.27 1.27)) (justify left) hide)
-    )
-    (property "Arrow Part Number" "SRP4020TA-100M" (at 171.45 90.17 0)
-      (effects (font (size 1.27 1.27)) (justify left) hide)
-    )
-    (property "Arrow Price/Stock" "https://www.arrow.com/en/products/srp4020ta-100m/bourns?region=nac" (at 171.45 92.71 0)
-      (effects (font (size 1.27 1.27)) (justify left) hide)
-    )
-    (pin "1")
-    (pin "2")
-    (instances
-      (project "VXDash"
-        (path "/f2858fc4-50de-4ff0-a01c-5b985ee14aef/e4c69d46-7a64-435d-9e3a-d73acbe7ec2b"
-          (reference "L1") (unit 1)
-        )
-      )
-    )
-  )
   (symbol (lib_id "power:GND") (at 87.63 58.42 180) (unit 1)
     (in_bom yes) (on_board yes) (dnp no) (fields_autoplaced)
@@
   (symbol (lib_id "SamacSys_Parts:AP63200WU-7") (at 107.95 68.58 0) (unit 1)
     (in_bom yes) (on_board yes) (dnp no) (fields_autoplaced)
-    (property "Reference" "PS1" (at 120.65 62.23 0)
+    (property "Reference" "PS2" (at 120.65 62.23 0)
       (effects (font (size 1.27 1.27)))
     )
@@
       (effects (font (size 1.27 1.27)))
     )
-    (property "Footprint" "SOT95P280X100-6N" (at 129.54 66.04 0)
+    (property "Footprint" "SamacSys_Parts:SOT95P280X100-6N" (at 129.54 66.04 0)
       (effects (font (size 1.27 1.27)) (justify left) hide)
     )
@@
       (project "VXDash"
         (path "/f2858fc4-50de-4ff0-a01c-5b985ee14aef/e4c69d46-7a64-435d-9e3a-d73acbe7ec2b"
-          (reference "PS1") (unit 1)
-        )
-      )
+          (reference "PS2") (unit 1)
+        )
+      )
+    )
+  )
+  (symbol (lib_id "SamacSys_Parts:SRP4020TA-100M") (at 154.94 71.12 0) (unit 1)
+    (in_bom yes) (on_board yes) (dnp no) (fields_autoplaced)
+    (property "Reference" "L1" (at 165.1 66.04 0)
+      (effects (font (size 1.27 1.27)))
+    )
+    (property "Value" "SRP4020TA-100M" (at 165.1 68.58 0)
+      (effects (font (size 1.27 1.27)))
+    )
+    (property "Footprint" "SamacSys_Parts:INDPM4441X200N" (at 171.45 69.85 0)
+      (effects (font (size 1.27 1.27)) (justify left) hide)
+    )
+    (property "Datasheet" "http://www.bourns.com/docs/Product-Datasheets/SRP4020TA.pdf" (at 171.45 72.39 0)
+      (effects (font (size 1.27 1.27)) (justify left) hide)
+    )
+    (property "Description" "Bourns SRP4020TA Series Shielded Wire-wound SMD Inductor with a Carbonyl Powder Core, 10 uH +/-20% 1.8A Idc" (at 171.45 74.93 0)
+      (effects (font (size 1.27 1.27)) (justify left) hide)
+    )
+    (property "Height" "2" (at 171.45 77.47 0)
+      (effects (font (size 1.27 1.27)) (justify left) hide)
+    )
+    (property "Manufacturer_Name" "Bourns" (at 171.45 80.01 0)
+      (effects (font (size 1.27 1.27)) (justify left) hide)
+    )
+    (property "Manufacturer_Part_Number" "SRP4020TA-100M" (at 171.45 82.55 0)
+      (effects (font (size 1.27 1.27)) (justify left) hide)
+    )
+    (property "Mouser Part Number" "652-SRP4020TA-100M" (at 171.45 85.09 0)
+      (effects (font (size 1.27 1.27)) (justify left) hide)
+    )
+    (property "Mouser Price/Stock" "https://www.mouser.co.uk/ProductDetail/Bourns/SRP4020TA-100M?qs=Ph8%2FHnX6CQx3wposaLflWQ%3D%3D" (at 171.45 87.63 0)
+      (effects (font (size 1.27 1.27)) (justify left) hide)
+    )
+    (property "Arrow Part Number" "SRP4020TA-100M" (at 171.45 90.17 0)
+      (effects (font (size 1.27 1.27)) (justify left) hide)
+    )
+    (property "Arrow Price/Stock" "https://www.arrow.com/en/products/srp4020ta-100m/bourns?region=nac" (at 171.45 92.71 0)
+      (effects (font (size 1.27 1.27)) (justify left) hide)
+    )
+    (pin "1")
+    (pin "2")
+    (instances
+      (project "VXDash"
+        (path "/f2858fc4-50de-4ff0-a01c-5b985ee14aef/e4c69d46-7a64-435d-9e3a-d73acbe7ec2b"
+          (reference "L1") (unit 1)
+        )
+      )

Commit message: WIP commit
Parts:
- renumbered PS2 to PS1
Connections:
- net at C12.1, C13.1, C14.1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: now also C11.2, R4.2
- net at C10.2, L1.1, PS1.5 (SW): no longer C11.2, R4.2
Other:
- moved on the sheet: C11
Changed lines of the file:
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@@
   (junction (at 242.57 71.12) (diameter 0) (color 0 0 0 0)
   )
+  (junction (at 87.63 58.42) (diameter 0) (color 0 0 0 0)
+  )
+  (junction (at 208.28 78.74) (diameter 0) (color 0 0 0 0)
+  )
+  (junction (at 175.26 78.74) (diameter 0) (color 0 0 0 0)
+  )
+  (junction (at 142.24 55.88) (diameter 0) (color 0 0 0 0)
+  )
+  (junction (at 191.77 78.74) (diameter 0) (color 0 0 0 0)
+  )
+  (junction (at 208.28 71.12) (diameter 0) (color 0 0 0 0)
+  )
+  (junction (at 69.85 58.42) (diameter 0) (color 0 0 0 0)
+  )
+  (junction (at 191.77 71.12) (diameter 0) (color 0 0 0 0)
+  )
+  (junction (at 87.63 73.66) (diameter 0) (color 0 0 0 0)
+  )
+  (junction (at 175.26 71.12) (diameter 0) (color 0 0 0 0)
+  )
+  (junction (at 154.94 55.88) (diameter 0) (color 0 0 0 0)
+  )
+  (junction (at 36.83 52.07) (diameter 0) (color 0 0 0 0)
+  )
   (junction (at 154.94 63.5) (diameter 0) (color 0 0 0 0)
   )
-  (junction (at 87.63 58.42) (diameter 0) (color 0 0 0 0)
-  )
-  (junction (at 208.28 78.74) (diameter 0) (color 0 0 0 0)
-  )
-  (junction (at 175.26 78.74) (diameter 0) (color 0 0 0 0)
-  )
-  (junction (at 191.77 78.74) (diameter 0) (color 0 0 0 0)
-  )
-  (junction (at 208.28 71.12) (diameter 0) (color 0 0 0 0)
-  )
-  (junction (at 69.85 58.42) (diameter 0) (color 0 0 0 0)
-  )
-  (junction (at 191.77 71.12) (diameter 0) (color 0 0 0 0)
-  )
-  (junction (at 154.94 71.12) (diameter 0) (color 0 0 0 0)
-  )
-  (junction (at 87.63 73.66) (diameter 0) (color 0 0 0 0)
-  )
-  (junction (at 175.26 71.12) (diameter 0) (color 0 0 0 0)
-  )
-  (junction (at 154.94 55.88) (diameter 0) (color 0 0 0 0)
-  )
-  (junction (at 36.83 52.07) (diameter 0) (color 0 0 0 0)
-  )
   (junction (at 224.79 71.12) (diameter 0) (color 0 0 0 0)
   )
@@
     (stroke (width 0) (type default))
   )
-  (wire (pts (xy 154.94 63.5) (xy 154.94 71.12))
-    (stroke (width 0) (type default))
-  )
   (wire (pts (xy 191.77 78.74) (xy 175.26 78.74))
     (stroke (width 0) (type default))
@@
     (stroke (width 0) (type default))
   )
-  (wire (pts (xy 105.41 55.88) (xy 154.94 55.88))
+  (wire (pts (xy 105.41 55.88) (xy 142.24 55.88))
     (stroke (width 0) (type default))
   )
@@
     (stroke (width 0) (type default))
   )
-  (wire (pts (xy 154.94 63.5) (xy 170.18 63.5))
-    (stroke (width 0) (type default))
-  )
-  (wire (pts (xy 154.94 55.88) (xy 170.18 55.88))
+  (wire (pts (xy 175.26 63.5) (xy 175.26 71.12))
+    (stroke (width 0) (type default))
+  )
+  (wire (pts (xy 154.94 63.5) (xy 142.24 63.5))
+    (stroke (width 0) (type default))
+  )
+  (wire (pts (xy 154.94 55.88) (xy 142.24 55.88))
     (stroke (width 0) (type default))
   )
@@
   )
   (wire (pts (xy 69.85 58.42) (xy 87.63 58.42))
+    (stroke (width 0) (type default))
+  )
+  (wire (pts (xy 154.94 63.5) (xy 175.26 63.5))
     (stroke (width 0) (type default))
   )
@@
   (symbol (lib_id "SamacSys_Parts:AP63200WU-7") (at 107.95 68.58 0) (unit 1)
     (in_bom yes) (on_board yes) (dnp no) (fields_autoplaced)
-    (property "Reference" "PS2" (at 120.65 62.23 0)
+    (property "Reference" "PS1" (at 120.65 62.23 0)
       (effects (font (size 1.27 1.27)))
     )
@@
       (project "VXDash"
         (path "/f2858fc4-50de-4ff0-a01c-5b985ee14aef/e4c69d46-7a64-435d-9e3a-d73acbe7ec2b"
-          (reference "PS2") (unit 1)
+          (reference "PS1") (unit 1)
         )
       )
@@
     )
   )
-  (symbol (lib_id "Device:C") (at 170.18 59.69 0) (unit 1)
-    (in_bom yes) (on_board yes) (dnp no) (fields_autoplaced)
-    (property "Reference" "C11" (at 173.99 59.055 0)
-      (effects (font (size 1.27 1.27)) (justify left))
-    )
-    (property "Value" "100pF" (at 173.99 61.595 0)
-      (effects (font (size 1.27 1.27)) (justify left))
-    )
-    (property "Footprint" "Capacitor_SMD:C_0402_1005Metric" (at 171.1452 63.5 0)
-      (effects (font (size 1.27 1.27)) hide)
-    )
-    (property "Datasheet" "~" (at 170.18 59.69 0)
-      (effects (font (size 1.27 1.27)) hide)
-    )
-    (property "Description" "CAP CHIP 0402 100pF 50V C0G 10%" (at 170.18 59.69 0)
-      (effects (font (size 1.27 1.27)) hide)
-    )
-    (property "Manufacturer_Part_Number" "CC0402JRNPO9BN101" (at 170.18 59.69 0)
-      (effects (font (size 1.27 1.27)) hide)
-    )
+  (symbol (lib_id "Device:C") (at 142.24 59.69 0) (unit 1)
+    (in_bom yes) (on_board yes) (dnp no) (fields_autoplaced)
+    (property "Reference" "C11" (at 146.05 59.055 0)
+      (effects (font (size 1.27 1.27)) (justify left))
+    )
+    (property "Value" "100pF" (at 146.05 61.595 0)
+      (effects (font (size 1.27 1.27)) (justify left))
+    )
+    (property "Footprint" "Capacitor_SMD:C_0402_1005Metric" (at 143.2052 63.5 0)
+      (effects (font (size 1.27 1.27)) hide)
+    )
+    (property "Datasheet" "~" (at 142.24 59.69 0)
+      (effects (font (size 1.27 1.27)) hide)
+    )
+    (property "Description" "CAP CHIP 0402 100pF 50V C0G 10%" (at 142.24 59.69 0)
+      (effects (font (size 1.27 1.27)) hide)
+    )
+    (property "Manufacturer_Part_Number" "CC0402JRNPO9BN101" (at 142.24 59.69 0)
+      (effects (font (size 1.27 1.27)) hide)
+    )

Commit message: v1.0
- First PCB layout publication
- Titled schematics
- Added Revisions to Schematics and PCB
- iBOM release
- PDF export of PCB design
Other:
- title: (none) -> 12V to 5V conversion
Changed lines of the file:
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@@
 (kicad_sch (version 20230121) (generator eeschema)
   (paper "A4")
+  (title_block
+    (title "12V to 5V conversion")
+    (date "2023-04-10")
+    (rev "1.0")
+    (comment 1 "https://github.com/martinroger/VXDash")
+    (comment 2 "https://cadlab.io/projects/vxdash")
+  )
   (junction (at 69.85 73.66) (diameter 0) (color 0 0 0 0)
   )

Commit message: PNP resistor sensing circuits
Major updates :
 - PNP (BC807) based constant current supply-and-sense circuit for the passive resistor inputs

Minor updates :
- Added TODO for current consumption check on PNP-based circuits
- Changed from French notation to British notation for resistance values
Parts:
- R1: value 5.1K -> 5K1
- R2, R3: value 19.1K -> 19K1
Changed lines of the file:
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@@
       (effects (font (size 1.27 1.27)) (justify left))
     )
-    (property "Value" "19.1K" (at 157.48 48.895 0)
+    (property "Value" "19K1" (at 157.48 48.895 0)
       (effects (font (size 1.27 1.27)) (justify left))
     )
@@
       (effects (font (size 1.27 1.27)) (justify left))
     )
-    (property "Value" "19.1K" (at 39.37 67.945 0)
+    (property "Value" "19K1" (at 39.37 67.945 0)
       (effects (font (size 1.27 1.27)) (justify left))
     )
@@
       (effects (font (size 1.27 1.27)) (justify left))
     )
-    (property "Value" "5.1K" (at 39.37 47.625 0)
-      (effects (font (size 1.27 1.27)) (justify left))
-    )
+    (property "Value" "5K1" (at 39.37 47.625 0)
+      (effects (font (size 1.27 1.27)) (justify left))
+    )

Commit message: Replaced input capacitors before PS1
Parts:
- removed C7, C8: 10µF 25V, Capacitor_SMD:C_0603_1608Metric, symbol Device:C
- C5, C6: value 10µF 25V -> 22µF 25V; footprint Capacitor_SMD:C_0603_1608Metric -> Capacitor_SMD:C_1210_3225Metric; Manufacturer_Part_Number GRM188R61E106MA73J -> TMK325B7226KM-PR
Connections:
- net 12V_IN: now also C5.2
- net GND: now also C6.1
Other:
- moved on the sheet: C6
Changed lines of the file:
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@@
   (junction (at 208.28 71.12) (diameter 0) (color 0 0 0 0)
   )
+  (junction (at 191.77 71.12) (diameter 0) (color 0 0 0 0)
+  )
+  (junction (at 87.63 73.66) (diameter 0) (color 0 0 0 0)
+  )
+  (junction (at 175.26 71.12) (diameter 0) (color 0 0 0 0)
+  )
+  (junction (at 154.94 55.88) (diameter 0) (color 0 0 0 0)
+  )
+  (junction (at 36.83 52.07) (diameter 0) (color 0 0 0 0)
+  )
+  (junction (at 154.94 63.5) (diameter 0) (color 0 0 0 0)
+  )
   (junction (at 69.85 58.42) (diameter 0) (color 0 0 0 0)
   )
-  (junction (at 191.77 71.12) (diameter 0) (color 0 0 0 0)
-  )
-  (junction (at 87.63 73.66) (diameter 0) (color 0 0 0 0)
-  )
-  (junction (at 175.26 71.12) (diameter 0) (color 0 0 0 0)
-  )
-  (junction (at 154.94 55.88) (diameter 0) (color 0 0 0 0)
-  )
-  (junction (at 36.83 52.07) (diameter 0) (color 0 0 0 0)
-  )
-  (junction (at 154.94 63.5) (diameter 0) (color 0 0 0 0)
-  )
   (junction (at 224.79 71.12) (diameter 0) (color 0 0 0 0)
   )
@@
     (stroke (width 0) (type default))
   )
+  (wire (pts (xy 52.07 58.42) (xy 52.07 60.96))
+    (stroke (width 0) (type default))
+  )
   (wire (pts (xy 191.77 78.74) (xy 175.26 78.74))
     (stroke (width 0) (type default))
@@
     (stroke (width 0) (type default))
   )
+  (wire (pts (xy 69.85 58.42) (xy 87.63 58.42))
+    (stroke (width 0) (type default))
+  )
   (wire (pts (xy 105.41 55.88) (xy 142.24 55.88))
     (stroke (width 0) (type default))
@@
     (stroke (width 0) (type default))
   )
+  (wire (pts (xy 69.85 58.42) (xy 69.85 60.96))
+    (stroke (width 0) (type default))
+  )
   (wire (pts (xy 107.95 68.58) (xy 105.41 68.58))
     (stroke (width 0) (type default))
@@
     (stroke (width 0) (type default))
   )
+  (wire (pts (xy 69.85 68.58) (xy 69.85 73.66))
+    (stroke (width 0) (type default))
+  )
   (wire (pts (xy 260.35 71.12) (xy 270.51 71.12))
     (stroke (width 0) (type default))
@@
     (stroke (width 0) (type default))
   )
-  (wire (pts (xy 69.85 58.42) (xy 87.63 58.42))
-    (stroke (width 0) (type default))
-  )
   (wire (pts (xy 154.94 63.5) (xy 175.26 63.5))
     (stroke (width 0) (type default))
@@
   )
   (wire (pts (xy 242.57 71.12) (xy 252.73 71.12))
+    (stroke (width 0) (type default))
+  )
+  (wire (pts (xy 52.07 68.58) (xy 52.07 73.66))
     (stroke (width 0) (type default))
   )
@@
     )
   )
-  (symbol (lib_id "Device:C") (at 52.07 62.23 0) (unit 1)
-    (in_bom yes) (on_board yes) (dnp no) (fields_autoplaced)
-    (property "Reference" "C5" (at 55.88 61.595 0)
-      (effects (font (size 1.27 1.27)) (justify left))
-    )
-    (property "Value" "10µF 25V" (at 55.88 64.135 0)
-      (effects (font (size 1.27 1.27)) (justify left))
-    )
-    (property "Footprint" "Capacitor_SMD:C_0603_1608Metric" (at 53.0352 66.04 0)
-      (effects (font (size 1.27 1.27)) hide)
-    )
-    (property "Datasheet" "~" (at 52.07 62.23 0)
-      (effects (font (size 1.27 1.27)) hide)
-    )
-    (property "Description" "CAP CHIP 0603 10uF 25V X5R 20%" (at 52.07 62.23 0)
-      (effects (font (size 1.27 1.27)) hide)
-    )
-    (property "Manufacturer_Part_Number" "GRM188R61E106MA73J" (at 52.07 62.23 0)
-      (effects (font (size 1.27 1.27)) hide)
-    )
-    (pin "1")
-    (pin "2")
-    (instances
-      (project "VXDash"
-        (path "/f2858fc4-50de-4ff0-a01c-5b985ee14aef/e4c69d46-7a64-435d-9e3a-d73acbe7ec2b"
-          (reference "C5") (unit 1)
-        )
-      )
-    )
-  )
   (symbol (lib_id "power:GND") (at 134.62 77.47 0) (unit 1)
     (in_bom yes) (on_board yes) (dnp no) (fields_autoplaced)
@@
     )
   )
-  (symbol (lib_id "Device:C") (at 69.85 62.23 0) (unit 1)
-    (in_bom yes) (on_board yes) (dnp no) (fields_autoplaced)
-    (property "Reference" "C7" (at 73.66 61.595 0)
-      (effects (font (size 1.27 1.27)) (justify left))
-    )
-    (property "Value" "10µF 25V" (at 73.66 64.135 0)
-      (effects (font (size 1.27 1.27)) (justify left))
-    )
-    (property "Footprint" "Capacitor_SMD:C_0603_1608Metric" (at 70.8152 66.04 0)
-      (effects (font (size 1.27 1.27)) hide)
-    )
-    (property "Datasheet" "~" (at 69.85 62.23 0)
-      (effects (font (size 1.27 1.27)) hide)
-    )
-    (property "Description" "CAP CHIP 0603 10uF 25V X5R 20%" (at 69.85 62.23 0)
-      (effects (font (size 1.27 1.27)) hide)
-    )
-    (property "Manufacturer_Part_Number" "GRM188R61E106MA73J" (at 69.85 62.23 0)
-      (effects (font (size 1.27 1.27)) hide)
-    )
-    (pin "1")
-    (pin "2")
-    (instances
-      (project "VXDash"
-        (path "/f2858fc4-50de-4ff0-a01c-5b985ee14aef/e4c69d46-7a64-435d-9e3a-d73acbe7ec2b"
-          (reference "C7") (unit 1)
-        )
-      )
-    )
-  )
   (symbol (lib_id "Device:R") (at 154.94 59.69 0) (unit 1)
     (in_bom yes) (on_board yes) (dnp no) (fields_autoplaced)
@@
     )
   )
-  (symbol (lib_id "Device:C") (at 52.07 69.85 0) (unit 1)
-    (in_bom yes) (on_board yes) (dnp no) (fields_autoplaced)
-    (property "Reference" "C6" (at 55.88 69.215 0)
-      (effects (font (size 1.27 1.27)) (justify left))
-    )
-    (property "Value" "10µF 25V" (at 55.88 71.755 0)
-      (effects (font (size 1.27 1.27)) (justify left))
-    )
-    (property "Footprint" "Capacitor_SMD:C_0603_1608Metric" (at 53.0352 73.66 0)
-      (effects (font (size 1.27 1.27)) hide)
-    )
-    (property "Datasheet" "~" (at 52.07 69.85 0)
-      (effects (font (size 1.27 1.27)) hide)
-    )
-    (property "Description" "CAP CHIP 0603 10uF 25V X5R 20%" (at 52.07 69.85 0)
-      (effects (font (size 1.27 1.27)) hide)
-    )
-    (property "Manufacturer_Part_Number" "GRM188R61E106MA73J" (at 52.07 69.85 0)
+  (symbol (lib_id "Device:C") (at 52.07 64.77 0) (unit 1)
+    (in_bom yes) (on_board yes) (dnp no) (fields_autoplaced)
+    (property "Reference" "C6" (at 55.88 64.135 0)
+      (effects (font (size 1.27 1.27)) (justify left))
+    )
+    (property "Value" "22µF 25V" (at 55.88 66.675 0)
+      (effects (font (size 1.27 1.27)) (justify left))
+    )
+    (property "Footprint" "Capacitor_SMD:C_1210_3225Metric" (at 53.0352 68.58 0)
+      (effects (font (size 1.27 1.27)) hide)
+    )
+    (property "Datasheet" "~" (at 52.07 64.77 0)
+      (effects (font (size 1.27 1.27)) hide)
+    )
+    (property "Description" "CAP CER 22UF 25V X7R 1210" (at 52.07 64.77 0)
+      (effects (font (size 1.27 1.27)) hide)
+    )
+    (property "Manufacturer_Part_Number" "TMK325B7226KM-PR" (at 52.07 64.77 0)
       (effects (font (size 1.27 1.27)) hide)
     )
@@
     )
   )
-  (symbol (lib_id "Device:C") (at 69.85 69.85 0) (unit 1)
-    (in_bom yes) (on_board yes) (dnp no) (fields_autoplaced)
-    (property "Reference" "C8" (at 73.66 69.215 0)
-      (effects (font (size 1.27 1.27)) (justify left))
-    )
-    (property "Value" "10µF 25V" (at 73.66 71.755 0)
-      (effects (font (size 1.27 1.27)) (justify left))
-    )
-    (property "Footprint" "Capacitor_SMD:C_0603_1608Metric" (at 70.8152 73.66 0)
-      (effects (font (size 1.27 1.27)) hide)
-    )
-    (property "Datasheet" "~" (at 69.85 69.85 0)
-      (effects (font (size 1.27 1.27)) hide)
-    )
-    (property "Description" "CAP CHIP 0603 10uF 25V X5R 20%" (at 69.85 69.85 0)
-      (effects (font (size 1.27 1.27)) hide)
-    )
-    (property "Manufacturer_Part_Number" "GRM188R61E106MA73J" (at 69.85 69.85 0)
-      (effects (font (size 1.27 1.27)) hide)
-    )
-    (pin "1")
-    (pin "2")
-    (instances
-      (project "VXDash"
-        (path "/f2858fc4-50de-4ff0-a01c-5b985ee14aef/e4c69d46-7a64-435d-9e3a-d73acbe7ec2b"
-          (reference "C8") (unit 1)
-        )
-      )
-    )
-  )
   (symbol (lib_id "power:GND") (at 154.94 43.18 180) (unit 1)
     (in_bom yes) (on_board yes) (dnp no) (fields_autoplaced)
@@
         )
       )
+    )
+  )
+  (symbol (lib_id "Device:C") (at 69.85 64.77 0) (unit 1)
+    (in_bom yes) (on_board yes) (dnp no) (fields_autoplaced)
+    (property "Reference" "C5" (at 73.66 64.135 0)
+      (effects (font (size 1.27 1.27)) (justify left))
+    )
+    (property "Value" "22µF 25V" (at 73.66 66.675 0)
+      (effects (font (size 1.27 1.27)) (justify left))
+    )
+    (property "Footprint" "Capacitor_SMD:C_1210_3225Metric" (at 70.8152 68.58 0)
+      (effects (font (size 1.27 1.27)) hide)
+    )
+    (property "Datasheet" "~" (at 69.85 64.77 0)
+      (effects (font (size 1.27 1.27)) hide)
+    )
+    (property "Description" "CAP CER 22UF 25V X7R 1210" (at 69.85 64.77 0)
+      (effects (font (size 1.27 1.27)) hide)
+    )
+    (property "Manufacturer_Part_Number" "TMK325B7226KM-PR" (at 69.85 64.77 0)
+      (effects (font (size 1.27 1.27)) hide)
+    )
+    (pin "1")
+    (pin "2")
+    (instances
+      (project "VXDash"
+        (path "/f2858fc4-50de-4ff0-a01c-5b985ee14aef/e4c69d46-7a64-435d-9e3a-d73acbe7ec2b"
+          (reference "C5") (unit 1)
+        )
+      )
