File: KiCad PCB Files/VXDash.kicad_pcb (KiCad board)
At the start: 2 copper layers, 105 x 95 mm, 137 parts, among them IC1 CD74HC4050M96, IC2 SP721ABG, IC3 74HC4067BQ-Q100J, IC4 MP2322GQH-Z, J1 MX34036UF2, J2 Conn_01x04_Socket, K1 G6L-1P-DC12, K2 G6L-1P-DC12, U1 SFH617A-2X009T, U10 SFH617A-2X009T, U11 SFH617A-2X009T, U12 SFH617A-2X009T, U13 SFH617A-2X009T, U14 SFH617A-2X009T, U15 SFH617A-2X009T, U16 ESP32-DevKitC, U2 SFH617A-2X009T, U3 SFH617A-2X009T, U4 SFH617A-2X009T, U5 SFH617A-2X009T, U6 SFH617A-2X009T, U7 SFH617A-2X009T, U8 SFH617A-2X009T, U9 SFH617A-2X009T

Commit message: Power conversion split, work prep
-3V3 supply now in parallel with 5V stage
- Reorganisation of hierarchical sheets
- WaterT sense is indeed a PWM so is singled out in the hierarchical sheet
Connections:
- C17 pad 1: CONV_5V+ -> PROTECTED_12V+
- C18 pad 1: CONV_5V+ -> PROTECTED_12V+
- C19 pad 1: CONV_5V+ -> PROTECTED_12V+
- IC4 pad 2: CONV_5V+ -> PROTECTED_12V+
- R36 pad 1: CONV_5V+ -> PROTECTED_12V+
Routing:
- net PROTECTED_12V+: track 143.4 -> 174.3 mm, vias 5 -> 11
- net CONV_5V+: track 113.4 -> 108.6 mm, vias 6 -> 4
- removed copper zone on F.Cu, net CONV_5V+

Commit message: PCB adaptation
- Updated footprints
- Started grouping
- Hid a few references
Parts:
- removed D8: PMEG3010EH, Diode_SMD:D_SOD-123F
- removed K1, K2: G6L-1P-DC12, SamacSys_Parts:G6L-1P_2
- added C33: 0.1µF, Capacitor_SMD:C_0603_1608Metric, F.Cu at (229.9, 87.5)
- added C34: 0.1µF, Capacitor_SMD:C_0603_1608Metric, F.Cu at (229.9, 90.0)
- added C35: 0.1µF, Capacitor_SMD:C_0603_1608Metric, F.Cu at (229.9, 92.5)
- added C36: 1uF, Capacitor_SMD:C_0603_1608Metric, F.Cu at (229.9, 95.0)
- added C37: 0.1µF, Capacitor_SMD:C_0603_1608Metric, F.Cu at (229.9, 97.5)
- added D10: 18V, Diode_SMD:D_SOD-123, F.Cu at (239.7, 96.3)
- added F2: 0ZRB0250FF1E, Fuse:Fuse_BelFuse_0ZRE0033FF_L11.4mm_W3.8mm, F.Cu at (231.8, 82.7)
- added FB1: 120R@100MHz, Inductor_SMD:L_0805_2012Metric, F.Cu at (244.8, 98.6)
- added FB2: 120R@100MHz, Inductor_SMD:L_0805_2012Metric, F.Cu at (244.8, 101.3)
- added Q1: 2N7002, Package_TO_SOT_SMD:SOT-23, F.Cu at (234.3, 93.5)
- added Q2: PJA3441, Package_TO_SOT_SMD:SOT-23, F.Cu at (234.3, 98.0)
- added Q3: BC807, Package_TO_SOT_SMD:SOT-23, F.Cu at (163.5, -28.8)
- added Q4: BC807, Package_TO_SOT_SMD:SOT-23, F.Cu at (168.6, -28.8)
- added Q5: BC807, Package_TO_SOT_SMD:SOT-23, F.Cu at (173.7, -28.8)
- added Q6: BC807, Package_TO_SOT_SMD:SOT-23, F.Cu at (178.7, -28.8)
- added Q7: BC807, Package_TO_SOT_SMD:SOT-23, F.Cu at (158.4, -28.8)
- added Q8: BC807, Package_TO_SOT_SMD:SOT-23, F.Cu at (183.8, -28.8)
- added R62: 1K, Resistor_SMD:R_0805_2012Metric, F.Cu at (244.8, 92.8)
- added R63: 100K, Resistor_SMD:R_0402_1005Metric, F.Cu at (238.2, 99.0)
- added R64: 1K, Resistor_SMD:R_0805_2012Metric, F.Cu at (244.8, 95.7)
- added R65: 100K, Resistor_SMD:R_0402_1005Metric, F.Cu at (238.2, 101.0)
- added R66: 270R, Resistor_SMD:R_0603_1608Metric, F.Cu at (163.4, -35.6)
- added R67: 270R, Resistor_SMD:R_0603_1608Metric, F.Cu at (168.5, -35.6)
- added R68: 270R, Resistor_SMD:R_0603_1608Metric, F.Cu at (173.5, -35.6)
- added R69: 270R, Resistor_SMD:R_0603_1608Metric, F.Cu at (178.6, -35.6)
- added R70: 270R, Resistor_SMD:R_0603_1608Metric, F.Cu at (158.3, -35.6)
- added R71: 3K3, Resistor_SMD:R_0603_1608Metric, F.Cu at (184.9, -33.0)
- D1: value S5GC-13-F -> 18V; footprint Diode_SMD:D_SMC -> Diode_SMD:D_SOD-123
- D2: value SMCJ17A -> PMEG3010EH; footprint Diode_SMD:D_SMC -> Diode_SMD:D_SOD-123F
- R1: value 5.1K -> 5K1
- R2, R3: value 19.1K -> 19K1
- R48, R50, R52: value 220R -> 3K3; footprint Resistor_SMD:R_0805_2012Metric -> Resistor_SMD:R_0603_1608Metric
- R49, R51: value 1K -> 3K3; footprint Resistor_SMD:R_0805_2012Metric -> Resistor_SMD:R_0603_1608Metric
- R53, R55, R57: value 1K -> 2K2; footprint Resistor_SMD:R_0805_2012Metric -> Resistor_SMD:R_0603_1608Metric
- R54, R56: value 220R -> 2K2; footprint Resistor_SMD:R_0805_2012Metric -> Resistor_SMD:R_0603_1608Metric
- R58: value 220R -> 510R; footprint Resistor_SMD:R_0805_2012Metric -> Resistor_SMD:R_0603_1608Metric
- R59: value 2.7K -> 2K2; footprint Resistor_SMD:R_0805_2012Metric -> Resistor_SMD:R_0603_1608Metric
- RV1: value ERZV10D220 -> MOV-07D220K; footprint SamacSys_Parts:ERZV10D220 -> Varistor:RV_Disc_D9mm_W3.5mm_P5mm
- moved R56 114.9 mm to (177.8, -33.0)
- moved R58 114.7 mm to (183.7, -35.6), turned to 180 degrees
- moved R50 112.6 mm to (174.7, -33.0), turned to 90 degrees
- moved R48 112.0 mm to (164.6, -33.0), turned to 90 degrees
- moved R52 111.6 mm to (159.5, -33.0), turned to 90 degrees
- moved R54 111.5 mm to (167.6, -33.0)
- moved R51 109.5 mm to (179.8, -33.0)
- moved D2 109.3 mm to (184.3, -23.6), turned to 90 degrees
- moved R49 108.5 mm to (169.7, -33.0)
- moved R59 108.0 mm to (182.9, -33.0), turned to -90 degrees
- moved R57 107.7 mm to (157.5, -33.0), turned to -90 degrees
- moved R55 107.6 mm to (172.7, -33.0), turned to -90 degrees
- moved R53 107.4 mm to (162.6, -33.0), turned to -90 degrees
- moved D6 107.3 mm to (179.2, -23.6)
- moved D5 107.2 mm to (174.2, -23.6)
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Connections:
- D1 pad 1: PROTECTED_12V+ -> Net-(D1-K)
- D1 pad 2: SWITCHED_12V+ -> GND
- D2 pad 1: PROTECTED_12V+ -> AnalogKR_1
- D2 pad 2: GND -> sensor_KR_1
- R48 pad 1: REG_3.3V+ -> Net-(Q3-B)
- R48 pad 2: sensor_R_1 -> GND
- R49 pad 1: sensor_R_1 -> Net-(Q4-B)
- R50 pad 1: REG_3.3V+ -> Net-(Q5-B)
- R50 pad 2: sensor_R_2 -> GND
- R51 pad 1: sensor_R_2 -> Net-(Q6-B)
- R52 pad 1: REG_3.3V+ -> Net-(Q7-B)
- R52 pad 2: sensor_R_3 -> GND
- R53 pad 1: sensor_R_3 -> REG_3.3V+
- R53 pad 2: GND -> Net-(Q3-B)
- R54 pad 2: sensor_R_4 -> Net-(Q4-B)
- R55 pad 1: sensor_R_4 -> REG_3.3V+
- R55 pad 2: GND -> Net-(Q5-B)
- R56 pad 2: fuel_level -> Net-(Q6-B)
- R57 pad 1: fuel_level -> REG_3.3V+
- R57 pad 2: GND -> Net-(Q7-B)
- R58 pad 2: sensor_KR_1 -> Net-(Q8-E)
- R59 pad 1: sensor_KR_1 -> REG_3.3V+
- R59 pad 2: GND -> Net-(Q8-B)
- RV1 pad 1: BATT12V+ -> GND
- RV1 pad 2: GND -> Net-(Q2-D)
Routing:
- net fuel_level: track 28.9 -> 2.83 mm
- net AnalogKR_1: track 20.9 -> 0.00 mm
- net sensor_R_4: track 21.6 -> 2.83 mm, vias 0 -> 1
- net AnalogR_4: track 17.0 -> 0.00 mm
- net AnalogR_1: track 16.1 -> 0.00 mm
- net sensor_R_3: track 18.6 -> 2.83 mm, vias 0 -> 1
- net sensor_KR_1: track 18.7 -> 3.08 mm, vias 0 -> 1
- net AnalogR_2: track 15.6 -> 0.00 mm
- net sensor_R_2: track 17.7 -> 2.83 mm, vias 0 -> 1
- net AnalogR_3: track 13.9 -> 0.00 mm
- net sensor_R_1: track 15.1 -> 2.83 mm, vias 0 -> 1
- net FUEL_LVL_Rsense: track 11.5 -> 0.00 mm
- net Net-(Q5-E): track 0.00 -> 6.63 mm
- net Net-(Q3-E): track 0.00 -> 6.63 mm
- net Net-(Q7-E): track 0.00 -> 6.63 mm
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- removed copper zone on B.Cu, net BATT12V+
- removed copper zone on F.Cu, net SWITCHED_12V+

Commit message: Update VXDash.kicad_pcb
Positioning of the PNP groups
Parts:
- moved D2 108.7 mm to (176.6, 84.8)
- moved R59 108.7 mm to (175.2, 75.4)
- moved R71 108.7 mm to (177.2, 75.4)
- moved Q8 108.7 mm to (176.1, 79.5)
- moved R58 108.7 mm to (176.0, 72.8)
- moved D6 108.2 mm to (172.1, 84.3)
- moved Q6 108.2 mm to (171.6, 79.1)
- moved R51 108.2 mm to (172.7, 74.9)
- moved R56 108.2 mm to (170.7, 74.9)
- moved R69 108.2 mm to (171.5, 72.3)
- moved D5 108.2 mm to (167.6, 84.3)
- moved Q5 108.2 mm to (167.1, 79.1)
- moved R50 108.2 mm to (168.1, 74.9)
- moved R55 108.2 mm to (166.1, 74.9)
- moved R68 108.2 mm to (166.9, 72.3)
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Routing:
- net PROTECTED_12V+: track 174.3 -> 126.2 mm, vias 11 -> 2
- net right_turn: track 135.2 -> 125.5 mm
- net left_turn: track 144.5 -> 140.8 mm
- net CONV_5V+: track 108.6 -> 112.3 mm
- net S0: track 96.9 -> 98.8 mm
- net S3: track 113.2 -> 112.6 mm

Commit message: 1.1HW and Schematics -> PR
- Updated all dates in title blocks
- Added both FET based new power supply and protection circuits - completely winged the zones
- Completed PCB layout, passes DRCs --> Needs review
- Updated PCB metadata
- Relocated 5th mounting hole a bit
- Regenerated interactive BOM
Parts:
- moved R65 51.1 mm to (189.7, 85.0), turned to -90 degrees
- moved FB1 50.4 mm to (196.8, 83.4)
- moved FB2 50.2 mm to (196.8, 87.0)
- moved Q2 49.0 mm to (187.1, 85.0), turned to 180 degrees
- moved RV1 48.7 mm to (186.4, 94.2)
- moved D10 47.4 mm to (193.7, 85.0), turned to -90 degrees
- moved F2 46.8 mm to (187.9, 98.9)
- moved R62 46.2 mm to (200.5, 105.8), turned to 90 degrees
- moved R64 44.9 mm to (200.1, 91.6), turned to 180 degrees
- moved D1 40.8 mm to (199.8, 101.7)
- moved C37 40.7 mm to (191.2, 85.0), turned to 90 degrees
- moved R63 38.4 mm to (199.8, 99.7)
- moved C33 35.8 mm to (195.0, 95.4), turned to -90 degrees
- moved Q1 34.5 mm to (199.8, 95.0), turned to 90 degrees
- moved C35 31.3 mm to (199.8, 83.9), turned to 90 degrees
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Routing:
- net PROTECTED_12V+: track 126.2 -> 182.6 mm, vias 2 -> 9
- net fuel_level: track 2.83 -> 27.9 mm
- net AnalogKR_1: track 0.00 -> 24.4 mm
- net REG_3.3V+: track 478.6 -> 500.4 mm
- net AnalogR_4: track 0.00 -> 21.6 mm
- net sensor_R_4: track 2.83 -> 23.1 mm
- net AnalogR_3: track 0.00 -> 19.1 mm
- net sensor_R_3: track 2.83 -> 21.2 mm
- net sensor_KR_1: track 3.08 -> 20.5 mm
- net AnalogR_2: track 0.00 -> 16.7 mm
- net sensor_R_2: track 2.83 -> 19.2 mm
- net sensor_R_1: track 2.83 -> 18.3 mm
- net Net-(Q2-D): track 0.00 -> 15.5 mm
- net AnalogR_1: track 0.00 -> 15.2 mm
- net FUEL_LVL_Rsense: track 0.00 -> 14.4 mm
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- added copper zone on F.Cu, net /Power_Input/SWITCHED_12V+
- added copper zone on F.Cu, net Net-(D1-K)
- added copper zone on F.Cu, net Net-(D10-A)
- added copper zone on F.Cu, net Net-(Q2-D)

Commit message: B06 renamed to BCKLIGHT
Connections:
- net B06_ActHI renamed BCKLIGHT_ActHI
- net b06 renamed backlight
Changed lines of the file:
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@@
   (net 58 "coolant")
   (net 59 "full_beams")
-  (net 60 "b06")
+  (net 60 "backlight")
   (net 61 "ignition")
   (net 62 "abs")
@@
   (net 69 "/ESP32/RX1")
   (net 70 "5V_SENSOR")
-  (net 71 "B06_ActHI")
+  (net 71 "BCKLIGHT_ActHI")
   (net 72 "R_TURN_ActHI")
   (net 73 "L_TURN_ActHI")
@@
       (net 61 "ignition") (pinfunction "Y15") (pintype "passive") (thermal_bridge_angle 45))
     (pad "17" smd rect (at 0.75 -1.8 270) (size 0.29 0.9) (layers "F.Cu" "F.Paste" "F.Mask")
-      (net 60 "b06") (pinfunction "Y14") (pintype "passive") (thermal_bridge_angle 45))
+      (net 60 "backlight") (pinfunction "Y14") (pintype "passive") (thermal_bridge_angle 45))
     (pad "18" smd rect (at 0.25 -1.8 270) (size 0.29 0.9) (layers "F.Cu" "F.Paste" "F.Mask")
       (net 59 "full_beams") (pinfunction "Y13") (pintype "passive") (thermal_bridge_angle 45))
@@
       (stroke (width 0.1) (type solid)) (layer "F.Fab"))
     (pad "1" smd roundrect (at -0.9125 0 270) (size 1.025 1.4) (layers "F.Cu" "F.Paste" "F.Mask") (roundrect_rratio 0.243902439)
-      (net 71 "B06_ActHI") (pintype "passive"))
+      (net 71 "BCKLIGHT_ActHI") (pintype "passive"))
     (pad "2" smd roundrect (at 0.9125 0 270) (size 1.025 1.4) (layers "F.Cu" "F.Paste" "F.Mask") (roundrect_rratio 0.243902439)
       (net 102 "Net-(R34-Pad2)") (pintype "passive"))
@@
       (net 2 "GND") (pintype "passive"))
     (pad "4" smd rect (at 3.81 -1.27 270) (size 2 1.78) (layers "F.Cu" "F.Paste" "F.Mask")
-      (net 60 "b06") (pintype "passive"))
+      (net 60 "backlight") (pintype "passive"))
     (model "${KICAD6_3DMODEL_DIR}/Package_DIP.3dshapes/SMDIP-4_W7.62mm.wrl"
       (offset (xyz 0 0 0))
@@
       (stroke (width 0.1) (type solid)) (layer "F.Fab"))
     (pad "1" smd roundrect (at -0.9125 0 270) (size 1.025 1.4) (layers "F.Cu" "F.Paste" "F.Mask") (roundrect_rratio 0.243902439)
-      (net 60 "b06") (pintype "passive"))
+      (net 60 "backlight") (pintype "passive"))
     (pad "2" smd roundrect (at 0.9125 0 270) (size 1.025 1.4) (layers "F.Cu" "F.Paste" "F.Mask") (roundrect_rratio 0.243902439)
       (net 42 "REG_3.3V+") (pintype "passive"))
@@
       (net 75 "IGNITION_ActHI") (pinfunction "2") (pintype "passive"))
     (pad "3" thru_hole circle (at -4.4 0 270) (size 1.5 1.5) (drill 1) (layers "*.Cu" "*.Mask" "B.SilkS")
-      (net 71 "B06_ActHI") (pinfunction "3") (pintype "passive"))
+      (net 71 "BCKLIGHT_ActHI") (pinfunction "3") (pintype "passive"))
     (pad "4" thru_hole circle (at -6.6 0 270) (size 1.5 1.5) (drill 1) (layers "*.Cu" "*.Mask" "B.SilkS")
       (net 74 "FBEAMS_ActHI") (pinfunction "4") (pintype "passive"))

Commit message: Update VXDash.kicad_pcb
Implemented current schematic changes
Capacitors near PS1
Capacitors for Water T sense
Water T sense relocated to the CMOS
Parts:
- removed C7, C8: 10µF 25V, Capacitor_SMD:C_0603_1608Metric
- removed D9: PMEG3010EH, Diode_SMD:D_SOD-123F
- removed R60: 220R, Resistor_SMD:R_0805_2012Metric
- removed R61: 1K, Resistor_SMD:R_0805_2012Metric
- added C38: 0.1µF, Capacitor_SMD:C_0603_1608Metric, F.Cu at (121.7, 89.0)
- added C39: 0.1µF 50V, Capacitor_SMD:C_0603_1608Metric, F.Cu at (123.6, 89.0)
- C5, C6: value 10µF 25V -> 22µF 25V; footprint Capacitor_SMD:C_0603_1608Metric -> Capacitor_SMD:C_1210_3225Metric
- moved C5 9.47 mm to (192.0, 76.6), turned to 0 degrees
- moved C6 2.05 mm to (198.8, 76.3)
Connections:
- C5 pad 2: Net-(C5-Pad2) -> PROTECTED_12V+
- C6 pad 1: Net-(C5-Pad2) -> GND
- IC1 pad 10: unconnected-(IC1-4Y-Pad10) -> water_T
- IC1 pad 9: GND -> WATER_T_Rsense
Routing:
- net water_T: track 23.8 -> 43.6 mm, vias 1 -> 2
- net WATER_T_Rsense: track 10.2 -> 27.1 mm
- net REG_3.3V+: track 500.4 -> 497.9 mm
- net Net-(C7-Pad2): track 2.01 -> 0.00 mm
- net Net-(C5-Pad2): track 2.01 -> 0.00 mm
Other:
- board size 105 x 95 mm -> 115 x 95 mm
