File: KiCad PCB Files/R-KRsensing_Pair.kicad_sch (KiCad schematic)
At the start: 14 parts, among them IC5 LM358BAIDGKR, Q10 BC807, Q9 BC807, U18 LM4040DBZ-4.1

Commit message: PCB layout update 1.2.1
Updated with OpAmp circuitry plus some component identification
Parts:
- removed R52: 220R, Resistor_SMD:R_0603_1608Metric, symbol Device:R
- added R61: 470R, Resistor_SMD:R_0603_1608Metric, symbol Device:R
Connections:
- net CONV_5V+: now also R61.1
- net at IC5.6 (IN2-), Q10.2 (E): now also R61.2
- net Analog_IN_2 renamed Analog_K_IN_2
- net Analog_OUT_2 renamed Analog_K_OUT_2
Other:
- note added: "Current is set as follows : - LM4040DBZ-4.1 sets voltage at 4.096V on a good day - Assuming we have 5V this makes a reference voltage of 0.904V - Reference resistence is currently 470R -> Reference current is 0.904/470 = 1.92mA approx - For high K sensors (70-2000Ohm), that gives a sensor voltage of anywhere between 0.1344V and 3.84V - Practically the maximum voltage that can be is 4.096V-0.550V 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"
- moved on the sheet: C6, D2, D9, IC5, Q10, Q9, R60, R72, R73, R74, R75, R76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

Commit message: Comments
@Alex-XNR
Just confirmed with comments to educate me.
I think the only point that remains open is the question of Rf and Ri ? I can't remember where I saw they were included and I can't see, to find anymore.
For the higher resistance I/O I think I will try with a higher Iset resistor ? With my crappy simulator it seems to run.
Parts:
- removed C6: 0.1uF 50V, Capacitor_SMD:C_0603_1608Metric, symbol Device:C
- removed Q10, Q9: BC807, Package_TO_SOT_SMD:SOT-23, symbol Transistor_BJT:BC807
- removed R61: 470R, Resistor_SMD:R_0603_1608Metric, symbol Device:R
- removed U18: LM4040DBZ-4.1, Package_TO_SOT_SMD:SOT-23, symbol Reference_Voltage:LM4040DBZ-4.1
- added C6 (x2): 0.1uF 50V, Capacitor_SMD:C_0603_1608Metric, symbol Device:C
- added Q7, Q8: DMG2301L, Package_TO_SOT_SMD:SOT-23, symbol Device:Q_PMOS_GSD
- added R52: 51R, Resistor_SMD:R_0603_1608Metric, symbol Device:R
- added R58: 330k, Resistor_SMD:R_0603_1608Metric, symbol Device:R
- R60: value 220R -> 22R; Manufacturer_Name Stackpole Electronics Inc -> (none); Manufacturer_Part_Number RMCF0603FT220R -> (none)
- R72: value 910R -> 6k8; Manufacturer_Name Yageo -> (none); Manufacturer_Part_Number RC0603FR-07910RL -> (none)
- R73, R75: value 2K2 -> 2k7; Manufacturer_Name Yageo -> (none); Manufacturer_Part_Number RC0603FR-072K2L -> (none)
- R74, R76: value 9K1 -> 5k1; Manufacturer_Name Yageo -> (none); Manufacturer_Part_Number RC0603FR-079K1L -> (none)
Connections:
- net CONV_5V+: now also C6.2, R52.2
- net GND: now also C6.1, C6.1, R58.2
- net at D9.2 (A), R75.1: now also Q8.3 (D)
- net at IC5.1 (OUT1): now also Q7.1 (G)
- net at IC5.2 (IN1-), R60.2: now also Q7.2 (S)
- net at IC5.3 (IN1+), IC5.5 (IN2+), R72.2: now also C6.2, R58.1
- net at IC5.6 (IN2-): now also Q8.2 (S), R52.1
- net at IC5.7 (OUT2): now also Q8.1 (G)
- net at D2.2 (A), R73.1: now also Q7.3 (D)
Other:
- note added: "Current is set as follows : - 100mV across 22R = ~4.54mA. MOSFET used to avoid influence from additional base current. - For fuel level and common sensors (0-250Ohm), that gives a sensor voltage of anywhere between 0 and 1.135V - Practically the maximum voltage that can be is 4.9V-0.550V = 4.35V (the schottky typical Vf, although usually lower) - That means that in this current setup the maximum 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"
- note added: "Full-scale 5V = just under 3V3 (~3.27V)"
- note added: "Ideas/issues : - How to account for variations in the Vf of PMEG3010EH Alex: At ~4.5mA, Vf varies by ~120mV from -40 to 80degC. This equates to ~24ohm error over a large temp Martin : gotcha - 5V may not be true 5V -> Zener regulator there too ? evaluate possible swings Alex: Used a Vref that follows any variation of 5V. More worried about keeping a set V across the current set resistor. - Design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"
- note added: "Rf and Ri useful ? 47K, but apparently LM358B/BA integrates Rf and Ri Alex: Standard TI LM358B or BA doesn't include resistors from what I can find. Martin: Dang, I can't find where I read that Rf and Ri at 1k were integrated to simplify application. I guess let's add some then ?"
- note added: "Vref set to 4.9V As the divider follows the supply, its less susceptible to supply variation than a fixed voltage (zener). i.e. always close to 100mV across Iset resistor."
- note removed: "Current is set as follows : - LM4040DBZ-4.1 sets voltage at 4.096V on a good day - Assuming we have 5V this makes a reference voltage of 0.904V - Reference resistence is currently 220R -> Reference current is 0.904/220 = 4.1mA approx - For fuel level and common sensors (0-250Ohm), that gives a sensor voltage of anywhere between 0 and 1.025V - Practically the maximum voltage that can be is 4.096V-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"
- note removed: "Current is set as follows : - LM4040DBZ-4.1 sets voltage at 4.096V on a good day - Assuming we have 5V this makes a reference voltage of 0.904V - Reference resistence is currently 470R -> Reference current is 0.904/470 = 1.92mA approx - For high K sensors (70-2000Ohm), that gives a sensor voltage of anywhere between 0.1344V and 3.84V - Practically the maximum voltage that can be is 4.096V-0.550V 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"
- note removed: "Ideas/issues : - How to account for variations in the Vf of PMEG3010EH - 5V may not be true 5V -> Zener regulator there too ? evaluate possible swings - Design is a bit limited to be usable on >750Ohm sensors like ECU sensors - Something better than PMEG3010EH to use ?"
- note removed: "Rf and Ri useful ? 47K, but apparently LM358B/BA integrates Rf and Ri"
