File: KiCad PCB Files/Opto_ActHi.kicad_sch (KiCad schematic)
At the start: 3 parts, among them U1 SFH617A-2X009T

Commit message: v1.0
- First PCB layout publication
- Titled schematics
- Added Revisions to Schematics and PCB
- iBOM release
- PDF export of PCB design
Other:
- title: (none) -> Active Hi Optocoupler circuit
Changed lines of the file:
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@@
 (kicad_sch (version 20230121) (generator eeschema)
   (paper "A4")
+  (title_block
+    (title "Active Hi Optocoupler circuit")
+    (date "2023-04-10")
+    (rev "1.0")
+    (comment 1 "https://github.com/martinroger/VXDash")
+    (comment 2 "https://cadlab.io/projects/vxdash")
+  )
   (junction (at 116.84 110.49) (diameter 0) (color 0 0 0 0)
   )

Commit message: PCB layout update 1.2.1
Updated with OpAmp circuitry plus some component identification
Parts:
- U1: Manufacturer_Name (none) -> Vishay; Manufacturer_Part_Number (none) -> SFH617A-2X009T
Changed lines of the file:
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@@
   (title_block
     (title "Active Hi Optocoupler circuit")
-    (date "2023-05-01")
-    (rev "1.2")
+    (date "2023-05-14")
+    (rev "1.2.1")
     (comment 1 "https://github.com/martinroger/VXDash")
     (comment 2 "https://cadlab.io/projects/vxdash")
@@
       (effects (font (size 1.27 1.27)) hide)
     )
-    (property "Datasheet" "http://www.vishay.com/docs/83740/sfh617a.pdf" (at 121.92 85.09 0)
+    (property "Datasheet" "https://www.vishay.com/docs/83740/sfh617a.pdf" (at 121.92 85.09 0)
       (effects (font (size 1.27 1.27)) hide)
     )
+    (property "Description" "OPTOISOLATOR 5.3KV TRANS 4SMD" (at 114.3 93.98 0)
+      (effects (font (size 1.27 1.27)) hide)
+    )
+    (property "Manufacturer_Name" "Vishay" (at 114.3 93.98 0)
+      (effects (font (size 1.27 1.27)) hide)
+    )
+    (property "Manufacturer_Part_Number" "SFH617A-2X009T" (at 114.3 93.98 0)
+      (effects (font (size 1.27 1.27)) hide)
+    )
