File: KiCad PCB Files/Power_Input.kicad_sch (KiCad schematic)
At the start: 16 parts, among them Q1 PJA3441, Q2 2N7002

Commit message: Added first draft of Op-amp based circuitry
Also some rationalisation of the components to avoid near-duplicates (e.g. 0.1uF 50V caps)
Parts:
- C6: value 0.1µF -> 0.1uF 50V
Changed lines of the file:
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@@
   (title_block
     (title "Power switching and protection")
-    (date "2023-04-25")
+    (date "2023-05-01")
     (rev "1.2")
     (comment 1 "https://github.com/martinroger/VXDash")
@@
       (effects (font (size 1.27 1.27)) (justify left))
     )
-    (property "Value" "0.1µF" (at 101.6 55.8801 0)
+    (property "Value" "0.1uF 50V" (at 101.6 55.8801 0)
       (effects (font (size 1.27 1.27)) (justify left))
     )
@@
       (effects (font (size 1.27 1.27)) (justify left))
     )
-    (property "Value" "0.1µF" (at 166.37 74.93 0)
+    (property "Value" "0.1uF 50V" (at 166.37 74.93 0)
       (effects (font (size 1.27 1.27)) (justify left))
     )
@@
       (effects (font (size 1.27 1.27)) (justify left))
     )
-    (property "Value" "0.1µF" (at 109.22 91.44 0)
+    (property "Value" "0.1uF 50V" (at 109.22 91.44 0)
       (effects (font (size 1.27 1.27)) (justify left))
     )
@@
       (effects (font (size 1.27 1.27)) (justify left))
     )
-    (property "Value" "0.1µF" (at 146.05 74.93 0)
-      (effects (font (size 1.27 1.27)) (justify left))
-    )
+    (property "Value" "0.1uF 50V" (at 146.05 74.93 0)
+      (effects (font (size 1.27 1.27)) (justify left))
+    )

Commit message: PCB layout update 1.2.1
Updated with OpAmp circuitry plus some component identification
Parts:
- C36: Manufacturer_Name (none) -> Taiyo Yuden; Manufacturer_Part_Number (none) -> UMK107BJ105KA-T
- R4: Manufacturer_Name (none) -> Vishay Dale
Changed lines of the file:
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@@
   (title_block
     (title "Power switching and protection")
-    (date "2023-05-01")
-    (rev "1.2")
+    (date "2023-05-14")
+    (rev "1.2.1")
     (comment 1 "https://github.com/martinroger/VXDash")
     (comment 2 "https://cadlab.io/projects/vxdash")
@@
       (effects (font (size 1.27 1.27)) hide)
     )
-    (property "Datasheet" "~" (at 153.67 48.26 0)
+    (property "Datasheet" "https://www.we-online.com/katalog/datasheet/742792023.pdf" (at 153.67 48.26 0)
       (effects (font (size 1.27 1.27)) hide)
     )
@@
     )
     (property "Manufacturer_Part_Number" "742792023" (at 153.67 48.26 0)
+      (effects (font (size 1.27 1.27)) hide)
+    )
+    (property "Description" "FERRITE BEAD 120 OHM 0805 1LN" (at 153.67 48.26 0)
       (effects (font (size 1.27 1.27)) hide)
     )
@@
       (effects (font (size 1.27 1.27)) hide)
     )
-    (property "Datasheet" "~" (at 96.52 88.9 0)
+    (property "Datasheet" "https://www.vishay.com/docs/28773/crcwce3.pdf" (at 96.52 88.9 0)
       (effects (font (size 1.27 1.27)) hide)
     )
@@
     )
     (property "Manufacturer_Part_Number" "CRCW0402100KFKEDC" (at 96.52 88.9 0)
+      (effects (font (size 1.27 1.27)) hide)
+    )
+    (property "Manufacturer_Name" "Vishay Dale" (at 96.52 88.9 0)
       (effects (font (size 1.27 1.27)) hide)
     )
@@
       (effects (font (size 1.27 1.27)) hide)
     )
-    (property "Datasheet" "~" (at 134.62 53.34 0)
+    (property "Datasheet" "https://www.mccsemi.com/pdf/Products/BZT52C2V4~BZT52C75(500mW)(SOD-123).pdf" (at 134.62 53.34 0)
       (effects (font (size 1.27 1.27)) hide)
     )
@@
     )
     (property "Manufacturer_Part_Number" "BZT52C18-TP" (at 134.62 53.34 0)
+      (effects (font (size 1.27 1.27)) hide)
+    )
+    (property "Description" "DIODE ZENER 18V 200MW SOD123" (at 134.62 53.34 0)
       (effects (font (size 1.27 1.27)) hide)
     )
@@
       (effects (font (size 1.27 1.27)) hide)
     )
-    (property "Datasheet" "~" (at 118.11 50.8 0)
+    (property "Datasheet" "https://www.panjit.com.tw/upload/datasheet/PJA3441.pdf" (at 118.11 50.8 0)
       (effects (font (size 1.27 1.27)) hide)
     )
@@
     )
     (property "Manufacturer_Part_Number" "PJA3441_R1_00001" (at 118.11 50.8 0)
+      (effects (font (size 1.27 1.27)) hide)
+    )
+    (property "Description" "P-Channel 40 V 3.1A (Ta) 1.25W (Ta) Surface Mount SOT-23" (at 118.11 50.8 0)
       (effects (font (size 1.27 1.27)) hide)
     )
@@
       (effects (font (size 1.27 1.27)) hide)
     )
-    (property "Datasheet" "~" (at 175.26 73.66 0)
+    (property "Datasheet" "https://www.yuden.co.jp/productdata/catalog/mlcc06_e.pdf" (at 175.26 73.66 0)
       (effects (font (size 1.27 1.27)) hide)
     )
@@
     )
     (property "Tolerance" "10%" (at 175.26 73.66 0)
+      (effects (font (size 1.27 1.27)) hide)
+    )
+    (property "Description" "CAP CER 1UF 50V X5R 0603" (at 175.26 73.66 0)
+      (effects (font (size 1.27 1.27)) hide)
+    )
+    (property "Manufacturer_Name" "Taiyo Yuden" (at 175.26 73.66 0)
+      (effects (font (size 1.27 1.27)) hide)
+    )
+    (property "Manufacturer_Part_Number" "UMK107BJ105KA-T" (at 175.26 73.66 0)
       (effects (font (size 1.27 1.27)) hide)
     )
@@
       (effects (font (size 1.27 1.27)) hide)
     )
-    (property "Datasheet" "~" (at 115.57 81.28 0)
+    (property "Datasheet" "https://www.mccsemi.com/pdf/Products/2N7002(SOT-23).PDF" (at 115.57 81.28 0)
       (effects (font (size 1.27 1.27)) hide)
     )
@@
     )
     (property "Manufacturer_Part_Number" "2N7002-TP" (at 115.57 81.28 0)
+      (effects (font (size 1.27 1.27)) hide)
+    )
+    (property "Description" "MOSFET N-CH 60V 115MA SOT23" (at 115.57 81.28 0)
       (effects (font (size 1.27 1.27)) hide)
     )
@@
       (effects (font (size 1.27 1.27)) hide)
     )
-    (property "Datasheet" "~" (at 91.44 88.9 0)
+    (property "Datasheet" "https://www.mccsemi.com/pdf/Products/BZT52C2V4~BZT52C75(500mW)(SOD-123).pdf" (at 91.44 88.9 0)
       (effects (font (size 1.27 1.27)) hide)
     )
@@
     )
     (property "Manufacturer_Part_Number" "BZT52C18-TP" (at 91.44 88.9 0)
+      (effects (font (size 1.27 1.27)) hide)
+    )
+    (property "Description" "DIODE ZENER 18V 200MW SOD123" (at 91.44 88.9 0)
       (effects (font (size 1.27 1.27)) hide)
     )
@@
       (effects (font (size 1.27 1.27)) hide)
     )
-    (property "Datasheet" "~" (at 125.73 53.34 0)
+    (property "Datasheet" "https://www.vishay.com/docs/28773/crcwce3.pdf" (at 125.73 53.34 0)
       (effects (font (size 1.27 1.27)) hide)
     )
@@
     )
     (property "Manufacturer_Part_Number" "CRCW0402100KFKEDC" (at 125.73 53.34 0)
+      (effects (font (size 1.27 1.27)) hide)
+    )
+    (property "Manufacturer_Name" "Vishay Dale" (at 125.73 53.34 0)
       (effects (font (size 1.27 1.27)) hide)
     )
@@
       (effects (font (size 1.27 1.27)) (justify left) hide)
     )
-    (property "Datasheet" "~" (at 82.55 48.26 0)
+    (property "Datasheet" "https://www.belfuse.com/resources/datasheets/circuitprotection/ds-cp-0zrb-series.pdf" (at 82.55 48.26 0)
       (effects (font (size 1.27 1.27)) hide)
     )
@@
     )
     (property "Manufacturer_Part_Number" "0ZRB0250FF1E" (at 82.55 48.26 0)
+      (effects (font (size 1.27 1.27)) hide)
+    )
+    (property "Description" "PTC RESET FUSE 30V 2.5A RADIAL" (at 82.55 48.26 0)
       (effects (font (size 1.27 1.27)) hide)
     )
@@
       (effects (font (size 1.27 1.27)) hide)
     )
-    (property "Datasheet" "~" (at 91.44 55.88 0)
+    (property "Datasheet" "https://www.bourns.com/docs/Product-Datasheets/MOV07D.pdf" (at 91.44 55.88 0)
       (effects (font (size 1.27 1.27)) hide)
     )
@@
       (effects (font (size 1.27 1.27)) hide)
     )
+    (property "Description" "VARISTOR 22V 250A DISC 7MM" (at 91.44 55.88 0)
+      (effects (font (size 1.27 1.27)) hide)
+    )
