File: KiCad PCB Files/R_bank.kicad_sch (KiCad schematic)
At the start: 14 parts, among them SW1 SW_DIP_x12

Commit message: General update
- Mosfet for OP AMP circuits
- Components all have PNs now
- Externalised Rset
Parts:
- R58, R59, R61, R70, R71, R79, R80, R81, R82, R83, R84, R85: Manufacturer_Name (none) -> Yageo; Manufacturer_Part_Number (none) -> RC0603FR-07270RL
Changed lines of the file:
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@@
       (effects (font (size 1.27 1.27)) hide)
     )
-    (property "Datasheet" "~" (at 125.73 139.7 0)
+    (property "Datasheet" "https://www.yageo.com/upload/media/product/productsearch/datasheet/rchip/PYu-RC_Group_51_RoHS_L_12.pdf" (at 125.73 139.7 0)
+      (effects (font (size 1.27 1.27)) hide)
+    )
+    (property "Description" "RES 270 OHM 1% 1/10W 0603" (at 125.73 139.7 0)
+      (effects (font (size 1.27 1.27)) hide)
+    )
+    (property "Manufacturer_Name" "Yageo" (at 125.73 139.7 0)
+      (effects (font (size 1.27 1.27)) hide)
+    )
+    (property "Manufacturer_Part_Number" "RC0603FR-07270RL" (at 125.73 139.7 0)
       (effects (font (size 1.27 1.27)) hide)
     )
@@
       (effects (font (size 1.27 1.27)) hide)
     )
-    (property "Datasheet" "~" (at 125.73 101.6 0)
+    (property "Datasheet" "https://www.yageo.com/upload/media/product/productsearch/datasheet/rchip/PYu-RC_Group_51_RoHS_L_12.pdf" (at 125.73 101.6 0)
+      (effects (font (size 1.27 1.27)) hide)
+    )
+    (property "Description" "RES 270 OHM 1% 1/10W 0603" (at 125.73 101.6 0)
+      (effects (font (size 1.27 1.27)) hide)
+    )
+    (property "Manufacturer_Name" "Yageo" (at 125.73 101.6 0)
+      (effects (font (size 1.27 1.27)) hide)
+    )
+    (property "Manufacturer_Part_Number" "RC0603FR-07270RL" (at 125.73 101.6 0)
       (effects (font (size 1.27 1.27)) hide)
     )
@@
       (effects (font (size 1.27 1.27)) hide)
     )
-    (property "Datasheet" "~" (at 125.73 93.98 0)
+    (property "Datasheet" "https://www.yageo.com/upload/media/product/productsearch/datasheet/rchip/PYu-RC_Group_51_RoHS_L_12.pdf" (at 125.73 93.98 0)
+      (effects (font (size 1.27 1.27)) hide)
+    )
+    (property "Description" "RES 270 OHM 1% 1/10W 0603" (at 125.73 93.98 0)
+      (effects (font (size 1.27 1.27)) hide)
+    )
+    (property "Manufacturer_Name" "Yageo" (at 125.73 93.98 0)
+      (effects (font (size 1.27 1.27)) hide)
+    )
+    (property "Manufacturer_Part_Number" "RC0603FR-07270RL" (at 125.73 93.98 0)
       (effects (font (size 1.27 1.27)) hide)
     )
@@
       (effects (font (size 1.27 1.27)) hide)
     )
-    (property "Datasheet" "~" (at 125.73 86.36 0)
+    (property "Datasheet" "https://www.yageo.com/upload/media/product/productsearch/datasheet/rchip/PYu-RC_Group_51_RoHS_L_12.pdf" (at 125.73 86.36 0)
+      (effects (font (size 1.27 1.27)) hide)
+    )
+    (property "Description" "RES 270 OHM 1% 1/10W 0603" (at 125.73 86.36 0)
+      (effects (font (size 1.27 1.27)) hide)
+    )
+    (property "Manufacturer_Name" "Yageo" (at 125.73 86.36 0)
+      (effects (font (size 1.27 1.27)) hide)
+    )
+    (property "Manufacturer_Part_Number" "RC0603FR-07270RL" (at 125.73 86.36 0)
       (effects (font (size 1.27 1.27)) hide)
     )
@@
       (effects (font (size 1.27 1.27)) hide)
     )
-    (property "Datasheet" "~" (at 125.73 124.46 0)
+    (property "Datasheet" "https://www.yageo.com/upload/media/product/productsearch/datasheet/rchip/PYu-RC_Group_51_RoHS_L_12.pdf" (at 125.73 124.46 0)
+      (effects (font (size 1.27 1.27)) hide)
+    )
+    (property "Description" "RES 270 OHM 1% 1/10W 0603" (at 125.73 124.46 0)
+      (effects (font (size 1.27 1.27)) hide)
+    )
+    (property "Manufacturer_Name" "Yageo" (at 125.73 124.46 0)
+      (effects (font (size 1.27 1.27)) hide)
+    )
+    (property "Manufacturer_Part_Number" "RC0603FR-07270RL" (at 125.73 124.46 0)
       (effects (font (size 1.27 1.27)) hide)
     )
@@
       (effects (font (size 1.27 1.27)) hide)
     )
-    (property "Datasheet" "~" (at 125.73 147.32 0)
+    (property "Datasheet" "https://www.yageo.com/upload/media/product/productsearch/datasheet/rchip/PYu-RC_Group_51_RoHS_L_12.pdf" (at 125.73 147.32 0)
+      (effects (font (size 1.27 1.27)) hide)
+    )
+    (property "Description" "RES 270 OHM 1% 1/10W 0603" (at 125.73 147.32 0)
+      (effects (font (size 1.27 1.27)) hide)
+    )
+    (property "Manufacturer_Name" "Yageo" (at 125.73 147.32 0)
+      (effects (font (size 1.27 1.27)) hide)
+    )
+    (property "Manufacturer_Part_Number" "RC0603FR-07270RL" (at 125.73 147.32 0)
       (effects (font (size 1.27 1.27)) hide)
     )
@@
       (effects (font (size 1.27 1.27)) hide)
     )
-    (property "Datasheet" "~" (at 125.73 78.74 0)
+    (property "Datasheet" "https://www.yageo.com/upload/media/product/productsearch/datasheet/rchip/PYu-RC_Group_51_RoHS_L_12.pdf" (at 125.73 78.74 0)
+      (effects (font (size 1.27 1.27)) hide)
+    )
+    (property "Description" "RES 270 OHM 1% 1/10W 0603" (at 125.73 78.74 0)
+      (effects (font (size 1.27 1.27)) hide)
+    )
+    (property "Manufacturer_Name" "Yageo" (at 125.73 78.74 0)
+      (effects (font (size 1.27 1.27)) hide)
+    )
+    (property "Manufacturer_Part_Number" "RC0603FR-07270RL" (at 125.73 78.74 0)
       (effects (font (size 1.27 1.27)) hide)
     )
@@
       (effects (font (size 1.27 1.27)) hide)
     )
-    (property "Datasheet" "~" (at 125.73 154.94 0)
+    (property "Datasheet" "https://www.yageo.com/upload/media/product/productsearch/datasheet/rchip/PYu-RC_Group_51_RoHS_L_12.pdf" (at 125.73 154.94 0)
+      (effects (font (size 1.27 1.27)) hide)
+    )
+    (property "Description" "RES 270 OHM 1% 1/10W 0603" (at 125.73 154.94 0)
+      (effects (font (size 1.27 1.27)) hide)
+    )
+    (property "Manufacturer_Name" "Yageo" (at 125.73 154.94 0)
+      (effects (font (size 1.27 1.27)) hide)
+    )
+    (property "Manufacturer_Part_Number" "RC0603FR-07270RL" (at 125.73 154.94 0)
       (effects (font (size 1.27 1.27)) hide)
     )
@@
       (effects (font (size 1.27 1.27)) hide)
     )
-    (property "Datasheet" "~" (at 125.73 132.08 0)
+    (property "Datasheet" "https://www.yageo.com/upload/media/product/productsearch/datasheet/rchip/PYu-RC_Group_51_RoHS_L_12.pdf" (at 125.73 132.08 0)
+      (effects (font (size 1.27 1.27)) hide)
+    )
+    (property "Description" "RES 270 OHM 1% 1/10W 0603" (at 125.73 132.08 0)
+      (effects (font (size 1.27 1.27)) hide)
+    )
+    (property "Manufacturer_Name" "Yageo" (at 125.73 132.08 0)
+      (effects (font (size 1.27 1.27)) hide)
+    )
+    (property "Manufacturer_Part_Number" "RC0603FR-07270RL" (at 125.73 132.08 0)
       (effects (font (size 1.27 1.27)) hide)
     )
@@
       (effects (font (size 1.27 1.27)) hide)
     )
-    (property "Datasheet" "~" (at 125.73 109.22 0)
+    (property "Datasheet" "https://www.yageo.com/upload/media/product/productsearch/datasheet/rchip/PYu-RC_Group_51_RoHS_L_12.pdf" (at 125.73 109.22 0)
+      (effects (font (size 1.27 1.27)) hide)
+    )
+    (property "Description" "RES 270 OHM 1% 1/10W 0603" (at 125.73 109.22 0)
+      (effects (font (size 1.27 1.27)) hide)
+    )
+    (property "Manufacturer_Name" "Yageo" (at 125.73 109.22 0)
+      (effects (font (size 1.27 1.27)) hide)
+    )
+    (property "Manufacturer_Part_Number" "RC0603FR-07270RL" (at 125.73 109.22 0)
       (effects (font (size 1.27 1.27)) hide)
     )
@@
       (effects (font (size 1.27 1.27)) hide)
     )
-    (property "Datasheet" "~" (at 125.73 71.12 0)
+    (property "Datasheet" "https://www.yageo.com/upload/media/product/productsearch/datasheet/rchip/PYu-RC_Group_51_RoHS_L_12.pdf" (at 125.73 71.12 0)
+      (effects (font (size 1.27 1.27)) hide)
+    )
+    (property "Description" "RES 270 OHM 1% 1/10W 0603" (at 125.73 71.12 0)
+      (effects (font (size 1.27 1.27)) hide)
+    )
+    (property "Manufacturer_Name" "Yageo" (at 125.73 71.12 0)
+      (effects (font (size 1.27 1.27)) hide)
+    )
+    (property "Manufacturer_Part_Number" "RC0603FR-07270RL" (at 125.73 71.12 0)
       (effects (font (size 1.27 1.27)) hide)
     )
@@
       (effects (font (size 1.27 1.27)) hide)
     )
-    (property "Datasheet" "~" (at 125.73 116.84 0)
-      (effects (font (size 1.27 1.27)) hide)
-    )
+    (property "Datasheet" "https://www.yageo.com/upload/media/product/productsearch/datasheet/rchip/PYu-RC_Group_51_RoHS_L_12.pdf" (at 125.73 116.84 0)
+      (effects (font (size 1.27 1.27)) hide)
+    )
+    (property "Description" "RES 270 OHM 1% 1/10W 0603" (at 125.73 116.84 0)
+      (effects (font (size 1.27 1.27)) hide)
+    )
+    (property "Manufacturer_Name" "Yageo" (at 125.73 116.84 0)
+      (effects (font (size 1.27 1.27)) hide)
+    )
+    (property "Manufacturer_Part_Number" "RC0603FR-07270RL" (at 125.73 116.84 0)
+      (effects (font (size 1.27 1.27)) hide)
+    )

Commit message: v1.2.3
- Removed one 270R resistor otherwise the pots serve no purpose
- Added some silkscreen references
- Regenerated PDFs
Parts:
- R85: now not fitted; now left out of the parts list
Changed lines of the file:
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@@
   (title_block
     (title "270R divider")
-    (date "2023-05-14")
-    (rev "1.2.2")
+    (date "2023-06-18")
+    (rev "1.2.3")
     (comment 1 "https://github.com/martinroger/VXDash")
     (comment 2 "https://cadlab.io/projects/vxdash")
@@
   )
   (symbol (lib_id "Device:R") (at 125.73 154.94 90) (unit 1)
-    (in_bom yes) (on_board yes) (dnp no) (fields_autoplaced)
+    (in_bom no) (on_board yes) (dnp yes) (fields_autoplaced)
     (property "Reference" "R85" (at 125.73 149.86 90)
       (effects (font (size 1.27 1.27)))
