File: KiCad PCB Files/3V3_SMPS.kicad_sch (KiCad schematic)
At the start: 13 parts, among them IC4 AP62200

Commit message: Schematic pre-review
WIP - final TODOs needed before review
Connections:
- net 12V_IN renamed 12V_in
- net 3V3_OUT renamed 3V3_out
Changed lines of the file:
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@@
 		(title "5 to 3V3 stage")
 		(date "2025-07-19")
-		(rev "1.3.1")
+		(rev "1.4")
 		(comment 1 "https://github.com/martinroger/VXDash")
 		(comment 2 "https://cadlab.io/projects/vxdash")
@@
 		)
 	)
-	(hierarchical_label "3V3_OUT"
+	(hierarchical_label "3V3_out"
 		(shape output)
 		(at 207.01 60.96 0)
@@
 		)
 	)
-	(hierarchical_label "12V_IN"
+	(hierarchical_label "12V_in"
 		(shape input)
 		(at 76.2 55.88 180)
@@
 			)
 		)
-		(property "Description" "Ceremic capacitor"
+		(property "Description" ""
 			(at 168.91 66.04 0)
 			(effects
@@
 			)
 		)
-		(property "Description" "Resistor"
+		(property "Description" ""
 			(at 160.02 77.47 0)
 			(effects
@@
 			)
 		)
-		(property "Description" "Ceremic capacitor"
+		(property "Description" ""
 			(at 99.06 62.23 0)
 			(effects
@@
 			)
 		)
-		(property "Description" "Resistor"
+		(property "Description" ""
 			(at 160.02 66.04 0)
 			(effects
@@
 			)
 		)
-		(property "Description" "Resistor"
+		(property "Description" ""
 			(at 88.9 63.5 0)
 			(effects
@@
 			)
 		)
-		(property "Description" "Ceremic capacitor"
+		(property "Description" ""
 			(at 200.66 66.04 0)
 			(effects
@@
 			)
 		)
-		(property "Description" "Ceremic capacitor"
+		(property "Description" ""
 			(at 193.04 66.04 0)
 			(effects
@@
 			)
 		)
-		(property "Description" "Inductor"
+		(property "Description" ""
 			(at 153.67 63.5 0)
 			(effects
@@
 			)
 		)
-		(property "Description" "Resistor"
+		(property "Description" ""
 			(at 88.9 76.2 0)
 			(effects
@@
 			)
 		)
-		(property "Description" "Ceremic capacitor"
+		(property "Description" ""
 			(at 106.68 62.23 0)
 			(effects
@@
 			)
 		)
-		(property "Description" "Ceremic capacitor"
+		(property "Description" ""
 			(at 140.97 55.88 0)
 			(effects
@@
 			)
 		)
-		(property "Description" "Ceremic capacitor"
+		(property "Description" ""
 			(at 185.42 66.04 0)
 			(effects
