File: KiCad PCB Files/5V_SMPS.kicad_sch (KiCad schematic)
At the start: 13 parts, among them IC8 AP62200

Commit message: Schematic pre-review
WIP - final TODOs needed before review
Connections:
- net 12V_EN renamed 5V_en
- net 12V_IN renamed 12V_in
- net 5V_OUT renamed 5V_out
Changed lines of the file:
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@@
 		(title "12V to 5V conversion")
 		(date "2025-07-19")
-		(rev "1.3.1")
+		(rev "1.4")
 		(comment 1 "https://github.com/martinroger/VXDash")
 		(comment 2 "https://cadlab.io/projects/vxdash")
@@
 		)
 	)
-	(hierarchical_label "12V_IN"
+	(hierarchical_label "12V_in"
 		(shape input)
 		(at 67.31 76.2 180)
@@
 		)
 	)
-	(hierarchical_label "5V_OUT"
+	(hierarchical_label "5V_out"
 		(shape output)
 		(at 195.58 81.28 0)
@@
 		)
 	)
-	(hierarchical_label "12V_EN"
+	(hierarchical_label "5V_en"
 		(shape input)
 		(at 67.31 91.44 180)
@@
 		(dnp no)
 		(fields_autoplaced yes)
-		(property "Reference" "#PWR012"
+		(property "Reference" "#PWR"
 			(at 113.03 114.3 0)
 			(effects
@@
 		)
 		(instances
-			(project ""
-				(path "/f2858fc4-50de-4ff0-a01c-5b985ee14aef/08acef39-2886-400a-86d2-7f8ed30d55fe"
+			(project "VXDash"
+				(path "/f2858fc4-50de-4ff0-a01c-5b985ee14aef/1e710dfa-ec27-4a4d-bb24-4bffb525a2be"
 					(reference "#PWR013")
-					(unit 1)
-				)
-				(path "/f2858fc4-50de-4ff0-a01c-5b985ee14aef/e4c69d46-7a64-435d-9e3a-d73acbe7ec2b"
-					(reference "#PWR012")
 					(unit 1)
 				)
@@
 			)
 		)
-		(property "Description" "Ceremic capacitor"
+		(property "Description" ""
 			(at 157.48 86.36 0)
 			(effects
@@
 		(instances
 			(project "VXDash"
-				(path "/f2858fc4-50de-4ff0-a01c-5b985ee14aef/08acef39-2886-400a-86d2-7f8ed30d55fe"
+				(path "/f2858fc4-50de-4ff0-a01c-5b985ee14aef/1e710dfa-ec27-4a4d-bb24-4bffb525a2be"
 					(reference "C28")
 					(unit 1)
@@
 			)
 		)
-		(property "Description" "Ceremic capacitor"
+		(property "Description" ""
 			(at 90.17 82.55 0)
 			(effects
@@
 		(instances
 			(project "VXDash"
-				(path "/f2858fc4-50de-4ff0-a01c-5b985ee14aef/08acef39-2886-400a-86d2-7f8ed30d55fe"
+				(path "/f2858fc4-50de-4ff0-a01c-5b985ee14aef/1e710dfa-ec27-4a4d-bb24-4bffb525a2be"
 					(reference "C23")
 					(unit 1)
@@
 			)
 		)
-		(property "Description" "Ceremic capacitor"
+		(property "Description" ""
 			(at 189.23 86.36 0)
 			(effects
@@
 		(instances
 			(project "VXDash"
-				(path "/f2858fc4-50de-4ff0-a01c-5b985ee14aef/08acef39-2886-400a-86d2-7f8ed30d55fe"
-					(reference "C58")
+				(path "/f2858fc4-50de-4ff0-a01c-5b985ee14aef/1e710dfa-ec27-4a4d-bb24-4bffb525a2be"
+					(reference "C50")
 					(unit 1)
 				)
@@
 			)
 		)
-		(property "Description" "Ceremic capacitor"
+		(property "Description" ""
 			(at 181.61 86.36 0)
 			(effects
@@
 		(instances
 			(project "VXDash"
-				(path "/f2858fc4-50de-4ff0-a01c-5b985ee14aef/08acef39-2886-400a-86d2-7f8ed30d55fe"
+				(path "/f2858fc4-50de-4ff0-a01c-5b985ee14aef/1e710dfa-ec27-4a4d-bb24-4bffb525a2be"
 					(reference "C32")
 					(unit 1)
@@
 		(instances
 			(project "VXDash"
-				(path "/f2858fc4-50de-4ff0-a01c-5b985ee14aef/08acef39-2886-400a-86d2-7f8ed30d55fe"
-					(reference "IC9")
+				(path "/f2858fc4-50de-4ff0-a01c-5b985ee14aef/1e710dfa-ec27-4a4d-bb24-4bffb525a2be"
+					(reference "IC7")
 					(unit 1)
 				)
@@
 			)
 		)
-		(property "Datasheet" "~"
+		(property "Datasheet" ""
 			(at 74.93 91.44 0)
 			(effects
@@
 			)
 		)
-		(property "Description" "Resistor"
+		(property "Description" ""
 			(at 74.93 91.44 0)
 			(effects
@@
 		(instances
 			(project "VXDash"
-				(path "/f2858fc4-50de-4ff0-a01c-5b985ee14aef/08acef39-2886-400a-86d2-7f8ed30d55fe"
+				(path "/f2858fc4-50de-4ff0-a01c-5b985ee14aef/1e710dfa-ec27-4a4d-bb24-4bffb525a2be"
 					(reference "R79")
 					(unit 1)
@@
 			)
 		)
-		(property "Description" "Inductor"
+		(property "Description" ""
 			(at 142.24 83.82 0)
 			(effects
@@
 		(instances
 			(project "VXDash"
-				(path "/f2858fc4-50de-4ff0-a01c-5b985ee14aef/08acef39-2886-400a-86d2-7f8ed30d55fe"
+				(path "/f2858fc4-50de-4ff0-a01c-5b985ee14aef/1e710dfa-ec27-4a4d-bb24-4bffb525a2be"
 					(reference "L3")
 					(unit 1)
@@
 			)
 		)
-		(property "Description" "Ceremic capacitor"
+		(property "Description" ""
 			(at 129.54 76.2 0)
 			(effects
@@
 		(instances
 			(project "VXDash"
-				(path "/f2858fc4-50de-4ff0-a01c-5b985ee14aef/08acef39-2886-400a-86d2-7f8ed30d55fe"
+				(path "/f2858fc4-50de-4ff0-a01c-5b985ee14aef/1e710dfa-ec27-4a4d-bb24-4bffb525a2be"
 					(reference "C26")
 					(unit 1)
@@
 			)
 		)
-		(property "Description" "Ceremic capacitor"
+		(property "Description" ""
 			(at 173.99 86.36 0)
 			(effects
@@
 		(instances
 			(project "VXDash"
-				(path "/f2858fc4-50de-4ff0-a01c-5b985ee14aef/08acef39-2886-400a-86d2-7f8ed30d55fe"
+				(path "/f2858fc4-50de-4ff0-a01c-5b985ee14aef/1e710dfa-ec27-4a4d-bb24-4bffb525a2be"
 					(reference "C30")
 					(unit 1)
@@
 			)
 		)
-		(property "Description" "Resistor"
+		(property "Description" ""
 			(at 148.59 97.79 0)
 			(effects
@@
 		(instances
 			(project "VXDash"
-				(path "/f2858fc4-50de-4ff0-a01c-5b985ee14aef/08acef39-2886-400a-86d2-7f8ed30d55fe"
+				(path "/f2858fc4-50de-4ff0-a01c-5b985ee14aef/1e710dfa-ec27-4a4d-bb24-4bffb525a2be"
 					(reference "R82")
 					(unit 1)
@@
 			)
 		)
-		(property "Description" "Ceremic capacitor"
+		(property "Description" ""
 			(at 82.55 82.55 0)
 			(effects
@@
 		(instances
 			(project "VXDash"
-				(path "/f2858fc4-50de-4ff0-a01c-5b985ee14aef/08acef39-2886-400a-86d2-7f8ed30d55fe"
+				(path "/f2858fc4-50de-4ff0-a01c-5b985ee14aef/1e710dfa-ec27-4a4d-bb24-4bffb525a2be"
 					(reference "C22")
 					(unit 1)
@@
 			)
 		)
-		(property "Description" "Resistor"
+		(property "Description" ""
 			(at 100.33 96.52 0)
 			(effects
@@
 		(instances
 			(project "VXDash"
-				(path "/f2858fc4-50de-4ff0-a01c-5b985ee14aef/08acef39-2886-400a-86d2-7f8ed30d55fe"
+				(path "/f2858fc4-50de-4ff0-a01c-5b985ee14aef/1e710dfa-ec27-4a4d-bb24-4bffb525a2be"
 					(reference "R80")
 					(unit 1)
@@
 			)
 		)
-		(property "Description" "Resistor"
+		(property "Description" ""
 			(at 148.59 86.36 0)
 			(effects
@@
 		(instances
 			(project "VXDash"
-				(path "/f2858fc4-50de-4ff0-a01c-5b985ee14aef/08acef39-2886-400a-86d2-7f8ed30d55fe"
+				(path "/f2858fc4-50de-4ff0-a01c-5b985ee14aef/1e710dfa-ec27-4a4d-bb24-4bffb525a2be"
 					(reference "R81")
 					(unit 1)
