File: KiCad PCB Files/Rsensing_Pair.kicad_sch (KiCad schematic)
At the start: 13 parts, among them IC5 AD8542ARMZ-REEL, Q7 DMG2301L, Q8 DMG2301L

Commit message: Using calibratred AnalogReadMilliVolts
Parts:
- added C6 (x2): 0.1uF 50V, Capacitor_SMD:C_0603_1608Metric, symbol Device:C_Small
Connections:
- net Analog_OUT_1: now also C6.1
- net Analog_OUT_2: now also C6.2
- net GND: now also C6.1, C6.2
Other:
- note removed: "Rf and Ri useful ? 47K, but apparently LM358B/BA integrates Rf and Ri Alex: Standard TI LM358B or BA doesn't include resistors from what I can find. Martin: Dang, I can't find where I read that Rf and Ri at 1k were integrated to simplify application. I guess let's add some then ?"
Changed lines of the file:
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@@
   (junction (at 113.03 90.17) (diameter 0) (color 0 0 0 0)
   )
+  (junction (at 151.13 100.33) (diameter 0) (color 0 0 0 0)
+  )
   (junction (at 139.7 100.33) (diameter 0) (color 0 0 0 0)
   )
@@
   (junction (at 82.55 135.89) (diameter 0) (color 0 0 0 0)
   )
+  (junction (at 139.7 90.17) (diameter 0) (color 0 0 0 0)
+  )
   (junction (at 53.34 96.52) (diameter 0) (color 0 0 0 0)
   )
   (junction (at 24.13 110.49) (diameter 0) (color 0 0 0 0)
   )
+  (junction (at 139.7 153.67) (diameter 0) (color 0 0 0 0)
+  )
   (junction (at 113.03 100.33) (diameter 0) (color 0 0 0 0)
   )
+  (junction (at 151.13 146.05) (diameter 0) (color 0 0 0 0)
+  )
   (junction (at 34.29 96.52) (diameter 0) (color 0 0 0 0)
   )
@@
     (stroke (width 0) (type default))
   )
+  (wire (pts (xy 151.13 153.67) (xy 151.13 146.05))
+    (stroke (width 0) (type default))
+  )
   (wire (pts (xy 113.03 146.05) (xy 113.03 144.78))
     (stroke (width 0) (type default))
@@
     (stroke (width 0) (type default))
   )
-  (wire (pts (xy 139.7 146.05) (xy 139.7 152.4))
+  (wire (pts (xy 139.7 146.05) (xy 139.7 153.67))
     (stroke (width 0) (type default))
   )
@@
     (stroke (width 0) (type default))
   )
+  (wire (pts (xy 151.13 90.17) (xy 151.13 100.33))
+    (stroke (width 0) (type default))
+  )
+  (wire (pts (xy 139.7 90.17) (xy 143.51 90.17))
+    (stroke (width 0) (type default))
+  )
   (wire (pts (xy 24.13 110.49) (xy 34.29 110.49))
     (stroke (width 0) (type default))
@@
     (stroke (width 0) (type default))
   )
-  (wire (pts (xy 139.7 93.98) (xy 139.7 100.33))
+  (wire (pts (xy 139.7 83.82) (xy 139.7 90.17))
     (stroke (width 0) (type default))
   )
@@
     (stroke (width 0) (type default))
   )
+  (wire (pts (xy 139.7 90.17) (xy 139.7 100.33))
+    (stroke (width 0) (type default))
+  )
   (wire (pts (xy 72.39 90.17) (xy 113.03 90.17))
     (stroke (width 0) (type default))
   )
+  (wire (pts (xy 148.59 153.67) (xy 151.13 153.67))
+    (stroke (width 0) (type default))
+  )
   (wire (pts (xy 67.31 142.24) (xy 53.34 142.24))
     (stroke (width 0) (type default))
@@
     (stroke (width 0) (type default))
   )
+  (wire (pts (xy 139.7 153.67) (xy 143.51 153.67))
+    (stroke (width 0) (type default))
+  )
   (wire (pts (xy 74.93 95.25) (xy 105.41 95.25))
     (stroke (width 0) (type default))
@@
     (stroke (width 0) (type default))
   )
+  (wire (pts (xy 139.7 153.67) (xy 139.7 162.56))
+    (stroke (width 0) (type default))
+  )
   (wire (pts (xy 24.13 80.01) (xy 24.13 83.82))
     (stroke (width 0) (type default))
@@
   )
   (wire (pts (xy 34.29 96.52) (xy 34.29 100.33))
+    (stroke (width 0) (type default))
+  )
+  (wire (pts (xy 148.59 90.17) (xy 151.13 90.17))
     (stroke (width 0) (type default))
   )
@@
     (effects (font (size 1.27 1.27)) (justify left bottom))
   )
-  (text "Rf and Ri useful ? 47K, but apparently LM358B/BA integrates Rf and Ri\nAlex: Standard TI LM358B or BA doesn't include resistors from what I can find.\nMartin: Dang, I can't find where I read that Rf and Ri at 1k were integrated to simplify application. \nI guess let's add some then ?"
-    (at 154.94 88.9 0)
-    (effects (font (size 1.27 1.27)) (justify left bottom))
-  )
   (global_label "CONV_5V+" (shape bidirectional) (at 87.63 135.89 0) (fields_autoplaced)
     (effects (font (size 1.27 1.27)) (justify left))
@@
     (effects (font (size 1.27 1.27)) (justify left))
   )
-  (hierarchical_label "Analog_OUT_1" (shape output) (at 139.7 93.98 90) (fields_autoplaced)
+  (hierarchical_label "Analog_OUT_1" (shape output) (at 139.7 83.82 90) (fields_autoplaced)
     (effects (font (size 1.27 1.27)) (justify left))
   )
-  (hierarchical_label "Analog_OUT_2" (shape output) (at 139.7 152.4 270) (fields_autoplaced)
+  (hierarchical_label "Analog_OUT_2" (shape output) (at 139.7 162.56 270) (fields_autoplaced)
     (effects (font (size 1.27 1.27)) (justify right))
   )
@@
     )
   )
+  (symbol (lib_id "Device:C_Small") (at 146.05 153.67 270) (unit 1)
+    (in_bom yes) (on_board yes) (dnp no)
+    (property "Reference" "C6" (at 147.3201 157.48 0)
+      (effects (font (size 1.27 1.27)) (justify left))
+    )
+    (property "Value" "0.1uF 50V" (at 144.7801 157.48 0)
+      (effects (font (size 1.27 1.27)) (justify left))
+    )
+    (property "Footprint" "Capacitor_SMD:C_0603_1608Metric" (at 142.24 154.6352 0)
+      (effects (font (size 1.27 1.27)) hide)
+    )
+    (property "Datasheet" "https://media.digikey.com/pdf/Data%20Sheets/Samsung%20PDFs/CL10B104KB8NNWC_Spec.pdf" (at 146.05 153.67 0)
+      (effects (font (size 1.27 1.27)) hide)
+    )
+    (property "Manufacturer_Part_Number" "CL10B104KB8NNWC" (at 146.05 153.67 0)
+      (effects (font (size 1.27 1.27)) hide)
+    )
+    (property "Manufacturer_Name" "Samsung" (at 146.05 153.67 0)
+      (effects (font (size 1.27 1.27)) hide)
+    )
+    (property "Description" "CAP CER 0.1UF 50V X7R 0603" (at 146.05 153.67 0)
+      (effects (font (size 1.27 1.27)) hide)
+    )
+    (pin "1")
+    (pin "2")
+    (instances
+      (project "DashSpy"
+        (path "/215a03d8-0cac-4df9-aae9-9174d39cedfe"
+          (reference "C6") (unit 1)
+        )
+      )
+      (project "VXDash"
+        (path "/f2858fc4-50de-4ff0-a01c-5b985ee14aef"
+          (reference "C1") (unit 1)
+        )
+        (path "/f2858fc4-50de-4ff0-a01c-5b985ee14aef/d1068bfa-7fca-483b-992f-259828068143"
+          (reference "C45") (unit 1)
+        )
+        (path "/f2858fc4-50de-4ff0-a01c-5b985ee14aef/ab8a9460-71cd-4862-ab5b-7fd199f4cc91"
+          (reference "C46") (unit 1)
+        )
+        (path "/f2858fc4-50de-4ff0-a01c-5b985ee14aef/326d91f1-1d34-43d4-aac6-11bd9692edf0"
+          (reference "C47") (unit 1)
+        )
+      )
+    )
+  )
   (symbol (lib_id "Device:R") (at 134.62 100.33 90) (unit 1)
     (in_bom yes) (on_board yes) (dnp no) (fields_autoplaced)
@@
         )
       )
+    )
+  )
+  (symbol (lib_id "Device:C_Small") (at 146.05 90.17 90) (unit 1)
+    (in_bom yes) (on_board yes) (dnp no)
+    (property "Reference" "C6" (at 144.7799 86.36 0)
+      (effects (font (size 1.27 1.27)) (justify left))
+    )
+    (property "Value" "0.1uF 50V" (at 147.3199 86.36 0)
+      (effects (font (size 1.27 1.27)) (justify left))
+    )
+    (property "Footprint" "Capacitor_SMD:C_0603_1608Metric" (at 149.86 89.2048 0)
+      (effects (font (size 1.27 1.27)) hide)
+    )
+    (property "Datasheet" "https://media.digikey.com/pdf/Data%20Sheets/Samsung%20PDFs/CL10B104KB8NNWC_Spec.pdf" (at 146.05 90.17 0)
+      (effects (font (size 1.27 1.27)) hide)
+    )
+    (property "Manufacturer_Part_Number" "CL10B104KB8NNWC" (at 146.05 90.17 0)
+      (effects (font (size 1.27 1.27)) hide)
+    )
+    (property "Manufacturer_Name" "Samsung" (at 146.05 90.17 0)
+      (effects (font (size 1.27 1.27)) hide)
+    )
+    (property "Description" "CAP CER 0.1UF 50V X7R 0603" (at 146.05 90.17 0)
+      (effects (font (size 1.27 1.27)) hide)
+    )
+    (pin "1")
+    (pin "2")
+    (instances
+      (project "DashSpy"
+        (path "/215a03d8-0cac-4df9-aae9-9174d39cedfe"
+          (reference "C6") (unit 1)
+        )
+      )
+      (project "VXDash"
+        (path "/f2858fc4-50de-4ff0-a01c-5b985ee14aef"
+          (reference "C1") (unit 1)
+        )
+        (path "/f2858fc4-50de-4ff0-a01c-5b985ee14aef/d1068bfa-7fca-483b-992f-259828068143"
+          (reference "C24") (unit 1)
+        )
+        (path "/f2858fc4-50de-4ff0-a01c-5b985ee14aef/ab8a9460-71cd-4862-ab5b-7fd199f4cc91"
+          (reference "C43") (unit 1)
+        )
+        (path "/f2858fc4-50de-4ff0-a01c-5b985ee14aef/326d91f1-1d34-43d4-aac6-11bd9692edf0"
+          (reference "C44") (unit 1)
+        )
+      )

Commit message: 1.3.1 Decoupling capacitors on the ADC inputs
Parts:
- removed C6 (x2): 0.1uF 50V, Capacitor_SMD:C_0603_1608Metric, symbol Device:C_Small

Commit message: Continuing migration
Parts:
- IC6: renamed from IC5; footprint SOP65P490X110-8N -> DIY:SOP65P490X110-8N; symbol SamacSys_Parts:AD8542ARMZ-REEL -> DIY:AD8542ARMZ-REEL
- Q3: renamed from Q7; symbol Device:Q_PMOS_GSD -> Transistor_FET:Q_PMOS_GSD
- Q4: renamed from Q8; symbol Device:Q_PMOS_GSD -> Transistor_FET:Q_PMOS_GSD
- renumbered C6 to C14, C6 to C40, D2 to D3, D9 to D4, R72 to R48, R73 to R51, R75 to R53, R74 to R54, R76 to R55, R58 to R57

Commit message: WIP
Main schematic re-layout.
Updated 12V power input circuit.
SMPS regulators changed.
Updated analogue voltage circuit.
Parts:
- removed C14, C40: 0.1uF 50V, Capacitor_SMD:C_0603_1608Metric, symbol Device:C
- removed D3, D4: PMEG3010EH, Diode_SMD:D_SOD-123F, symbol Diode:PMEG3010EH
- removed IC6: AD8542ARMZ-REEL, DIY:SOP65P490X110-8N, symbol DIY:AD8542ARMZ-REEL
- removed Q3, Q4: DMG2301L, Package_TO_SOT_SMD:SOT-23, symbol Transistor_FET:Q_PMOS_GSD
- removed R48: 6k8, Resistor_SMD:R_0603_1608Metric, symbol Device:R
- removed R51, R53: 27k, Resistor_SMD:R_0603_1608Metric, symbol Device:R
- removed R54, R55: 51k, Resistor_SMD:R_0603_1608Metric, symbol Device:R
- removed R57: 330k, Resistor_SMD:R_0603_1608Metric, symbol Device:R
Other:
- note removed: "Current is set as follows : - 100mV across 22R = ~4.54mA. MOSFET used to avoid influence from additional base current. - For fuel level and common sensors (0-250Ohm), that gives a sensor voltage of anywhere between 0 and 1.135V - Practically the maximum voltage that can be is 4.9V-0.550V = 4.35V (the schottky typical Vf, although usually lower) - That means that in this current setup the maximum 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"
- note removed: "Full-scale 5V = just under 3V3 (~3.27V)"
- note removed: "Ideas/issues : - How to account for variations in the Vf of PMEG3010EH Alex: At ~4.5mA, Vf varies by ~120mV from -40 to 80degC. This equates to ~24ohm error over a large temp Martin : gotcha - 5V may not be true 5V -> Zener regulator there too ? evaluate possible swings Alex: Used a Vref that follows any variation of 5V. More worried about keeping a set V across the current set resistor. - Design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"
- note removed: "Vref set to 4.9V As the divider follows the supply, its less susceptible to supply variation than a fixed voltage (zener). i.e. always close to 100mV across Iset resistor."

Commit message: Schematic pre-review
WIP - final TODOs needed before review
Parts:
- added C41: 100n, Capacitor_SMD:C_0603_1608Metric_Pad1.08x0.95mm_HandSolder, symbol VXDash_passives:Cap_MLCC
- added C42, C43: 33n, Capacitor_SMD:C_0603_1608Metric_Pad1.08x0.95mm_HandSolder, symbol VXDash_passives:Cap_MLCC
- added D11, D7, D8, D9: BAT54, Diode_SMD:D_SOD-123, symbol VXDash_diodes:D_Schottky
- added IC2, IC5: AS2333_OpAmp, Package_SO:MSOP-8_3x3mm_P0.65mm, symbol VXDash_ICs:AS2333_OpAmp
- added Q3, Q4, Q5, Q6: DMP3099L, Package_TO_SOT_SMD:SOT-23, symbol Transistor_FET:Q_PMOS_GSD
- added R55, R56, R66, R67: 1k, Resistor_SMD:R_0603_1608Metric_Pad0.98x0.95mm_HandSolder, symbol VXDash_passives:Res
- added R57, R68: 18R, Resistor_SMD:R_0603_1608Metric_Pad0.98x0.95mm_HandSolder, symbol VXDash_passives:Res
- added R58, R69: 0R, Resistor_SMD:R_0603_1608Metric_Pad0.98x0.95mm_HandSolder, symbol VXDash_passives:Res
- added R59, R70: 1k, Resistor_SMD:R_1206_3216Metric_Pad1.30x1.75mm_HandSolder, symbol VXDash_passives:Res
- added R60, R71: 160R, Resistor_SMD:R_0603_1608Metric_Pad0.98x0.95mm_HandSolder, symbol VXDash_passives:Res
- added R61, R72: 6R8, Resistor_SMD:R_0603_1608Metric_Pad0.98x0.95mm_HandSolder, symbol VXDash_passives:Res
Connections:
- new net: Q5.1 (G), R67.2
- new net: D9.2 (A), Q6.3 (D)
- new net: Q3.2 (S), R57.1
- new net: Q3.1 (G), R56.2
- new net: Q5.2 (S), R68.1
- new net: Q5.3 (D), R69.2, R72.1
- new net: Q3.3 (D), R58.2, R61.1
- new net: R60.1, R61.2
- new net: IC5.3 (+), Q6.2 (S), R69.1
- new net: R71.1, R72.2
- new net: D7.2 (A), Q4.3 (D)
- new net: IC2.1, R55.1
- new net: IC2.3 (+), Q4.2 (S), R58.1
- new net: IC5.1, R66.1
- new net: Q6.1 (G), R66.2
- new net: Q4.1 (G), R55.2
- new net +3V3: C41.2, D11.1 (K), D8.1 (K), IC2.8
- new net ADC_A: C42.2, D8.2 (A), R59.2
- new net ADC_B: C43.2, D11.2 (A), R70.2
- new net GND: C41.1, C42.1, C43.1, IC2.4
- new net HighResiSet_A: R56.1
- new net HighResiSet_B: R67.1
- new net Sender_A: D7.1 (K), R59.1
- new net Sender_B: D9.1 (K), R70.1
- new net SensorSupply: R57.2, R60.2, R68.2, R71.2
- new net Vref: IC2.2 (-), IC5.2 (-)
