File: Vehicle Emulator Board/12V_to_3V3_MP2322GQH.kicad_sch (KiCad schematic)
At the start: 12 parts, among them IC4 MP2322GQH-Z

Commit message: VEB
Other:
- title: 5 to 3V3 stage -> Vehicle Emulator Board
Changed lines of the file:
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@@
   (paper "A4")
   (title_block
-    (title "5 to 3V3 stage")
-    (date "2024-10-06")
-    (rev "1.3.1")
+    (title "Vehicle Emulator Board")
+    (date "2025-03-09")
+    (rev "1.0.0")
     (comment 1 "https://github.com/martinroger/VXDash")
     (comment 2 "https://cadlab.io/projects/vxdash")
@@
     (pin "2")
     (instances
-      (project "VXDash"
+      (project "Vehicle Emulator Board"
         (path "/f2858fc4-50de-4ff0-a01c-5b985ee14aef/e4c69d46-7a64-435d-9e3a-d73acbe7ec2b"
           (reference "C8") (unit 1)
@@
     (pin "2")
     (instances
-      (project "VXDash"
+      (project "Vehicle Emulator Board"
         (path "/f2858fc4-50de-4ff0-a01c-5b985ee14aef/21f2fd69-aa93-4550-8877-dde4aa3e5582"
           (reference "C22") (unit 1)
@@
     (pin "1")
     (instances
-      (project "VXDash"
+      (project "Vehicle Emulator Board"
         (path "/f2858fc4-50de-4ff0-a01c-5b985ee14aef/21f2fd69-aa93-4550-8877-dde4aa3e5582"
           (reference "#PWR042") (unit 1)
@@
     (pin "1")
     (instances
-      (project "VXDash"
+      (project "Vehicle Emulator Board"
         (path "/f2858fc4-50de-4ff0-a01c-5b985ee14aef/21f2fd69-aa93-4550-8877-dde4aa3e5582"
           (reference "#PWR036") (unit 1)
@@
     (pin "1")
     (instances
-      (project "VXDash"
+      (project "Vehicle Emulator Board"
         (path "/f2858fc4-50de-4ff0-a01c-5b985ee14aef/21f2fd69-aa93-4550-8877-dde4aa3e5582"
           (reference "#PWR037") (unit 1)
@@
     (pin "1")
     (instances
-      (project "VXDash"
+      (project "Vehicle Emulator Board"
         (path "/f2858fc4-50de-4ff0-a01c-5b985ee14aef/21f2fd69-aa93-4550-8877-dde4aa3e5582"
           (reference "#PWR035") (unit 1)
@@
     (pin "1")
     (instances
-      (project "VXDash"
+      (project "Vehicle Emulator Board"
         (path "/f2858fc4-50de-4ff0-a01c-5b985ee14aef/21f2fd69-aa93-4550-8877-dde4aa3e5582"
           (reference "#PWR039") (unit 1)
@@
     (pin "2")
     (instances
-      (project "VXDash"
+      (project "Vehicle Emulator Board"
         (path "/f2858fc4-50de-4ff0-a01c-5b985ee14aef/21f2fd69-aa93-4550-8877-dde4aa3e5582"
           (reference "L2") (unit 1)
@@
     (pin "1")
     (instances
-      (project "VXDash"
+      (project "Vehicle Emulator Board"
         (path "/f2858fc4-50de-4ff0-a01c-5b985ee14aef/21f2fd69-aa93-4550-8877-dde4aa3e5582"
           (reference "#PWR040") (unit 1)
@@
     (pin "2")
     (instances
-      (project "VXDash"
+      (project "Vehicle Emulator Board"
         (path "/f2858fc4-50de-4ff0-a01c-5b985ee14aef/21f2fd69-aa93-4550-8877-dde4aa3e5582"
           (reference "R39") (unit 1)
@@
     (pin "8")
     (instances
-      (project "VXDash"
+      (project "Vehicle Emulator Board"
         (path "/f2858fc4-50de-4ff0-a01c-5b985ee14aef/21f2fd69-aa93-4550-8877-dde4aa3e5582"
           (reference "IC4") (unit 1)
@@
     (pin "2")
     (instances
-      (project "VXDash"
+      (project "Vehicle Emulator Board"
         (path "/f2858fc4-50de-4ff0-a01c-5b985ee14aef/21f2fd69-aa93-4550-8877-dde4aa3e5582"
           (reference "C20") (unit 1)
@@
     (pin "1")
     (instances
-      (project "VXDash"
+      (project "Vehicle Emulator Board"
         (path "/f2858fc4-50de-4ff0-a01c-5b985ee14aef/21f2fd69-aa93-4550-8877-dde4aa3e5582"
           (reference "#PWR038") (unit 1)
@@
     (pin "2")
     (instances
-      (project "VXDash"
+      (project "Vehicle Emulator Board"
         (path "/f2858fc4-50de-4ff0-a01c-5b985ee14aef/21f2fd69-aa93-4550-8877-dde4aa3e5582"
           (reference "C21") (unit 1)
@@
     (pin "2")
     (instances
-      (project "VXDash"
+      (project "Vehicle Emulator Board"
         (path "/f2858fc4-50de-4ff0-a01c-5b985ee14aef/21f2fd69-aa93-4550-8877-dde4aa3e5582"
           (reference "C23") (unit 1)
@@
     (pin "2")
     (instances
-      (project "VXDash"
+      (project "Vehicle Emulator Board"
         (path "/f2858fc4-50de-4ff0-a01c-5b985ee14aef/21f2fd69-aa93-4550-8877-dde4aa3e5582"
           (reference "C17") (unit 1)
@@
     (pin "2")
     (instances
-      (project "VXDash"
+      (project "Vehicle Emulator Board"
         (path "/f2858fc4-50de-4ff0-a01c-5b985ee14aef/21f2fd69-aa93-4550-8877-dde4aa3e5582"
           (reference "R37") (unit 1)
@@
     (pin "2")
     (instances
-      (project "VXDash"
+      (project "Vehicle Emulator Board"
         (path "/f2858fc4-50de-4ff0-a01c-5b985ee14aef/21f2fd69-aa93-4550-8877-dde4aa3e5582"
           (reference "R38") (unit 1)
@@
     (pin "2")
     (instances
-      (project "VXDash"
+      (project "Vehicle Emulator Board"
         (path "/f2858fc4-50de-4ff0-a01c-5b985ee14aef/e4c69d46-7a64-435d-9e3a-d73acbe7ec2b"
           (reference "C8") (unit 1)
