File: Vehicle Emulator Board/Opto_ActLo.kicad_sch (KiCad schematic)
At the start: 3 parts, among them U1 SFH617A-2X009T

Commit message: VEB
Other:
- title: Active Low Optocoupler circuit -> Vehicle Emulator Board
Changed lines of the file:
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@@
   (paper "A4")
   (title_block
-    (title "Active Low Optocoupler circuit")
-    (date "2024-10-06")
-    (rev "1.3.1")
+    (title "Vehicle Emulator Board")
+    (date "2025-03-09")
+    (rev "1.0.0")
     (comment 1 "https://github.com/martinroger/VXDash")
     (comment 2 "https://cadlab.io/projects/vxdash")
@@
         )
       )
-      (project "VXDash"
+      (project "Vehicle Emulator Board"
         (path "/f2858fc4-50de-4ff0-a01c-5b985ee14aef/2079de5b-2f3f-4362-a932-421ac573d68a"
           (reference "R7") (unit 1)
@@
         )
       )
-      (project "VXDash"
+      (project "Vehicle Emulator Board"
         (path "/f2858fc4-50de-4ff0-a01c-5b985ee14aef/2079de5b-2f3f-4362-a932-421ac573d68a"
           (reference "R6") (unit 1)
@@
     (pin "1")
     (instances
-      (project "VXDash"
+      (project "Vehicle Emulator Board"
         (path "/f2858fc4-50de-4ff0-a01c-5b985ee14aef/2079de5b-2f3f-4362-a932-421ac573d68a"
           (reference "#PWR015") (unit 1)
@@
         )
       )
-      (project "VXDash"
+      (project "Vehicle Emulator Board"
         (path "/f2858fc4-50de-4ff0-a01c-5b985ee14aef"
           (reference "U1") (unit 1)
