File: Vehicle Emulator Board/Rsensing_Pair.kicad_sch (KiCad schematic)
At the start: 13 parts, among them IC5 AD8542ARMZ-REEL, Q7 DMG2301L, Q8 DMG2301L

Commit message: VEB
Other:
- title: Dual Op-Amp Constant current source resistive sensor -> Vehicle Emulator Board
Changed lines of the file:
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@@
   (paper "A4")
   (title_block
-    (title "Dual Op-Amp Constant current source resistive sensor")
-    (date "2024-10-06")
-    (rev "1.3.1")
+    (title "Vehicle Emulator Board")
+    (date "2025-03-09")
+    (rev "1.0.0")
     (comment 1 "https://github.com/martinroger/VXDash")
     (comment 2 "https://cadlab.io/projects/vxdash")
@@
     (pin "1")
     (instances
-      (project "VXDash"
+      (project "Vehicle Emulator Board"
         (path "/f2858fc4-50de-4ff0-a01c-5b985ee14aef/326d91f1-1d34-43d4-aac6-11bd9692edf0"
           (reference "#PWR071") (unit 1)
@@
     (pin "3")
     (instances
-      (project "VXDash"
+      (project "Vehicle Emulator Board"
         (path "/f2858fc4-50de-4ff0-a01c-5b985ee14aef/326d91f1-1d34-43d4-aac6-11bd9692edf0"
           (reference "Q8") (unit 1)
@@
     (pin "1")
     (instances
-      (project "VXDash"
+      (project "Vehicle Emulator Board"
         (path "/f2858fc4-50de-4ff0-a01c-5b985ee14aef/326d91f1-1d34-43d4-aac6-11bd9692edf0"
           (reference "#PWR069") (unit 1)
@@
     (pin "1")
     (instances
-      (project "VXDash"
+      (project "Vehicle Emulator Board"
         (path "/f2858fc4-50de-4ff0-a01c-5b985ee14aef/326d91f1-1d34-43d4-aac6-11bd9692edf0"
           (reference "#PWR072") (unit 1)
@@
     (pin "2")
     (instances
-      (project "VXDash"
+      (project "Vehicle Emulator Board"
         (path "/f2858fc4-50de-4ff0-a01c-5b985ee14aef/326d91f1-1d34-43d4-aac6-11bd9692edf0"
           (reference "D9") (unit 1)
@@
     (pin "8")
     (instances
-      (project "VXDash"
+      (project "Vehicle Emulator Board"
         (path "/f2858fc4-50de-4ff0-a01c-5b985ee14aef/326d91f1-1d34-43d4-aac6-11bd9692edf0"
           (reference "IC5") (unit 1)
@@
     (pin "2")
     (instances
-      (project "VXDash"
+      (project "Vehicle Emulator Board"
         (path "/f2858fc4-50de-4ff0-a01c-5b985ee14aef/326d91f1-1d34-43d4-aac6-11bd9692edf0"
           (reference "R72") (unit 1)
@@
     (pin "2")
     (instances
-      (project "VXDash"
+      (project "Vehicle Emulator Board"
         (path "/f2858fc4-50de-4ff0-a01c-5b985ee14aef/326d91f1-1d34-43d4-aac6-11bd9692edf0"
           (reference "R74") (unit 1)
@@
     (pin "2")
     (instances
-      (project "VXDash"
+      (project "Vehicle Emulator Board"
         (path "/f2858fc4-50de-4ff0-a01c-5b985ee14aef/326d91f1-1d34-43d4-aac6-11bd9692edf0"
           (reference "R73") (unit 1)
@@
         )
       )
-      (project "VXDash"
+      (project "Vehicle Emulator Board"
         (path "/f2858fc4-50de-4ff0-a01c-5b985ee14aef"
           (reference "C35") (unit 1)
@@
     (pin "1")
     (instances
-      (project "VXDash"
+      (project "Vehicle Emulator Board"
         (path "/f2858fc4-50de-4ff0-a01c-5b985ee14aef/326d91f1-1d34-43d4-aac6-11bd9692edf0"
           (reference "#PWR070") (unit 1)
@@
     (pin "2")
     (instances
-      (project "VXDash"
+      (project "Vehicle Emulator Board"
         (path "/f2858fc4-50de-4ff0-a01c-5b985ee14aef/326d91f1-1d34-43d4-aac6-11bd9692edf0"
           (reference "R75") (unit 1)
@@
     (pin "3")
     (instances
-      (project "VXDash"
+      (project "Vehicle Emulator Board"
         (path "/f2858fc4-50de-4ff0-a01c-5b985ee14aef/326d91f1-1d34-43d4-aac6-11bd9692edf0"
           (reference "Q7") (unit 1)
@@
     (pin "1")
     (instances
-      (project "VXDash"
+      (project "Vehicle Emulator Board"
         (path "/f2858fc4-50de-4ff0-a01c-5b985ee14aef/326d91f1-1d34-43d4-aac6-11bd9692edf0"
           (reference "#PWR064") (unit 1)
@@
     (pin "2")
     (instances
-      (project "VXDash"
+      (project "Vehicle Emulator Board"
         (path "/f2858fc4-50de-4ff0-a01c-5b985ee14aef/326d91f1-1d34-43d4-aac6-11bd9692edf0"
           (reference "R76") (unit 1)
@@
         )
       )
-      (project "VXDash"
+      (project "Vehicle Emulator Board"
         (path "/f2858fc4-50de-4ff0-a01c-5b985ee14aef"
           (reference "C35") (unit 1)
@@
     (pin "2")
     (instances
-      (project "VXDash"
+      (project "Vehicle Emulator Board"
         (path "/f2858fc4-50de-4ff0-a01c-5b985ee14aef/326d91f1-1d34-43d4-aac6-11bd9692edf0"
           (reference "R58") (unit 1)
@@
     (pin "2")
     (instances
-      (project "VXDash"
+      (project "Vehicle Emulator Board"
         (path "/f2858fc4-50de-4ff0-a01c-5b985ee14aef/326d91f1-1d34-43d4-aac6-11bd9692edf0"
           (reference "D2") (unit 1)
