File: Vehicle Emulator Board/Vehicle Emulator Board.kicad_sch (KiCad schematic)
At the start: 18 parts, among them IC1 CD74HC4050M96, IC2 SP721ABG, IC5 74HC4067BQ-Q100J, J1 MX34036UF2, J2 Conn_01x04_Socket

Commit message: VEB
Parts:
- removed C10 (x2), C6, C8, C9 (x2): 0.1uF 50V, Capacitor_SMD:C_0603_1608Metric, symbol Device:C
- removed IC1: CD74HC4050M96, SamacSys_Parts:SOIC127P600X175-16N, symbol SamacSys_Parts:CD74HC4050M96
- removed IC5: 74HC4067BQ-Q100J, SamacSys_Parts:74HC4067BQQ100J, symbol SamacSys_Parts:74HC4067BQ-Q100J
- removed J2: Conn_01x04_Socket, Connector_JST:JST_XH_S4B-XH-A-1_1x04_P2.50mm_Horizontal, symbol Connector:Conn_01x04_Socket
- added Q9: BC847, Package_TO_SOT_SMD:SOT-23, symbol Transistor_BJT:BC847
- added R36: 10K, symbol Device:R_Small
- added R71: 1K, symbol Device:R_Small
Connections:
- net GND: now also Q9.2 (E)
- new net: Q9.3 (C), R36.2
- new net: Q9.1 (B), R71.2
- no-connect marks 16 -> 8
Other:
- removed sheet ESP32
- note removed: "50mA max consumption"
- note removed: "Allocated 100mA, may be more like 50mA DO NOT TURN ON WIFI/RF"
- note removed: "Nextion Up to 500mA"
- title: Main architecture -> Vehicle Emulator Board
- moved on the sheet: F1, J1
