File: KiCad PCB Files/VXDash/ESP32.kicad_sch (KiCad schematic)
At the start: 4 parts, among them J2 Spare_GPIO, U16 ESP32-DevKitC

Commit message: Moved VXDash project into sub folder
Parts:
- removed U16: ESP32-DevKitC, PCM_Espressif:ESP32-DevKitC, symbol PCM_Espressif:ESP32-DevKitC
- added U16: ESP32-S3-WROOM-1, RF_Module:ESP32-S3-WROOM-1, symbol RF_Module:ESP32-S3-WROOM-1
- J2: value Spare_GPIO -> Expansion
- renumbered C24 to C21, R83 to R41
Connections:
- net +3V3: now also U16.2 (3V3); no longer R41.2
- net GND: now also U16.1 (GND), U16.40 (GND), U16.41 (GND)
- net UART0_RX: now also U16.36 (RXD0)
- net UART0_TX: now also U16.37 (TXD0)
- no-connect marks 7 -> 0
Other:
- moved on the sheet: C21
