File: KiCad PCB Files/VXDash/Analogue.kicad_sch (KiCad schematic)
At the start: 12 parts, among them U17 ADS1115IDGS

Commit message: Grape shot additions
- Added 0R to the VCC pin on the CAN transceiver for pin compatibility with other transceiver
- Updated TODO box
- Rename ADC_SDA and ADC_SCL to SDA and SCL
- Official symbol and footprint from ESP, using ESP32-S3-WROOM-1-N16R8
- Reassigned Coolant LOW to active HI
- Replaced MUX with i²C TCA9555 IO Expander
- Resequenced Active His and Lows to match current SW definition
- Resequenced ADC channels to match current SW definition
- Added simple peripherals for MCU
- Added RESET and BOOT buttons circuits
- Added CAN transceivers for each display, and Termination resistor
- Added USB C
Connections:
- net ADC_SDL renamed ADC_SCL
Other:
- company: (none) -> Alex Miller & Martin Roger
- title: (none) -> Main architecture
Changed lines of the file:
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@@
 	(paper "A3")
 	(title_block
-		(date "2025-08-08")
+		(title "Main architecture")
+		(date "2025-08-10")
 		(rev "1.4")
+		(company "Alex Miller & Martin Roger")
 		(comment 1 "https://github.com/martinroger/VXDash")
 		(comment 2 "https://cadlab.io/projects/vxdash")
@@
 		)
 	)
-	(hierarchical_label "ADC_SDL"
+	(hierarchical_label "ADC_SCL"
 		(shape input)
 		(at 88.9 134.62 180)

Commit message: Minor changes
- Connection for the caliber selection on the sensing circuit
- Typo
Connections:
- no-connect marks 0 -> 3
Changed lines of the file:
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@@
 		(color 0 0 0 0)
 	)
+	(no_connect
+		(at 194.31 107.95)
+	)
+	(no_connect
+		(at 162.56 107.95)
+	)
+	(no_connect
+		(at 194.31 110.49)
+	)
 	(wire
 		(pts
@@
 	(wire
 		(pts
+			(xy 191.77 107.95) (xy 194.31 107.95)
+		)
+		(stroke
+			(width 0)
+			(type default)
+		)
+	)
+	(wire
+		(pts
 			(xy 147.32 127) (xy 292.1 127)
 		)
@@
 	(wire
 		(pts
+			(xy 191.77 100.33) (xy 194.31 100.33)
+		)
+		(stroke
+			(width 0)
+			(type default)
+		)
+	)
+	(wire
+		(pts
 			(xy 137.16 120.65) (xy 137.16 119.38)
 		)
@@
 		(pts
 			(xy 137.16 110.49) (xy 132.08 110.49)
+		)
+		(stroke
+			(width 0)
+			(type default)
+		)
+	)
+	(wire
+		(pts
+			(xy 191.77 110.49) (xy 194.31 110.49)
 		)
 		(stroke
@@
 		)
 	)
+	(hierarchical_label "Set_Hi_Chan_A"
+		(shape input)
+		(at 194.31 100.33 0)
+		(effects
+			(font
+				(size 1.27 1.27)
+			)
+			(justify left)
+		)
+	)

Commit message: PCB layout in progress
Changed some pin assignments to aid routing.
Parts:
- C33: renamed from C26; footprint (none) -> Capacitor_SMD:C_0603_1608Metric_Pad1.08x0.95mm_HandSolder
- C35: renamed from C29; footprint (none) -> Capacitor_SMD:C_0603_1608Metric_Pad1.08x0.95mm_HandSolder
- C36: renamed from C30; footprint (none) -> Capacitor_SMD:C_0603_1608Metric_Pad1.08x0.95mm_HandSolder
- renumbered C65 to C34, D3 to D5, R130 to R62, R131 to R63, R50 to R64, R51 to R65, R52 to R66, R53 to R67, U17 to U19
Changed lines of the file:
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@@
 		(dnp no)
 		(fields_autoplaced yes)
-		(property "Reference" "R53"
+		(property "Reference" "R67"
 			(at 308.61 132.0799 0)
 			(effects
@@
 		)
 		(property "MFT_PN" ""
+			(at 306.07 133.35 0)
+			(effects
+				(font
+					(size 1.27 1.27)
+				)
+				(hide yes)
+			)
+		)
+		(property "Tolerance" ""
 			(at 306.07 133.35 0)
 			(effects
@@
 			(project "VXDash"
 				(path "/f2858fc4-50de-4ff0-a01c-5b985ee14aef/024f3b9c-af80-4b8c-9e91-7ad2b6b7f854"
-					(reference "R53")
+					(reference "R67")
 					(unit 1)
 				)
@@
 		(dnp no)
 		(fields_autoplaced yes)
-		(property "Reference" "R50"
+		(property "Reference" "R64"
 			(at 298.45 120.65 90)
 			(effects
@@
 		(property "MFT_PN" ""
 			(at 298.45 127 0)
+			(effects
+				(font
+					(size 1.27 1.27)
+				)
+				(hide yes)
+			)
+		)
+		(property "Tolerance" ""
+			(at 298.45 127 90)
 			(effects
 				(font
@@
 			(project "VXDash"
 				(path "/f2858fc4-50de-4ff0-a01c-5b985ee14aef/024f3b9c-af80-4b8c-9e91-7ad2b6b7f854"
-					(reference "R50")
+					(reference "R64")
 					(unit 1)
 				)
@@
 		(on_board yes)
 		(dnp no)
-		(property "Reference" "C30"
+		(property "Reference" "C36"
 			(at 327.66 124.4599 0)
 			(effects
@@
 			)
 		)
-		(property "Footprint" ""
+		(property "Footprint" "Capacitor_SMD:C_0603_1608Metric_Pad1.08x0.95mm_HandSolder"
 			(at 322.8848 123.19 0)
 			(effects
@@
 				)
 				(justify right)
+			)
+		)
+		(property "Tolerance" ""
+			(at 323.85 127 0)
+			(effects
+				(font
+					(size 1.27 1.27)
+				)
+				(hide yes)
 			)
 		)
@@
 			(project "VXDash"
 				(path "/f2858fc4-50de-4ff0-a01c-5b985ee14aef/024f3b9c-af80-4b8c-9e91-7ad2b6b7f854"
-					(reference "C30")
+					(reference "C36")
 					(unit 1)
 				)
@@
 		(dnp no)
 		(fields_autoplaced yes)
-		(property "Reference" "R130"
+		(property "Reference" "R62"
 			(at 228.6 91.4399 0)
 			(effects
@@
 		)
 		(property "MFT_PN" ""
+			(at 226.06 92.71 0)
+			(effects
+				(font
+					(size 1.27 1.27)
+				)
+				(hide yes)
+			)
+		)
+		(property "Tolerance" ""
 			(at 226.06 92.71 0)
 			(effects
@@
 			(project "VXDash"
 				(path "/f2858fc4-50de-4ff0-a01c-5b985ee14aef/024f3b9c-af80-4b8c-9e91-7ad2b6b7f854"
-					(reference "R130")
+					(reference "R62")
 					(unit 1)
 				)
@@
 		(dnp no)
 		(fields_autoplaced yes)
-		(property "Reference" "R52"
+		(property "Reference" "R66"
 			(at 308.61 119.3799 0)
 			(effects
@@
 		)
 		(property "MFT_PN" ""
+			(at 306.07 120.65 0)
+			(effects
+				(font
+					(size 1.27 1.27)
+				)
+				(hide yes)
+			)
+		)
+		(property "Tolerance" ""
 			(at 306.07 120.65 0)
 			(effects
@@
 			(project "VXDash"
 				(path "/f2858fc4-50de-4ff0-a01c-5b985ee14aef/024f3b9c-af80-4b8c-9e91-7ad2b6b7f854"
-					(reference "R52")
+					(reference "R66")
 					(unit 1)
 				)
@@
 		(dnp no)
 		(fields_autoplaced yes)
-		(property "Reference" "C29"
+		(property "Reference" "C35"
 			(at 288.29 129.5399 0)
 			(effects
@@
 			)
 		)
-		(property "Footprint" ""
+		(property "Footprint" "Capacitor_SMD:C_0603_1608Metric_Pad1.08x0.95mm_HandSolder"
 			(at 293.0652 128.27 0)
 			(effects
@@
 				)
 				(justify right)
+			)
+		)
+		(property "Tolerance" ""
+			(at 292.1 132.08 0)
+			(effects
+				(font
+					(size 1.27 1.27)
+				)
+				(hide yes)
 			)
 		)
@@
 			(project "VXDash"
 				(path "/f2858fc4-50de-4ff0-a01c-5b985ee14aef/024f3b9c-af80-4b8c-9e91-7ad2b6b7f854"
-					(reference "C29")
+					(reference "C35")
 					(unit 1)
 				)
@@
 		(dnp no)
 		(fields_autoplaced yes)
-		(property "Reference" "#PWR046"
+		(property "Reference" "#PWR056"
 			(at 318.77 147.32 0)
 			(effects
@@
 			(project "VXDash"
 				(path "/f2858fc4-50de-4ff0-a01c-5b985ee14aef/024f3b9c-af80-4b8c-9e91-7ad2b6b7f854"
-					(reference "#PWR046")
+					(reference "#PWR056")
 					(unit 1)
 				)
@@
 		(on_board yes)
 		(dnp no)
-		(property "Reference" "D3"
+		(property "Reference" "D5"
 			(at 316.23 126.365 90)
 			(effects
@@
 		)
 		(property "MFT_PN" "BZT52C18-TP"
+			(at 318.77 127 90)
+			(effects
+				(font
+					(size 1.27 1.27)
+				)
+				(hide yes)
+			)
+		)
+		(property "Tolerance" ""
 			(at 318.77 127 90)
 			(effects
@@
 			(project "VXDash"
 				(path "/f2858fc4-50de-4ff0-a01c-5b985ee14aef/024f3b9c-af80-4b8c-9e91-7ad2b6b7f854"
-					(reference "D3")
+					(reference "D5")
 					(unit 1)
 				)
@@
 		(on_board yes)
 		(dnp no)
-		(property "Reference" "C26"
+		(property "Reference" "C33"
 			(at 139.7 113.03 0)
 			(effects
@@
 			)
 		)
-		(property "Footprint" ""
+		(property "Footprint" "Capacitor_SMD:C_0603_1608Metric_Pad1.08x0.95mm_HandSolder"
 			(at 136.1948 119.38 0)
 			(effects
@@
 				)
 				(justify right)
+			)
+		)
+		(property "Tolerance" ""
+			(at 137.16 115.57 0)
+			(effects
+				(font
+					(size 1.27 1.27)
+				)
+				(hide yes)
 			)
 		)
@@
 			(project "VXDash"
 				(path "/f2858fc4-50de-4ff0-a01c-5b985ee14aef/024f3b9c-af80-4b8c-9e91-7ad2b6b7f854"
-					(reference "C26")
+					(reference "C33")
 					(unit 1)
 				)
@@
 		(dnp no)
 		(fields_autoplaced yes)
-		(property "Reference" "R131"
+		(property "Reference" "R63"
 			(at 223.52 107.9501 0)
 			(effects
@@
 		)
 		(property "MFT_PN" ""
+			(at 226.06 106.68 0)
+			(effects
+				(font
+					(size 1.27 1.27)
+				)
+				(hide yes)
+			)
+		)
+		(property "Tolerance" ""
 			(at 226.06 106.68 0)
 			(effects
@@
 			(project "VXDash"
 				(path "/f2858fc4-50de-4ff0-a01c-5b985ee14aef/024f3b9c-af80-4b8c-9e91-7ad2b6b7f854"
-					(reference "R131")
+					(reference "R63")
 					(unit 1)
 				)
@@
 		(on_board yes)
 		(dnp no)
-		(property "Reference" "U17"
+		(property "Reference" "U19"
 			(at 129.9367 119.38 0)
 			(effects
@@
 		)
 		(property "Description" "Ultra-Small, Low-Power, I2C-Compatible, 860-SPS, 16-Bit ADCs With Internal Reference, Oscillator, and Programmable Comparator, VSSOP-10"
+			(at 132.08 134.62 0)
+			(effects
+				(font
+					(size 1.27 1.27)
+				)
+				(hide yes)
+			)
+		)
+		(property "Tolerance" ""
 			(at 132.08 134.62 0)
 			(effects
@@
 			(project "VXDash"
 				(path "/f2858fc4-50de-4ff0-a01c-5b985ee14aef/024f3b9c-af80-4b8c-9e91-7ad2b6b7f854"
-					(reference "U17")
+					(reference "U19")
 					(unit 1)
 				)
@@
 		(dnp no)
 		(fields_autoplaced yes)
-		(property "Reference" "R51"
+		(property "Reference" "R65"
 			(at 308.61 107.9499 0)
 			(effects
@@
 		)
 		(property "MFT_PN" ""
+			(at 306.07 109.22 0)
+			(effects
+				(font
+					(size 1.27 1.27)
+				)
+				(hide yes)
+			)
+		)
+		(property "Tolerance" ""
 			(at 306.07 109.22 0)
 			(effects
@@
 			(project "VXDash"
 				(path "/f2858fc4-50de-4ff0-a01c-5b985ee14aef/024f3b9c-af80-4b8c-9e91-7ad2b6b7f854"
-					(reference "R51")
+					(reference "R65")
 					(unit 1)
 				)
@@
 		(dnp no)
 		(fields_autoplaced yes)
-		(property "Reference" "#PWR071"
+		(property "Reference" "#PWR055"
 			(at 226.06 119.38 0)
 			(effects
@@
 			(project "VXDash"
 				(path "/f2858fc4-50de-4ff0-a01c-5b985ee14aef/024f3b9c-af80-4b8c-9e91-7ad2b6b7f854"
-					(reference "#PWR071")
+					(reference "#PWR055")
 					(unit 1)
 				)
@@
 		(on_board yes)
 		(dnp no)
-		(property "Reference" "#PWR043"
+		(property "Reference" "#PWR054"
 			(at 137.16 127 0)
 			(effects
@@
 			(project "VXDash"
 				(path "/f2858fc4-50de-4ff0-a01c-5b985ee14aef/024f3b9c-af80-4b8c-9e91-7ad2b6b7f854"
-					(reference "#PWR043")
+					(reference "#PWR054")
 					(unit 1)
 				)
@@
 		(dnp no)
 		(fields_autoplaced yes)
-		(property "Reference" "#PWR040"
+		(property "Reference" "#PWR053"
 			(at 132.08 153.67 0)
 			(effects
@@
 			(project "VXDash"
 				(path "/f2858fc4-50de-4ff0-a01c-5b985ee14aef/024f3b9c-af80-4b8c-9e91-7ad2b6b7f854"
-					(reference "#PWR040")
+					(reference "#PWR053")
 					(unit 1)
 				)
@@
 		(dnp no)
 		(fields_autoplaced yes)
-		(property "Reference" "C65"
+		(property "Reference" "C34"
 			(at 236.22 104.1399 0)
 			(effects
@@
 		)
 		(property "MFT_PN" ""
+			(at 232.41 106.68 0)
+			(effects
+				(font
+					(size 1.27 1.27)
+				)
+				(hide yes)
+			)
+		)
+		(property "Tolerance" ""
 			(at 232.41 106.68 0)
 			(effects
@@
 			(project "VXDash"
 				(path "/f2858fc4-50de-4ff0-a01c-5b985ee14aef/024f3b9c-af80-4b8c-9e91-7ad2b6b7f854"
-					(reference "C65")
+					(reference "C34")
 					(unit 1)
 				)

Commit message: ERC corrections, idiot lights
- VXDash : added idiot lights (also to emulator board)
- VXDash : corrected some ERC violations
Connections:
- no-connect marks 3 -> 4
Changed lines of the file:
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@@
+	)
+	(no_connect
+		(at 121.92 129.54)
 	)
 	(no_connect

Commit message: New main dash PCB - WIP inc. CAD
Parts:
- R64, R66, R67: footprint Resistor_SMD:R_0805_2012Metric_Pad1.20x1.40mm_HandSolder -> Resistor_SMD:R_0603_1608Metric_Pad0.98x0.95mm_HandSolder

Commit message: Large schematic update
- Fascia pass-through connector
- Load emulators for all but turn signals
- Test points
- Additional caps for decoupling
- Regrouped display connectors in single unit
- Added CAN debug connector
Parts:
- added TP8: ADS_VREF, TestPoint:TestPoint_Pad_D2.0mm, symbol Connector:TestPoint
Connections:
- net v_ref: now also TP8.1
Changed lines of the file:
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@@
+	(wire
+		(pts
+			(xy 227.33 68.58) (xy 227.33 73.66)
+		)
+		(stroke
+			(width 0)
+			(type default)
+		)
+	)
 	(wire
 		(pts
@@
 			)
 			(justify right bottom)
+		)
+	)
+	(label "v_ref"
+		(at 227.33 73.66 0)
+		(effects
+			(font
+				(size 1.27 1.27)
+			)
+			(justify left bottom)
 		)
 	)
@@
 					(unit 1)
 				)
+			)
+		)
+	)
+	(symbol
+		(lib_id "Connector:TestPoint")
+		(at 227.33 68.58 0)
+		(unit 1)
+		(exclude_from_sim no)
+		(in_bom yes)
+		(on_board yes)
+		(dnp no)
+		(fields_autoplaced yes)
+		(property "Reference" "TP8"
+			(at 229.87 64.0079 0)
+			(effects
+				(font
+					(size 1.27 1.27)
+				)
+				(justify left)
+			)
+		)
+		(property "Value" "ADS_VREF"
+			(at 229.87 66.5479 0)
+			(effects
+				(font
+					(size 1.27 1.27)
+				)
+				(justify left)
+			)
+		)
+		(property "Footprint" "TestPoint:TestPoint_Pad_D2.0mm"
+			(at 232.41 68.58 0)
+			(effects
+				(font
+					(size 1.27 1.27)
+				)
+				(hide yes)
+			)
+		)
+		(property "Datasheet" "~"
+			(at 232.41 68.58 0)
+			(effects
+				(font
+					(size 1.27 1.27)
+				)
+				(hide yes)
+			)
+		)
+		(property "Description" "test point"
+			(at 227.33 68.58 0)
+			(effects
+				(font
+					(size 1.27 1.27)
+				)
+				(hide yes)
+			)
+		)
+		(pin "1"
+		)
+		(instances
+			(project "VXDash"
+				(path "/f2858fc4-50de-4ff0-a01c-5b985ee14aef/024f3b9c-af80-4b8c-9e91-7ad2b6b7f854"
+					(reference "TP8")
+					(unit 1)
+				)

Commit message: BOM first pass
- Still missing some internal connectors definitions
- Alternative to use a 4x4ch opto config instead of 16x1 ?
- Alternative LiteOn optos identified (easier to source on LCSC)
Parts:
- C33, C34, C36: LCSC (none) -> C16194176; MFT (none) -> Samsung Electro-Mechanics; MFT_PN (none) -> CL10B104KB8NNWC
- C35: LCSC (none) -> C100042; MFT (none) -> Yageo; MFT_PN (none) -> CC0603KRX7R9BB103
- D5: ALT_MFT_PN_1 (none) -> BZT52C18-E3-08; LCSC (none) -> C668896; LCSC alt (none) -> C467525
- R62: LCSC (none) -> C163424; MFT (none) -> Yageo; MFT_PN (none) -> RC0603FR-0739KL
- R63: LCSC (none) -> C141684; MFT (none) -> Yageo; MFT_PN (none) -> RC0603FR-07820KL
- R64: value 1K -> 1k; LCSC (none) -> C22548; MFT (none) -> Yageo; MFT_PN (none) -> RC0603FR-071KL
- R65: LCSC (none) -> C105577; MFT (none) -> Yageo; MFT_PN (none) -> RC0805FR-07100RL; Power 100mW -> 125mW
- R66: value 1Meg -> 1M; LCSC (none) -> C105578; MFT (none) -> Yageo; MFT_PN (none) -> RC0603FR-071ML
- R67: LCSC (none) -> C123420; MFT (none) -> Yageo; MFT_PN (none) -> RC0603FR-07220KL
- TP8: now left out of the parts list
- U19: LCSC (none) -> C37593; MFT (none) -> Texas Instruments; MFT_PN (none) -> ADS1115IDGSR
