File: KiCad PCB Files/VXDash/Opto_ActHi.kicad_sch (KiCad schematic)
At the start: 3 parts

Commit message: Moved VXDash project into sub folder
Parts:
- removed R6: 8k2, Resistor_SMD:R_0805_2012Metric_Pad1.20x1.40mm_HandSolder, symbol VXDash_passives:Res
- removed R7: 10k, Resistor_SMD:R_0805_2012Metric_Pad1.20x1.40mm_HandSolder, symbol VXDash_passives:Res
- removed U1: ~, Package_DIP:SMDIP-4_W7.62mm, symbol Isolator:SFH617A-2X009T
- added R27: 8k2, Resistor_SMD:R_0805_2012Metric_Pad1.20x1.40mm_HandSolder, symbol VXDash_passives:Res
- added R28: 10k, Resistor_SMD:R_0805_2012Metric_Pad1.20x1.40mm_HandSolder, symbol VXDash_passives:Res
- added U11: ~, Package_DIP:SMDIP-4_W7.62mm, symbol Isolator:SFH617A-2X009T
Connections:
- net +3V3: now also R28.1
- net GND: now also U11.2, U11.3
- new net: R27.2, U11.1
- new net HL_Input: R27.1
- new net ~{LL_output}: R28.2, U11.4
Other:
- title: Active Low Optocoupler circuit -> Active Hi Optocoupler circuit

Commit message: Grape shot additions
- Added 0R to the VCC pin on the CAN transceiver for pin compatibility with other transceiver
- Updated TODO box
- Rename ADC_SDA and ADC_SCL to SDA and SCL
- Official symbol and footprint from ESP, using ESP32-S3-WROOM-1-N16R8
- Reassigned Coolant LOW to active HI
- Replaced MUX with i²C TCA9555 IO Expander
- Resequenced Active His and Lows to match current SW definition
- Resequenced ADC channels to match current SW definition
- Added simple peripherals for MCU
- Added RESET and BOOT buttons circuits
- Added CAN transceivers for each display, and Termination resistor
- Added USB C
Parts:
- renumbered R27 to R41, R28 to R68, U11 to U16
Other:
- company: (none) -> Alex Miller & Martin Roger
- title: Active Hi Optocoupler circuit -> Main architecture
Changed lines of the file:
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@@
 	(paper "A4")
 	(title_block
-		(title "Active Hi Optocoupler circuit")
-		(date "2025-08-08")
+		(title "Main architecture")
+		(date "2025-08-10")
 		(rev "1.4")
+		(company "Alex Miller & Martin Roger")
 		(comment 1 "https://github.com/martinroger/VXDash")
 		(comment 2 "https://cadlab.io/projects/vxdash")
@@
 		(dnp no)
 		(fields_autoplaced yes)
-		(property "Reference" "U11"
+		(property "Reference" "U16"
 			(at 138.43 92.71 0)
 			(effects
@@
 		(instances
 			(project "VXDash"
+				(path "/f2858fc4-50de-4ff0-a01c-5b985ee14aef/0e70c286-e2c1-42eb-aaa1-5a4ab22bb424"
+					(reference "U19")
+					(unit 1)
+				)
 				(path "/f2858fc4-50de-4ff0-a01c-5b985ee14aef/36ea4b64-9158-43b1-97c6-20da8346f32e"
 					(reference "U14")
@@
 				(path "/f2858fc4-50de-4ff0-a01c-5b985ee14aef/6cef8934-8b7c-410b-8d9f-f073b93271b8"
 					(reference "U11")
+					(unit 1)
+				)
+				(path "/f2858fc4-50de-4ff0-a01c-5b985ee14aef/771becef-f508-42ea-9fb3-6952fb053001"
+					(reference "U16")
 					(unit 1)
 				)
@@
 		(dnp no)
 		(fields_autoplaced yes)
-		(property "Reference" "R28"
+		(property "Reference" "R68"
 			(at 152.4 85.0899 0)
 			(effects
@@
 		(instances
 			(project "VXDash"
+				(path "/f2858fc4-50de-4ff0-a01c-5b985ee14aef/0e70c286-e2c1-42eb-aaa1-5a4ab22bb424"
+					(reference "R70")
+					(unit 1)
+				)
 				(path "/f2858fc4-50de-4ff0-a01c-5b985ee14aef/36ea4b64-9158-43b1-97c6-20da8346f32e"
 					(reference "R34")
@@
 				(path "/f2858fc4-50de-4ff0-a01c-5b985ee14aef/6cef8934-8b7c-410b-8d9f-f073b93271b8"
 					(reference "R28")
+					(unit 1)
+				)
+				(path "/f2858fc4-50de-4ff0-a01c-5b985ee14aef/771becef-f508-42ea-9fb3-6952fb053001"
+					(reference "R68")
 					(unit 1)
 				)
@@
 		(dnp no)
 		(fields_autoplaced yes)
-		(property "Reference" "#PWR024"
+		(property "Reference" "#PWR037"
 			(at 149.86 113.03 0)
 			(effects
@@
 		(instances
 			(project "VXDash"
+				(path "/f2858fc4-50de-4ff0-a01c-5b985ee14aef/0e70c286-e2c1-42eb-aaa1-5a4ab22bb424"
+					(reference "#PWR039")
+					(unit 1)
+				)
 				(path "/f2858fc4-50de-4ff0-a01c-5b985ee14aef/36ea4b64-9158-43b1-97c6-20da8346f32e"
 					(reference "#PWR030")
@@
 				(path "/f2858fc4-50de-4ff0-a01c-5b985ee14aef/6cef8934-8b7c-410b-8d9f-f073b93271b8"
 					(reference "#PWR024")
+					(unit 1)
+				)
+				(path "/f2858fc4-50de-4ff0-a01c-5b985ee14aef/771becef-f508-42ea-9fb3-6952fb053001"
+					(reference "#PWR037")
 					(unit 1)
 				)
@@
 		(dnp no)
 		(fields_autoplaced yes)
-		(property "Reference" "R27"
+		(property "Reference" "R41"
 			(at 129.54 85.0899 0)
 			(effects
@@
 		(instances
 			(project "VXDash"
+				(path "/f2858fc4-50de-4ff0-a01c-5b985ee14aef/0e70c286-e2c1-42eb-aaa1-5a4ab22bb424"
+					(reference "R69")
+					(unit 1)
+				)
 				(path "/f2858fc4-50de-4ff0-a01c-5b985ee14aef/36ea4b64-9158-43b1-97c6-20da8346f32e"
 					(reference "R33")
@@
 				(path "/f2858fc4-50de-4ff0-a01c-5b985ee14aef/6cef8934-8b7c-410b-8d9f-f073b93271b8"
 					(reference "R27")
+					(unit 1)
+				)
+				(path "/f2858fc4-50de-4ff0-a01c-5b985ee14aef/771becef-f508-42ea-9fb3-6952fb053001"
+					(reference "R41")
 					(unit 1)
 				)
@@
 		(dnp no)
 		(fields_autoplaced yes)
-		(property "Reference" "#PWR023"
+		(property "Reference" "#PWR035"
 			(at 127 113.03 0)
 			(effects
@@
 		(instances
 			(project "VXDash"
+				(path "/f2858fc4-50de-4ff0-a01c-5b985ee14aef/0e70c286-e2c1-42eb-aaa1-5a4ab22bb424"
+					(reference "#PWR038")
+					(unit 1)
+				)
 				(path "/f2858fc4-50de-4ff0-a01c-5b985ee14aef/36ea4b64-9158-43b1-97c6-20da8346f32e"
 					(reference "#PWR029")
@@
 					(unit 1)
 				)
+				(path "/f2858fc4-50de-4ff0-a01c-5b985ee14aef/771becef-f508-42ea-9fb3-6952fb053001"
+					(reference "#PWR035")
+					(unit 1)
+				)

Commit message: Emulator board refinements
- Is there stupid with the Active Hi Optos so that the logic is not inverted ?
- Added N-Mosfet activatable resistors. Stupidly simple ? Better MOSFET recommendation ?
Changed lines of the file:
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@@
 	)
 	(global_label "+3V3"
-		(shape bidirectional)
+		(shape input)
 		(at 157.48 81.28 0)
 		(fields_autoplaced yes)
@@
 		)
 		(property "Intersheetrefs" "${INTERSHEET_REFS}"
-			(at 171.1049 81.28 0)
+			(at 164.891 81.28 0)
 			(effects
 				(font

Commit message: PCB layout in progress
Changed some pin assignments to aid routing.
Parts:
- U7: renamed from U16; value ~ -> DPC817; footprint Package_DIP:SMDIP-4_W7.62mm -> Package_DIP:SMDIP-4_W9.53mm; ALT_MFT_PN_1 (none) -> DPC817S-C-TR; MFT (none) -> Diodes Inc; MFT_PN (none) -> DPC817S-B-TR
- renumbered R41 to R19, R68 to R20
Changed lines of the file:
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@@
 		(dnp no)
 		(fields_autoplaced yes)
-		(property "Reference" "U16"
+		(property "Reference" "U7"
+			(at 138.43 90.17 0)
+			(effects
+				(font
+					(size 1.27 1.27)
+				)
+			)
+		)
+		(property "Value" "DPC817"
 			(at 138.43 92.71 0)
 			(effects
@@
 			)
 		)
-		(property "Value" "~"
-			(at 139.6999 93.98 90)
-			(effects
-				(font
-					(size 1.27 1.27)
-				)
-				(justify left)
-			)
-		)
-		(property "Footprint" "Package_DIP:SMDIP-4_W7.62mm"
+		(property "Footprint" "Package_DIP:SMDIP-4_W9.53mm"
 			(at 138.43 106.68 0)
 			(effects
@@
 			)
 		)
-		(property "MFT" ""
+		(property "MFT" "Diodes Inc"
 			(at 138.43 99.06 90)
 			(effects
@@
 			)
 		)
-		(property "MFT_PN" ""
+		(property "MFT_PN" "DPC817S-B-TR"
 			(at 138.43 99.06 90)
+			(effects
+				(font
+					(size 1.27 1.27)
+				)
+				(hide yes)
+			)
+		)
+		(property "Tolerance" ""
+			(at 138.43 99.06 0)
+			(effects
+				(font
+					(size 1.27 1.27)
+				)
+				(hide yes)
+			)
+		)
+		(property "ALT_MFT_PN_1" "DPC817S-C-TR"
+			(at 138.43 99.06 0)
 			(effects
 				(font
@@
 			(project "VXDash"
 				(path "/f2858fc4-50de-4ff0-a01c-5b985ee14aef/0e70c286-e2c1-42eb-aaa1-5a4ab22bb424"
-					(reference "U19")
+					(reference "U18")
 					(unit 1)
 				)
 				(path "/f2858fc4-50de-4ff0-a01c-5b985ee14aef/36ea4b64-9158-43b1-97c6-20da8346f32e"
+					(reference "U16")
+					(unit 1)
+				)
+				(path "/f2858fc4-50de-4ff0-a01c-5b985ee14aef/4633f9da-2230-4b15-802a-f9ef806e5330"
+					(reference "U15")
+					(unit 1)
+				)
+				(path "/f2858fc4-50de-4ff0-a01c-5b985ee14aef/6cef8934-8b7c-410b-8d9f-f073b93271b8"
+					(reference "U13")
+					(unit 1)
+				)
+				(path "/f2858fc4-50de-4ff0-a01c-5b985ee14aef/771becef-f508-42ea-9fb3-6952fb053001"
+					(reference "U7")
+					(unit 1)
+				)
+				(path "/f2858fc4-50de-4ff0-a01c-5b985ee14aef/c35a8a47-33e6-4037-9210-ef0a9877c6bd"
 					(reference "U14")
 					(unit 1)
 				)
-				(path "/f2858fc4-50de-4ff0-a01c-5b985ee14aef/4633f9da-2230-4b15-802a-f9ef806e5330"
-					(reference "U13")
-					(unit 1)
-				)
-				(path "/f2858fc4-50de-4ff0-a01c-5b985ee14aef/6cef8934-8b7c-410b-8d9f-f073b93271b8"
-					(reference "U11")
-					(unit 1)
-				)
-				(path "/f2858fc4-50de-4ff0-a01c-5b985ee14aef/771becef-f508-42ea-9fb3-6952fb053001"
-					(reference "U16")
-					(unit 1)
-				)
-				(path "/f2858fc4-50de-4ff0-a01c-5b985ee14aef/c35a8a47-33e6-4037-9210-ef0a9877c6bd"
-					(reference "U12")
-					(unit 1)
-				)
 				(path "/f2858fc4-50de-4ff0-a01c-5b985ee14aef/df7be051-e61b-464b-85a0-ebedf6cc1666"
-					(reference "U15")
+					(reference "U17")
 					(unit 1)
 				)
@@
 		(dnp no)
 		(fields_autoplaced yes)
-		(property "Reference" "R68"
+		(property "Reference" "R20"
 			(at 152.4 85.0899 0)
 			(effects
@@
 		)
 		(property "MFT_PN" ""
+			(at 149.86 86.36 0)
+			(effects
+				(font
+					(size 1.27 1.27)
+				)
+				(hide yes)
+			)
+		)
+		(property "Tolerance" ""
 			(at 149.86 86.36 0)
 			(effects
@@
 			(project "VXDash"
 				(path "/f2858fc4-50de-4ff0-a01c-5b985ee14aef/0e70c286-e2c1-42eb-aaa1-5a4ab22bb424"
-					(reference "R70")
+					(reference "R46")
 					(unit 1)
 				)
 				(path "/f2858fc4-50de-4ff0-a01c-5b985ee14aef/36ea4b64-9158-43b1-97c6-20da8346f32e"
+					(reference "R38")
+					(unit 1)
+				)
+				(path "/f2858fc4-50de-4ff0-a01c-5b985ee14aef/4633f9da-2230-4b15-802a-f9ef806e5330"
+					(reference "R36")
+					(unit 1)
+				)
+				(path "/f2858fc4-50de-4ff0-a01c-5b985ee14aef/6cef8934-8b7c-410b-8d9f-f073b93271b8"
+					(reference "R32")
+					(unit 1)
+				)
+				(path "/f2858fc4-50de-4ff0-a01c-5b985ee14aef/771becef-f508-42ea-9fb3-6952fb053001"
+					(reference "R20")
+					(unit 1)
+				)
+				(path "/f2858fc4-50de-4ff0-a01c-5b985ee14aef/c35a8a47-33e6-4037-9210-ef0a9877c6bd"
 					(reference "R34")
 					(unit 1)
 				)
-				(path "/f2858fc4-50de-4ff0-a01c-5b985ee14aef/4633f9da-2230-4b15-802a-f9ef806e5330"
-					(reference "R32")
-					(unit 1)
-				)
-				(path "/f2858fc4-50de-4ff0-a01c-5b985ee14aef/6cef8934-8b7c-410b-8d9f-f073b93271b8"
-					(reference "R28")
-					(unit 1)
-				)
-				(path "/f2858fc4-50de-4ff0-a01c-5b985ee14aef/771becef-f508-42ea-9fb3-6952fb053001"
-					(reference "R68")
-					(unit 1)
-				)
-				(path "/f2858fc4-50de-4ff0-a01c-5b985ee14aef/c35a8a47-33e6-4037-9210-ef0a9877c6bd"
-					(reference "R30")
-					(unit 1)
-				)
 				(path "/f2858fc4-50de-4ff0-a01c-5b985ee14aef/df7be051-e61b-464b-85a0-ebedf6cc1666"
-					(reference "R36")
+					(reference "R40")
 					(unit 1)
 				)
@@
 		(dnp no)
 		(fields_autoplaced yes)
-		(property "Reference" "#PWR037"
+		(property "Reference" "#PWR028"
 			(at 149.86 113.03 0)
 			(effects
@@
 			(project "VXDash"
 				(path "/f2858fc4-50de-4ff0-a01c-5b985ee14aef/0e70c286-e2c1-42eb-aaa1-5a4ab22bb424"
+					(reference "#PWR046")
+					(unit 1)
+				)
+				(path "/f2858fc4-50de-4ff0-a01c-5b985ee14aef/36ea4b64-9158-43b1-97c6-20da8346f32e"
+					(reference "#PWR041")
+					(unit 1)
+				)
+				(path "/f2858fc4-50de-4ff0-a01c-5b985ee14aef/4633f9da-2230-4b15-802a-f9ef806e5330"
 					(reference "#PWR039")
 					(unit 1)
 				)
-				(path "/f2858fc4-50de-4ff0-a01c-5b985ee14aef/36ea4b64-9158-43b1-97c6-20da8346f32e"
-					(reference "#PWR030")
-					(unit 1)
-				)
-				(path "/f2858fc4-50de-4ff0-a01c-5b985ee14aef/4633f9da-2230-4b15-802a-f9ef806e5330"
+				(path "/f2858fc4-50de-4ff0-a01c-5b985ee14aef/6cef8934-8b7c-410b-8d9f-f073b93271b8"
+					(reference "#PWR035")
+					(unit 1)
+				)
+				(path "/f2858fc4-50de-4ff0-a01c-5b985ee14aef/771becef-f508-42ea-9fb3-6952fb053001"
 					(reference "#PWR028")
 					(unit 1)
 				)
-				(path "/f2858fc4-50de-4ff0-a01c-5b985ee14aef/6cef8934-8b7c-410b-8d9f-f073b93271b8"
-					(reference "#PWR024")
-					(unit 1)
-				)
-				(path "/f2858fc4-50de-4ff0-a01c-5b985ee14aef/771becef-f508-42ea-9fb3-6952fb053001"
+				(path "/f2858fc4-50de-4ff0-a01c-5b985ee14aef/c35a8a47-33e6-4037-9210-ef0a9877c6bd"
 					(reference "#PWR037")
 					(unit 1)
 				)
-				(path "/f2858fc4-50de-4ff0-a01c-5b985ee14aef/c35a8a47-33e6-4037-9210-ef0a9877c6bd"
-					(reference "#PWR026")
-					(unit 1)
-				)
 				(path "/f2858fc4-50de-4ff0-a01c-5b985ee14aef/df7be051-e61b-464b-85a0-ebedf6cc1666"
-					(reference "#PWR032")
+					(reference "#PWR043")
 					(unit 1)
 				)
@@
 		(dnp no)
 		(fields_autoplaced yes)
-		(property "Reference" "R41"
+		(property "Reference" "R19"
 			(at 129.54 85.0899 0)
 			(effects
@@
 		)
 		(property "MFT_PN" ""
+			(at 127 86.36 0)
+			(effects
+				(font
+					(size 1.27 1.27)
+				)
+				(hide yes)
+			)
+		)
+		(property "Tolerance" ""
 			(at 127 86.36 0)
 			(effects
@@
 			(project "VXDash"
 				(path "/f2858fc4-50de-4ff0-a01c-5b985ee14aef/0e70c286-e2c1-42eb-aaa1-5a4ab22bb424"
-					(reference "R69")
+					(reference "R45")
 					(unit 1)
 				)
 				(path "/f2858fc4-50de-4ff0-a01c-5b985ee14aef/36ea4b64-9158-43b1-97c6-20da8346f32e"
+					(reference "R37")
+					(unit 1)
+				)
+				(path "/f2858fc4-50de-4ff0-a01c-5b985ee14aef/4633f9da-2230-4b15-802a-f9ef806e5330"
+					(reference "R35")
+					(unit 1)
+				)
+				(path "/f2858fc4-50de-4ff0-a01c-5b985ee14aef/6cef8934-8b7c-410b-8d9f-f073b93271b8"
+					(reference "R31")
+					(unit 1)
+				)
+				(path "/f2858fc4-50de-4ff0-a01c-5b985ee14aef/771becef-f508-42ea-9fb3-6952fb053001"
+					(reference "R19")
+					(unit 1)
+				)
+				(path "/f2858fc4-50de-4ff0-a01c-5b985ee14aef/c35a8a47-33e6-4037-9210-ef0a9877c6bd"
 					(reference "R33")
 					(unit 1)
 				)
-				(path "/f2858fc4-50de-4ff0-a01c-5b985ee14aef/4633f9da-2230-4b15-802a-f9ef806e5330"
-					(reference "R31")
-					(unit 1)
-				)
-				(path "/f2858fc4-50de-4ff0-a01c-5b985ee14aef/6cef8934-8b7c-410b-8d9f-f073b93271b8"
-					(reference "R27")
-					(unit 1)
-				)
-				(path "/f2858fc4-50de-4ff0-a01c-5b985ee14aef/771becef-f508-42ea-9fb3-6952fb053001"
-					(reference "R41")
-					(unit 1)
-				)
-				(path "/f2858fc4-50de-4ff0-a01c-5b985ee14aef/c35a8a47-33e6-4037-9210-ef0a9877c6bd"
-					(reference "R29")
-					(unit 1)
-				)
 				(path "/f2858fc4-50de-4ff0-a01c-5b985ee14aef/df7be051-e61b-464b-85a0-ebedf6cc1666"
-					(reference "R35")
+					(reference "R39")
 					(unit 1)
 				)
@@
 		(dnp no)
 		(fields_autoplaced yes)
-		(property "Reference" "#PWR035"
+		(property "Reference" "#PWR027"
 			(at 127 113.03 0)
 			(effects
@@
 			(project "VXDash"
 				(path "/f2858fc4-50de-4ff0-a01c-5b985ee14aef/0e70c286-e2c1-42eb-aaa1-5a4ab22bb424"
+					(reference "#PWR045")
+					(unit 1)
+				)
+				(path "/f2858fc4-50de-4ff0-a01c-5b985ee14aef/36ea4b64-9158-43b1-97c6-20da8346f32e"
+					(reference "#PWR040")
+					(unit 1)
+				)
+				(path "/f2858fc4-50de-4ff0-a01c-5b985ee14aef/4633f9da-2230-4b15-802a-f9ef806e5330"
 					(reference "#PWR038")
 					(unit 1)
 				)
-				(path "/f2858fc4-50de-4ff0-a01c-5b985ee14aef/36ea4b64-9158-43b1-97c6-20da8346f32e"
-					(reference "#PWR029")
-					(unit 1)
-				)
-				(path "/f2858fc4-50de-4ff0-a01c-5b985ee14aef/4633f9da-2230-4b15-802a-f9ef806e5330"
+				(path "/f2858fc4-50de-4ff0-a01c-5b985ee14aef/6cef8934-8b7c-410b-8d9f-f073b93271b8"
+					(reference "#PWR034")
+					(unit 1)
+				)
+				(path "/f2858fc4-50de-4ff0-a01c-5b985ee14aef/771becef-f508-42ea-9fb3-6952fb053001"
 					(reference "#PWR027")
 					(unit 1)
 				)
-				(path "/f2858fc4-50de-4ff0-a01c-5b985ee14aef/6cef8934-8b7c-410b-8d9f-f073b93271b8"
-					(reference "#PWR023")
-					(unit 1)
-				)
-				(path "/f2858fc4-50de-4ff0-a01c-5b985ee14aef/771becef-f508-42ea-9fb3-6952fb053001"
-					(reference "#PWR035")
-					(unit 1)
-				)
 				(path "/f2858fc4-50de-4ff0-a01c-5b985ee14aef/c35a8a47-33e6-4037-9210-ef0a9877c6bd"
-					(reference "#PWR025")
+					(reference "#PWR036")
 					(unit 1)
 				)
 				(path "/f2858fc4-50de-4ff0-a01c-5b985ee14aef/df7be051-e61b-464b-85a0-ebedf6cc1666"
-					(reference "#PWR031")
-					(unit 1)
-				)
+					(reference "#PWR042")
+					(unit 1)
+				)

Commit message: ERC corrections, idiot lights
- VXDash : added idiot lights (also to emulator board)
- VXDash : corrected some ERC violations
Connections:
- net ~{LL_output} renamed ~{LL_Output}
Changed lines of the file:
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@@
 		)
 	)
-	(hierarchical_label "~{LL_output}"
+	(hierarchical_label "~{LL_Output}"
 		(shape output)
 		(at 157.48 96.52 0)

Commit message: BOM first pass
- Still missing some internal connectors definitions
- Alternative to use a 4x4ch opto config instead of 16x1 ?
- Alternative LiteOn optos identified (easier to source on LCSC)
Parts:
- R19: footprint Resistor_SMD:R_0805_2012Metric_Pad1.20x1.40mm_HandSolder -> Resistor_SMD:R_0603_1608Metric_Pad0.98x0.95mm_HandSolder; LCSC (none) -> C114637; MFT (none) -> Yageo; MFT_PN (none) -> RC0603FR-078K2L
- R20: footprint Resistor_SMD:R_0805_2012Metric_Pad1.20x1.40mm_HandSolder -> Resistor_SMD:R_0603_1608Metric_Pad0.98x0.95mm_HandSolder; LCSC (none) -> C98220; MFT (none) -> Yageo; MFT_PN (none) -> RC0603FR-0710KL
- U7: LCSC (none) -> C22454766; LCSC alt (none) -> C125121
Changed lines of the file:
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@@
 		(comment 2 "https://cadlab.io/projects/vxdash")
+	)
+	(text_box "Single channel alternative : LiteOn LTV-817S"
+		(exclude_from_sim no)
+		(at 120.65 115.57 0)
+		(size 52.07 5.08)
+		(margins 0.9525 0.9525 0.9525 0.9525)
+		(stroke
+			(width 0)
+			(type solid)
+		)
+		(fill
+			(type none)
+		)
+		(effects
+			(font
+				(size 1.27 1.27)
+			)
+			(justify left top)
+		)
 	)
 	(text_box "Assume 50% CTR w.c.\nVf = 1.2V @1mA\nLowest battery = 10V\n\nCircuit CTR:\nIf = (10V-1.2V)/1mA = 8.8k. \nLower closest 8k2 = 1.07mA\nIc = 3.3/10k = 330uA\nCTRc = 0.33/1.07 = 30.8%\n\nOpto is always in saturation\n"
@@
 			)
 		)
-		(property "LCSC" ""
-			(at 138.43 99.06 0)
-			(effects
-				(font
-					(size 1.27 1.27)
-				)
-				(hide yes)
-			)
-		)
-		(property "LCSC alt" ""
+		(property "LCSC" "C22454766"
+			(at 138.43 99.06 0)
+			(effects
+				(font
+					(size 1.27 1.27)
+				)
+				(hide yes)
+			)
+		)
+		(property "LCSC alt" "C125121"
 			(at 138.43 99.06 0)
 			(effects
@@
 				)
 				(hide yes)
+			)
+		)
+		(property "Ippm" ""
+			(at 138.43 99.06 0)
+			(effects
+				(font
+					(size 1.27 1.27)
+				)
+			)
+		)
+		(property "Vbr" ""
+			(at 138.43 99.06 0)
+			(effects
+				(font
+					(size 1.27 1.27)
+				)
+			)
+		)
+		(property "Vwm" ""
+			(at 138.43 99.06 0)
+			(effects
+				(font
+					(size 1.27 1.27)
+				)
 			)
 		)
@@
 			)
 		)
-		(property "Footprint" "Resistor_SMD:R_0805_2012Metric_Pad1.20x1.40mm_HandSolder"
+		(property "Footprint" "Resistor_SMD:R_0603_1608Metric_Pad0.98x0.95mm_HandSolder"
 			(at 148.082 86.36 90)
 			(effects
@@
 			)
 		)
-		(property "Datasheet" ""
+		(property "Datasheet" "http://datasheet.octopart.com/RC0603FR-0710KL-Yageo-datasheet-141265859.pdf"
 			(at 149.86 86.36 0)
 			(effects
@@
 			)
 		)
-		(property "MFT" ""
-			(at 149.86 86.36 0)
-			(effects
-				(font
-					(size 1.27 1.27)
-				)
-				(hide yes)
-			)
-		)
-		(property "MFT_PN" ""
+		(property "MFT" "Yageo"
+			(at 149.86 86.36 0)
+			(effects
+				(font
+					(size 1.27 1.27)
+				)
+				(hide yes)
+			)
+		)
+		(property "MFT_PN" "RC0603FR-0710KL"
 			(at 149.86 86.36 0)
 			(effects
@@
 			)
 		)
-		(property "LCSC" ""
+		(property "LCSC" "C98220"
 			(at 149.86 86.36 0)
 			(effects
@@
 				)
 				(hide yes)
+			)
+		)
+		(property "Ippm" ""
+			(at 149.86 86.36 0)
+			(effects
+				(font
+					(size 1.27 1.27)
+				)
+			)
+		)
+		(property "Vbr" ""
+			(at 149.86 86.36 0)
+			(effects
+				(font
+					(size 1.27 1.27)
+				)
+			)
+		)
+		(property "Vwm" ""
+			(at 149.86 86.36 0)
+			(effects
+				(font
+					(size 1.27 1.27)
+				)
 			)
 		)
@@
 			)
 		)
-		(property "Footprint" "Resistor_SMD:R_0805_2012Metric_Pad1.20x1.40mm_HandSolder"
+		(property "Footprint" "Resistor_SMD:R_0603_1608Metric_Pad0.98x0.95mm_HandSolder"
 			(at 125.222 86.36 90)
 			(effects
@@
 			)
 		)
-		(property "Datasheet" ""
+		(property "Datasheet" "http://datasheet.octopart.com/RC0603FR-078K2L-Yageo-datasheet-164759695.pdf"
 			(at 127 86.36 0)
 			(effects
@@
 			)
 		)
-		(property "MFT" ""
-			(at 127 86.36 0)
-			(effects
-				(font
-					(size 1.27 1.27)
-				)
-				(hide yes)
-			)
-		)
-		(property "MFT_PN" ""
+		(property "MFT" "Yageo"
+			(at 127 86.36 0)
+			(effects
+				(font
+					(size 1.27 1.27)
+				)
+				(hide yes)
+			)
+		)
+		(property "MFT_PN" "RC0603FR-078K2L"
 			(at 127 86.36 0)
 			(effects
@@
 			)
 		)
-		(property "LCSC" ""
+		(property "LCSC" "C114637"
 			(at 127 86.36 0)
 			(effects
@@
 			)
 		)
+		(property "Ippm" ""
+			(at 127 86.36 0)
+			(effects
+				(font
+					(size 1.27 1.27)
+				)
+			)
+		)
+		(property "Vbr" ""
+			(at 127 86.36 0)
+			(effects
+				(font
+					(size 1.27 1.27)
+				)
+			)
+		)
+		(property "Vwm" ""
+			(at 127 86.36 0)
+			(effects
+				(font
+					(size 1.27 1.27)
+				)
+			)
+		)
