File: KiCad PCB Files/VXDash/Rsensing_Pair.kicad_sch (KiCad schematic)
At the start: 27 parts, among them IC2 AS2333_OpAmp, IC5 AS2333_OpAmp, Q3 DMP3099L, Q4 DMP3099L, Q5 DMP3099L, Q6 DMP3099L

Commit message: Moved VXDash project into sub folder
Parts:
- renumbered C41 to C22, C42 to C23, C43 to C24, D7 to D1, D8 to D2, D9 to D6, D11 to D7, IC2 to IC5, IC5 to IC6, Q3 to Q1, Q4 to Q2, Q5 to Q3, Q6 to Q4, R55 to R42, R56 to R43, R57 to R44, R58 to R45, R59 to R46, R60 to R47, R61 to R48, R66 to R49, R67 to R54, R68 to R55, R69 to R64, R70 to R65, R71 to R66, R72 to R67

Commit message: Grape shot additions
- Added 0R to the VCC pin on the CAN transceiver for pin compatibility with other transceiver
- Updated TODO box
- Rename ADC_SDA and ADC_SCL to SDA and SCL
- Official symbol and footprint from ESP, using ESP32-S3-WROOM-1-N16R8
- Reassigned Coolant LOW to active HI
- Replaced MUX with i²C TCA9555 IO Expander
- Resequenced Active His and Lows to match current SW definition
- Resequenced ADC channels to match current SW definition
- Added simple peripherals for MCU
- Added RESET and BOOT buttons circuits
- Added CAN transceivers for each display, and Termination resistor
- Added USB C
Other:
- company: (none) -> Alex Miller & Martin Roger
- title: Dual Op-Amp Constant current source resistive sensor -> Main architecture
Changed lines of the file:
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@@
 	(paper "A4")
 	(title_block
-		(title "Dual Op-Amp Constant current source resistive sensor")
-		(date "2025-08-08")
+		(title "Main architecture")
+		(date "2025-08-10")
 		(rev "1.4")
+		(company "Alex Miller & Martin Roger")
 		(comment 1 "https://github.com/martinroger/VXDash")
 		(comment 2 "https://cadlab.io/projects/vxdash")

Commit message: Minor changes
- Connection for the caliber selection on the sensing circuit
- Typo
Changed lines of the file:
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@@
 		)
 	)
-	(text_box "ADC range 2.7V. Allows for reasonable voltage drop across current source and diode.\n300R and 3k max sensor resistance per range.\nLow range = 2.7 / 300 = 9mA,\nHigh range = 2.7 / 3k = 900uA.\n150mV Vref. \nLow range = 150mV / 9mA = 16.666 ohm\nHigh range 150mA / 900uA = 166.666 ohm\n\nHigh range = 160R + 6R8 = 166R8 = 899.2uA\nLow range = 18R || 166R8 = 16.247R = 9.232mA\n"
+	(text_box "ADC range 2.7V. Allows for reasonable voltage drop across current source and diode.\n300R and 3k max sensor resistance per range.\nLow range = 2.7 / 300 = 9mA,\nHigh range = 2.7 / 3k = 900uA.\n150mV Vref. \nLow range = 150mV / 9mA = 16.666 ohm\nHigh range 150mV / 900uA = 166.666 ohm\n\nHigh range = 160R + 6R8 = 166R8 = 899.2uA\nLow range = 18R || 166R8 = 16.247R = 9.232mA\n"
 		(exclude_from_sim no)
 		(at 118.11 49.53 0)

Commit message: PCB layout in progress
Changed some pin assignments to aid routing.
Parts:
- renumbered C22 to C27, C23 to C28, C24 to C29, D6 to D3, D7 to D4, IC5 to IC4, IC6 to IC5, R42 to R47, R43 to R48, R44 to R49, R45 to R50, R46 to R51, R47 to R52, R48 to R53, R49 to R54, R54 to R55, R55 to R56, R64 to R57, R65 to R58, R66 to R59, R67 to R60

Commit message: ERC corrections, idiot lights
- VXDash : added idiot lights (also to emulator board)
- VXDash : corrected some ERC violations
Parts:
- removed IC5: AS2333_OpAmp, Package_SO:MSOP-8_3x3mm_P0.65mm, symbol VXDash_ICs:AS2333_OpAmp
Connections:
- net Vref: now also IC4.6 (-)
- net at Q4.2 (S), R57.1: now also IC4.5 (+)
- net at R54.1: now also IC4.7
Changed lines of the file:
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@@
+	(symbol
+		(lib_id "VXDash_ICs:AS2333_OpAmp")
+		(at 184.15 96.52 0)
+		(unit 2)
+		(exclude_from_sim no)
+		(in_bom yes)
+		(on_board yes)
+		(dnp no)
+		(fields_autoplaced yes)
+		(property "Reference" "IC4"
+			(at 184.15 86.36 0)
+			(effects
+				(font
+					(size 1.27 1.27)
+				)
+			)
+		)
+		(property "Value" "AS2333_OpAmp"
+			(at 184.15 88.9 0)
+			(effects
+				(font
+					(size 1.27 1.27)
+				)
+			)
+		)
+		(property "Footprint" "Package_SO:MSOP-8_3x3mm_P0.65mm"
+			(at 184.15 83.82 0)
+			(effects
+				(font
+					(size 1.27 1.27)
+				)
+				(hide yes)
+			)
+		)
+		(property "Datasheet" "https://www.diodes.com/assets/Datasheets/AS2333.pdf"
+			(at 184.15 81.28 0)
+			(effects
+				(font
+					(size 1.27 1.27)
+				)
+				(hide yes)
+			)
+		)
+		(property "Description" "1.8V, MICROPOWER CMOS ZERO-DRIFT OPERATIONAL AMPLIFIERS"
+			(at 184.15 78.74 0)
+			(effects
+				(font
+					(size 1.27 1.27)
+				)
+				(hide yes)
+			)
+		)
+		(property "MFT" "Diode Inc"
+			(at 184.15 73.66 0)
+			(effects
+				(font
+					(size 1.27 1.27)
+				)
+				(hide yes)
+			)
+		)
+		(property "MFT_PN" "AS2333M8-13"
+			(at 184.15 76.2 0)
+			(effects
+				(font
+					(size 1.27 1.27)
+				)
+				(hide yes)
+			)
+		)
+		(property "Tolerance" ""
+			(at 184.15 96.52 0)
+			(effects
+				(font
+					(size 1.27 1.27)
+				)
+				(hide yes)
+			)
+		)
+		(pin "2"
+		)
+		(pin "4"
+		)
+		(pin "7"
+		)
+		(pin "3"
+		)
+		(pin "8"
+		)
+		(pin "1"
+		)
+		(pin "5"
+		)
+		(pin "6"
+		)
+		(instances
+			(project "VXDash"
+				(path "/f2858fc4-50de-4ff0-a01c-5b985ee14aef/024f3b9c-af80-4b8c-9e91-7ad2b6b7f854/17fb3549-8ca7-418f-beb2-9d5e3767d202"
+					(reference "IC4")
+					(unit 2)
+				)
+			)
+		)
+	)
 	(symbol
 		(lib_id "VXDash_ICs:AS2333_OpAmp")
@@
 					(unit 1)
 				)
-			)
-		)
-	)
-	(symbol
-		(lib_id "VXDash_ICs:AS2333_OpAmp")
-		(at 184.15 96.52 0)
-		(unit 1)
-		(exclude_from_sim no)
-		(in_bom yes)
-		(on_board yes)
-		(dnp no)
-		(fields_autoplaced yes)
-		(property "Reference" "IC5"
-			(at 184.15 86.36 0)
-			(effects
-				(font
-					(size 1.27 1.27)
-				)
-			)
-		)
-		(property "Value" "AS2333_OpAmp"
-			(at 184.15 88.9 0)
-			(effects
-				(font
-					(size 1.27 1.27)
-				)
-			)
-		)
-		(property "Footprint" "Package_SO:MSOP-8_3x3mm_P0.65mm"
-			(at 184.15 83.82 0)
-			(effects
-				(font
-					(size 1.27 1.27)
-				)
-				(hide yes)
-			)
-		)
-		(property "Datasheet" "https://www.diodes.com/assets/Datasheets/AS2333.pdf"
-			(at 184.15 81.28 0)
-			(effects
-				(font
-					(size 1.27 1.27)
-				)
-				(hide yes)
-			)
-		)
-		(property "Description" "1.8V, MICROPOWER CMOS ZERO-DRIFT OPERATIONAL AMPLIFIERS"
-			(at 184.15 78.74 0)
-			(effects
-				(font
-					(size 1.27 1.27)
-				)
-				(hide yes)
-			)
-		)
-		(property "MFT" "Diode Inc"
-			(at 184.15 73.66 0)
-			(effects
-				(font
-					(size 1.27 1.27)
-				)
-				(hide yes)
-			)
-		)
-		(property "MFT_PN" "AS2333M8-13"
-			(at 184.15 76.2 0)
-			(effects
-				(font
-					(size 1.27 1.27)
-				)
-				(hide yes)
-			)
-		)
-		(property "Tolerance" ""
-			(at 184.15 96.52 0)
-			(effects
-				(font
-					(size 1.27 1.27)
-				)
-				(hide yes)
-			)
-		)
-		(pin "2"
-		)
-		(pin "4"
-		)
-		(pin "7"
-		)
-		(pin "3"
-		)
-		(pin "8"
-		)
-		(pin "1"
-		)
-		(pin "5"
-		)
-		(pin "6"
-		)
-		(instances
-			(project "VXDash"
-				(path "/f2858fc4-50de-4ff0-a01c-5b985ee14aef/024f3b9c-af80-4b8c-9e91-7ad2b6b7f854/17fb3549-8ca7-418f-beb2-9d5e3767d202"
-					(reference "IC5")
-					(unit 1)
-				)

Commit message: New main dash PCB - WIP inc. CAD
Parts:
- added unit 1 of IC4
Connections:
- net +3V3: now also IC4.8; no longer IC4.8
- net GND: now also IC4.4; no longer IC4.4
- net Vref: now also IC4.2 (-); no longer IC4.2 (-)
- net at R47.1: now also IC4.1; no longer IC4.1
- net at Q2.2 (S), R50.1: now also IC4.3 (+); no longer IC4.3 (+)

Commit message: Fields updates
Parts:
- IC4: LCSC (none) -> C5948553

Commit message: BOM first pass
- Still missing some internal connectors definitions
- Alternative to use a 4x4ch opto config instead of 16x1 ?
- Alternative LiteOn optos identified (easier to source on LCSC)
Parts:
- C27: LCSC (none) -> C16194176; MFT (none) -> Samsung Electro-Mechanics; MFT_PN (none) -> CL10B104KB8NNWC
- C28, C29: LCSC (none) -> C106856; MFT (none) -> Yageo; MFT_PN (none) -> CC0603KRX7R9BB333
- D1, D2, D3, D4: LCSC (none) -> C152458
- Q1, Q2, Q3, Q4: LCSC (none) -> C155244
- R47, R48, R54, R55: LCSC (none) -> C22548; MFT (none) -> Yageo; MFT_PN (none) -> RC0603FR-071KL
- R49, R56: LCSC (none) -> C245924; MFT (none) -> Yageo; MFT_PN (none) -> RC0603FR-0718RL
- R50, R57: LCSC (none) -> C21189; MFT (none) -> Royal Ohm; MFT_PN (none) -> 0603WAF0000T5E
- R51, R58: LCSC (none) -> C131398; MFT (none) -> Yageo; MFT_PN (none) -> RC1206FR-071KL
- R52, R59: LCSC (none) -> C185369; MFT (none) -> Yageo; MFT_PN (none) -> RC0603FR-07160RL
- R53, R60: LCSC (none) -> C23214; MFT (none) -> Royal Ohm; MFT_PN (none) -> 0603WAF680KT5E
