File: KiCad PCB Files/VXDash/VXDash.kicad_pcb (KiCad board)
At the start: 4 copper layers, 245.2 x 136.8 mm, 233 parts, among them IC1 CD74HC4050M96, IC2 AP62200, IC3 AP62200, IC4 AS2333_OpAmp, IC5 AP62200, IC6 ATA6561, IC7 ATA6561, IC9 ATA6561, J1 Header_VX220_RightAngle, J10 CANbus, J2 Alarm port, J3 I²C debug, J4 UART0 debug, J5 LD_CAN, J6 RD_CAN, J7 USB4105-GF-A, J8 LD_UART, J9 RD_UART, Q1 DMP3099L, Q2 DMP3099L, Q3 DMP3099L, Q4 DMP3099L, Q5 2N7002, Q6 PJA3441, Q7 PJA3441, U1 TCA9555PWR, U10 DPC817, U11 DPC817, U12 DPC817, U13 DPC817, U14 DPC817, U15 DPC817, U16 DPC817, U17 DPC817, U18 DPC817, U19 ADS1115IDGS, U2 ESP32-S3-WROOM-1, U3 DPC817, U4 DPC817, U5 DPC817, U6 DPC817, U7 DPC817, U8 DPC817, U9 DPC817

Commit message: PCB refresh from schematic
Parts:
- added C53: 100n, Capacitor_SMD:C_0603_1608Metric_Pad1.08x0.95mm_HandSolder, B.Cu at (283.5, 104.0)
- added C54: 100n, Capacitor_SMD:C_0603_1608Metric_Pad1.08x0.95mm_HandSolder, B.Cu at (283.5, 106.5)
- added C55: 100n, Capacitor_SMD:C_0603_1608Metric_Pad1.08x0.95mm_HandSolder, B.Cu at (283.5, 109.0)
- added C56: 100n, Capacitor_SMD:C_0603_1608Metric_Pad1.08x0.95mm_HandSolder, B.Cu at (283.5, 111.5)
- added C61: 100n, Capacitor_SMD:C_0603_1608Metric_Pad1.08x0.95mm_HandSolder, B.Cu at (283.5, 114.0)
- added C62: 100n, Capacitor_SMD:C_0603_1608Metric_Pad1.08x0.95mm_HandSolder, B.Cu at (283.5, 116.5)
- added D22: BAT54, Diode_SMD:D_SOD-123, B.Cu at (242.4, 131.1)
- added D23: BAT54, Diode_SMD:D_SOD-123, B.Cu at (242.4, 108.6)
- added D24: BAT54, Diode_SMD:D_SOD-123, B.Cu at (230.1, 131.1)
- added D25: BAT54, Diode_SMD:D_SOD-123, B.Cu at (258.2, 151.6)
- added D26: BAT54, Diode_SMD:D_SOD-123, B.Cu at (230.1, 119.8)
- added D27: BAT54, Diode_SMD:D_SOD-123, B.Cu at (270.5, 151.6)
- added D28: BAT54, Diode_SMD:D_SOD-123, B.Cu at (282.8, 151.6)
- added D29: BAT54, Diode_SMD:D_SOD-123, B.Cu at (230.1, 108.6)
- added D30: BAT54, Diode_SMD:D_SOD-123, B.Cu at (242.4, 119.8)
- added D31: BAT54, Diode_SMD:D_SOD-123, B.Cu at (250.4, 104.4)
- added D32: BAT54, Diode_SMD:D_SOD-123, B.Cu at (250.4, 107.7)
- added J11: LD connector, Connector_JST:JST_PH_S8B-PH-K_1x08_P2.00mm_Horizontal, B.Cu at (278.4, 105.1)
- added J12: RD connector, Connector_JST:JST_PH_S8B-PH-K_1x08_P2.00mm_Horizontal, B.Cu at (278.4, 114.7)
- added J2: FASCIA PASSTHRU, Connector_JST:JST_PHD_S16B-PHDSS_2x08_P2.00mm_Horizontal, B.Cu at (278.4, 123.6)
- added J5: CAN debug, Connector_PinHeader_2.54mm:PinHeader_1x03_P2.54mm_Vertical, B.Cu at (268.7, 136.0)
- added JP10: EN LOAD EMU, Jumper:SolderJumper-2_P1.3mm_Open_RoundedPad1.0x1.5mm, B.Cu at (224.9, 104.5)
- added JP11: EN LOAD EMU, Jumper:SolderJumper-2_P1.3mm_Open_RoundedPad1.0x1.5mm, B.Cu at (237.2, 115.7)
- added JP3: EN LOAD EMU, Jumper:SolderJumper-2_P1.3mm_Open_RoundedPad1.0x1.5mm, B.Cu at (237.2, 104.5)
- added JP4: EN LOAD EMU, Jumper:SolderJumper-2_P1.3mm_Open_RoundedPad1.0x1.5mm, B.Cu at (237.2, 126.9)
- added JP5: EN LOAD EMU, Jumper:SolderJumper-2_P1.3mm_Open_RoundedPad1.0x1.5mm, B.Cu at (224.9, 126.9)
- added JP6: EN LOAD EMU, Jumper:SolderJumper-2_P1.3mm_Open_RoundedPad1.0x1.5mm, B.Cu at (253.0, 147.5)
- added JP7: EN LOAD EMU, Jumper:SolderJumper-2_P1.3mm_Open_RoundedPad1.0x1.5mm, B.Cu at (224.9, 115.7)
- added JP8: EN LOAD EMU, Jumper:SolderJumper-2_P1.3mm_Open_RoundedPad1.0x1.5mm, B.Cu at (265.3, 147.5)
- added JP9: EN LOAD EMU, Jumper:SolderJumper-2_P1.3mm_Open_RoundedPad1.0x1.5mm, B.Cu at (277.6, 147.5)
- added R106: 47R, Resistor_SMD:R_0603_1608Metric_Pad0.98x0.95mm_HandSolder, B.Cu at (237.4, 108.2)
- added R107: 15R, Resistor_SMD:R_0603_1608Metric_Pad0.98x0.95mm_HandSolder, B.Cu at (237.4, 110.7)
- added R108: 680R, Resistor_SMD:R_1210_3225Metric_Pad1.30x2.65mm_HandSolder, B.Cu at (230.1, 127.3)
- added R109: 47R, Resistor_SMD:R_0603_1608Metric_Pad0.98x0.95mm_HandSolder, B.Cu at (225.1, 130.6)
- added R110: 15R, Resistor_SMD:R_0603_1608Metric_Pad0.98x0.95mm_HandSolder, B.Cu at (225.1, 133.1)
- added R111: 680R, Resistor_SMD:R_1210_3225Metric_Pad1.30x2.65mm_HandSolder, B.Cu at (258.1, 147.9)
- added R112: 47R, Resistor_SMD:R_0603_1608Metric_Pad0.98x0.95mm_HandSolder, B.Cu at (253.1, 151.2)
- added R113: 15R, Resistor_SMD:R_0603_1608Metric_Pad0.98x0.95mm_HandSolder, B.Cu at (253.1, 153.7)
- added R114: 680R, Resistor_SMD:R_1210_3225Metric_Pad1.30x2.65mm_HandSolder, B.Cu at (230.1, 116.0)
- added R115: 47R, Resistor_SMD:R_0603_1608Metric_Pad0.98x0.95mm_HandSolder, B.Cu at (225.1, 119.4)
- added R116: 15R, Resistor_SMD:R_0603_1608Metric_Pad0.98x0.95mm_HandSolder, B.Cu at (225.1, 121.9)
- added R117: 680R, Resistor_SMD:R_1210_3225Metric_Pad1.30x2.65mm_HandSolder, B.Cu at (270.4, 147.9)
- added R118: 47R, Resistor_SMD:R_0603_1608Metric_Pad0.98x0.95mm_HandSolder, B.Cu at (265.4, 151.2)
- added R119: 15R, Resistor_SMD:R_0603_1608Metric_Pad0.98x0.95mm_HandSolder, B.Cu at (265.4, 153.7)
- added R120: 680R, Resistor_SMD:R_1210_3225Metric_Pad1.30x2.65mm_HandSolder, B.Cu at (282.7, 147.9)
- added R121: 47R, Resistor_SMD:R_0603_1608Metric_Pad0.98x0.95mm_HandSolder, B.Cu at (277.7, 151.2)
- added R122: 15R, Resistor_SMD:R_0603_1608Metric_Pad0.98x0.95mm_HandSolder, B.Cu at (277.7, 153.7)
- added R123: 680R, Resistor_SMD:R_1210_3225Metric_Pad1.30x2.65mm_HandSolder, B.Cu at (230.1, 104.8)
- added R124: 47R, Resistor_SMD:R_0603_1608Metric_Pad0.98x0.95mm_HandSolder, B.Cu at (225.1, 108.2)
- added R125: 15R, Resistor_SMD:R_0603_1608Metric_Pad0.98x0.95mm_HandSolder, B.Cu at (225.1, 110.7)
- added R126: 680R, Resistor_SMD:R_1210_3225Metric_Pad1.30x2.65mm_HandSolder, B.Cu at (242.4, 116.0)
- added R127: 47R, Resistor_SMD:R_0603_1608Metric_Pad0.98x0.95mm_HandSolder, B.Cu at (237.4, 119.4)
- added R128: 15R, Resistor_SMD:R_0603_1608Metric_Pad0.98x0.95mm_HandSolder, B.Cu at (237.4, 121.9)
- added R129: 0R, Resistor_SMD:R_0805_2012Metric_Pad1.20x1.40mm_HandSolder, B.Cu at (264.0, 135.1)
- added R130: 10k, Resistor_SMD:R_0603_1608Metric_Pad0.98x0.95mm_HandSolder, B.Cu at (283.5, 121.5)
- added R131: 15R, Resistor_SMD:R_1206_3216Metric_Pad1.30x1.75mm_HandSolder, B.Cu at (250.3, 114.3)
- added R132: 100R, Resistor_SMD:R_2512_6332Metric_Pad1.40x3.35mm_HandSolder, B.Cu at (256.9, 124.5)
- added R133: 150R, Resistor_SMD:R_2512_6332Metric_Pad1.40x3.35mm_HandSolder, B.Cu at (256.9, 129.3)
- added R134: 100R, Resistor_SMD:R_2512_6332Metric_Pad1.40x3.35mm_HandSolder, B.Cu at (256.9, 134.2)
- added R135: 150R, Resistor_SMD:R_2512_6332Metric_Pad1.40x3.35mm_HandSolder, B.Cu at (256.9, 139.1)
- added R136: 120R, Resistor_SMD:R_0805_2012Metric_Pad1.20x1.40mm_HandSolder, B.Cu at (264.0, 138.1)
- added R137: 120R, Resistor_SMD:R_0805_2012Metric_Pad1.20x1.40mm_HandSolder, B.Cu at (264.0, 141.0)
- added R138: 10k, Resistor_SMD:R_0603_1608Metric_Pad0.98x0.95mm_HandSolder, B.Cu at (283.5, 124.0)
- added R139: 10k, Resistor_SMD:R_0603_1608Metric_Pad0.98x0.95mm_HandSolder, B.Cu at (283.5, 126.6)
- added R91: 10k, Resistor_SMD:R_0603_1608Metric_Pad0.98x0.95mm_HandSolder, B.Cu at (283.5, 119.0)
- added R94: 680R, Resistor_SMD:R_1210_3225Metric_Pad1.30x2.65mm_HandSolder, B.Cu at (242.4, 127.3)
- added R95: 47R, Resistor_SMD:R_0603_1608Metric_Pad0.98x0.95mm_HandSolder, B.Cu at (237.4, 130.6)
- added R96: 15R, Resistor_SMD:R_0603_1608Metric_Pad0.98x0.95mm_HandSolder, B.Cu at (237.4, 133.1)
- added R97: 15R, Resistor_SMD:R_1206_3216Metric_Pad1.30x1.75mm_HandSolder, B.Cu at (250.3, 111.1)
- added R98: 680R, Resistor_SMD:R_1210_3225Metric_Pad1.30x2.65mm_HandSolder, B.Cu at (242.4, 104.8)
- added SW1: RESET, Button_Switch_THT:SW_PUSH_1P1T_6x3.5mm_H5.0_APEM_MJTP1250, B.Cu at (279.4, 136.2)
- added SW2: BOOT, Button_Switch_THT:SW_PUSH_1P1T_6x3.5mm_H5.0_APEM_MJTP1250, B.Cu at (279.4, 141.2)
- added TP1: 5V, TestPoint:TestPoint_Pad_D2.0mm, B.Cu at (259.4, 104.7)
- added TP2: VBUS, TestPoint:TestPoint_Pad_D2.0mm, B.Cu at (259.4, 108.8)
- added TP3: EXP_INT, TestPoint:TestPoint_Pad_D2.0mm, B.Cu at (259.4, 112.8)
- added TP4: PROT_12V, TestPoint:TestPoint_Pad_D2.0mm, B.Cu at (259.4, 116.9)
- added TP5: 5V_A, TestPoint:TestPoint_Pad_D2.0mm, B.Cu at (255.3, 104.7)
- added TP6: 5V_B, TestPoint:TestPoint_Pad_D2.0mm, B.Cu at (255.3, 108.8)
- added TP7: 3V3, TestPoint:TestPoint_Pad_D2.0mm, B.Cu at (255.3, 112.8)
- added TP8: ADS_VREF, TestPoint:TestPoint_Pad_D2.0mm, B.Cu at (243.3, 138.4)
- D20, D21: moved to B.Cu
- R100, R89: value 620 -> 620R
- R101, R102, R103, R104, R105: value 270 -> 270R
- R11, R12, R13, R14, R15, R16, R17, R18, R19, R20, R21, R22, R23, R24, R25, R26, R27, R28, R29, R30, R31, R32, R33, R34, R35, R36, R37, R38, R39, R40, R45, R46: footprint Resistor_SMD:R_0805_2012Metric_Pad1.20x1.40mm_HandSolder -> Resistor_SMD:R_0603_1608Metric_Pad0.98x0.95mm_HandSolder
- R5, R6: value 60R -> 120R
- R64, R71, R75: value 1K -> 1k
- R66: value 1Meg -> 1M
- R92: value 270 -> 100R; footprint Resistor_SMD:R_1206_3216Metric_Pad1.30x1.75mm_HandSolder -> Resistor_SMD:R_2512_6332Metric_Pad1.40x3.35mm_HandSolder; moved to B.Cu
- R93: value 270 -> 150R; footprint Resistor_SMD:R_1206_3216Metric_Pad1.30x1.75mm_HandSolder -> Resistor_SMD:R_2512_6332Metric_Pad1.40x3.35mm_HandSolder; moved to B.Cu
- moved D20 10.2 mm to (149.6, 98.2)
- moved R92 8.50 mm to (151.2, 103.2)
- moved R93 8.50 mm to (159.8, 103.2)
- moved D21 6.83 mm to (158.1, 98.2)
Connections:
- net R_TURN_ActLO renamed R_TURN_ActHI
- C31 pad 1: +5V -> /Left Display CAN XCVR/V_SUPPLY
- C32 pad 1: +5V -> /Left Display CAN XCVR/V_SUPPLY
- R61 pad 2: +5V -> /Left Display CAN XCVR/V_SUPPLY
- R93 pad 1: Net-(D21-K) -> Net-(R93-Pad1)
- R93 pad 2: ABS_ActLO -> Net-(R131-Pad1)
- U2 pad 38: unconnected-(U2-GPIO2/TOUCH2/ADC1_CH1-Pad38) -> /RD_ALIVE
- U2 pad 39: unconnected-(U2-GPIO1/TOUCH1/ADC1_CH0-Pad39) -> /LD_ALIVE
Routing:
- net (no net): track 0.00 -> 11.2 mm
- net Net-(D6-A1): track 5.67 -> 0.00 mm
- net Net-(D7-A1): track 5.53 -> 0.00 mm

Commit message: Pre-grouping
Parts:
- removed the J2 at (165.8, 92.0)
- removed the J5 at (83.2, 101.2)
- removed J6: RD_CAN, Connector_PinHeader_2.54mm:PinHeader_1x03_P2.54mm_Vertical
- removed J8: LD_UART, Connector_PinHeader_2.54mm:PinHeader_1x04_P2.54mm_Vertical
- removed J9: RD_UART, Connector_PinHeader_2.54mm:PinHeader_1x04_P2.54mm_Vertical
- removed MTH1, MTH2, MTH4, MTH5: MountingHole_3.5mm_Pad_Via, MountingHole:MountingHole_3.5mm_Pad_Via
- removed the R91 at (83.2, 118.4)
- moved R136 246.2 mm to (18.0, 147.4)
- moved R137 246.2 mm to (18.0, 150.3)
- moved J5 245.6 mm to (26.3, 175.6)
- moved R129 231.4 mm to (35.1, 101.5)
- moved TP6 222.3 mm to (44.4, 38.7)
- moved TP5 215.8 mm to (49.7, 39.2)
- moved TP4 211.1 mm to (55.3, 63.0)
- moved TP7 210.1 mm to (58.6, 39.2)
- moved C55 189.3 mm to (104.6, 170.7)
- moved C62 189.3 mm to (104.6, 178.3)
- moved C53 189.3 mm to (104.6, 165.7)
- moved C54 189.3 mm to (104.6, 168.2)
- moved C56 189.3 mm to (104.6, 173.3)
- moved C61 189.3 mm to (104.6, 175.8)
- moved TP8 186.9 mm to (98.5, 20.4)
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