File: KiCad PCB Files/VXDash/Opto_ActLo.kicad_sch (KiCad schematic)
At the start: 3 parts

Commit message: Moved VXDash project into sub folder
Parts:
- removed R26: 8k2, Resistor_SMD:R_0805_2012Metric_Pad1.20x1.40mm_HandSolder, symbol VXDash_passives:Res
- removed R27: 10k, Resistor_SMD:R_0805_2012Metric_Pad1.20x1.40mm_HandSolder, symbol VXDash_passives:Res
- removed U11: ~, Package_DIP:SMDIP-4_W7.62mm, symbol Isolator:SFH617A-2X009T
- added R7: 8k2, Resistor_SMD:R_0805_2012Metric_Pad1.20x1.40mm_HandSolder, symbol VXDash_passives:Res
- added R8: 10k, Resistor_SMD:R_0805_2012Metric_Pad1.20x1.40mm_HandSolder, symbol VXDash_passives:Res
- added U1: ~, Package_DIP:SMDIP-4_W7.62mm, symbol Isolator:SFH617A-2X009T
Connections:
- net +3V3: now also R8.1
- net GND: now also U1.3
- new net: R7.2, U1.1
- new net PROTECTED_12V+: R7.1
- new net ~{HL_Input}: U1.2
- new net ~{LL_Output}: R8.2, U1.4
Other:
- title: Active Hi Optocoupler circuit -> Active Low Optocoupler circuit

Commit message: Grape shot additions
- Added 0R to the VCC pin on the CAN transceiver for pin compatibility with other transceiver
- Updated TODO box
- Rename ADC_SDA and ADC_SCL to SDA and SCL
- Official symbol and footprint from ESP, using ESP32-S3-WROOM-1-N16R8
- Reassigned Coolant LOW to active HI
- Replaced MUX with i²C TCA9555 IO Expander
- Resequenced Active His and Lows to match current SW definition
- Resequenced ADC channels to match current SW definition
- Added simple peripherals for MCU
- Added RESET and BOOT buttons circuits
- Added CAN transceivers for each display, and Termination resistor
- Added USB C
Other:
- company: (none) -> Alex Miller & Martin Roger
- title: Active Low Optocoupler circuit -> Main architecture
Changed lines of the file:
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@@
 	(paper "A4")
 	(title_block
-		(title "Active Low Optocoupler circuit")
-		(date "2025-08-08")
+		(title "Main architecture")
+		(date "2025-08-10")
 		(rev "1.4")
+		(company "Alex Miller & Martin Roger")
 		(comment 1 "https://github.com/martinroger/VXDash")
 		(comment 2 "https://cadlab.io/projects/vxdash")
@@
 					(unit 1)
 				)
-				(path "/f2858fc4-50de-4ff0-a01c-5b985ee14aef/643e93ce-074d-41b8-8267-8cd768a19e35"
-					(reference "R16")
-					(unit 1)
-				)
 				(path "/f2858fc4-50de-4ff0-a01c-5b985ee14aef/78ec3fed-e0f7-4c10-8e27-628198f4a0d7"
 					(reference "R14")
@@
 					(unit 1)
 				)
-				(path "/f2858fc4-50de-4ff0-a01c-5b985ee14aef/643e93ce-074d-41b8-8267-8cd768a19e35"
-					(reference "R15")
-					(unit 1)
-				)
 				(path "/f2858fc4-50de-4ff0-a01c-5b985ee14aef/78ec3fed-e0f7-4c10-8e27-628198f4a0d7"
 					(reference "R13")
@@
 					(unit 1)
 				)
-				(path "/f2858fc4-50de-4ff0-a01c-5b985ee14aef/643e93ce-074d-41b8-8267-8cd768a19e35"
-					(reference "#PWR017")
-					(unit 1)
-				)
 				(path "/f2858fc4-50de-4ff0-a01c-5b985ee14aef/78ec3fed-e0f7-4c10-8e27-628198f4a0d7"
 					(reference "#PWR016")
@@
 					(unit 1)
 				)
-				(path "/f2858fc4-50de-4ff0-a01c-5b985ee14aef/643e93ce-074d-41b8-8267-8cd768a19e35"
-					(reference "U5")
-					(unit 1)
-				)

Commit message: Emulator board refinements
- Is there stupid with the Active Hi Optos so that the logic is not inverted ?
- Added N-Mosfet activatable resistors. Stupidly simple ? Better MOSFET recommendation ?
Connections:
- net PROTECTED_12V+ renamed Protected_12V
Changed lines of the file:
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@@
+		)
+	)
+	(global_label "Protected_12V"
+		(shape input)
+		(at 124.46 85.09 180)
+		(fields_autoplaced yes)
+		(effects
+			(font
+				(size 1.27 1.27)
+			)
+			(justify right)
+		)
+		(property "Intersheetrefs" "${INTERSHEET_REFS}"
+			(at 108.5824 85.09 0)
+			(effects
+				(font
+					(size 1.27 1.27)
+				)
+				(justify right)
+				(hide yes)
+			)
 		)
 	)
 	(global_label "+3V3"
-		(shape bidirectional)
+		(shape input)
 		(at 167.64 85.09 0)
 		(fields_autoplaced yes)
@@
 		)
 		(property "Intersheetrefs" "${INTERSHEET_REFS}"
-			(at 181.2649 85.09 0)
+			(at 175.051 85.09 0)
 			(effects
 				(font
@@
 				(hide yes)
 			)
-		)
-	)
-	(global_label "PROTECTED_12V+"
-		(shape bidirectional)
-		(at 124.46 85.09 180)
-		(fields_autoplaced yes)
-		(effects
-			(font
-				(size 1.27 1.27)
-			)
-			(justify right)
-		)
-		(property "Intersheetrefs" "${INTERSHEET_REFS}"
-			(at 104.4852 85.09 0)
-			(effects
-				(font
-					(size 1.27 1.27)
-				)
-				(justify right)
-				(hide yes)
-			)

Commit message: PCB layout in progress
Changed some pin assignments to aid routing.
Parts:
- U3: renamed from U1; value ~ -> DPC817; footprint Package_DIP:SMDIP-4_W7.62mm -> Package_DIP:SMDIP-4_W9.53mm; ALT_MFT_PN_1 (none) -> DPC817S-C-TR; MFT (none) -> Diodes Inc; MFT_PN (none) -> DPC817S-B-TR
- renumbered R7 to R11, R8 to R12
Changed lines of the file:
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@@
 		(dnp no)
 		(fields_autoplaced yes)
-		(property "Reference" "R8"
+		(property "Reference" "R12"
 			(at 157.48 90.1699 0)
 			(effects
@@
 		)
 		(property "MFT_PN" ""
+			(at 154.94 91.44 0)
+			(effects
+				(font
+					(size 1.27 1.27)
+				)
+				(hide yes)
+			)
+		)
+		(property "Tolerance" ""
 			(at 154.94 91.44 0)
 			(effects
@@
 			(project "VXDash"
 				(path "/f2858fc4-50de-4ff0-a01c-5b985ee14aef/2079de5b-2f3f-4362-a932-421ac573d68a"
-					(reference "R8")
+					(reference "R12")
 					(unit 1)
 				)
 				(path "/f2858fc4-50de-4ff0-a01c-5b985ee14aef/22d7e4c3-2f98-48b1-822b-d87f9cb003dc"
+					(reference "R22")
+					(unit 1)
+				)
+				(path "/f2858fc4-50de-4ff0-a01c-5b985ee14aef/2c42d151-3f82-4e36-8ef6-a2a8856329ed"
+					(reference "R16")
+					(unit 1)
+				)
+				(path "/f2858fc4-50de-4ff0-a01c-5b985ee14aef/3c86231c-7b35-4b64-9413-492f9e109edd"
+					(reference "R28")
+					(unit 1)
+				)
+				(path "/f2858fc4-50de-4ff0-a01c-5b985ee14aef/4292c77c-6947-4703-ab55-15d783bb0dbb"
+					(reference "R24")
+					(unit 1)
+				)
+				(path "/f2858fc4-50de-4ff0-a01c-5b985ee14aef/78ec3fed-e0f7-4c10-8e27-628198f4a0d7"
 					(reference "R18")
 					(unit 1)
 				)
-				(path "/f2858fc4-50de-4ff0-a01c-5b985ee14aef/2c42d151-3f82-4e36-8ef6-a2a8856329ed"
-					(reference "R12")
-					(unit 1)
-				)
-				(path "/f2858fc4-50de-4ff0-a01c-5b985ee14aef/3c86231c-7b35-4b64-9413-492f9e109edd"
-					(reference "R24")
-					(unit 1)
-				)
-				(path "/f2858fc4-50de-4ff0-a01c-5b985ee14aef/4292c77c-6947-4703-ab55-15d783bb0dbb"
-					(reference "R20")
-					(unit 1)
-				)
-				(path "/f2858fc4-50de-4ff0-a01c-5b985ee14aef/78ec3fed-e0f7-4c10-8e27-628198f4a0d7"
+				(path "/f2858fc4-50de-4ff0-a01c-5b985ee14aef/b35c940f-baa6-46a1-adee-d5b5ad7f2de7"
 					(reference "R14")
 					(unit 1)
 				)
-				(path "/f2858fc4-50de-4ff0-a01c-5b985ee14aef/b35c940f-baa6-46a1-adee-d5b5ad7f2de7"
-					(reference "R10")
-					(unit 1)
-				)
 				(path "/f2858fc4-50de-4ff0-a01c-5b985ee14aef/eb0d7996-49da-4ffe-ae91-4b075a92eda1"
+					(reference "R30")
+					(unit 1)
+				)
+				(path "/f2858fc4-50de-4ff0-a01c-5b985ee14aef/ee13a136-3711-40c9-8966-5935214037ae"
 					(reference "R26")
-					(unit 1)
-				)
-				(path "/f2858fc4-50de-4ff0-a01c-5b985ee14aef/ee13a136-3711-40c9-8966-5935214037ae"
-					(reference "R22")
 					(unit 1)
 				)
@@
 		(dnp no)
 		(fields_autoplaced yes)
-		(property "Reference" "R7"
+		(property "Reference" "R11"
 			(at 134.62 90.1699 0)
 			(effects
@@
 		)
 		(property "MFT_PN" ""
+			(at 132.08 91.44 0)
+			(effects
+				(font
+					(size 1.27 1.27)
+				)
+				(hide yes)
+			)
+		)
+		(property "Tolerance" ""
 			(at 132.08 91.44 0)
 			(effects
@@
 			(project "VXDash"
 				(path "/f2858fc4-50de-4ff0-a01c-5b985ee14aef/2079de5b-2f3f-4362-a932-421ac573d68a"
-					(reference "R7")
+					(reference "R11")
 					(unit 1)
 				)
 				(path "/f2858fc4-50de-4ff0-a01c-5b985ee14aef/22d7e4c3-2f98-48b1-822b-d87f9cb003dc"
+					(reference "R21")
+					(unit 1)
+				)
+				(path "/f2858fc4-50de-4ff0-a01c-5b985ee14aef/2c42d151-3f82-4e36-8ef6-a2a8856329ed"
+					(reference "R15")
+					(unit 1)
+				)
+				(path "/f2858fc4-50de-4ff0-a01c-5b985ee14aef/3c86231c-7b35-4b64-9413-492f9e109edd"
+					(reference "R27")
+					(unit 1)
+				)
+				(path "/f2858fc4-50de-4ff0-a01c-5b985ee14aef/4292c77c-6947-4703-ab55-15d783bb0dbb"
+					(reference "R23")
+					(unit 1)
+				)
+				(path "/f2858fc4-50de-4ff0-a01c-5b985ee14aef/78ec3fed-e0f7-4c10-8e27-628198f4a0d7"
 					(reference "R17")
 					(unit 1)
 				)
-				(path "/f2858fc4-50de-4ff0-a01c-5b985ee14aef/2c42d151-3f82-4e36-8ef6-a2a8856329ed"
-					(reference "R11")
-					(unit 1)
-				)
-				(path "/f2858fc4-50de-4ff0-a01c-5b985ee14aef/3c86231c-7b35-4b64-9413-492f9e109edd"
-					(reference "R23")
-					(unit 1)
-				)
-				(path "/f2858fc4-50de-4ff0-a01c-5b985ee14aef/4292c77c-6947-4703-ab55-15d783bb0dbb"
-					(reference "R19")
-					(unit 1)
-				)
-				(path "/f2858fc4-50de-4ff0-a01c-5b985ee14aef/78ec3fed-e0f7-4c10-8e27-628198f4a0d7"
+				(path "/f2858fc4-50de-4ff0-a01c-5b985ee14aef/b35c940f-baa6-46a1-adee-d5b5ad7f2de7"
 					(reference "R13")
 					(unit 1)
 				)
-				(path "/f2858fc4-50de-4ff0-a01c-5b985ee14aef/b35c940f-baa6-46a1-adee-d5b5ad7f2de7"
-					(reference "R9")
-					(unit 1)
-				)
 				(path "/f2858fc4-50de-4ff0-a01c-5b985ee14aef/eb0d7996-49da-4ffe-ae91-4b075a92eda1"
+					(reference "R29")
+					(unit 1)
+				)
+				(path "/f2858fc4-50de-4ff0-a01c-5b985ee14aef/ee13a136-3711-40c9-8966-5935214037ae"
 					(reference "R25")
-					(unit 1)
-				)
-				(path "/f2858fc4-50de-4ff0-a01c-5b985ee14aef/ee13a136-3711-40c9-8966-5935214037ae"
-					(reference "R21")
 					(unit 1)
 				)
@@
 		(dnp no)
 		(fields_autoplaced yes)
-		(property "Reference" "#PWR013"
+		(property "Reference" "#PWR023"
 			(at 154.94 114.3 0)
 			(effects
@@
 			(project "VXDash"
 				(path "/f2858fc4-50de-4ff0-a01c-5b985ee14aef/2079de5b-2f3f-4362-a932-421ac573d68a"
-					(reference "#PWR013")
+					(reference "#PWR023")
 					(unit 1)
 				)
 				(path "/f2858fc4-50de-4ff0-a01c-5b985ee14aef/22d7e4c3-2f98-48b1-822b-d87f9cb003dc"
-					(reference "#PWR018")
+					(reference "#PWR029")
 					(unit 1)
 				)
 				(path "/f2858fc4-50de-4ff0-a01c-5b985ee14aef/2c42d151-3f82-4e36-8ef6-a2a8856329ed"
-					(reference "#PWR015")
+					(reference "#PWR025")
 					(unit 1)
 				)
 				(path "/f2858fc4-50de-4ff0-a01c-5b985ee14aef/3c86231c-7b35-4b64-9413-492f9e109edd"
-					(reference "#PWR021")
+					(reference "#PWR032")
 					(unit 1)
 				)
 				(path "/f2858fc4-50de-4ff0-a01c-5b985ee14aef/4292c77c-6947-4703-ab55-15d783bb0dbb"
-					(reference "#PWR019")
+					(reference "#PWR030")
 					(unit 1)
 				)
 				(path "/f2858fc4-50de-4ff0-a01c-5b985ee14aef/78ec3fed-e0f7-4c10-8e27-628198f4a0d7"
-					(reference "#PWR016")
+					(reference "#PWR026")
 					(unit 1)
 				)
 				(path "/f2858fc4-50de-4ff0-a01c-5b985ee14aef/b35c940f-baa6-46a1-adee-d5b5ad7f2de7"
-					(reference "#PWR014")
+					(reference "#PWR024")
 					(unit 1)
 				)
 				(path "/f2858fc4-50de-4ff0-a01c-5b985ee14aef/eb0d7996-49da-4ffe-ae91-4b075a92eda1"
-					(reference "#PWR022")
+					(reference "#PWR033")
 					(unit 1)
 				)
 				(path "/f2858fc4-50de-4ff0-a01c-5b985ee14aef/ee13a136-3711-40c9-8966-5935214037ae"
-					(reference "#PWR020")
+					(reference "#PWR031")
 					(unit 1)
 				)
@@
 		(dnp no)
 		(fields_autoplaced yes)
-		(property "Reference" "U1"
+		(property "Reference" "U3"
 			(at 144.78 92.71 0)
 			(effects
@@
 			)
 		)
-		(property "Value" "~"
+		(property "Value" "DPC817"
 			(at 144.78 95.25 0)
 			(effects
@@
 			)
 		)
-		(property "Footprint" "Package_DIP:SMDIP-4_W7.62mm"
+		(property "Footprint" "Package_DIP:SMDIP-4_W9.53mm"
 			(at 144.78 107.95 0)
 			(effects
@@
 			)
 		)
-		(property "MFT" ""
+		(property "MFT" "Diodes Inc"
 			(at 144.78 100.33 90)
 			(effects
@@
 			)
 		)
-		(property "MFT_PN" ""
+		(property "MFT_PN" "DPC817S-B-TR"
 			(at 144.78 100.33 90)
+			(effects
+				(font
+					(size 1.27 1.27)
+				)
+				(hide yes)
+			)
+		)
+		(property "Tolerance" ""
+			(at 144.78 100.33 0)
+			(effects
+				(font
+					(size 1.27 1.27)
+				)
+				(hide yes)
+			)
+		)
+		(property "ALT_MFT_PN_1" "DPC817S-C-TR"
+			(at 144.78 100.33 0)
 			(effects
 				(font
@@
 			(project "VXDash"
 				(path "/f2858fc4-50de-4ff0-a01c-5b985ee14aef/2079de5b-2f3f-4362-a932-421ac573d68a"
-					(reference "U1")
+					(reference "U3")
 					(unit 1)
 				)
 				(path "/f2858fc4-50de-4ff0-a01c-5b985ee14aef/22d7e4c3-2f98-48b1-822b-d87f9cb003dc"
+					(reference "U8")
+					(unit 1)
+				)
+				(path "/f2858fc4-50de-4ff0-a01c-5b985ee14aef/2c42d151-3f82-4e36-8ef6-a2a8856329ed"
+					(reference "U5")
+					(unit 1)
+				)
+				(path "/f2858fc4-50de-4ff0-a01c-5b985ee14aef/3c86231c-7b35-4b64-9413-492f9e109edd"
+					(reference "U11")
+					(unit 1)
+				)
+				(path "/f2858fc4-50de-4ff0-a01c-5b985ee14aef/4292c77c-6947-4703-ab55-15d783bb0dbb"
+					(reference "U9")
+					(unit 1)
+				)
+				(path "/f2858fc4-50de-4ff0-a01c-5b985ee14aef/78ec3fed-e0f7-4c10-8e27-628198f4a0d7"
 					(reference "U6")
 					(unit 1)
 				)
-				(path "/f2858fc4-50de-4ff0-a01c-5b985ee14aef/2c42d151-3f82-4e36-8ef6-a2a8856329ed"
-					(reference "U3")
-					(unit 1)
-				)
-				(path "/f2858fc4-50de-4ff0-a01c-5b985ee14aef/3c86231c-7b35-4b64-9413-492f9e109edd"
-					(reference "U9")
-					(unit 1)
-				)
-				(path "/f2858fc4-50de-4ff0-a01c-5b985ee14aef/4292c77c-6947-4703-ab55-15d783bb0dbb"
-					(reference "U7")
-					(unit 1)
-				)
-				(path "/f2858fc4-50de-4ff0-a01c-5b985ee14aef/78ec3fed-e0f7-4c10-8e27-628198f4a0d7"
+				(path "/f2858fc4-50de-4ff0-a01c-5b985ee14aef/b35c940f-baa6-46a1-adee-d5b5ad7f2de7"
 					(reference "U4")
 					(unit 1)
 				)
-				(path "/f2858fc4-50de-4ff0-a01c-5b985ee14aef/b35c940f-baa6-46a1-adee-d5b5ad7f2de7"
-					(reference "U2")
-					(unit 1)
-				)
 				(path "/f2858fc4-50de-4ff0-a01c-5b985ee14aef/eb0d7996-49da-4ffe-ae91-4b075a92eda1"
+					(reference "U12")
+					(unit 1)
+				)
+				(path "/f2858fc4-50de-4ff0-a01c-5b985ee14aef/ee13a136-3711-40c9-8966-5935214037ae"
 					(reference "U10")
 					(unit 1)
 				)
-				(path "/f2858fc4-50de-4ff0-a01c-5b985ee14aef/ee13a136-3711-40c9-8966-5935214037ae"
-					(reference "U8")
-					(unit 1)
-				)

Commit message: BOM first pass
- Still missing some internal connectors definitions
- Alternative to use a 4x4ch opto config instead of 16x1 ?
- Alternative LiteOn optos identified (easier to source on LCSC)
Parts:
- R11: footprint Resistor_SMD:R_0805_2012Metric_Pad1.20x1.40mm_HandSolder -> Resistor_SMD:R_0603_1608Metric_Pad0.98x0.95mm_HandSolder; LCSC (none) -> C114637; MFT (none) -> Yageo; MFT_PN (none) -> RC0603FR-078K2L
- R12: footprint Resistor_SMD:R_0805_2012Metric_Pad1.20x1.40mm_HandSolder -> Resistor_SMD:R_0603_1608Metric_Pad0.98x0.95mm_HandSolder; LCSC (none) -> C98220; MFT (none) -> Yageo; MFT_PN (none) -> RC0603FR-0710KL
- U3: LCSC (none) -> C22454766; LCSC alt (none) -> C125121
Changed lines of the file:
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@@
+		)
+	)
+	(text_box "Single channel alternative : LiteOn LTV-817S"
+		(exclude_from_sim no)
+		(at 123.19 115.57 0)
+		(size 52.07 5.08)
+		(margins 0.9525 0.9525 0.9525 0.9525)
+		(stroke
+			(width 0)
+			(type solid)
+		)
+		(fill
+			(type none)
+		)
+		(effects
+			(font
+				(size 1.27 1.27)
+			)
+			(justify left top)
 		)
 	)
@@
 			)
 		)
-		(property "Footprint" "Resistor_SMD:R_0805_2012Metric_Pad1.20x1.40mm_HandSolder"
+		(property "Footprint" "Resistor_SMD:R_0603_1608Metric_Pad0.98x0.95mm_HandSolder"
 			(at 153.162 91.44 90)
 			(effects
@@
 			)
 		)
-		(property "Datasheet" ""
+		(property "Datasheet" "http://datasheet.octopart.com/RC0603FR-0710KL-Yageo-datasheet-141265859.pdf"
 			(at 154.94 91.44 0)
 			(effects
@@
 			)
 		)
-		(property "MFT" ""
-			(at 154.94 91.44 0)
-			(effects
-				(font
-					(size 1.27 1.27)
-				)
-				(hide yes)
-			)
-		)
-		(property "MFT_PN" ""
+		(property "MFT" "Yageo"
+			(at 154.94 91.44 0)
+			(effects
+				(font
+					(size 1.27 1.27)
+				)
+				(hide yes)
+			)
+		)
+		(property "MFT_PN" "RC0603FR-0710KL"
 			(at 154.94 91.44 0)
 			(effects
@@
 			)
 		)
-		(property "LCSC" ""
+		(property "LCSC" "C98220"
 			(at 154.94 91.44 0)
 			(effects
@@
 				)
 				(hide yes)
+			)
+		)
+		(property "Ippm" ""
+			(at 154.94 91.44 0)
+			(effects
+				(font
+					(size 1.27 1.27)
+				)
+			)
+		)
+		(property "Vbr" ""
+			(at 154.94 91.44 0)
+			(effects
+				(font
+					(size 1.27 1.27)
+				)
+			)
+		)
+		(property "Vwm" ""
+			(at 154.94 91.44 0)
+			(effects
+				(font
+					(size 1.27 1.27)
+				)
 			)
 		)
@@
 			)
 		)
-		(property "Footprint" "Resistor_SMD:R_0805_2012Metric_Pad1.20x1.40mm_HandSolder"
+		(property "Footprint" "Resistor_SMD:R_0603_1608Metric_Pad0.98x0.95mm_HandSolder"
 			(at 130.302 91.44 90)
 			(effects
@@
 			)
 		)
-		(property "Datasheet" ""
+		(property "Datasheet" "http://datasheet.octopart.com/RC0603FR-078K2L-Yageo-datasheet-164759695.pdf"
 			(at 132.08 91.44 0)
 			(effects
@@
 			)
 		)
-		(property "MFT" ""
-			(at 132.08 91.44 0)
-			(effects
-				(font
-					(size 1.27 1.27)
-				)
-				(hide yes)
-			)
-		)
-		(property "MFT_PN" ""
+		(property "MFT" "Yageo"
+			(at 132.08 91.44 0)
+			(effects
+				(font
+					(size 1.27 1.27)
+				)
+				(hide yes)
+			)
+		)
+		(property "MFT_PN" "RC0603FR-078K2L"
 			(at 132.08 91.44 0)
 			(effects
@@
 			)
 		)
-		(property "LCSC" ""
+		(property "LCSC" "C114637"
 			(at 132.08 91.44 0)
 			(effects
@@
 				)
 				(hide yes)
+			)
+		)
+		(property "Ippm" ""
+			(at 132.08 91.44 0)
+			(effects
+				(font
+					(size 1.27 1.27)
+				)
+			)
+		)
+		(property "Vbr" ""
+			(at 132.08 91.44 0)
+			(effects
+				(font
+					(size 1.27 1.27)
+				)
+			)
+		)
+		(property "Vwm" ""
+			(at 132.08 91.44 0)
+			(effects
+				(font
+					(size 1.27 1.27)
+				)
 			)
 		)
@@
 			)
 		)
-		(property "LCSC" ""
-			(at 144.78 100.33 0)
-			(effects
-				(font
-					(size 1.27 1.27)
-				)
-				(hide yes)
-			)
-		)
-		(property "LCSC alt" ""
+		(property "LCSC" "C22454766"
+			(at 144.78 100.33 0)
+			(effects
+				(font
+					(size 1.27 1.27)
+				)
+				(hide yes)
+			)
+		)
+		(property "LCSC alt" "C125121"
 			(at 144.78 100.33 0)
 			(effects
@@
 			)
 		)
+		(property "Ippm" ""
+			(at 144.78 100.33 0)
+			(effects
+				(font
+					(size 1.27 1.27)
+				)
+			)
+		)
+		(property "Vbr" ""
+			(at 144.78 100.33 0)
+			(effects
+				(font
+					(size 1.27 1.27)
+				)
+			)
+		)
+		(property "Vwm" ""
+			(at 144.78 100.33 0)
+			(effects
+				(font
+					(size 1.27 1.27)
+				)
+			)
+		)

Commit message: OpAmp reversal corrected + LTSpice
- Need to relayout PCB
- OpAmp LT Spice model
Other:
- title: Main architecture -> Optoisolator Active Low Follower
Changed lines of the file:
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@@
 	(paper "A4")
 	(title_block
-		(title "Main architecture")
-		(date "2025-08-10")
-		(rev "1.4")
+		(title "Optoisolator Active Low Follower")
+		(date "2025-10-27")
+		(rev "2.0")
 		(company "Alex Miller & Martin Roger")
 		(comment 1 "https://github.com/martinroger/VXDash")
-		(comment 2 "https://cadlab.io/projects/vxdash")
 	)
 	(text_box "Assume 50% CTR w.c.\nVf = 1.2V @1mA\nLowest battery = 10V\n\nCircuit CTR:\nIf = (10V-1.2V)/1mA = 8.8k. \nLower closest 8k2 = 1.07mA\nIc = 3.3/10k = 330uA\nCTRc = 0.33/1.07 = 30.8%\n\nOpto is always in saturation\n"
