File: KiCad PCB Files/VXDash/Power_Input.kicad_sch (KiCad schematic)
At the start: 18 parts, among them Q1 2N7002, Q2 PJA3441, Q9 PJA3441

Commit message: Moved VXDash project into sub folder
Parts:
- renumbered C33 to C39, C34 to C40, C37 to C41, C35 to C42, C36 to C43, C53 to C44, D1 to D10, D10 to D11, Q1 to Q5, Q9 to Q6, Q2 to Q7, R62 to R78, R63 to R79, R64 to R80, R65 to R81

Commit message: Grape shot additions
- Added 0R to the VCC pin on the CAN transceiver for pin compatibility with other transceiver
- Updated TODO box
- Rename ADC_SDA and ADC_SCL to SDA and SCL
- Official symbol and footprint from ESP, using ESP32-S3-WROOM-1-N16R8
- Reassigned Coolant LOW to active HI
- Replaced MUX with i²C TCA9555 IO Expander
- Resequenced Active His and Lows to match current SW definition
- Resequenced ADC channels to match current SW definition
- Added simple peripherals for MCU
- Added RESET and BOOT buttons circuits
- Added CAN transceivers for each display, and Termination resistor
- Added USB C
Other:
- company: (none) -> Alex Miller & Martin Roger
- title: Power switching and protection -> Main architecture
Changed lines of the file:
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@@
 	(paper "A4")
 	(title_block
-		(title "Power switching and protection")
-		(date "2025-08-08")
+		(title "Main architecture")
+		(date "2025-08-10")
 		(rev "1.4")
+		(company "Alex Miller & Martin Roger")
 		(comment 1 "https://github.com/martinroger/VXDash")
 		(comment 2 "https://cadlab.io/projects/vxdash")
@@
 			)
 		)
-		(property "Datasheet" "~"
+		(property "Datasheet" "https://www.panjit.com.tw/upload/datasheet/PJA3441.pdf?srsltid=AfmBOorcXQifrwfHYhMWRYHvs2fEGINIyw20eErdW3fOG6z6g98X7-Kb"
 			(at 132.08 77.47 0)
 			(effects
@@
 			)
 		)
-		(property "Datasheet" "~"
+		(property "Datasheet" "https://www.panjit.com.tw/upload/datasheet/PJA3441.pdf?srsltid=AfmBOorcXQifrwfHYhMWRYHvs2fEGINIyw20eErdW3fOG6z6g98X7-Kb"
 			(at 160.02 77.47 0)
 			(effects

Commit message: PCB layout in progress
Changed some pin assignments to aid routing.
Parts:
- C44: renamed from C39; footprint (none) -> Capacitor_SMD:C_0603_1608Metric_Pad1.08x0.95mm_HandSolder
- C45: renamed from C40; footprint (none) -> Capacitor_SMD:C_0603_1608Metric_Pad1.08x0.95mm_HandSolder
- C49: renamed from C44; footprint (none) -> Capacitor_SMD:C_0603_1608Metric_Pad1.08x0.95mm_HandSolder
- R79: renamed from R80; footprint Resistor_SMD:R_0805_2012Metric_Pad1.20x1.40mm_HandSolder -> Resistor_SMD:R_0603_1608Metric_Pad0.98x0.95mm_HandSolder
- renumbered C41 to C46, C42 to C47, C43 to C48, D10 to D8, D11 to D9, F2 to F1, R78 to R77, R79 to R78, R81 to R80
Connections:
- net Power_Mid: now reaches D9.1 (K), Q6.2 (S), Q7.2 (S), R80.1

Commit message: New main dash PCB - WIP inc. CAD
Parts:
- added D12: BATT12V_ON, LED_SMD:LED_0603_1608Metric_Pad1.05x0.95mm_HandSolder, symbol VXDash_diodes:LED_Small
- added R99: 3k, Resistor_SMD:R_0603_1608Metric_Pad0.98x0.95mm_HandSolder, symbol VXDash_passives:Res
Connections:
- net GND: now also D12.1 (K)
- net Power_Fused: now also R99.1
- new net: D12.2 (A), R99.2
Other:
- note added: "PJA3441 40V Vds max 3.1A max Vgs-th 2.5V max 88mOhm max +-20V Vgs max"
- note removed: "PJA3441 40V Vds max 3.1A max Vgs-th 2.5V max 88mOhm max +-20V Vgs max Also provides reverse protection"
- moved on the sheet: C44, F1, RV1

Commit message: BOM first pass
- Still missing some internal connectors definitions
- Alternative to use a 4x4ch opto config instead of 16x1 ?
- Alternative LiteOn optos identified (easier to source on LCSC)
Parts:
- C44, C45, C49: LCSC (none) -> C16194176; MFT (none) -> Samsung Electro-Mechanics; MFT_PN (none) -> CL10B104KB8NNWC
- C46, C47, C48: LCSC (none) -> C14860; MFT (none) -> Samsung Electro-Mechanics; MFT_PN (none) -> CL31B106KAHNNNE
- D12: LCSC (none) -> C157740; MFT (none) -> Lite-On; MFT_PN (none) -> LTST-C190KFKT
- D8, D9: ALT_MFT_PN_1 (none) -> BZT52C18-E3-08; LCSC (none) -> C668896; LCSC alt (none) -> C467525
- F1: LCSC (none) -> C3761262; LCSC alt (none) -> C207101
- FB1: ALT_MFT_PN_1 (none) -> BLM21PG121SN1D; LCSC (none) -> N/A; LCSC alt (none) -> C79382
- Q5: LCSC (none) -> C78712
- Q6, Q7: LCSC (none) -> C313504
- R77: LCSC (none) -> C126352; MFT (none) -> Yageo; MFT_PN (none) -> RC0805FR-0730KL; Power 100mW -> 125mW
- R78, R79: LCSC (none) -> C98220; MFT (none) -> Yageo; MFT_PN (none) -> RC0603FR-0710KL
- R80: LCSC (none) -> C14675; MFT (none) -> Yageo; MFT_PN (none) -> RC0603FR-07100KL
- R99: LCSC (none) -> C126358; MFT (none) -> Yageo; MFT_PN (none) -> RC0603FR-073KL
- RV1: LCSC (none) -> C1528486

Commit message: OpAmp reversal corrected + LTSpice
- Need to relayout PCB
- OpAmp LT Spice model
Other:
- title: Main architecture -> Ignition and power protection
Changed lines of the file:
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@@
 	(paper "A4")
 	(title_block
-		(title "Main architecture")
-		(date "2025-08-10")
-		(rev "1.4")
+		(title "Ignition and power protection")
+		(date "2025-10-27")
+		(rev "2.0")
 		(company "Alex Miller & Martin Roger")
 		(comment 1 "https://github.com/martinroger/VXDash")
-		(comment 2 "https://cadlab.io/projects/vxdash")
 	)
 	(text "PJA3441\n40V Vds max\n3.1A max\nVgs-th 2.5V max\n88mOhm max\n+-20V Vgs max"
