File: KiCad PCB Files/VXDash/VXDash.kicad_sch (KiCad schematic)
At the start: 76 parts, among them IC1 CD74HC4050M96, J1 Header_VX220_RightAngle, J10 CANbus, J11 LD connector, J12 RD connector, J2 FASCIA PASSTHRU, J3 I²C debug, J4 UART0 debug, J5 CAN debug, SW1 RESET, SW2 BOOT, U1 TCA9555PWR, U2 ESP32-S3-WROOM-1

Commit message: Pre-grouping phase 1
Connections:
- net usb_dn renamed USB_DN
- net usb_dp renamed USB_DP
Other:
- note added: "Add 2P JST PH for the 3v3 and 5V internal reconnections ?"
Changed lines of the file:
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@@
 		)
 	)
+	(text "Add 2P JST PH for the 3v3 and 5V internal reconnections ?"
+		(exclude_from_sim no)
+		(at 335.026 93.726 0)
+		(effects
+			(font
+				(size 1.27 1.27)
+				(color 255 0 0 1)
+			)
+		)
+	)
 	(text "Rationale is to have :\n- latched\n- low profile\n- somewhat easy to DIY crimp with OTC pincers\n- 2A/pin (overkill)"
 		(exclude_from_sim no)
@@
 		)
 	)
-	(label "usb_dn"
+	(label "USB_DN"
 		(at 351.79 157.48 0)
 		(effects
@@
 		)
 	)
-	(label "usb_dp"
+	(label "USB_DP"
 		(at 351.79 154.94 0)
 		(effects

Commit message: Pre-grouping phase 2
It's tight yo
Connections:
- net ABS_ActLO: now also J2.3 (Pin_3); no longer J2.14 (Pin_14)
- net AIRBAG_ActLO: now also J2.10 (Pin_10); no longer J2.8 (Pin_8)
- net ALARM_ActHI: now also J2.4 (Pin_4); no longer J2.7 (Pin_7)
- net ALTERN_ActLO: now also J2.9 (Pin_9); no longer J2.16 (Pin_16)
- net BRAKE_ActLO: now also J2.16 (Pin_16); no longer J2.2 (Pin_2)
- net CEL_ActLO: now also J2.8 (Pin_8); no longer J2.10 (Pin_10)
- net COOLANT_ActHI: now also J2.2 (Pin_2); no longer J2.3 (Pin_3)
- net DOOR_ActLO: now also J2.1 (Pin_1); no longer J2.12 (Pin_12)
- net GND: now also J2.13 (Pin_13); no longer J2.15 (Pin_15)
- net H_BEAM_ActHI: now also J2.11 (Pin_11); no longer J2.5 (Pin_5)
- net L_BEAM_ActHI: now also J2.6 (Pin_6); no longer J2.9 (Pin_9)
- net L_TURN_ActHI: now also J2.7 (Pin_7); no longer J2.11 (Pin_11)
- net OIL_ALRM_ActLO: now also J2.12 (Pin_12); no longer J2.6 (Pin_6)
- net PARK_ActLO: now also J2.14 (Pin_14); no longer J2.4 (Pin_4)
- net Protected_12V: now also J2.15 (Pin_15); no longer J2.1 (Pin_1)
- net R_TURN_ActHI: now also J2.5 (Pin_5); no longer J2.13 (Pin_13)

Commit message: Finer placement
Parts:
- added TP10: Vsense2, TestPoint:TestPoint_Pad_D1.5mm, symbol Connector:TestPoint
- added TP9: Vsense1, TestPoint:TestPoint_Pad_D1.5mm, symbol Connector:TestPoint
Connections:
- net ANALOGUE/V_SENSOR_IN_1: now also TP9.1
- net ANALOGUE/V_SENSOR_IN_2: now also TP10.1
- no-connect marks 19 -> 17
Changed lines of the file:
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@@
 	)
 	(no_connect
-		(at 525.78 69.85)
-	)
-	(no_connect
 		(at 251.46 170.18)
 	)
@@
 	)
 	(no_connect
-		(at 525.78 67.31)
-	)
-	(no_connect
 		(at 152.4 54.61)
 	)
@@
 	(wire
 		(pts
-			(xy 525.78 69.85) (xy 523.24 69.85)
-		)
-		(stroke
-			(width 0)
-			(type default)
-		)
-	)
-	(wire
-		(pts
 			(xy 342.9 149.86) (xy 351.79 149.86)
 		)
@@
 	(wire
 		(pts
-			(xy 525.78 67.31) (xy 523.24 67.31)
+			(xy 523.24 67.31) (xy 543.56 67.31)
 		)
 		(stroke
@@
 	(wire
 		(pts
+			(xy 543.56 69.85) (xy 543.56 72.39)
+		)
+		(stroke
+			(width 0)
+			(type default)
+		)
+	)
+	(wire
+		(pts
 			(xy 248.92 377.19) (xy 262.89 377.19)
 		)
@@
 		)
 	)
+	(wire
+		(pts
+			(xy 523.24 69.85) (xy 543.56 69.85)
+		)
+		(stroke
+			(width 0)
+			(type default)
+		)
+	)
 	(table
 		(column_count 2)
@@
 	)
 	(symbol
+		(lib_id "Connector:TestPoint")
+		(at 543.56 67.31 270)
+		(unit 1)
+		(exclude_from_sim no)
+		(in_bom yes)
+		(on_board yes)
+		(dnp no)
+		(fields_autoplaced yes)
+		(property "Reference" "TP9"
+			(at 548.64 66.0399 90)
+			(effects
+				(font
+					(size 1.27 1.27)
+				)
+				(justify left)
+			)
+		)
+		(property "Value" "Vsense1"
+			(at 548.64 68.5799 90)
+			(effects
+				(font
+					(size 1.27 1.27)
+				)
+				(justify left)
+			)
+		)
+		(property "Footprint" "TestPoint:TestPoint_Pad_D1.5mm"
+			(at 543.56 72.39 0)
+			(effects
+				(font
+					(size 1.27 1.27)
+				)
+				(hide yes)
+			)
+		)
+		(property "Datasheet" "~"
+			(at 543.56 72.39 0)
+			(effects
+				(font
+					(size 1.27 1.27)
+				)
+				(hide yes)
+			)
+		)
+		(property "Description" "test point"
+			(at 543.56 67.31 0)
+			(effects
+				(font
+					(size 1.27 1.27)
+				)
+				(hide yes)
+			)
+		)
+		(pin "1"
+		)
+		(instances
+			(project ""
+				(path "/f2858fc4-50de-4ff0-a01c-5b985ee14aef"
+					(reference "TP9")
+					(unit 1)
+				)
+			)
+		)
+	)
+	(symbol
 		(lib_id "VXDash_passives:Cap_MLCC")
 		(at 280.67 326.39 270)
@@
 					(unit 1)
 				)
+			)
+		)
+	)
+	(symbol
+		(lib_id "Connector:TestPoint")
+		(at 543.56 72.39 270)
+		(unit 1)
+		(exclude_from_sim no)
+		(in_bom yes)
+		(on_board yes)
+		(dnp no)
+		(fields_autoplaced yes)
+		(property "Reference" "TP10"
+			(at 548.64 71.1199 90)
+			(effects
+				(font
+					(size 1.27 1.27)
+				)
+				(justify left)
+			)
+		)
+		(property "Value" "Vsense2"
+			(at 548.64 73.6599 90)
+			(effects
+				(font
+					(size 1.27 1.27)
+				)
+				(justify left)
+			)
+		)
+		(property "Footprint" "TestPoint:TestPoint_Pad_D1.5mm"
+			(at 543.56 77.47 0)
+			(effects
+				(font
+					(size 1.27 1.27)
+				)
+				(hide yes)
+			)
+		)
+		(property "Datasheet" "~"
+			(at 543.56 77.47 0)
+			(effects
+				(font
+					(size 1.27 1.27)
+				)
+				(hide yes)
+			)
+		)
+		(property "Description" "test point"
+			(at 543.56 72.39 0)
+			(effects
+				(font
+					(size 1.27 1.27)
+				)
+				(hide yes)
+			)
+		)
+		(pin "1"
+		)
+		(instances
+			(project "VXDash"
+				(path "/f2858fc4-50de-4ff0-a01c-5b985ee14aef"
+					(reference "TP10")
+					(unit 1)
+				)

Commit message: Advanced layout
Connections:
- net ABS_ActLO: now also J2.4 (Pin_4); no longer J2.3 (Pin_3)
- net AIRBAG_ActLO: now also J2.7 (Pin_7); no longer J2.10 (Pin_10)
- net ALARM_ActHI: now also J2.13 (Pin_13); no longer J2.4 (Pin_4)
- net ALTERN_ActLO: now also J2.16 (Pin_16); no longer J2.9 (Pin_9)
- net BRAKE_ActLO: now also J2.3 (Pin_3); no longer J2.16 (Pin_16)
- net CEL_ActLO: now also J2.9 (Pin_9); no longer J2.8 (Pin_8)
- net COOLANT_ActHI: now also J2.12 (Pin_12); no longer J2.2 (Pin_2)
- net DOOR_ActLO: now also J2.6 (Pin_6); no longer J2.1 (Pin_1)
- net GND: now also J2.2 (Pin_2); no longer J2.13 (Pin_13)
- net H_BEAM_ActHI: now also J2.15 (Pin_15); no longer J2.11 (Pin_11)
- net L_BEAM_ActHI: now also J2.11 (Pin_11); no longer J2.6 (Pin_6)
- net L_TURN_ActHI: now also J2.14 (Pin_14); no longer J2.7 (Pin_7)
- net OIL_ALRM_ActLO: now also J2.8 (Pin_8); no longer J2.12 (Pin_12)
- net PARK_ActLO: now also J2.5 (Pin_5); no longer J2.14 (Pin_14)
- net Protected_12V: now also J2.1 (Pin_1); no longer J2.15 (Pin_15)
- net R_TURN_ActHI: now also J2.10 (Pin_10); no longer J2.5 (Pin_5)
- net alternator: now also U1.15 (P12); no longer U1.14 (P11)
- net brakes: now also U1.4 (P00); no longer U1.5 (P01)
- net button: now also U1.14 (P11); no longer U1.15 (P12)
- net coolant: now also U1.16 (P13); no longer U1.17 (P14)
- net door: now also U1.18 (P15); no longer U1.19 (P16)
- net ignition: now also U1.6 (P02); no longer U1.4 (P00)
- net left_turn: now also U1.17 (P14); no longer U1.16 (P13)
- net parking: now also U1.5 (P01); no longer U1.6 (P02)
- net right_turn: now also U1.19 (P16); no longer U1.18 (P15)
Other:
- moved on the sheet: J2

Commit message: Primary layout done
- No ground stitching or pours
- Board edges to revise
- DRC to check
- BOM exclusions to check
Parts:
- removed J3: I²C debug, Connector_PinHeader_2.54mm:PinHeader_1x03_P2.54mm_Vertical, symbol Connector_Generic:Conn_01x03
- removed J4: UART0 debug, Connector_PinHeader_2.54mm:PinHeader_1x04_P2.54mm_Vertical, symbol Connector_Generic:Conn_01x04
- added TP11: SCL, TestPoint:TestPoint_Pad_D1.5mm, symbol Connector:TestPoint
- added TP12: SDA, TestPoint:TestPoint_Pad_D1.5mm, symbol Connector:TestPoint
- added TP13: TX0, TestPoint:TestPoint_Pad_D1.5mm, symbol Connector:TestPoint
- added TP14: RX0, TestPoint:TestPoint_Pad_D1.5mm, symbol Connector:TestPoint
- added TP16: GND, TestPoint:TestPoint_Pad_D1.5mm, symbol Connector:TestPoint
- TP1, TP2, TP3, TP4, TP5, TP6, TP7: footprint TestPoint:TestPoint_Pad_D2.0mm -> TestPoint:TestPoint_Pad_D1.5mm
- TP10, TP9: now left out of the parts list
Connections:
- net 5V_aux_enable: now also U2.24 (GPIO47/SPICLK_P/SUBSPICLK_P_DIFF); no longer U2.15 (GPIO3/TOUCH3/ADC1_CH2)
- net 5V_enable: now also U2.25 (GPIO48/SPICLK_N/SUBSPICLK_N_DIFF); no longer U2.11 (GPIO18/U1RXD/ADC2_CH7/CLK_OUT3)
- net CAN_rx: now also U2.31 (GPIO38/FSPIWP/SUBSPIWP); no longer U2.24 (GPIO47/SPICLK_P/SUBSPICLK_P_DIFF)
- net CAN_tx: now also U2.32 (MTCK/GPIO39/CLK_OUT3/SUBSPICS1); no longer U2.25 (GPIO48/SPICLK_N/SUBSPICLK_N_DIFF)
- net GND: now also TP16.1
- net LD_ALIVE: now also U2.20 (GPIO12/TOUCH12/ADC2_CH1/FSPICLK/FSPIIO6/SUBSPICLK); no longer U2.39 (GPIO1/TOUCH1/ADC1_CH0)
- net LD_GP0: now also U2.23 (GPIO21); no longer U2.10 (GPIO17/U1TXD/ADC2_CH6)
- net LD_RXD: now also U2.22 (GPIO14/TOUCH14/ADC2_CH3/FSPIWP/FSPIDQS/SUBSPIWP); no longer U2.8 (GPIO15/U0RTS/ADC2_CH4/XTAL_32K_P)
- net LD_TXD: now also U2.21 (GPIO13/TOUCH13/ADC2_CH2/FSPIQ/FSPIIO7/SUBSPIQ); no longer U2.9 (GPIO16/U0CTS/ADC2_CH5/XTAL_32K_N)
- net RD_GP0: now also U2.33 (MTDO/GPIO40/CLK_OUT2); no longer U2.32 (MTCK/GPIO39/CLK_OUT3/SUBSPICS1)
- net RD_RXD: now also U2.34 (MTDI/GPIO41/CLK_OUT1); no longer U2.33 (MTDO/GPIO40/CLK_OUT2)
- net RD_TXD: now also U2.35 (MTMS/GPIO42); no longer U2.34 (MTDI/GPIO41/CLK_OUT1)
- net SCL: now also U2.17 (GPIO9/TOUCH9/ADC1_CH8/FSPIHD/SUBSPIHD), TP11.1; no longer U2.21 (GPIO13/TOUCH13/ADC2_CH2/FSPIQ/FSPIIO7/SUBSPIQ)
- net SDA: now also U2.15 (GPIO3/TOUCH3/ADC1_CH2), TP12.1; no longer U2.20 (GPIO12/TOUCH12/ADC2_CH1/FSPICLK/FSPIIO6/SUBSPICLK)
- net Set_Hi_Chan_A: now also U2.8 (GPIO15/U0RTS/ADC2_CH4/XTAL_32K_P); no longer U2.4 (GPIO4/TOUCH4/ADC1_CH3)
- net expander_INT: now also U2.7 (GPIO7/TOUCH7/ADC1_CH6); no longer U2.19 (GPIO11/TOUCH11/ADC2_CH0/FSPID/FSPIIO5/SUBSPID)
- net full_beams: now also U2.19 (GPIO11/TOUCH11/ADC2_CH0/FSPID/FSPIIO5/SUBSPID); no longer U2.6 (GPIO6/TOUCH6/ADC1_CH5)
- net rpm: now also U2.6 (GPIO6/TOUCH6/ADC1_CH5); no longer U2.12 (GPIO8/TOUCH8/ADC1_CH7/SUBSPICS1)
- net speed: now also U2.5 (GPIO5/TOUCH5/ADC1_CH4); no longer U2.17 (GPIO9/TOUCH9/ADC1_CH8/FSPIHD/SUBSPIHD)
- net uart0_rx: now also TP14.1
- net uart0_tx: now also TP13.1
- net water_T: now also U2.4 (GPIO4/TOUCH4/ADC1_CH3); no longer U2.7 (GPIO7/TOUCH7/ADC1_CH6)

Commit message: OpAmp reversal corrected + LTSpice
- Need to relayout PCB
- OpAmp LT Spice model
Parts:
- added H1: MountingHole_Pad, MountingHole:MountingHole_3.7mm_Pad_Via, symbol Mechanical:MountingHole_Pad
Connections:
- net GND: now also H1.1
Changed lines of the file:
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@@
 	(title_block
 		(title "Main architecture")
-		(date "2025-08-10")
-		(rev "${PCB_REV}")
+		(date "2025-10-27")
+		(rev "2.0-proto")
 		(company "Alex Miller & Martin Roger")
 		(comment 1 "https://github.com/martinroger/VXDash")
-		(comment 2 "https://cadlab.io/projects/vxdash")
 	)
 	(text "Address is 0x20"
@@
 	(wire
 		(pts
+			(xy 27.94 398.78) (xy 27.94 401.32)
+		)
+		(stroke
+			(width 0)
+			(type default)
+		)
+	)
+	(wire
+		(pts
 			(xy 81.28 336.55) (xy 116.84 336.55)
 		)
@@
 	)
 	(symbol
+		(lib_id "Mechanical:MountingHole_Pad")
+		(at 27.94 396.24 0)
+		(unit 1)
+		(exclude_from_sim yes)
+		(in_bom no)
+		(on_board yes)
+		(dnp no)
+		(fields_autoplaced yes)
+		(property "Reference" "H1"
+			(at 30.48 393.6999 0)
+			(effects
+				(font
+					(size 1.27 1.27)
+				)
+				(justify left)
+			)
+		)
+		(property "Value" "MountingHole_Pad"
+			(at 30.48 396.2399 0)
+			(effects
+				(font
+					(size 1.27 1.27)
+				)
+				(justify left)
+			)
+		)
+		(property "Footprint" "MountingHole:MountingHole_3.7mm_Pad_Via"
+			(at 27.94 396.24 0)
+			(effects
+				(font
+					(size 1.27 1.27)
+				)
+				(hide yes)
+			)
+		)
+		(property "Datasheet" "~"
+			(at 27.94 396.24 0)
+			(effects
+				(font
+					(size 1.27 1.27)
+				)
+				(hide yes)
+			)
+		)
+		(property "Description" "Mounting Hole with connection"
+			(at 27.94 396.24 0)
+			(effects
+				(font
+					(size 1.27 1.27)
+				)
+				(hide yes)
+			)
+		)
+		(pin "1"
+		)
+		(instances
+			(project ""
+				(path "/f2858fc4-50de-4ff0-a01c-5b985ee14aef"
+					(reference "H1")
+					(unit 1)
+				)
+			)
+		)
+	)
+	(symbol
 		(lib_id "VXDash_diodes:LED_Small")
 		(at 156.21 349.25 180)
@@
 					(unit 1)
 				)
+			)
+		)
+	)
+	(symbol
+		(lib_id "power:GND")
+		(at 27.94 401.32 0)
+		(unit 1)
+		(exclude_from_sim no)
+		(in_bom yes)
+		(on_board yes)
+		(dnp no)
+		(property "Reference" "#PWR016"
+			(at 27.94 407.67 0)
+			(effects
+				(font
+					(size 1.27 1.27)
+				)
+				(hide yes)
+			)
+		)
+		(property "Value" "GND"
+			(at 29.718 405.384 0)
+			(effects
+				(font
+					(size 1.27 1.27)
+				)
+				(justify right)
+			)
+		)
+		(property "Footprint" ""
+			(at 27.94 401.32 0)
+			(effects
+				(font
+					(size 1.27 1.27)
+				)
+				(hide yes)
+			)
+		)
+		(property "Datasheet" ""
+			(at 27.94 401.32 0)
+			(effects
+				(font
+					(size 1.27 1.27)
+				)
+				(hide yes)
+			)
+		)
+		(property "Description" "Power symbol creates a global label with name \"GND\" , ground"
+			(at 27.94 401.32 0)
+			(effects
+				(font
+					(size 1.27 1.27)
+				)
+				(hide yes)
+			)
+		)
+		(pin "1"
+		)
+		(instances
+			(project "VXDash"
+				(path "/f2858fc4-50de-4ff0-a01c-5b985ee14aef"
+					(reference "#PWR016")
+					(unit 1)
+				)

Commit message: Corrected OpAmp routing + more sims
Parts:
- H1: footprint MountingHole:MountingHole_3.7mm_Pad_Via -> MountingHole:MountingHole_3.5mm_Pad_TopOnly
Changed lines of the file:
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@@
 			)
 		)
-		(property "Footprint" "MountingHole:MountingHole_3.7mm_Pad_Via"
+		(property "Footprint" "MountingHole:MountingHole_3.5mm_Pad_TopOnly"
 			(at 27.94 396.24 0)
 			(effects

Commit message: New PCB outline
- Corrected small issues with solder expansion mask
- Ground pour in place but no ground stitching
- No Silkscreen texts
Parts:
- added H3: MH_mid_left, MountingHole:MountingHole_3.5mm_Pad_Via, symbol Mechanical:MountingHole_Pad
- added H4: MH_mid_right, MountingHole:MountingHole_3.5mm_Pad_Via, symbol Mechanical:MountingHole_Pad
- added H5: MH_bottom_left, MountingHole:MountingHole_3.5mm_Pad_Via, symbol Mechanical:MountingHole_Pad
- added H6: MH_bottom_right, MountingHole:MountingHole_3.5mm_Pad_Via, symbol Mechanical:MountingHole_Pad
- added H7: MH_center, MountingHole:MountingHole_3.5mm_Pad_Via, symbol Mechanical:MountingHole_Pad
- H1: value MountingHole_Pad -> MH_top_right; footprint MountingHole:MountingHole_3.5mm_Pad_TopOnly -> MountingHole:MountingHole_3.5mm_Pad_Via; now not fitted
Connections:
- net GND: now also H3.1, H4.1, H5.1, H6.1, H7.1
