File: KiCad PCB Files/VXDash/3V3_SMPS.kicad_sch (KiCad schematic)
At the start: 13 parts, among them IC8 AP62200

Commit message: Moved VXDash project into sub folder
Parts:
- removed C12: 10u, Capacitor_SMD:C_1206_3216Metric_Pad1.33x1.80mm_HandSolder, symbol VXDash_passives:Cap_MLCC
- removed C21: 22u, Capacitor_SMD:C_1206_3216Metric_Pad1.33x1.80mm_HandSolder, symbol VXDash_passives:Cap_MLCC
- removed IC8: AP62200, Package_TO_SOT_SMD:TSOT-23-6_HandSoldering, symbol VXDash_regulators:AP62200
- removed R5: 1k, Resistor_SMD:R_0603_1608Metric_Pad0.98x0.95mm_HandSolder, symbol VXDash_passives:Res
- added C14: 10u, Capacitor_SMD:C_1206_3216Metric_Pad1.33x1.80mm_HandSolder, symbol VXDash_passives:Cap_MLCC
- added C15: 100n, symbol VXDash_passives:Cap_MLCC
- added IC4: AP62200, Package_TO_SOT_SMD:TSOT-23-6_HandSoldering, symbol VXDash_regulators:AP62200
- added R40: 24k, Resistor_SMD:R_0603_1608Metric_Pad0.98x0.95mm_HandSolder, symbol VXDash_passives:Res
- C17: value 100n -> 22p; footprint (none) -> Capacitor_SMD:C_0402_1005Metric_Pad0.74x0.62mm_HandSolder; Dielectric X7R -> C0G/NP0; now not fitted
- C18: value 22p -> 100n; footprint Capacitor_SMD:C_0402_1005Metric_Pad0.74x0.62mm_HandSolder -> (none); Dielectric C0G/NP0 -> X7R; now fitted
- C19: value 100n -> 22u; footprint (none) -> Capacitor_SMD:C_1206_3216Metric_Pad1.33x1.80mm_HandSolder; Tol 10% -> 20%; Voltage 50V -> 10V
- C20: Tol 10% -> 20%; Voltage 50V -> 10V
- L2: value 4u7 -> 3u3; footprint VXDash_inductors:Ind_5050 -> Inductor_SMD:L_Taiyo-Yuden_NR-50xx_HandSoldering; DCR 32mOhm -> 30mOhm; Irated 3.2A -> 3A; Isat 4.2A -> 3.6A; MFT Pulse Electronics -> Taiyo Yuden; MFT_PN BWVS005050404R7M00 -> NRS5030T3R3MMGJ; Tol (none) -> 20%; Tolerance 20% -> (none)
- R37: value 100k -> 820k
- R38: value 43k -> 120k
- R39: value 8k2 -> 75k
Connections:
- net 12V_in: now also R37.1, C14.2, C15.2, IC4.3 (VIN); no longer C16.2
- net GND: now also C18.1, C19.2, R38.2, C14.1, C15.1, IC4.1 (GND), R40.2; no longer C16.1, C19.1, R37.2, R39.2
- net 3V3_out: now reaches C18.2, R39.1
- net 3V3_out: now also C17.1, C19.1, C20.1, L2.2; no longer R38.2
- net at L2.1: now also C16.1, IC4.2 (SW); no longer C17.1
- net at C17.2: now also R39.2, IC4.4 (FB), R40.1
- removed net 5V_out: C18.1, C19.2, C20.1, L2.2, R38.1
- new net: IC4.5 (EN), R37.2, R38.1
- new net: C16.2, IC4.6 (BST)
Other:
- title: 12V to 5V conversion -> 5 to 3V3 stage

Commit message: Grape shot additions
- Added 0R to the VCC pin on the CAN transceiver for pin compatibility with other transceiver
- Updated TODO box
- Rename ADC_SDA and ADC_SCL to SDA and SCL
- Official symbol and footprint from ESP, using ESP32-S3-WROOM-1-N16R8
- Reassigned Coolant LOW to active HI
- Replaced MUX with i²C TCA9555 IO Expander
- Resequenced Active His and Lows to match current SW definition
- Resequenced ADC channels to match current SW definition
- Added simple peripherals for MCU
- Added RESET and BOOT buttons circuits
- Added CAN transceivers for each display, and Termination resistor
- Added USB C
Other:
- company: (none) -> Alex Miller & Martin Roger
- title: 5 to 3V3 stage -> Main architecture
Changed lines of the file:
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@@
 	(paper "A4")
 	(title_block
-		(title "5 to 3V3 stage")
-		(date "2025-08-08")
+		(title "Main architecture")
+		(date "2025-08-10")
 		(rev "1.4")
+		(company "Alex Miller & Martin Roger")
 		(comment 1 "https://github.com/martinroger/VXDash")
 		(comment 2 "https://cadlab.io/projects/vxdash")

Commit message: PCB layout in progress
Changed some pin assignments to aid routing.
Parts:
- C21: renamed from C15; footprint (none) -> Capacitor_SMD:C_0603_1608Metric_Pad1.08x0.95mm_HandSolder
- C22: renamed from C16; footprint (none) -> Capacitor_SMD:C_0603_1608Metric_Pad1.08x0.95mm_HandSolder
- C24: renamed from C18; footprint (none) -> Capacitor_SMD:C_0603_1608Metric_Pad1.08x0.95mm_HandSolder
- renumbered C14 to C20, C17 to C23, C19 to C25, C20 to C26, IC4 to IC3, R37 to R41, R38 to R42, R39 to R43, R40 to R44
Connections:
- net 3V3_SW: now reaches C22.1, IC3.2 (SW), L2.1
- net 3V3_FB: now reaches C23.2, IC3.4 (FB), R43.2, R44.1
- net 3V3_EN: now reaches IC3.5 (EN), R41.2, R42.1
- net 12V_in renamed V_IN
- net 3V3_out renamed 3V3_OUT
Changed lines of the file:
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@@
 		)
 	)
-	(hierarchical_label "3V3_out"
+	(label "3V3_EN"
+		(at 102.87 71.12 0)
+		(effects
+			(font
+				(size 1.27 1.27)
+			)
+			(justify left bottom)
+		)
+	)
+	(label "3V3_SW"
+		(at 140.97 60.96 0)
+		(effects
+			(font
+				(size 1.27 1.27)
+			)
+			(justify left bottom)
+		)
+	)
+	(label "3V3_FB"
+		(at 144.78 71.12 0)
+		(effects
+			(font
+				(size 1.27 1.27)
+			)
+			(justify left bottom)
+		)
+	)
+	(hierarchical_label "3V3_OUT"
 		(shape output)
 		(at 207.01 60.96 0)
@@
 		)
 	)
-	(hierarchical_label "12V_in"
+	(hierarchical_label "V_IN"
 		(shape input)
 		(at 76.2 55.88 180)
@@
 		(dnp no)
 		(fields_autoplaced yes)
-		(property "Reference" "#PWR033"
+		(property "Reference" "#PWR044"
 			(at 124.46 93.98 0)
 			(effects
@@
 			(project ""
 				(path "/f2858fc4-50de-4ff0-a01c-5b985ee14aef/21f2fd69-aa93-4550-8877-dde4aa3e5582"
-					(reference "#PWR033")
+					(reference "#PWR044")
 					(unit 1)
 				)
@@
 		(dnp no)
 		(fields_autoplaced yes)
-		(property "Reference" "IC4"
+		(property "Reference" "IC3"
 			(at 124.46 48.26 0)
 			(effects
@@
 		(property "MFT_PN" "AP62200WU-7"
 			(at 124.46 38.1 0)
+			(effects
+				(font
+					(size 1.27 1.27)
+				)
+				(hide yes)
+			)
+		)
+		(property "Tolerance" ""
+			(at 124.46 53.34 0)
 			(effects
 				(font
@@
 			(project ""
 				(path "/f2858fc4-50de-4ff0-a01c-5b985ee14aef/21f2fd69-aa93-4550-8877-dde4aa3e5582"
-					(reference "IC4")
+					(reference "IC3")
 					(unit 1)
 				)
@@
 		(dnp yes)
 		(fields_autoplaced yes)
-		(property "Reference" "C17"
+		(property "Reference" "C23"
 			(at 172.72 63.4999 0)
 			(effects
@@
 		)
 		(property "MFT_PN" ""
+			(at 168.91 66.04 0)
+			(effects
+				(font
+					(size 1.27 1.27)
+				)
+				(hide yes)
+			)
+		)
+		(property "Tolerance" ""
 			(at 168.91 66.04 0)
 			(effects
@@
 			(project ""
 				(path "/f2858fc4-50de-4ff0-a01c-5b985ee14aef/21f2fd69-aa93-4550-8877-dde4aa3e5582"
-					(reference "C17")
+					(reference "C23")
 					(unit 1)
 				)
@@
 		(dnp no)
 		(fields_autoplaced yes)
-		(property "Reference" "R40"
+		(property "Reference" "R44"
 			(at 162.56 76.1999 0)
 			(effects
@@
 		)
 		(property "MFT_PN" ""
+			(at 160.02 77.47 0)
+			(effects
+				(font
+					(size 1.27 1.27)
+				)
+				(hide yes)
+			)
+		)
+		(property "Tolerance" ""
 			(at 160.02 77.47 0)
 			(effects
@@
 			(project "VXDash"
 				(path "/f2858fc4-50de-4ff0-a01c-5b985ee14aef/21f2fd69-aa93-4550-8877-dde4aa3e5582"
-					(reference "R40")
+					(reference "R44")
 					(unit 1)
 				)
@@
 		(on_board yes)
 		(dnp no)
-		(property "Reference" "C14"
+		(property "Reference" "C20"
 			(at 97.79 48.26 0)
 			(effects
@@
 				)
 				(justify left)
+			)
+		)
+		(property "Tolerance" ""
+			(at 99.06 62.23 0)
+			(effects
+				(font
+					(size 1.27 1.27)
+				)
+				(hide yes)
 			)
 		)
@@
 			(project "VXDash"
 				(path "/f2858fc4-50de-4ff0-a01c-5b985ee14aef/21f2fd69-aa93-4550-8877-dde4aa3e5582"
-					(reference "C14")
+					(reference "C20")
 					(unit 1)
 				)
@@
 		(dnp no)
 		(fields_autoplaced yes)
-		(property "Reference" "R39"
+		(property "Reference" "R43"
 			(at 162.56 64.7699 0)
 			(effects
@@
 		)
 		(property "MFT_PN" ""
+			(at 160.02 66.04 0)
+			(effects
+				(font
+					(size 1.27 1.27)
+				)
+				(hide yes)
+			)
+		)
+		(property "Tolerance" ""
 			(at 160.02 66.04 0)
 			(effects
@@
 			(project ""
 				(path "/f2858fc4-50de-4ff0-a01c-5b985ee14aef/21f2fd69-aa93-4550-8877-dde4aa3e5582"
-					(reference "R39")
+					(reference "R43")
 					(unit 1)
 				)
@@
 		(dnp no)
 		(fields_autoplaced yes)
-		(property "Reference" "R37"
+		(property "Reference" "R41"
 			(at 91.44 62.2299 0)
 			(effects
@@
 		)
 		(property "MFT_PN" ""
+			(at 88.9 63.5 0)
+			(effects
+				(font
+					(size 1.27 1.27)
+				)
+				(hide yes)
+			)
+		)
+		(property "Tolerance" ""
 			(at 88.9 63.5 0)
 			(effects
@@
 			(project "VXDash"
 				(path "/f2858fc4-50de-4ff0-a01c-5b985ee14aef/21f2fd69-aa93-4550-8877-dde4aa3e5582"
-					(reference "R37")
+					(reference "R41")
 					(unit 1)
 				)
@@
 		(on_board yes)
 		(dnp no)
-		(property "Reference" "C20"
+		(property "Reference" "C26"
 			(at 199.39 53.34 0)
 			(effects
@@
 		)
 		(property "MFT_PN" ""
+			(at 200.66 66.04 0)
+			(effects
+				(font
+					(size 1.27 1.27)
+				)
+				(hide yes)
+			)
+		)
+		(property "Tolerance" ""
 			(at 200.66 66.04 0)
 			(effects
@@
 			(project "VXDash"
 				(path "/f2858fc4-50de-4ff0-a01c-5b985ee14aef/21f2fd69-aa93-4550-8877-dde4aa3e5582"
-					(reference "C20")
+					(reference "C26")
 					(unit 1)
 				)
@@
 		(on_board yes)
 		(dnp no)
-		(property "Reference" "C19"
+		(property "Reference" "C25"
 			(at 191.77 53.34 0)
 			(effects
@@
 		)
 		(property "MFT_PN" ""
+			(at 193.04 66.04 0)
+			(effects
+				(font
+					(size 1.27 1.27)
+				)
+				(hide yes)
+			)
+		)
+		(property "Tolerance" ""
 			(at 193.04 66.04 0)
 			(effects
@@
 			(project ""
 				(path "/f2858fc4-50de-4ff0-a01c-5b985ee14aef/21f2fd69-aa93-4550-8877-dde4aa3e5582"
-					(reference "C19")
+					(reference "C25")
 					(unit 1)
 				)
@@
 			)
 		)
+		(property "Tolerance" ""
+			(at 153.67 60.96 0)
+			(effects
+				(font
+					(size 1.27 1.27)
+				)
+				(hide yes)
+			)
+		)
 		(pin "2"
 		)
@@
 		(dnp no)
 		(fields_autoplaced yes)
-		(property "Reference" "R38"
+		(property "Reference" "R42"
 			(at 91.44 74.9299 0)
 			(effects
@@
 		)
 		(property "MFT_PN" ""
+			(at 88.9 76.2 0)
+			(effects
+				(font
+					(size 1.27 1.27)
+				)
+				(hide yes)
+			)
+		)
+		(property "Tolerance" ""
 			(at 88.9 76.2 0)
 			(effects
@@
 			(project "VXDash"
 				(path "/f2858fc4-50de-4ff0-a01c-5b985ee14aef/21f2fd69-aa93-4550-8877-dde4aa3e5582"
-					(reference "R38")
+					(reference "R42")
 					(unit 1)
 				)
@@
 		(on_board yes)
 		(dnp no)
-		(property "Reference" "C15"
+		(property "Reference" "C21"
 			(at 105.41 48.26 0)
 			(effects
@@
 			)
 		)
-		(property "Footprint" ""
+		(property "Footprint" "Capacitor_SMD:C_0603_1608Metric_Pad1.08x0.95mm_HandSolder"
 			(at 107.6452 58.42 0)
 			(effects
@@
 				)
 				(justify left)
+			)
+		)
+		(property "Tolerance" ""
+			(at 106.68 62.23 0)
+			(effects
+				(font
+					(size 1.27 1.27)
+				)
+				(hide yes)
 			)
 		)
@@
 			(project "VXDash"
 				(path "/f2858fc4-50de-4ff0-a01c-5b985ee14aef/21f2fd69-aa93-4550-8877-dde4aa3e5582"
-					(reference "C15")
+					(reference "C21")
 					(unit 1)
 				)
@@
 		(dnp no)
 		(fields_autoplaced yes)
-		(property "Reference" "C16"
+		(property "Reference" "C22"
 			(at 140.97 45.72 90)
 			(effects
@@
 			)
 		)
-		(property "Footprint" ""
+		(property "Footprint" "Capacitor_SMD:C_0603_1608Metric_Pad1.08x0.95mm_HandSolder"
 			(at 137.16 54.9148 0)
 			(effects
@@
 					(size 1.27 1.27)
 				)
+			)
+		)
+		(property "Tolerance" ""
+			(at 140.97 55.88 90)
+			(effects
+				(font
+					(size 1.27 1.27)
+				)
+				(hide yes)
 			)
 		)
@@
 			(project "VXDash"
 				(path "/f2858fc4-50de-4ff0-a01c-5b985ee14aef/21f2fd69-aa93-4550-8877-dde4aa3e5582"
-					(reference "C16")
+					(reference "C22")
 					(unit 1)
 				)
@@
 		(on_board yes)
 		(dnp no)
-		(property "Reference" "C18"
+		(property "Reference" "C24"
 			(at 184.15 53.34 0)
 			(effects
@@
 			)
 		)
-		(property "Footprint" ""
+		(property "Footprint" "Capacitor_SMD:C_0603_1608Metric_Pad1.08x0.95mm_HandSolder"
 			(at 186.3852 62.23 0)
 			(effects
@@
 				)
 				(justify left)
+			)
+		)
+		(property "Tolerance" ""
+			(at 185.42 66.04 0)
+			(effects
+				(font
+					(size 1.27 1.27)
+				)
+				(hide yes)
 			)
 		)
@@
 			(project "VXDash"
 				(path "/f2858fc4-50de-4ff0-a01c-5b985ee14aef/21f2fd69-aa93-4550-8877-dde4aa3e5582"
-					(reference "C18")
+					(reference "C24")
 					(unit 1)
 				)

Commit message: Fields updates
Parts:
- IC3: LCSC (none) -> C1323282; LCSC alt (none) -> C1323282

Commit message: BOM first pass
- Still missing some internal connectors definitions
- Alternative to use a 4x4ch opto config instead of 16x1 ?
- Alternative LiteOn optos identified (easier to source on LCSC)
Parts:
- C20: LCSC (none) -> C14860; MFT (none) -> Samsung Electro-Mechanics; MFT_PN (none) -> CL31B106KAHNNNE
- C21, C22, C24: LCSC (none) -> C16194176; MFT (none) -> Samsung Electro-Mechanics; MFT_PN (none) -> CL10B104KB8NNWC
- C23: LCSC (none) -> C1882706; MFT (none) -> KEMET; MFT_PN (none) -> C0402C220J5GAC7411
- C25, C26: LCSC (none) -> C87996; MFT (none) -> Samsung Electro-Mechanics; MFT_PN (none) -> CL31B226KPHNNNE
- L2: LCSC (none) -> C222937
- R41: LCSC (none) -> C141684; MFT (none) -> Yageo; MFT_PN (none) -> RC0603FR-07820KL
- R42: LCSC (none) -> C114607; MFT (none) -> Yageo; MFT_PN (none) -> RC0603FR-07120KL
- R43: LCSC (none) -> C114636; MFT (none) -> Yageo; MFT_PN (none) -> RC0603FR-0775KL
- R44: LCSC (none) -> C137760; MFT (none) -> Yageo; MFT_PN (none) -> RC0603FR-0724KL

Commit message: OpAmp reversal corrected + LTSpice
- Need to relayout PCB
- OpAmp LT Spice model
Other:
- title: Main architecture -> 3V3 SMPS
Changed lines of the file:
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@@
 	(paper "A4")
 	(title_block
-		(title "Main architecture")
-		(date "2025-08-10")
-		(rev "1.4")
+		(title "3V3 SMPS")
+		(date "2025-10-27")
+		(rev "2.0")
 		(company "Alex Miller & Martin Roger")
 		(comment 1 "https://github.com/martinroger/VXDash")
-		(comment 2 "https://cadlab.io/projects/vxdash")
 	)
 	(text_box "Ven = 1.2V type. 1.25V max\nMust enable at 10V.\nRtop = 820k, Rbtm = 120k.\nVen = 9.4V @1.2V typ., ~9.8V @1.25V max."
