File: KiCad PCB Files/VXDash/5V_SMPS.kicad_sch (KiCad schematic)
At the start: 13 parts, among them IC4 AP62200

Commit message: Moved VXDash project into sub folder
Parts:
- removed C5: 100n, symbol VXDash_passives:Cap_MLCC
- removed C6: 22p, Capacitor_SMD:C_0402_1005Metric_Pad0.74x0.62mm_HandSolder, symbol VXDash_passives:Cap_MLCC
- removed IC4: AP62200, Package_TO_SOT_SMD:TSOT-23-6_HandSoldering, symbol VXDash_regulators:AP62200
- removed R1: 75k, Resistor_SMD:R_0603_1608Metric_Pad0.98x0.95mm_HandSolder, symbol VXDash_passives:Res
- removed R2: 24k, Resistor_SMD:R_0603_1608Metric_Pad0.98x0.95mm_HandSolder, symbol VXDash_passives:Res
- added C12, C13: 22u, Capacitor_SMD:C_1206_3216Metric_Pad1.33x1.80mm_HandSolder, symbol VXDash_passives:Cap_MLCC
- added IC3: AP62200, Package_TO_SOT_SMD:TSOT-23-6_HandSoldering, symbol VXDash_regulators:AP62200
- added R5: 43k, Resistor_SMD:R_0603_1608Metric_Pad0.98x0.95mm_HandSolder, symbol VXDash_passives:Res
- added R6: 8k2, Resistor_SMD:R_0603_1608Metric_Pad0.98x0.95mm_HandSolder, symbol VXDash_passives:Res
- C10: value 10u -> 22p; footprint Capacitor_SMD:C_1206_3216Metric_Pad1.33x1.80mm_HandSolder -> Capacitor_SMD:C_0402_1005Metric_Pad0.74x0.62mm_HandSolder; Dielectric X7R -> C0G/NP0; Voltage 25V -> 50V; now not fitted
- C7: value 22u -> 10u; Voltage 50V -> 25V
- C9: value 22u -> 100n; footprint Capacitor_SMD:C_1206_3216Metric_Pad1.33x1.80mm_HandSolder -> (none)
- L1: value 3u3 -> 4u7; footprint Inductor_SMD:L_Taiyo-Yuden_NR-50xx_HandSoldering -> VXDash_inductors:Ind_5050; DCR 30mOhm -> 32mOhm; Irated 3A -> 3.2A; Isat 3.6A -> 4.2A; MFT Taiyo Yuden -> Pulse Electronics; MFT_PN NRS5030T3R3MMGJ -> BWVS005050404R7M00; Tol (none) -> 20%; Tolerance 20% -> (none)
- R3: value 820k -> 1k
- R4: value 120k -> 100k
Connections:
- net 12V_in: now also C7.2, C8.2, IC3.3 (VIN); no longer C10.2, C11.2, R3.1
- net GND: now also C7.1, C12.2, C13.2, IC3.1 (GND), R6.2; no longer C10.1, C7.2, C9.2
- net at L1.1: now also C9.1, IC3.2 (SW)
- net at R3.2, R4.1: now also IC3.5 (EN)
- removed net 3V3_out: C7.1, C8.2, C9.1, L1.2
- new net: C10.2, IC3.4 (FB), R5.2, R6.1
- new net: C9.2, IC3.6 (BST)
- new net 5V_en: R3.1
- new net 5V_out: C10.1, C11.2, C12.1, C13.1, L1.2, R5.1
Other:
- title: 5 to 3V3 stage -> 12V to 5V conversion

Commit message: Grape shot additions
- Added 0R to the VCC pin on the CAN transceiver for pin compatibility with other transceiver
- Updated TODO box
- Rename ADC_SDA and ADC_SCL to SDA and SCL
- Official symbol and footprint from ESP, using ESP32-S3-WROOM-1-N16R8
- Reassigned Coolant LOW to active HI
- Replaced MUX with i²C TCA9555 IO Expander
- Resequenced Active His and Lows to match current SW definition
- Resequenced ADC channels to match current SW definition
- Added simple peripherals for MCU
- Added RESET and BOOT buttons circuits
- Added CAN transceivers for each display, and Termination resistor
- Added USB C
Other:
- company: (none) -> Alex Miller & Martin Roger
- title: 12V to 5V conversion -> Main architecture
Changed lines of the file:
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@@
 	(paper "A4")
 	(title_block
-		(title "12V to 5V conversion")
-		(date "2025-08-08")
+		(title "Main architecture")
+		(date "2025-08-10")
 		(rev "1.4")
+		(company "Alex Miller & Martin Roger")
 		(comment 1 "https://github.com/martinroger/VXDash")
 		(comment 2 "https://cadlab.io/projects/vxdash")

Commit message: PCB layout in progress
Changed some pin assignments to aid routing.
Parts:
- C14: renamed from C8; footprint (none) -> Capacitor_SMD:C_0603_1608Metric_Pad1.08x0.95mm_HandSolder
- C15: renamed from C9; footprint (none) -> Capacitor_SMD:C_0603_1608Metric_Pad1.08x0.95mm_HandSolder
- C17: renamed from C11; footprint (none) -> Capacitor_SMD:C_0603_1608Metric_Pad1.08x0.95mm_HandSolder
- renumbered C7 to C13, C10 to C16, C12 to C18, C13 to C19, IC3 to IC2, R6 to R10, R3 to R7, R4 to R8, R5 to R9
Connections:
- net 5V_FB: now reaches C16.2, IC2.4 (FB), R10.1, R9.2
- net 5V_SW: now reaches C15.1, IC2.2 (SW), L1.1
- net 12V_in renamed V_IN
- net 5V_en renamed 5V_EN
- net 5V_out renamed 5V_OUT

Commit message: Fields updates
Parts:
- IC2: LCSC (none) -> C1323282; LCSC alt (none) -> C1323282

Commit message: BOM first pass
- Still missing some internal connectors definitions
- Alternative to use a 4x4ch opto config instead of 16x1 ?
- Alternative LiteOn optos identified (easier to source on LCSC)
Parts:
- C13: LCSC (none) -> C14860; MFT (none) -> Samsung Electro-Mechanics; MFT_PN (none) -> CL31B106KAHNNNE
- C14, C15, C17: LCSC (none) -> C16194176; MFT (none) -> Samsung Electro-Mechanics; MFT_PN (none) -> CL10B104KB8NNWC
- C16: LCSC (none) -> C1882706; MFT (none) -> KEMET; MFT_PN (none) -> C0402C220J5GAC7411
- C18, C19: LCSC (none) -> C87996; MFT (none) -> Samsung Electro-Mechanics; MFT_PN (none) -> CL31B226KPHNNNE
- L1: LCSC (none) -> C2838218
- R10: LCSC (none) -> C114637; MFT (none) -> Yageo; MFT_PN (none) -> RC0603FR-078K2L
- R7: LCSC (none) -> C22548; MFT (none) -> Yageo; MFT_PN (none) -> RC0603FR-071KL
- R8: LCSC (none) -> C14675; MFT (none) -> Yageo; MFT_PN (none) -> RC0603FR-07100KL
- R9: LCSC (none) -> C137719; MFT (none) -> Yageo; MFT_PN (none) -> RC0603FR-0743KL

Commit message: OpAmp reversal corrected + LTSpice
- Need to relayout PCB
- OpAmp LT Spice model
Other:
- title: Main architecture -> 5V SMPS
Changed lines of the file:
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@@
 	(paper "A4")
 	(title_block
-		(title "Main architecture")
-		(date "2025-08-10")
-		(rev "1.4")
+		(title "5V SMPS")
+		(date "2025-10-27")
+		(rev "2.0")
 		(company "Alex Miller & Martin Roger")
 		(comment 1 "https://github.com/martinroger/VXDash")
-		(comment 2 "https://cadlab.io/projects/vxdash")
 	)
 	(text_box "Vfb = 0.8V, +/-2% w.c.\nRtop = 43k, Rbtm = 8k2\n4.995V out typ. min ~4.86V, max ~5.12V"
