File: KiCad PCB Files/VXDash/AnalogV_Divider.kicad_sch (KiCad schematic)
At the start: 7 parts

Commit message: BOM first pass
- Still missing some internal connectors definitions
- Alternative to use a 4x4ch opto config instead of 16x1 ?
- Alternative LiteOn optos identified (easier to source on LCSC)
Parts:
- C37: LCSC (none) -> C16194176; MFT (none) -> Samsung Electro-Mechanics; MFT_PN (none) -> CL10B104KB8NNWC
- C38: LCSC (none) -> C100042; MFT (none) -> Yageo; MFT_PN (none) -> CC0603KRX7R9BB103
- D6: LCSC (none) -> C152458
- R68: LCSC (none) -> C17415; MFT (none) -> Royal Ohm; MFT_PN (none) -> 0805W8F100JT5E; Power 100mW -> 125mW
- R69: LCSC (none) -> C14675; MFT (none) -> Yageo; MFT_PN (none) -> RC0603FR-07100KL
- R70: LCSC (none) -> C114660; MFT (none) -> Yageo; MFT_PN (none) -> RC0603FR-07150KL
- R71: value 1K -> 1k; LCSC (none) -> C22548; MFT (none) -> Yageo; MFT_PN (none) -> RC0603FR-071KL
Changed lines of the file:
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@@
 			)
 		)
-		(property "Value" "1K"
+		(property "Value" "1k"
 			(at 173.99 92.71 90)
 			(effects
@@
 			)
 		)
-		(property "Datasheet" ""
+		(property "Datasheet" "http://datasheet.octopart.com/RC0603FR-071KL-Yageo-datasheet-141265859.pdf"
 			(at 173.99 96.52 0)
 			(effects
@@
 			)
 		)
-		(property "MFT" ""
+		(property "MFT" "Yageo"
 			(at 173.99 96.52 0)
 			(effects
@@
 			)
 		)
-		(property "MFT_PN" ""
+		(property "MFT_PN" "RC0603FR-071KL"
 			(at 173.99 96.52 0)
 			(effects
@@
 			)
 		)
-		(property "LCSC" ""
+		(property "LCSC" "C22548"
 			(at 173.99 96.52 0)
 			(effects
@@
 				)
 				(hide yes)
+			)
+		)
+		(property "Ippm" ""
+			(at 173.99 96.52 0)
+			(effects
+				(font
+					(size 1.27 1.27)
+				)
+			)
+		)
+		(property "Vbr" ""
+			(at 173.99 96.52 0)
+			(effects
+				(font
+					(size 1.27 1.27)
+				)
+			)
+		)
+		(property "Vwm" ""
+			(at 173.99 96.52 0)
+			(effects
+				(font
+					(size 1.27 1.27)
+				)
 			)
 		)
@@
 			)
 		)
-		(property "Datasheet" ""
+		(property "Datasheet" "https://www.lcsc.com/datasheet/C114660.pdf"
 			(at 146.05 105.41 0)
 			(effects
@@
 			)
 		)
-		(property "MFT" ""
-			(at 146.05 105.41 0)
-			(effects
-				(font
-					(size 1.27 1.27)
-				)
-				(hide yes)
-			)
-		)
-		(property "MFT_PN" ""
+		(property "MFT" "Yageo"
+			(at 146.05 105.41 0)
+			(effects
+				(font
+					(size 1.27 1.27)
+				)
+				(hide yes)
+			)
+		)
+		(property "MFT_PN" "RC0603FR-07150KL"
 			(at 146.05 105.41 0)
 			(effects
@@
 			)
 		)
-		(property "LCSC" ""
+		(property "LCSC" "C114660"
 			(at 146.05 105.41 0)
 			(effects
@@
 				)
 				(hide yes)
+			)
+		)
+		(property "Ippm" ""
+			(at 146.05 105.41 0)
+			(effects
+				(font
+					(size 1.27 1.27)
+				)
+			)
+		)
+		(property "Vbr" ""
+			(at 146.05 105.41 0)
+			(effects
+				(font
+					(size 1.27 1.27)
+				)
+			)
+		)
+		(property "Vwm" ""
+			(at 146.05 105.41 0)
+			(effects
+				(font
+					(size 1.27 1.27)
+				)
 			)
 		)
@@
 			)
 		)
-		(property "LCSC" ""
+		(property "LCSC" "C152458"
 			(at 179.07 91.44 0)
 			(effects
@@
 				)
 				(hide yes)
+			)
+		)
+		(property "Ippm" ""
+			(at 179.07 91.44 0)
+			(effects
+				(font
+					(size 1.27 1.27)
+				)
+			)
+		)
+		(property "Vbr" ""
+			(at 179.07 91.44 0)
+			(effects
+				(font
+					(size 1.27 1.27)
+				)
+			)
+		)
+		(property "Vwm" ""
+			(at 179.07 91.44 0)
+			(effects
+				(font
+					(size 1.27 1.27)
+				)
 			)
 		)
@@
 			)
 		)
-		(property "Datasheet" ""
+		(property "Datasheet" "https://www.lcsc.com/datasheet/C17415.pdf"
 			(at 116.84 77.47 0)
 			(effects
@@
 			)
 		)
-		(property "Power" "100mW"
+		(property "Power" "125mW"
 			(at 116.84 77.47 0)
 			(effects
@@
 			)
 		)
-		(property "MFT" ""
+		(property "MFT" "Royal Ohm"
 			(at 116.84 77.47 0)
 			(effects
@@
 			)
 		)
-		(property "MFT_PN" ""
+		(property "MFT_PN" "0805W8F100JT5E"
 			(at 116.84 77.47 0)
 			(effects
@@
 			)
 		)
-		(property "LCSC" ""
+		(property "LCSC" "C17415"
 			(at 116.84 77.47 0)
 			(effects
@@
 				)
 				(hide yes)
+			)
+		)
+		(property "Ippm" ""
+			(at 116.84 77.47 0)
+			(effects
+				(font
+					(size 1.27 1.27)
+				)
+			)
+		)
+		(property "Vbr" ""
+			(at 116.84 77.47 0)
+			(effects
+				(font
+					(size 1.27 1.27)
+				)
+			)
+		)
+		(property "Vwm" ""
+			(at 116.84 77.47 0)
+			(effects
+				(font
+					(size 1.27 1.27)
+				)
 			)
 		)
@@
 			)
 		)
-		(property "Datasheet" "~"
+		(property "Datasheet" "https://www.lcsc.com/datasheet/C100042.pdf"
 			(at 180.34 105.41 0)
 			(effects
@@
 			)
 		)
-		(property "MFT" ""
-			(at 180.34 105.41 0)
-			(effects
-				(font
-					(size 1.27 1.27)
-				)
-				(hide yes)
-			)
-		)
-		(property "MFT_PN" ""
+		(property "MFT" "Yageo"
+			(at 180.34 105.41 0)
+			(effects
+				(font
+					(size 1.27 1.27)
+				)
+				(hide yes)
+			)
+		)
+		(property "MFT_PN" "CC0603KRX7R9BB103"
 			(at 180.34 105.41 0)
 			(effects
@@
 			)
 		)
-		(property "LCSC" ""
+		(property "LCSC" "C100042"
 			(at 180.34 105.41 0)
 			(effects
@@
 				)
 				(hide yes)
+			)
+		)
+		(property "Ippm" ""
+			(at 180.34 105.41 0)
+			(effects
+				(font
+					(size 1.27 1.27)
+				)
+			)
+		)
+		(property "Vbr" ""
+			(at 180.34 105.41 0)
+			(effects
+				(font
+					(size 1.27 1.27)
+				)
+			)
+		)
+		(property "Vwm" ""
+			(at 180.34 105.41 0)
+			(effects
+				(font
+					(size 1.27 1.27)
+				)
 			)
 		)
@@
 			)
 		)
-		(property "Datasheet" ""
+		(property "Datasheet" "http://datasheet.octopart.com/RC0603FR-07100KL-Yageo-datasheet-141265859.pdf"
 			(at 146.05 86.36 0)
 			(effects
@@
 			)
 		)
-		(property "MFT" ""
-			(at 146.05 86.36 0)
-			(effects
-				(font
-					(size 1.27 1.27)
-				)
-				(hide yes)
-			)
-		)
-		(property "MFT_PN" ""
+		(property "MFT" "Yageo"
+			(at 146.05 86.36 0)
+			(effects
+				(font
+					(size 1.27 1.27)
+				)
+				(hide yes)
+			)
+		)
+		(property "MFT_PN" "RC0603FR-07100KL"
 			(at 146.05 86.36 0)
 			(effects
@@
 			)
 		)
-		(property "LCSC" ""
+		(property "LCSC" "C14675"
 			(at 146.05 86.36 0)
 			(effects
@@
 				)
 				(hide yes)
+			)
+		)
+		(property "Ippm" ""
+			(at 146.05 86.36 0)
+			(effects
+				(font
+					(size 1.27 1.27)
+				)
+			)
+		)
+		(property "Vbr" ""
+			(at 146.05 86.36 0)
+			(effects
+				(font
+					(size 1.27 1.27)
+				)
+			)
+		)
+		(property "Vwm" ""
+			(at 146.05 86.36 0)
+			(effects
+				(font
+					(size 1.27 1.27)
+				)
 			)
 		)
@@
 			)
 		)
-		(property "Datasheet" "~"
+		(property "Datasheet" "http://datasheet.octopart.com/CL10B104KB8NNWC-Samsung-datasheet-8326407.pdf"
 			(at 128.27 82.55 0)
 			(effects
@@
 			)
 		)
-		(property "MFT" ""
-			(at 128.27 82.55 0)
-			(effects
-				(font
-					(size 1.27 1.27)
-				)
-				(hide yes)
-			)
-		)
-		(property "MFT_PN" ""
+		(property "MFT" "Samsung Electro-Mechanics"
+			(at 128.27 82.55 0)
+			(effects
+				(font
+					(size 1.27 1.27)
+				)
+				(hide yes)
+			)
+		)
+		(property "MFT_PN" "CL10B104KB8NNWC"
 			(at 128.27 82.55 0)
 			(effects
@@
 			)
 		)
-		(property "LCSC" ""
+		(property "LCSC" "C16194176"
 			(at 128.27 82.55 0)
 			(effects
@@
 			)
 		)
+		(property "Ippm" ""
+			(at 128.27 82.55 0)
+			(effects
+				(font
+					(size 1.27 1.27)
+				)
+			)
+		)
+		(property "Vbr" ""
+			(at 128.27 82.55 0)
+			(effects
+				(font
+					(size 1.27 1.27)
+				)
+			)
+		)
+		(property "Vwm" ""
+			(at 128.27 82.55 0)
+			(effects
+				(font
+					(size 1.27 1.27)
+				)
+			)
+		)

Commit message: OpAmp reversal corrected + LTSpice
- Need to relayout PCB
- OpAmp LT Spice model
Other:
- title: Main architecture -> Analog V divider
Changed lines of the file:
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@@
 	(paper "A4")
 	(title_block
-		(title "Main architecture")
-		(date "2025-08-10")
-		(rev "1.4")
+		(title "Analog V divider")
+		(date "2025-10-27")
+		(rev "1.1")
 		(company "Alex Miller & Martin Roger")
 		(comment 1 "https://github.com/martinroger/VXDash")
-		(comment 2 "https://cadlab.io/projects/vxdash")
 	)
 	(text_box "Place near ADC\n~16kHz RC"
