File: KiCad PCB Files/VXDash/USBC.kicad_sch (KiCad schematic)
At the start: 7 parts, among them J5 USB4105-GF-A

Commit message: PCB layout in progress
Changed some pin assignments to aid routing.
Parts:
- C57: renamed from C12; footprint Capacitor_SMD:C_0603_1608Metric -> Capacitor_SMD:C_0603_1608Metric_Pad1.08x0.95mm_HandSolder; Type SMD -> (none)
- J7: renamed from J5; footprint DIY:GCT_USB4105-GF-A -> VXDash_connectors:GCT_USB4105-GF-A; MANUFACTURER GCT -> (none); MAXIMUM_PACKAGE_HEIGHT 3.31 mm -> (none); MFT (none) -> GCT; MFT_PN (none) -> USB4105-GF-A; Manufacturer_Name GCT -> (none); Manufacturer_Part_Number USB4105-GF-A -> (none); PARTREV B4 -> (none); STANDARD Manufacturer Recommendations -> (none)
- R85: renamed from R72; footprint (none) -> Resistor_SMD:R_0603_1608Metric_Pad0.98x0.95mm_HandSolder
- R86: renamed from R71; value 0 -> 0R; footprint (none) -> Resistor_SMD:R_0603_1608Metric_Pad0.98x0.95mm_HandSolder
- R87: renamed from R73; footprint (none) -> Resistor_SMD:R_0603_1608Metric_Pad0.98x0.95mm_HandSolder
- renumbered D7 to D10, D10 to D11
Connections:
- net USB_DN: now also D10.3 (K); no longer D10.4 (K)
- net USB_DP: now also D10.4 (K); no longer D10.3 (K)
Changed lines of the file:
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@@
 	(hierarchical_label "USB_DP"
 		(shape passive)
-		(at 118.11 100.33 90)
+		(at 120.65 100.33 90)
 		(effects
 			(font
@@
 	(hierarchical_label "USB_DN"
 		(shape passive)
-		(at 120.65 100.33 90)
+		(at 118.11 100.33 90)
 		(effects
 			(font
@@
 		(dnp no)
 		(fields_autoplaced yes)
-		(property "Reference" "R71"
+		(property "Reference" "R86"
 			(at 115.57 73.6599 0)
 			(effects
@@
 			)
 		)
-		(property "Value" "0"
+		(property "Value" "0R"
 			(at 115.57 76.1999 0)
 			(effects
@@
 			)
 		)
-		(property "Footprint" ""
+		(property "Footprint" "Resistor_SMD:R_0603_1608Metric_Pad0.98x0.95mm_HandSolder"
 			(at 111.252 74.93 90)
 			(effects
@@
 		)
 		(property "MFT_PN" ""
+			(at 113.03 74.93 0)
+			(effects
+				(font
+					(size 1.27 1.27)
+				)
+				(hide yes)
+			)
+		)
+		(property "Tolerance" ""
 			(at 113.03 74.93 0)
 			(effects
@@
 			(project "VXDash"
 				(path "/f2858fc4-50de-4ff0-a01c-5b985ee14aef/2e212a69-c846-4621-91af-cd3a20f77307"
-					(reference "R71")
+					(reference "R86")
 					(unit 1)
 				)
@@
 		(dnp no)
 		(fields_autoplaced yes)
-		(property "Reference" "J5"
+		(property "Reference" "J7"
 			(at 85.09 40.64 0)
 			(effects
@@
 			)
 		)
-		(property "Footprint" "DIY:GCT_USB4105-GF-A"
+		(property "Footprint" "VXDash_connectors:GCT_USB4105-GF-A"
 			(at 85.09 58.42 0)
 			(effects
@@
 			)
 		)
-		(property "PARTREV" "B4"
+		(property "MFT" "GCT"
 			(at 85.09 58.42 0)
 			(effects
@@
 					(size 1.27 1.27)
 				)
-				(justify bottom)
-				(hide yes)
-			)
-		)
-		(property "STANDARD" "Manufacturer Recommendations"
+				(hide yes)
+			)
+		)
+		(property "MFT_PN" "USB4105-GF-A"
 			(at 85.09 58.42 0)
 			(effects
@@
 					(size 1.27 1.27)
 				)
-				(justify bottom)
-				(hide yes)
-			)
-		)
-		(property "MAXIMUM_PACKAGE_HEIGHT" "3.31 mm"
+				(hide yes)
+			)
+		)
+		(property "Type" "SMD"
 			(at 85.09 58.42 0)
 			(effects
@@
 					(size 1.27 1.27)
 				)
-				(justify bottom)
-				(hide yes)
-			)
-		)
-		(property "MANUFACTURER" "GCT"
-			(at 85.09 58.42 0)
-			(effects
-				(font
-					(size 1.27 1.27)
-				)
-				(justify bottom)
-				(hide yes)
-			)
-		)
-		(property "Manufacturer_Name" "GCT"
-			(at 85.09 58.42 0)
-			(effects
-				(font
-					(size 1.27 1.27)
-				)
-				(hide yes)
-			)
-		)
-		(property "Manufacturer_Part_Number" "USB4105-GF-A"
-			(at 85.09 58.42 0)
-			(effects
-				(font
-					(size 1.27 1.27)
-				)
-				(hide yes)
-			)
-		)
-		(property "Instructions/Notes" ""
-			(at 85.09 58.42 0)
-			(effects
-				(font
-					(size 1.27 1.27)
-				)
-				(hide yes)
-			)
-		)
-		(property "Type" "SMD"
+				(hide yes)
+			)
+		)
+		(property "Tolerance" ""
 			(at 85.09 58.42 0)
 			(effects
@@
 			(project "a1s-mini"
 				(path "/f2858fc4-50de-4ff0-a01c-5b985ee14aef/2e212a69-c846-4621-91af-cd3a20f77307"
-					(reference "J5")
+					(reference "J7")
 					(unit 1)
 				)
@@
 		(dnp no)
 		(fields_autoplaced yes)
-		(property "Reference" "D10"
+		(property "Reference" "D11"
 			(at 168.91 25.4 0)
 			(effects
@@
 				)
 				(justify left)
+				(hide yes)
+			)
+		)
+		(property "Tolerance" ""
+			(at 176.53 33.02 0)
+			(effects
+				(font
+					(size 1.27 1.27)
+				)
 				(hide yes)
 			)
@@
 			(project "a1s-mini"
 				(path "/f2858fc4-50de-4ff0-a01c-5b985ee14aef/2e212a69-c846-4621-91af-cd3a20f77307"
-					(reference "D10")
+					(reference "D11")
 					(unit 1)
 				)
@@
 		(dnp no)
 		(fields_autoplaced yes)
-		(property "Reference" "R73"
+		(property "Reference" "R87"
 			(at 124.46 49.53 90)
 			(effects
@@
 			)
 		)
-		(property "Footprint" ""
+		(property "Footprint" "Resistor_SMD:R_0603_1608Metric_Pad0.98x0.95mm_HandSolder"
 			(at 124.46 57.658 90)
 			(effects
@@
 		(property "MFT_PN" ""
 			(at 124.46 55.88 0)
+			(effects
+				(font
+					(size 1.27 1.27)
+				)
+				(hide yes)
+			)
+		)
+		(property "Tolerance" ""
+			(at 124.46 55.88 90)
 			(effects
 				(font
@@
 			(project "VXDash"
 				(path "/f2858fc4-50de-4ff0-a01c-5b985ee14aef/2e212a69-c846-4621-91af-cd3a20f77307"
-					(reference "R73")
+					(reference "R87")
 					(unit 1)
 				)
@@
 		(dnp no)
 		(fields_autoplaced yes)
-		(property "Reference" "R72"
+		(property "Reference" "R85"
 			(at 58.42 46.99 90)
 			(effects
@@
 			)
 		)
-		(property "Footprint" ""
+		(property "Footprint" "Resistor_SMD:R_0603_1608Metric_Pad0.98x0.95mm_HandSolder"
 			(at 58.42 55.118 90)
 			(effects
@@
 		(property "MFT_PN" ""
 			(at 58.42 53.34 0)
+			(effects
+				(font
+					(size 1.27 1.27)
+				)
+				(hide yes)
+			)
+		)
+		(property "Tolerance" ""
+			(at 58.42 53.34 90)
 			(effects
 				(font
@@
 			(project "VXDash"
 				(path "/f2858fc4-50de-4ff0-a01c-5b985ee14aef/2e212a69-c846-4621-91af-cd3a20f77307"
-					(reference "R72")
+					(reference "R85")
 					(unit 1)
 				)
@@
 		(dnp no)
 		(fields_autoplaced yes)
-		(property "Reference" "C12"
+		(property "Reference" "C57"
 			(at 187.96 53.3399 0)
 			(effects
@@
 			)
 		)
-		(property "Footprint" "Capacitor_SMD:C_0603_1608Metric"
+		(property "Footprint" "Capacitor_SMD:C_0603_1608Metric_Pad1.08x0.95mm_HandSolder"
 			(at 183.1848 52.07 0)
 			(effects
@@
 			)
 		)
-		(property "Type" "SMD"
+		(property "Type" ""
 			(at 184.15 55.88 0)
 			(effects
@@
 		)
 		(property "MFT_PN" ""
+			(at 184.15 55.88 0)
+			(effects
+				(font
+					(size 1.27 1.27)
+				)
+				(hide yes)
+			)
+		)
+		(property "Tolerance" ""
 			(at 184.15 55.88 0)
 			(effects
@@
 			(project "a1s-mini"
 				(path "/f2858fc4-50de-4ff0-a01c-5b985ee14aef/2e212a69-c846-4621-91af-cd3a20f77307"
-					(reference "C12")
+					(reference "C57")
 					(unit 1)
 				)
@@
 		(dnp no)
 		(fields_autoplaced yes)
-		(property "Reference" "D7"
+		(property "Reference" "D10"
 			(at 124.46 109.855 0)
 			(effects
@@
 		)
 		(property "Type" "SMD"
+			(at 118.11 110.49 0)
+			(effects
+				(font
+					(size 1.27 1.27)
+				)
+				(hide yes)
+			)
+		)
+		(property "Tolerance" ""
 			(at 118.11 110.49 0)
 			(effects
@@
 			(project "a1s-mini"
 				(path "/f2858fc4-50de-4ff0-a01c-5b985ee14aef/2e212a69-c846-4621-91af-cd3a20f77307"
-					(reference "D7")
-					(unit 1)
-				)
+					(reference "D10")
+					(unit 1)
+				)

Commit message: Fields updates
Parts:
- D11: LCSC (none) -> C82544
Changed lines of the file:
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@@
+			)
+		)
+		(property "LCSC" ""
+			(at 113.03 74.93 0)
+			(effects
+				(font
+					(size 1.27 1.27)
+				)
+				(hide yes)
+			)
+		)
+		(property "LCSC alt" ""
+			(at 113.03 74.93 0)
+			(effects
+				(font
+					(size 1.27 1.27)
+				)
+				(hide yes)
+			)
+		)
+		(property "JLCPCB" ""
+			(at 113.03 74.93 0)
+			(effects
+				(font
+					(size 1.27 1.27)
+				)
+				(hide yes)
 			)
 		)
@@
 			)
 		)
+		(property "LCSC" "C82544"
+			(at 176.53 33.02 0)
+			(effects
+				(font
+					(size 1.27 1.27)
+				)
+				(hide yes)
+			)
+		)
+		(property "LCSC alt" ""
+			(at 176.53 33.02 0)
+			(effects
+				(font
+					(size 1.27 1.27)
+				)
+				(hide yes)
+			)
+		)
+		(property "JLCPCB" ""
+			(at 176.53 33.02 0)
+			(effects
+				(font
+					(size 1.27 1.27)
+				)
+				(hide yes)
+			)
+		)
 		(pin "1"
 		)
@@
 			)
 		)
+		(property "LCSC" ""
+			(at 124.46 55.88 0)
+			(effects
+				(font
+					(size 1.27 1.27)
+				)
+				(hide yes)
+			)
+		)
+		(property "LCSC alt" ""
+			(at 124.46 55.88 0)
+			(effects
+				(font
+					(size 1.27 1.27)
+				)
+				(hide yes)
+			)
+		)
+		(property "JLCPCB" ""
+			(at 124.46 55.88 0)
+			(effects
+				(font
+					(size 1.27 1.27)
+				)
+				(hide yes)
+			)
+		)
 		(pin "1"
 		)
@@
 			)
 		)
+		(property "LCSC" ""
+			(at 58.42 53.34 0)
+			(effects
+				(font
+					(size 1.27 1.27)
+				)
+				(hide yes)
+			)
+		)
+		(property "LCSC alt" ""
+			(at 58.42 53.34 0)
+			(effects
+				(font
+					(size 1.27 1.27)
+				)
+				(hide yes)
+			)
+		)
+		(property "JLCPCB" ""
+			(at 58.42 53.34 0)
+			(effects
+				(font
+					(size 1.27 1.27)
+				)
+				(hide yes)
+			)
+		)
 		(pin "1"
 		)
@@
 			(at 184.15 55.88 0)
 			(effects
+				(font
+					(size 1.27 1.27)
+				)
+				(hide yes)
+			)
+		)
+		(property "LCSC" ""
+			(at 184.15 55.88 0)
+			(effects
+				(font
+					(size 1.27 1.27)
+				)
+				(hide yes)
+			)
+		)
+		(property "LCSC alt" ""
+			(at 184.15 55.88 0)
+			(effects
+				(font
+					(size 1.27 1.27)
+				)
+				(hide yes)
+			)
+		)
+		(property "JLCPCB" ""
+			(at 184.15 55.88 0)
+			(effects

Commit message: BOM first pass
- Still missing some internal connectors definitions
- Alternative to use a 4x4ch opto config instead of 16x1 ?
- Alternative LiteOn optos identified (easier to source on LCSC)
Parts:
- C57: LCSC (none) -> C19702; LCSC alt (none) -> C6119842; MFT (none) -> Samsung Electro-Mechanics; MFT_PN (none) -> CL10A106KP8NNNC
- D10: LCSC (none) -> C7074; MFT (none) -> Littelfuse; MFT_PN (none) -> SP0503BAHTG
- J7: LCSC (none) -> C3020560
- R85, R87: LCSC (none) -> C105580; LCSC alt (none) -> C23186; MFT (none) -> Yageo; MFT_PN (none) -> RC0603FR-075K1L
- R86: LCSC (none) -> C21189; MFT (none) -> Royal Ohm; MFT_PN (none) -> 0603WAF0000T5E

Commit message: Pre-grouping phase 1
Connections:
- net USB_DN: now also D10.4 (K); no longer D10.3 (K)
- net USB_DP: now also D10.3 (K); no longer D10.4 (K)
Changed lines of the file:
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@@
+	(wire
+		(pts
+			(xy 118.11 100.33) (xy 118.11 105.41)
+		)
+		(stroke
+			(width 0)
+			(type default)
+		)
+	)
 	(wire
 		(pts
@@
 	(wire
 		(pts
+			(xy 120.65 100.33) (xy 120.65 105.41)
+		)
+		(stroke
+			(width 0)
+			(type default)
+		)
+	)
+	(wire
+		(pts
 			(xy 105.41 71.12) (xy 113.03 71.12)
 		)
@@
 	(wire
 		(pts
-			(xy 120.65 100.33) (xy 120.65 105.41)
-		)
-		(stroke
-			(width 0)
-			(type default)
-		)
-	)
-	(wire
-		(pts
-			(xy 118.11 100.33) (xy 118.11 105.41)
-		)
-		(stroke
-			(width 0)
-			(type default)
-		)
-	)
-	(wire
-		(pts
 			(xy 105.41 50.8) (xy 113.03 50.8)
 		)
@@
 	(hierarchical_label "USB_DP"
 		(shape passive)
+		(at 118.11 100.33 90)
+		(effects
+			(font
+				(size 1.27 1.27)
+			)
+			(justify left)
+		)
+	)
+	(hierarchical_label "USB_DN"
+		(shape passive)
+		(at 46.99 58.42 180)
+		(effects
+			(font
+				(size 1.27 1.27)
+			)
+			(justify right)
+		)
+	)
+	(hierarchical_label "VBUS"
+		(shape passive)
+		(at 115.57 95.25 90)
+		(effects
+			(font
+				(size 1.27 1.27)
+			)
+			(justify left)
+		)
+	)
+	(hierarchical_label "USB_DN"
+		(shape passive)
 		(at 120.65 100.33 90)
 		(effects
@@
 		)
 	)
-	(hierarchical_label "USB_DN"
-		(shape passive)
-		(at 46.99 58.42 180)
-		(effects
-			(font
-				(size 1.27 1.27)
-			)
-			(justify right)
-		)
-	)
-	(hierarchical_label "VBUS"
-		(shape passive)
-		(at 115.57 95.25 90)
-		(effects
-			(font
-				(size 1.27 1.27)
-			)
-			(justify left)
-		)
-	)
-	(hierarchical_label "USB_DN"
-		(shape passive)
-		(at 118.11 100.33 90)
-		(effects
-			(font
-				(size 1.27 1.27)
-			)
-			(justify left)
-		)
-	)
 	(hierarchical_label "USB_DP"
 		(shape passive)
@@
 		)
 	)
-	(netclass_flag ""
-		(length 2.54)
-		(shape round)
-		(at 35.56 55.88 0)
-		(fields_autoplaced yes)
-		(effects
-			(font
-				(size 1.27 1.27)
-			)
-			(justify left bottom)
-		)
-		(property "Netclass" "10mil"
-			(at 36.1696 53.34 0)
-			(effects
-				(font
-					(size 1.27 1.27)
-					(italic yes)
-				)
-				(justify left)
-			)
-		)
-	)
-	(netclass_flag ""
-		(length 2.54)
-		(shape round)
-		(at 53.34 58.42 180)
-		(fields_autoplaced yes)
-		(effects
-			(font
-				(size 1.27 1.27)
-			)
-			(justify right bottom)
-		)
-		(property "Netclass" "10mil"
-			(at 53.9496 60.96 0)
-			(effects
-				(font
-					(size 1.27 1.27)
-					(italic yes)
-				)
-				(justify left)
-			)
-		)
-	)

Commit message: OpAmp reversal corrected + LTSpice
- Need to relayout PCB
- OpAmp LT Spice model
Other:
- company: Martin Roger -> Alex Miller & Martin Roger
Changed lines of the file:
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@@
 	(title_block
 		(title "A1S Mini Board")
-		(date "2025-08-10")
-		(rev "0.3.0")
-		(company "Martin Roger")
-		(comment 2 "https://cadlab.io/projects/vxdash")
+		(date "2025-10-27")
+		(rev "1.5")
+		(company "Alex Miller & Martin Roger")
+		(comment 1 "https://github.com/martinroger/VXDash")
 	)
 	(junction
