File: KiCad PCB Files/VXDash/Telltale load emulation.kicad_sch (KiCad schematic)
At the start: 4 parts

Commit message: Large schematic update
- Fascia pass-through connector
- Load emulators for all but turn signals
- Test points
- Additional caps for decoupling
- Regrouped display connectors in single unit
- Added CAN debug connector
Parts:
- added JP3: EN LOAD EMU, symbol Jumper:SolderJumper_2_Open
- renumbered D22 to D23, R95 to R106, R96 to R107, R94 to R98
Connections:
- net V+: now also JP3.2 (B); no longer D23.2 (A)
- new net: D23.2 (A), JP3.1 (A)

Commit message: Added TLs load emulator
50mA and sinking into one another
Parts:
- R98: footprint Resistor_SMD:R_1206_3216Metric_Pad1.30x1.75mm_HandSolder -> Resistor_SMD:R_1210_3225Metric_Pad1.30x2.65mm_HandSolder; Power 250mW -> 500mW
Changed lines of the file:
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@@
 			)
 		)
-		(property "Footprint" "Resistor_SMD:R_1206_3216Metric_Pad1.30x1.75mm_HandSolder"
+		(property "Footprint" "Resistor_SMD:R_1210_3225Metric_Pad1.30x2.65mm_HandSolder"
 			(at 126.238 95.25 90)
 			(effects
@@
 			)
 		)
-		(property "Power" "250mW"
+		(property "Power" "500mW"
 			(at 124.46 95.25 0)
 			(effects

Commit message: BOM first pass
- Still missing some internal connectors definitions
- Alternative to use a 4x4ch opto config instead of 16x1 ?
- Alternative LiteOn optos identified (easier to source on LCSC)
Parts:
- D23: LCSC (none) -> C152458
- JP3: footprint (none) -> Jumper:SolderJumper-2_P1.3mm_Open_RoundedPad1.0x1.5mm
- R106: value 47 -> 47R; LCSC (none) -> C114623; MFT (none) -> Yageo; MFT_PN (none) -> RC0603FR-0747RL
- R107: value 15 -> 15R; LCSC (none) -> C128059; MFT (none) -> Yageo; MFT_PN (none) -> RC0603FR-0715RL
- R98: value 680 -> 680R; LCSC (none) -> C163351; MFT (none) -> Yageo; MFT_PN (none) -> RC1210FR-07680RL
Changed lines of the file:
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@@
 			)
 		)
-		(property "Value" "680"
+		(property "Value" "680R"
 			(at 127.254 96.266 90)
 			(effects
@@
 			)
 		)
-		(property "Datasheet" ""
+		(property "Datasheet" "https://www.lcsc.com/datasheet/C163351.pdf"
 			(at 124.46 95.25 0)
 			(effects
@@
 			)
 		)
-		(property "MFT" ""
-			(at 124.46 95.25 0)
-			(effects
-				(font
-					(size 1.27 1.27)
-				)
-				(hide yes)
-			)
-		)
-		(property "MFT_PN" ""
+		(property "MFT" "Yageo"
+			(at 124.46 95.25 0)
+			(effects
+				(font
+					(size 1.27 1.27)
+				)
+				(hide yes)
+			)
+		)
+		(property "MFT_PN" "RC1210FR-07680RL"
 			(at 124.46 95.25 0)
 			(effects
@@
 			)
 		)
-		(property "LCSC" ""
+		(property "LCSC" "C163351"
 			(at 124.46 95.25 0)
 			(effects
@@
 				)
 				(hide yes)
+			)
+		)
+		(property "Ippm" ""
+			(at 124.46 95.25 0)
+			(effects
+				(font
+					(size 1.27 1.27)
+				)
+			)
+		)
+		(property "Vbr" ""
+			(at 124.46 95.25 0)
+			(effects
+				(font
+					(size 1.27 1.27)
+				)
+			)
+		)
+		(property "Vwm" ""
+			(at 124.46 95.25 0)
+			(effects
+				(font
+					(size 1.27 1.27)
+				)
 			)
 		)
@@
 			)
 		)
-		(property "Value" "15"
+		(property "Value" "15R"
 			(at 127.254 116.586 90)
 			(effects
@@
 			)
 		)
-		(property "Datasheet" ""
+		(property "Datasheet" "https://www.lcsc.com/datasheet/C128059.pdf"
 			(at 124.46 115.57 0)
 			(effects
@@
 			)
 		)
-		(property "MFT" ""
-			(at 124.46 115.57 0)
-			(effects
-				(font
-					(size 1.27 1.27)
-				)
-				(hide yes)
-			)
-		)
-		(property "MFT_PN" ""
+		(property "MFT" "Yageo"
+			(at 124.46 115.57 0)
+			(effects
+				(font
+					(size 1.27 1.27)
+				)
+				(hide yes)
+			)
+		)
+		(property "MFT_PN" " RC0603FR-0715RL"
 			(at 124.46 115.57 0)
 			(effects
@@
 			)
 		)
-		(property "LCSC" ""
+		(property "LCSC" "C128059"
 			(at 124.46 115.57 0)
 			(effects
@@
 				)
 				(hide yes)
+			)
+		)
+		(property "Ippm" ""
+			(at 124.46 115.57 0)
+			(effects
+				(font
+					(size 1.27 1.27)
+				)
+			)
+		)
+		(property "Vbr" ""
+			(at 124.46 115.57 0)
+			(effects
+				(font
+					(size 1.27 1.27)
+				)
+			)
+		)
+		(property "Vwm" ""
+			(at 124.46 115.57 0)
+			(effects
+				(font
+					(size 1.27 1.27)
+				)
 			)
 		)
@@
 			)
 		)
-		(property "Value" "47"
+		(property "Value" "47R"
 			(at 127.254 106.426 90)
 			(effects
@@
 			)
 		)
-		(property "Datasheet" ""
+		(property "Datasheet" "https://www.lcsc.com/datasheet/C114623.pdf"
 			(at 124.46 105.41 0)
 			(effects
@@
 			)
 		)
-		(property "MFT" ""
-			(at 124.46 105.41 0)
-			(effects
-				(font
-					(size 1.27 1.27)
-				)
-				(hide yes)
-			)
-		)
-		(property "MFT_PN" ""
+		(property "MFT" "Yageo"
+			(at 124.46 105.41 0)
+			(effects
+				(font
+					(size 1.27 1.27)
+				)
+				(hide yes)
+			)
+		)
+		(property "MFT_PN" "RC0603FR-0747RL"
 			(at 124.46 105.41 0)
 			(effects
@@
 			)
 		)
-		(property "LCSC" ""
+		(property "LCSC" "C114623"
 			(at 124.46 105.41 0)
 			(effects
@@
 				)
 				(hide yes)
+			)
+		)
+		(property "Ippm" ""
+			(at 124.46 105.41 0)
+			(effects
+				(font
+					(size 1.27 1.27)
+				)
+			)
+		)
+		(property "Vbr" ""
+			(at 124.46 105.41 0)
+			(effects
+				(font
+					(size 1.27 1.27)
+				)
+			)
+		)
+		(property "Vwm" ""
+			(at 124.46 105.41 0)
+			(effects
+				(font
+					(size 1.27 1.27)
+				)
 			)
 		)
@@
 			)
 		)
-		(property "LCSC" ""
+		(property "LCSC" "C152458"
 			(at 124.46 86.36 0)
 			(effects
@@
 				)
 				(hide yes)
+			)
+		)
+		(property "Ippm" ""
+			(at 124.46 86.36 0)
+			(effects
+				(font
+					(size 1.27 1.27)
+				)
+			)
+		)
+		(property "Vbr" ""
+			(at 124.46 86.36 0)
+			(effects
+				(font
+					(size 1.27 1.27)
+				)
+			)
+		)
+		(property "Vwm" ""
+			(at 124.46 86.36 0)
+			(effects
+				(font
+					(size 1.27 1.27)
+				)
 			)
 		)
@@
 			)
 		)
-		(property "Footprint" ""
+		(property "Footprint" "Jumper:SolderJumper-2_P1.3mm_Open_RoundedPad1.0x1.5mm"
 			(at 124.46 76.2 0)
 			(effects
@@
 			)
 		)
+		(property "Ippm" ""
+			(at 124.46 76.2 0)
+			(effects
+				(font
+					(size 1.27 1.27)
+				)
+			)
+		)
+		(property "Vbr" ""
+			(at 124.46 76.2 0)
+			(effects
+				(font
+					(size 1.27 1.27)
+				)
+			)
+		)
+		(property "Vwm" ""
+			(at 124.46 76.2 0)
+			(effects
+				(font
+					(size 1.27 1.27)
+				)
+			)
+		)

Commit message: OpAmp reversal corrected + LTSpice
- Need to relayout PCB
- OpAmp LT Spice model
Other:
- company: (none) -> Alex Miller & Martin Roger
- title: (none) -> Telltale Load Emulator 17mA
Changed lines of the file:
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@@
 	(paper "A4")
 	(title_block
-		(date "2025-08-10")
-		(rev "${PCB_REV}")
+		(title "Telltale Load Emulator 17mA")
+		(date "2025-10-27")
+		(rev "1.0")
+		(company "Alex Miller & Martin Roger")
+		(comment 1 "https://github.com/martinroger/VXDash")
 	)
 	(text "Approximately calculated for 17mA drop at 13V feed\nVf @20mA is approximately 0.38V\nVf @10mA is approximately 0.35V\n\n13-0.38 = 12,62V and 12.62/742 = 17mA\n13-0.35 = 12.65V and 12.65/742 = 17,04mA"

Commit message: Minor PR updates
- Updated revision number in schematic
- Minor change of track layout to avoid ground island
- DRC OK and ERC OK
- Removed stale notes from schematic
- Updated PCB silkscreen
Parts:
- R107: MFT_PN RC0603FR-0715RL -> RC0603FR-0715RL
Changed lines of the file:
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@@
 		(title "Telltale Load Emulator 17mA")
 		(date "2026-01-08")
-		(rev "2.0-proto-B")
+		(rev "2.0-proto-C")
 		(company "Alex Miller & Martin Roger")
 		(comment 1 "https://github.com/martinroger/VXDash")
@@
 			)
 		)
-		(property "MFT_PN" " RC0603FR-0715RL"
-			(at 124.46 115.57 0)
-			(effects
+		(property "MFT_PN" "RC0603FR-0715RL"
+			(at 124.46 115.57 0)
+			(effects
