File: KiCad PCB Files/VXDash/Buzzer.kicad_sch (KiCad schematic)
At the start: 5 parts, among them Q8 PJA3441

Commit message: Minor PR updates
- Updated revision number in schematic
- Minor change of track layout to avoid ground island
- DRC OK and ERC OK
- Removed stale notes from schematic
- Updated PCB silkscreen
Parts:
- R140: LCSC (none) -> C107702; MFT (none) -> Yageo; MFT_PN (none) -> RC0805FR-0722RL; Power 100mW -> 125mW
Changed lines of the file:
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@@
 		(title "Buzzer")
 		(date "2026-01-08")
-		(rev "2.0-proto-B")
+		(rev "2.0-proto-C")
 		(company "Alex Miller & Martin Roger")
 		(comment 1 "https://github.com/martinroger/VXDash")
@@
 			)
 		)
-		(property "Datasheet" "~"
+		(property "Datasheet" "https://www.lcsc.com/datasheet/C107702.pdf"
 			(at 191.77 92.71 0)
 			(effects
@@
 			)
 		)
-		(property "Power" "100mW"
+		(property "Power" "125mW"
 			(at 191.77 92.71 0)
 			(effects
@@
 			)
 		)
-		(property "MFT" ""
+		(property "MFT" "Yageo"
 			(at 191.77 92.71 0)
 			(effects
@@
 			)
 		)
-		(property "MFT_PN" ""
+		(property "MFT_PN" "RC0805FR-0722RL"
 			(at 191.77 92.71 0)
 			(effects
@@
 			)
 		)
-		(property "LCSC" ""
+		(property "LCSC" "C107702"
 			(at 191.77 92.71 0)
 			(effects
