File: KiCad PCB Files/VXDash/Buzzer.kicad_sch (KiCad schematic)
At the start: 5 parts, among them Q8 PJA3441

Commit message: AISLER MPN field
Adding an AISLER MPN field for fast BOM setup with Aisler.
Parts:
- BZ1: AISLER_MPN (none) -> TMB12A12
- D33: AISLER_MPN (none) -> BAT54T1G
- Q8: AISLER_MPN (none) -> PJA3441_R1_00001
- R140: AISLER_MPN (none) -> RC0805FR-0722RL
- R141: AISLER_MPN (none) -> RC0603FR-0710KL
Changed lines of the file:
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@@
+			)
+		)
+		(property "AISLER_MPN" "PJA3441_R1_00001"
+			(at 176.53 88.9 90)
+			(effects
+				(font
+					(size 1.27 1.27)
+				)
+				(hide yes)
 			)
 		)
@@
 					(size 1.27 1.27)
 				)
+			)
+		)
+		(property "AISLER_MPN" "BAT54T1G"
+			(at 186.69 86.36 0)
+			(effects
+				(font
+					(size 1.27 1.27)
+				)
+				(hide yes)
 			)
 		)
@@
 			)
 		)
+		(property "AISLER_MPN" "RC0603FR-0710KL"
+			(at 171.45 97.79 90)
+			(effects
+				(font
+					(size 1.27 1.27)
+				)
+				(hide yes)
+			)
+		)
 		(pin "1"
 		)
@@
 			)
 		)
+		(property "AISLER_MPN" "RC0805FR-0722RL"
+			(at 191.77 92.71 0)
+			(effects
+				(font
+					(size 1.27 1.27)
+				)
+				(hide yes)
+			)
+		)
 		(pin "2"
 		)
@@
 			(at 196.85 102.87 0)
 			(effects
+				(font
+					(size 1.27 1.27)
+				)
+				(hide yes)
+			)
+		)
+		(property "AISLER_MPN" "TMB12A12"
+			(at 196.85 102.87 0)
+			(effects
