File: KiCad PCB Files/VXDash_Emulator/AnalogV_Divider.kicad_sch (KiCad schematic)
At the start: 5 parts, among them IC10 ATA6561

Commit message: More changes (Primarily Remote ECU)
- Emulator board project to a functional skeleton
- Connectors board with ignition routing on CAN pin 4 to have switched signal available in the harness.
- Remote ECU : added 12V reduced protection circuit (to be reviewed)
- Remote ECU : Removed integrated CAN termination (should be on harness)
- Remote ECU : added CAN passthrough
- Remote ECU : added MCPWM channels
- Remote ECU : Added some opto inputs
- Remote ECU : Added internal USB C (overkill ?)
Parts:
- removed C58, C59: 100n, symbol VXDash_passives:Cap_MLCC
- removed C60: 22u, Capacitor_SMD:C_1206_3216Metric_Pad1.33x1.80mm_HandSolder, symbol VXDash_passives:Cap_MLCC
- removed IC10: ATA6561, Package_SO:SOIC-8_3.9x4.9mm_P1.27mm, symbol VXDash_ICs:ATA6561
- removed R116: 0R, Resistor_SMD:R_0805_2012Metric_Pad1.20x1.40mm_HandSolder, symbol VXDash_passives:Res
- added C32: 100n, symbol VXDash_passives:Cap_MLCC
- added C33: 10n, symbol VXDash_passives:Cap_MLCC
- added D4: 5.5V, Diode_SMD:D_SOD-323_HandSoldering, symbol VXDash_diodes:TVS_Uni
- added R56: 10R, Resistor_SMD:R_0805_2012Metric_Pad1.20x1.40mm_HandSolder, symbol VXDash_passives:Res
- added R57: 100k, Resistor_SMD:R_0805_2012Metric_Pad1.20x1.40mm_HandSolder, symbol VXDash_passives:Res
- added R58: 150k, Resistor_SMD:R_0805_2012Metric_Pad1.20x1.40mm_HandSolder, symbol VXDash_passives:Res
- added R59: 1K, Resistor_SMD:R_0805_2012Metric_Pad1.20x1.40mm_HandSolder, symbol VXDash_passives:Res
Connections:
- net GND: now also C32.1, C33.1, D4.2 (A2), R58.1
- new net: R57.2, R58.2, R59.1
- new net: C32.2, D4.1 (A1), R56.2, R57.1
- new net Analog_IN: R56.1
- new net Analog_OUT: C33.2, R59.2
Other:
- note removed: "Internal pull-up. Pull low to enable!"
- company: (none) -> Alex Miller & Martin Roger
- title: VXDash RemoteECU -> Main architecture
