File: KiCad PCB Files/VXDash_Emulator/can_xcvr.kicad_sch (KiCad schematic)
At the start: 5 parts, among them IC10 ATA6561

Commit message: More changes (Primarily Remote ECU)
- Emulator board project to a functional skeleton
- Connectors board with ignition routing on CAN pin 4 to have switched signal available in the harness.
- Remote ECU : added 12V reduced protection circuit (to be reviewed)
- Remote ECU : Removed integrated CAN termination (should be on harness)
- Remote ECU : added CAN passthrough
- Remote ECU : added MCPWM channels
- Remote ECU : Added some opto inputs
- Remote ECU : Added internal USB C (overkill ?)
Parts:
- renumbered C58 to C62, C59 to C63, C60 to C64, IC10 to IC11, R116 to R118
Other:
- note added: "0R resistor added for convenience and pin-compatibility with other transceivers."
- company: (none) -> Alex Miller & Martin Roger
- title: VXDash RemoteECU -> Main architecture
- moved on the sheet: C63, C64
