File: KiCad PCB Files/VXDash_Emulator/Opto_ActHi.kicad_sch (KiCad schematic)
At the start: 3 parts

Commit message: Emulator board refinements
- Is there stupid with the Active Hi Optos so that the logic is not inverted ?
- Added N-Mosfet activatable resistors. Stupidly simple ? Better MOSFET recommendation ?
Parts:
- R41: value 8k2 -> 33k
- R42: renamed from R68; value 10k -> 2k
Connections:
- net +3V3: now also R42.2; no longer R42.1
- net GND: no longer U16.2
- net at U16.1: now also R42.1; no longer R41.2
- net HL_Input renamed BATT12V+
- net ~{LL_output} renamed HL_output
- net HL_output: now also R41.2; no longer R42.2
- new net LL_input: U16.2
Other:
- moved on the sheet: R41, R42, U16

Commit message: ERC corrections, idiot lights
- VXDash : added idiot lights (also to emulator board)
- VXDash : corrected some ERC violations
Parts:
- added D4: HL State, LED_SMD:LED_0603_1608Metric_Pad1.05x0.95mm_HandSolder, symbol VXDash_diodes:LED_Small
- added R102: 270, Resistor_SMD:R_0603_1608Metric_Pad0.98x0.95mm_HandSolder, symbol VXDash_passives:Res
- added TP16: TP_LL, TestPoint:TestPoint_Pad_D2.0mm, symbol Connector:TestPoint_Small
- added TP9: TP_HL, TestPoint:TestPoint_Pad_D2.0mm, symbol Connector:TestPoint_Small
Connections:
- net GND: now also D4.1 (K)
- net HL_output: now also TP9.1
- net LL_input: now also R102.1, TP16.1
- new net: D4.2 (A), R102.2

Commit message: Emulator : ERC and footprints
Also moving some 0402 capacitors to 0603...
Parts:
- renumbered D4 to D13, R41 to R58, R42 to R59, R102 to R60, TP16 to TP10, U16 to U8
