File: KiCad PCB Files/VXDash_Emulator/Opto_ActLo.kicad_sch (KiCad schematic)
At the start: 3 parts

Commit message: Emulator board refinements
- Is there stupid with the Active Hi Optos so that the logic is not inverted ?
- Added N-Mosfet activatable resistors. Stupidly simple ? Better MOSFET recommendation ?
Parts:
- removed R7: 8k2, Resistor_SMD:R_0805_2012Metric_Pad1.20x1.40mm_HandSolder, symbol VXDash_passives:Res
- removed R8: 10k, Resistor_SMD:R_0805_2012Metric_Pad1.20x1.40mm_HandSolder, symbol VXDash_passives:Res
- removed U1: ~, Package_DIP:SMDIP-4_W7.62mm, symbol Isolator:SFH617A-2X009T
- added R72: 33k, Resistor_SMD:R_0805_2012Metric_Pad1.20x1.40mm_HandSolder, symbol VXDash_passives:Res
- added R73: 2k, Resistor_SMD:R_0805_2012Metric_Pad1.20x1.40mm_HandSolder, symbol VXDash_passives:Res
- added U33: ~, Package_DIP:SMDIP-4_W7.62mm, symbol Isolator:SFH617A-2X009T
Connections:
- net GND: now also U33.2, U33.3
- new net: R73.1, U33.1
- new net BATT12V+: R72.1
- new net LL_input: R73.2
- new net ~{HL_output}: R72.2, U33.4

Commit message: ERC corrections, idiot lights
- VXDash : added idiot lights (also to emulator board)
- VXDash : corrected some ERC violations
Parts:
- added D13: HL State, LED_SMD:LED_0603_1608Metric_Pad1.05x0.95mm_HandSolder, symbol VXDash_diodes:LED_Small
- added R109: 270, Resistor_SMD:R_0603_1608Metric_Pad0.98x0.95mm_HandSolder, symbol VXDash_passives:Res
Connections:
- net LL_input: now also D13.1 (K)
- new net: D13.2 (A), R109.2
- new net +3V3: R109.1

Commit message: Emulator : ERC and footprints
Also moving some 0402 capacitors to 0603...
Parts:
- renumbered D13 to D9, R72 to R46, R73 to R47, R109 to R48, U33 to U4

Commit message: Additional TP for Emulator board
Parts:
- added TP23: ~{TP_HL}, TestPoint:TestPoint_Pad_D2.0mm, symbol Connector:TestPoint_Small
- added TP24: TP_LL, TestPoint:TestPoint_Pad_D2.0mm, symbol Connector:TestPoint_Small
Connections:
- net ~{HL_output}: now also TP23.1
- net at R47.1, U4.1: now also TP24.1
