File: KiCad PCB Files/VXDash_Emulator/VXDash_Emulator.kicad_pcb (KiCad board)
At the start: 2 copper layers, 115 x 95 mm, 370 parts, among them IC1 CD74HC4050M96, IC10 ATA6561, IC2 74HC4067BQ-Q100J, IC2 SP721ABG, IC3 AP62200, IC4 AP62200, IC4 MP2322GQH-Z, IC5 AD8542ARMZ-REEL, IC5 AS2333_OpAmp, IC6 AD8542ARMZ-REEL, IC6 AS2333_OpAmp, IC7 AD8542ARMZ-REEL, IC7 AS2333_OpAmp, IC8 AP62200, IC9 AS2333_OpAmp, J1 Conn_02x10_Odd_Even, J1 MX34036UF2, J2 Conn_01x04_Socket, J2 Expansion, Q1 DMP3099L, Q10 DMP3099L, Q11 DMP3099L, Q12 DMP3099L, Q13 DMP3099L, Q14 DMP3099L, Q15 DMP3099L, Q2 DMP3099L, Q3 DMG2301L, Q3 DMP3099L, Q4 DMG2301L, Q4 DMP3099L, Q5 2N7002, Q5 DMG2301L, Q6 DMG2301L, Q6 PJA3441, Q7 DMG2301L, Q7 PJA3441, Q8 DMG2301L, Q8 DMP3099L, Q9 DMP3099L, U10 SFH617A-2X009T, U11 SFH617A-2X009T, U12 SFH617A-2X009T, U13 SFH617A-2X009T, U15 SFH617A-2X009T, U16 ESP32-DevKitC, U16 ESP32-S3-WROOM-1, U17 ADS1115IDGS, U18 ADS1115IDGS, U19 ADS1115IDGS, U2 SFH617A-2X009T, U3 SFH617A-2X009T, U4 SFH617A-2X009T, U5 SFH617A-2X009T, U6 SFH617A-2X009T, U7 SFH617A-2X009T, U8 SFH617A-2X009T, U9 SFH617A-2X009T

Commit message: Emulator : power stages layout
Parts:
- removed the C10 at (59.4, 50.3)
- removed the C10 at (201.8, 65.8)
- removed the C12 at (53.9, 58.9)
- removed the C12 at (192.8, 66.0)
- removed the C13 at (153.9, 75.9)
- removed the C13 at (53.9, 62.2)
- removed the C14 at (167.4, 75.9)
- removed the C14 at (-4.33, 118.9)
- removed the C17 at (4.64, 118.2)
- removed the C17 at (201.2, 52.1)
- removed the C19 at (-4.33, 122.3)
- removed the C19 at (192.0, 54.4)
- removed the C20 at (-4.33, 125.6)
- removed the C20 at (199.6, 50.5)
- removed C23: 100nF 50V, Capacitor_SMD:C_0402_1005Metric
- removed C24, C25, C26, C27, C28, C29, C30, C31, C32, C35, C40, C41, C42, C43, C44, C45, C46, C47, C48, C49, C50, C51, C52: 0.1uF 50V, Capacitor_SMD:C_0603_1608Metric
- removed C31, C36, C45, C55: 100n, Capacitor_SMD:C_0603_1608Metric_Pad1.08x0.95mm_HandSolder
- removed C36: 1uF, Capacitor_SMD:C_0603_1608Metric
- removed C37, C38, C46, C47, C56, C57: 33n, Capacitor_SMD:C_0603_1608Metric_Pad1.08x0.95mm_HandSolder
- removed C39, C40: 100n, Capacitor_SMD:C_0603_1608Metric
- removed C41, C42, C43, C48: 10u, Capacitor_SMD:C_1206_3216Metric_Pad1.33x1.80mm_HandSolder
- removed the C5 at (197.4, 66.0)
- removed the C5 at (118.9, 89.9)
- removed C51: 22p, Capacitor_SMD:C_0402_1005Metric_Pad0.74x0.62mm_HandSolder
- removed C53, C54, C60: 22u, Capacitor_SMD:C_1206_3216Metric_Pad1.33x1.80mm_HandSolder
- removed the C6 at (122.2, 88.9)
- removed the C6 at (204.6, 74.0)
- removed the C7 at (195.1, 66.0)
- removed the C7 at (53.9, 55.5)
- removed the D2 at (143.4, 88.1)
- removed the D2 at (57.9, 95.0)
- removed the D3 at (2.54, 95.2)
- removed the D3 at (157.0, 88.1)
- removed the D4 at (57.9, 109.5)
- removed the D4 at (167.2, 88.1)
- removed the D5 at (57.9, 138.6)
- removed the D5 at (170.4, 88.1)
- removed the D6 at (32.6, 51.0)
- removed the D6 at (180.6, 88.1)
- removed the D9 at (153.6, 88.1)
- removed the D9 at (32.6, 61.0)
- removed F2: 0ZRB0250FF1E, Fuse:Fuse_BelFuse_0ZRE0033FF_L11.4mm_W3.8mm
- removed IC10: ATA6561, Package_SO:SOIC-8_3.9x4.9mm_P1.27mm
- removed the IC2 at (152.1, 128.4)
- removed the IC2 at (119.5, 76.7)
- removed IC3, IC4, IC8: AP62200, Package_TO_SOT_SMD:TSOT-23-6_HandSoldering
- removed IC4: MP2322GQH-Z, DIY:MP2322GQHZ
- removed IC5, IC6, IC7: AD8542ARMZ-REEL, DIY:SOP65P490X110-8N
- removed IC5, IC6, IC7, IC9: AS2333_OpAmp, Package_SO:MSOP-8_3x3mm_P0.65mm
- removed the J1 at (15.6, 95.9)
- removed the J1 at (170.1, 97.4)
- removed the J2 at (115.6, 55.3)
- removed the J2 at (18.0, 51.6)
- removed the L2 at (196.8, 55.9)
- removed the L2 at (-3.06, 114.0)
- removed MTH1, MTH2, MTH3, MTH4, MTH5, MTH6: MountingHole_3.5mm_Pad_Via, MountingHole:MountingHole_3.5mm_Pad_Via
- removed PS1: AP63200WU-7, DIY:SOT95P280X100-6N
- removed the Q3 at (157.7, 81.3)
- removed the Q3 at (27.3, 60.9)
- removed the Q4 at (166.4, 81.3)
- removed the Q4 at (27.3, 65.6)
- removed the Q5 at (205.0, 97.5)
- removed the Q5 at (171.2, 81.3)
- removed the Q6 at (59.1, 125.0)
- removed the Q6 at (179.8, 81.3)
- removed the Q7 at (144.3, 81.3)
- removed the Q7 at (202.9, 90.4)
- removed the Q8 at (152.9, 81.3)
- removed the Q8 at (-30.9, 95.9)
- removed the R1 at (20.0, 94.8)
- removed the R1 at (207.9, 67.1)
- removed the R10 at (39.8, 148.2)
- removed the R10 at (152.5, 106.0)
- removed the R11 at (26.6, 101.6)
- removed the R11 at (152.5, 121.2)
- removed the R12 at (146.2, 106.0)
- removed the R12 at (26.6, 104.6)
- removed the R13 at (146.2, 121.2)
- removed the R13 at (39.8, 130.7)
- removed the R14 at (39.8, 133.7)
- removed the R14 at (139.8, 106.0)
- removed the R15 at (26.6, 130.7)
- removed the R15 at (139.8, 121.2)
- removed the R16 at (133.5, 106.0)
- removed the R16 at (26.6, 133.7)
- removed the R17 at (13.1, 131.1)
- removed the R17 at (133.5, 121.2)
- removed the R18 at (127.1, 106.0)
- removed the R18 at (13.1, 134.0)
- removed the R19 at (127.1, 121.2)
- removed the R19 at (26.6, 116.2)
- removed the R2 at (20.0, 97.3)
- removed the R2 at (207.4, 68.7)
- removed the R20 at (26.6, 119.1)
- removed the R20 at (120.8, 106.0)
- removed the R21 at (120.8, 121.2)
- removed the R21 at (40.4, 81.1)
- removed the R22 at (114.4, 106.0)
- removed the R22 at (40.4, 84.1)
- removed the R23 at (114.4, 121.2)
- removed the R23 at (39.8, 101.6)
- removed the R24 at (39.8, 104.6)
- removed the R24 at (108.1, 106.0)
- removed the R25 at (108.1, 121.2)
- removed the R25 at (27.2, 81.1)
- removed the R26 at (27.2, 84.1)
- removed the R26 at (197.0, 105.8)
- removed the R27 at (197.0, 121.4)
- removed the R27 at (26.6, 145.2)
- removed the R28 at (184.3, 105.8)
- removed the R28 at (26.6, 148.2)
- removed the R29 at (184.3, 121.4)
- removed the R29 at (-4.96, 137.4)
- removed the R3 at (59.0, 55.1)
- removed the R3 at (201.8, 68.3)
- removed the R30 at (-4.96, 140.3)
- removed the R30 at (177.9, 105.8)
- removed the R31 at (39.8, 116.2)
- removed the R31 at (177.9, 121.4)
- removed the R34 at (190.6, 105.8)
- removed the R34 at (171.6, 121.4)
- removed the R35 at (-31.0, 144.0)
- removed the R35 at (190.6, 121.4)
- removed the R37 at (0.85, 118.5)
- removed the R37 at (198.1, 50.5)
- removed the R38 at (195.8, 51.1)
- removed the R38 at (0.85, 121.0)
- removed the R39 at (190.0, 55.4)
- removed the R39 at (0.85, 123.5)
- removed the R4 at (200.8, 68.3)
- removed the R4 at (59.0, 57.6)
- removed the R40 at (0.85, 126.0)
- removed the R40 at (127.1, 77.3)
- removed the R41 at (17.8, 72.9)
- removed the R41 at (127.1, 74.0)
- removed the R42 at (131.6, 77.3)
- removed the R42 at (13.1, 139.0)
- removed the R43 at (131.6, 74.0)
- removed the R43 at (13.1, 141.9)
- removed the R44 at (13.1, 144.9)
- removed the R44 at (136.0, 77.3)
- removed the R45 at (136.0, 74.0)
- removed the R45 at (13.1, 147.8)
- removed the R46 at (140.5, 77.3)
- removed the R46 at (53.0, 95.0)
- removed the R47 at (53.0, 98.0)
- removed the R47 at (140.5, 74.0)
- removed the R48 at (53.0, 100.9)
- removed the R48 at (162.6, 73.2)
- removed the R49 at (147.6, 73.2)
- removed the R49 at (53.0, 103.9)
- removed the R5 at (59.0, 60.1)
- removed the R5 at (191.8, 62.9)
- removed the R50 at (150.6, 73.2)
- removed the R50 at (1.99, 98.4)
- removed the R51 at (1.99, 101.3)
- removed the R51 at (158.5, 84.6)
- removed the R52 at (1.99, 104.3)
- removed the R52 at (161.0, 73.2)
- removed the R53 at (165.6, 84.6)
- removed the R53 at (1.99, 107.2)
- removed the R54 at (159.3, 87.4)
- removed the R54 at (6.54, 100.7)
- removed the R55 at (164.9, 87.4)
- removed the R55 at (6.54, 103.2)
- removed the R56 at (53.0, 109.5)
- removed the R56 at (176.0, 73.2)
- removed the R57 at (161.0, 80.8)
- removed the R57 at (53.0, 112.5)
- removed the R58 at (53.0, 115.4)
- removed the R58 at (147.6, 80.8)
- removed the R59 at (53.0, 118.4)
- removed the R59 at (174.5, 80.8)
- removed the R60 at (53.0, 138.6)
- removed the R60 at (164.1, 73.1)
- removed the R61 at (172.0, 84.6)
- removed the R61 at (53.0, 141.6)
- removed the R66 at (179.1, 84.6)
- removed the R66 at (42.0, 50.5)
- removed the R67 at (172.7, 87.4)
- removed the R67 at (42.0, 53.1)
- removed the R68 at (45.9, 63.5)
- removed the R68 at (178.3, 87.4)
- removed the R69 at (42.0, 55.6)
- removed the R69 at (174.5, 73.2)
- removed the R70 at (42.0, 58.1)
- removed the R70 at (177.5, 73.2)
- removed the R72 at (149.1, 73.2)
- removed the R72 at (46.4, 50.5)
- removed the R73 at (144.8, 84.6)
- removed the R73 at (46.4, 53.1)
- removed the R74 at (145.7, 87.4)
- removed the R74 at (46.4, 55.6)
- removed the R75 at (45.9, 66.8)
- removed the R75 at (152.1, 84.6)
- removed the R76 at (151.4, 87.4)
- removed the R76 at (46.4, 58.1)
- removed the R8 at (158.9, 106.0)
- removed the R8 at (165.2, 121.2)
- removed the R9 at (158.9, 121.2)
- removed the R9 at (39.8, 145.2)
- removed the U10 at (30.4, 76.4)
- removed the U10 at (106.8, 113.6)
- removed the U11 at (29.8, 140.4)
- removed the U11 at (195.7, 113.4)
- removed the U12 at (183.0, 113.4)
- removed the U12 at (-1.74, 132.6)
- removed the U13 at (43.0, 111.4)
- removed the U13 at (176.7, 113.4)
- removed the U15 at (189.4, 113.4)
- removed the U15 at (-27.8, 139.2)
- removed the U16 at (-8.87, 77.6)
- removed the U16 at (130.6, 69.0)
- removed the U2 at (43.0, 140.4)
- removed the U2 at (157.6, 113.6)
- removed the U3 at (151.3, 113.6)
- removed the U3 at (29.8, 96.9)
- removed the U4 at (144.9, 113.6)
- removed the U4 at (43.0, 125.9)
- removed the U5 at (29.8, 125.9)
- removed the U5 at (138.6, 113.6)
- removed the U6 at (16.3, 126.3)
- removed the U6 at (132.2, 113.6)
- removed the U7 at (125.9, 113.6)
- removed the U7 at (29.8, 111.4)
- removed the U8 at (119.5, 113.6)
- removed the U8 at (43.6, 76.4)
- removed the U9 at (43.0, 96.9)
- removed the U9 at (113.2, 113.6)
- added C10: 10u, Capacitor_SMD:C_1206_3216Metric_Pad1.33x1.80mm_HandSolder, F.Cu at (45.7, 69.1)
- added C12: 100n, Capacitor_SMD:C_0603_1608Metric_Pad1.08x0.95mm_HandSolder, F.Cu at (49.8, 80.8)
- added C13: 22p, Capacitor_SMD:C_0603_1608Metric_Pad1.08x0.95mm_HandSolder, F.Cu at (43.7, 77.2)
- added C14: 100n, Capacitor_SMD:C_0603_1608Metric_Pad1.08x0.95mm_HandSolder, F.Cu at (49.8, 70.6)
- added C17: 100n, Capacitor_SMD:C_0603_1608Metric_Pad1.08x0.95mm_HandSolder, F.Cu at (124.4, 107.5)
- added C19: 10u, Capacitor_SMD:C_1206_3216Metric_Pad1.33x1.80mm_HandSolder, F.Cu at (97.5, 105.7)
- added C20: 10u, Capacitor_SMD:C_1206_3216Metric_Pad1.33x1.80mm_HandSolder, F.Cu at (89.4, 105.2)
- added C5: 100n, Capacitor_SMD:C_0603_1608Metric_Pad1.08x0.95mm_HandSolder, F.Cu at (73.2, 80.8)
- added C6: 22p, Capacitor_SMD:C_0603_1608Metric_Pad1.08x0.95mm_HandSolder, F.Cu at (67.1, 77.2)
- added C7: 100n, Capacitor_SMD:C_0603_1608Metric_Pad1.08x0.95mm_HandSolder, F.Cu at (72.1, 70.6)
- added D2: ledc_chan_1_ON, LED_SMD:LED_0603_1608Metric_Pad1.05x0.95mm_HandSolder, F.Cu at (151.4, 87.3)
- added D20: HL State, LED_SMD:LED_0603_1608Metric_Pad1.05x0.95mm_HandSolder, F.Cu at (190.5, 80.0)
- added D21: HL State, LED_SMD:LED_0603_1608Metric_Pad1.05x0.95mm_HandSolder, F.Cu at (225.0, 41.2)
- added D22: HL State, LED_SMD:LED_0603_1608Metric_Pad1.05x0.95mm_HandSolder, F.Cu at (220.8, 63.3)
- added D23: HL State, LED_SMD:LED_0603_1608Metric_Pad1.05x0.95mm_HandSolder, F.Cu at (205.6, 80.0)
- added D24: HL State, LED_SMD:LED_0603_1608Metric_Pad1.05x0.95mm_HandSolder, F.Cu at (190.5, 63.3)
- added D25: ResON, LED_SMD:LED_0603_1608Metric_Pad1.05x0.95mm_HandSolder, F.Cu at (212.4, 136.9)
- added D26: ResON, LED_SMD:LED_0603_1608Metric_Pad1.05x0.95mm_HandSolder, F.Cu at (212.4, 109.3)
- added D27: ResON, LED_SMD:LED_0603_1608Metric_Pad1.05x0.95mm_HandSolder, F.Cu at (223.6, 127.7)
- added D28: ResON, LED_SMD:LED_0603_1608Metric_Pad1.05x0.95mm_HandSolder, F.Cu at (186.0, 138.3)
- added D29: ResON, LED_SMD:LED_0603_1608Metric_Pad1.05x0.95mm_HandSolder, F.Cu at (212.4, 118.5)
- added D3: BATT_ON, LED_SMD:LED_0603_1608Metric_Pad1.05x0.95mm_HandSolder, F.Cu at (151.4, 89.9)
- added D30: ResON, LED_SMD:LED_0603_1608Metric_Pad1.05x0.95mm_HandSolder, F.Cu at (172.3, 112.1)
- added D31: 18V, Diode_SMD:D_SOD-123, F.Cu at (93.0, 111.3)
- added D32: 18V, Diode_SMD:D_SOD-123, F.Cu at (106.7, 111.3)
- added D33: ResON, LED_SMD:LED_0603_1608Metric_Pad1.05x0.95mm_HandSolder, F.Cu at (212.4, 127.7)
- added D34: ResON, LED_SMD:LED_0603_1608Metric_Pad1.05x0.95mm_HandSolder, F.Cu at (223.6, 136.9)
- added D35: ResON, LED_SMD:LED_0603_1608Metric_Pad1.05x0.95mm_HandSolder, F.Cu at (223.6, 118.5)
- added D36: ResON, LED_SMD:LED_0603_1608Metric_Pad1.05x0.95mm_HandSolder, F.Cu at (128.8, 134.6)
- added D37: ResON, LED_SMD:LED_0603_1608Metric_Pad1.05x0.95mm_HandSolder, F.Cu at (172.3, 130.5)
- added D38: ResON, LED_SMD:LED_0603_1608Metric_Pad1.05x0.95mm_HandSolder, F.Cu at (199.2, 138.3)
- added D39: ResON, LED_SMD:LED_0603_1608Metric_Pad1.05x0.95mm_HandSolder, F.Cu at (223.6, 109.3)
- added D4: ledc_chan_0_ON, LED_SMD:LED_0603_1608Metric_Pad1.05x0.95mm_HandSolder, F.Cu at (151.4, 92.5)
- added D40: ResON, LED_SMD:LED_0603_1608Metric_Pad1.05x0.95mm_HandSolder, F.Cu at (140.0, 134.6)
- added D41: ResON, LED_SMD:LED_0603_1608Metric_Pad1.05x0.95mm_HandSolder, F.Cu at (153.0, 134.2)
- added D42: ResON, LED_SMD:LED_0603_1608Metric_Pad1.05x0.95mm_HandSolder, F.Cu at (172.3, 121.3)
- added D5: 5V_ON, LED_SMD:LED_0603_1608Metric_Pad1.05x0.95mm_HandSolder, F.Cu at (151.4, 95.1)
- added D6: 3V3_ON, LED_SMD:LED_0603_1608Metric_Pad1.05x0.95mm_HandSolder, F.Cu at (151.4, 97.7)
- added D9: HL State, LED_SMD:LED_0603_1608Metric_Pad1.05x0.95mm_HandSolder, F.Cu at (199.6, 125.8)
- added IC2: AP62200, Package_TO_SOT_SMD:TSOT-23-6_HandSoldering, F.Cu at (47.2, 76.7)
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Connections:
- C1 pad 1: /rpm -> GND
- C1 pad 2: GND -> +3V3
- C11 pad 1: /12V_to_5V_AP63200WU-7/5V_FB -> GND
- C11 pad 2: /12V_to_5V_AP63200WU-7/5V_REG_OUT -> Protected_12V
- C15 pad 1: GND -> /3V3_SMPS/3V3_OUT
- C15 pad 2: Net-(IC7-+IN_A) -> GND
- C16 pad 1: /12V_to_5V_AP63200WU-7/5V_REG_OUT -> /3V3_SMPS/3V3_OUT
- C18 pad 1: PROTECTED_12V+ -> GND
- C18 pad 2: GND -> Net-(D31-K)
- C2 pad 2: RPM_HALL -> +3V3
- C21 pad 1: Net-(IC4-BST) -> GND
- C21 pad 2: Net-(IC4-SW) -> Protected_12V
- C22 pad 1: Net-(IC4-FB) -> GND
- C22 pad 2: Net-(C19-Pad1) -> Protected_12V
- C3 pad 1: WATER_T_PWM -> GND
- C3 pad 2: GND -> Protected_12V
- C4 pad 1: /speed -> GND
- C4 pad 2: GND -> Protected_12V
- C8 pad 1: PROTECTED_12V+ -> /5V_SMPS_1/5V_OUT
- C9 pad 1: PROTECTED_12V+ -> /5V_SMPS_1/5V_OUT
- D1 pad 1: Net-(D1-A1) -> GND
- D1 pad 2: GND -> Net-(D1-A)
- D10 pad 1: Net-(D10-K) -> /parking
- D10 pad 2: GND -> Net-(D10-A)
- D11 pad 1: Net-(D11-K) -> /oil
- D12 pad 1: AnalogR_3 -> /airbag
- D13 pad 1: +3V3 -> GND
- D13 pad 2: /ANALOGUE/r_adc_3 -> Net-(D13-A)
- D14 pad 1: AnalogR_4 -> /cel
- D15 pad 1: +3V3 -> /abs
- D15 pad 2: /ANALOGUE/r_adc_4 -> Net-(D15-A)
- D16 pad 1: AnalogR_5 -> /door
- D17 pad 1: +3V3 -> /button
- D17 pad 2: /ANALOGUE/r_adc_5 -> Net-(D17-A)
- D18 pad 1: FUEL_LVL_Rsense -> /alternator
- D19 pad 1: +3V3 -> GND
- D19 pad 2: /ANALOGUE/r_adc_6 -> Net-(D19-A)
- D7 pad 1: +3V3 -> GND
- D7 pad 2: /ANALOGUE/r_adc_1 -> Net-(D7-A)
- D8 pad 1: AnalogR_2 -> GND
- F1 pad 1: +5V_1 -> BATT12V+
- F1 pad 2: 5V_SENSOR -> /POWER INPUT/Power_Fused
- IC1 pad 1: +3V3 -> GND
- IC1 pad 2: /rpm -> /5V_SMPS_1/5V_SW
- IC1 pad 3: RPM_HALL -> Protected_12V
- IC1 pad 4: unconnected-(IC1-2Y-Pad4) -> /5V_SMPS_1/5V_FB
- IC1 pad 5: GND -> Net-(IC1-EN)
- IC1 pad 6: unconnected-(IC1-3Y-Pad6) -> Net-(IC1-BST)
- L1 pad 1: /12V_to_5V_AP63200WU-7/5V_SW -> /5V_SMPS_1/5V_SW
- L1 pad 2: /12V_to_5V_AP63200WU-7/5V_REG_OUT -> /5V_SMPS_1/5V_OUT
- Q1 pad 2: Net-(Q1-S) -> GND
- Q1 pad 3: Net-(Q1-D) -> SPEED_HALL
- Q10 pad 1: Net-(Q10-G) -> Net-(D31-K)
- Q10 pad 2: Net-(Q10-S) -> GND
- Q11 pad 1: Net-(Q11-G) -> Net-(D32-A)
- Q11 pad 2: Net-(IC7B-+) -> /POWER INPUT/Power_Mid
- Q11 pad 3: Net-(D14-A) -> /POWER INPUT/Power_Fused
- Q12 pad 1: Net-(Q12-G) -> Net-(D32-A)
- Q12 pad 2: Net-(Q12-S) -> /POWER INPUT/Power_Mid
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Routing:
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- removed copper zone on F.Cu, net /12V_to_5V_AP63200WU-7/5V_REG_OUT
- removed copper zone on F.Cu, net /12V_to_5V_AP63200WU-7/5V_SW
- removed copper zone on F.Cu, net /POWER INPUT/Power_Pre-Filter
- removed copper zone on F.Cu, net /right_turn
- removed copper zone on B.Cu, net GND
- removed copper zone on F.Cu, net GND
- removed copper zone on F.Cu, net Net-(C19-Pad1)
- removed copper zone on F.Cu, net Net-(D11-K)
- removed copper zone on F.Cu, net Net-(IC4-SW)
- removed copper zone on F.Cu, net PROTECTED_12V+
Other:
- board text removed: "+5V"
- board text removed: "GND"
- board text removed: "RX"
- board text removed: "TX"

Commit message: Emulator : resistance banks layout
Parts:
- added J7: R bypass, Connector_PinSocket_2.54mm:PinSocket_1x02_P2.54mm_Vertical, F.Cu at (51.8, 138.9)
- R21: value 0 -> 270
- R22: value 10 -> 270
- R23: value 20 -> 270
- R24: value 30 -> 270
- R25: value 51 -> 270
- R26: value 91 -> 270
- R27: value 130 -> 270
- R28: value 180 -> 270
- R29: value 270 -> 2k
- R30: value 470 -> 2k
- R31: value 750 -> 2k
- R32: value 1k1 -> 2k
- R33: value 1k6 -> 2k
- R35: value 2k4 -> 2k
- R36: value 3k -> 2k
- moved D34 188.6 mm to (35.1, 141.3), turned to 180 degrees
- moved Q14 186.8 mm to (37.1, 138.8)
- moved R116 185.3 mm to (34.0, 138.8), turned to -90 degrees
- moved R117 184.2 mm to (35.1, 136.2)
- moved Q6 181.7 mm to (42.2, 124.6), turned to 180 degrees
- moved D27 179.5 mm to (44.2, 122.0)
- moved D25 178.2 mm to (35.0, 119.9), turned to 180 degrees
- moved Q4 176.3 mm to (37.0, 117.4)
- moved R103 175.0 mm to (44.2, 127.1), turned to 180 degrees
- moved R98 174.7 mm to (34.0, 117.4), turned to -90 degrees
- moved R99 174.2 mm to (35.0, 114.8)
- moved R102 174.0 mm to (45.2, 124.6), turned to 90 degrees
- moved Q8 171.3 mm to (42.2, 131.7), turned to 180 degrees
- moved Q13 171.1 mm to (42.2, 138.8), turned to 180 degrees
- moved Q5 170.9 mm to (42.2, 117.5), turned to 180 degrees
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Routing:
- net FUEL_LVL_Rsense: track 0.00 -> 68.7 mm
- net /Switchable Resistor 1/Res_ON: track 0.00 -> 27.9 mm, vias 0 -> 2
- net /Switchable Resistor 16/Res_ON: track 0.00 -> 24.6 mm, vias 0 -> 2
- net /Switchable Resistor 10/Res_ON: track 0.00 -> 24.3 mm, vias 0 -> 2
- net /Switchable Resistor 3/Res_ON: track 0.00 -> 22.0 mm, vias 0 -> 2
- net /Switchable Resistor 7/Res_ON: track 0.00 -> 21.8 mm, vias 0 -> 2
- net /Switchable Resistor 5/Res_ON: track 0.00 -> 21.7 mm, vias 0 -> 2
- net /Switchable Resistor 12/Res_ON: track 0.00 -> 20.6 mm, vias 0 -> 2
- net /Switchable Resistor 14/Res_ON: track 0.00 -> 20.6 mm, vias 0 -> 2
- net /Switchable Resistor 17/Res_ON: track 0.00 -> 16.1 mm
- net /Switchable Resistor 6/Res_ON: track 0.00 -> 13.9 mm
- net /Switchable Resistor 0/Res_ON: track 0.00 -> 12.3 mm
- net /Switchable Resistor11/Res_ON: track 0.00 -> 10.5 mm
- net /Switchable Resistor 15/Res_ON: track 0.00 -> 10.4 mm
- net /Switchable Resistor 4/Res_ON: track 0.00 -> 7.88 mm
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
Commit message: Additional TP for Emulator board
Parts:
- added TP23: ~{TP_HL}, TestPoint:TestPoint_Pad_D2.0mm, F.Cu at (187.2, 127.8)
- added TP24: TP_LL, TestPoint:TestPoint_Pad_D2.0mm, F.Cu at (172.0, 127.8)
- added TP25: ~{TP_HL}, TestPoint:TestPoint_Pad_D2.0mm, F.Cu at (186.7, 118.6)
- added TP26: TP_LL, TestPoint:TestPoint_Pad_D2.0mm, F.Cu at (171.4, 118.6)
- added TP27: ~{TP_HL}, TestPoint:TestPoint_Pad_D2.0mm, F.Cu at (163.6, 128.0)
- added TP28: TP_LL, TestPoint:TestPoint_Pad_D2.0mm, F.Cu at (148.3, 128.0)
- added TP29: ~{TP_HL}, TestPoint:TestPoint_Pad_D2.0mm, F.Cu at (162.6, 137.2)
- added TP30: TP_LL, TestPoint:TestPoint_Pad_D2.0mm, F.Cu at (147.3, 137.2)
- added TP31: ~{TP_HL}, TestPoint:TestPoint_Pad_D2.0mm, F.Cu at (164.1, 118.4)
- added TP32: TP_LL, TestPoint:TestPoint_Pad_D2.0mm, F.Cu at (148.8, 118.4)
- added TP33: ~{TP_HL}, TestPoint:TestPoint_Pad_D2.0mm, F.Cu at (186.4, 157.5)
- added TP34: TP_LL, TestPoint:TestPoint_Pad_D2.0mm, F.Cu at (171.2, 157.5)
- added TP35: ~{TP_HL}, TestPoint:TestPoint_Pad_D2.0mm, F.Cu at (187.2, 148.1)
- added TP36: TP_LL, TestPoint:TestPoint_Pad_D2.0mm, F.Cu at (172.0, 148.1)
- added TP37: ~{TP_HL}, TestPoint:TestPoint_Pad_D2.0mm, F.Cu at (162.1, 147.3)
- added TP38: TP_LL, TestPoint:TestPoint_Pad_D2.0mm, F.Cu at (146.8, 147.3)
- added TP39: ~{TP_HL}, TestPoint:TestPoint_Pad_D2.0mm, F.Cu at (187.5, 137.2)
- added TP40: TP_LL, TestPoint:TestPoint_Pad_D2.0mm, F.Cu at (172.2, 137.2)
- moved SW1 208.7 mm to (19.4, 192.7)
- moved R17 192.7 mm to (31.2, 191.0)
- moved R134 186.2 mm to (31.2, 193.9)
- moved R19 173.6 mm to (35.7, 190.8)
- moved U2 163.8 mm to (80.8, 164.6), turned to -90 degrees
- moved J6 133.0 mm to (132.6, 179.8)
- moved R40 114.2 mm to (114.4, 180.1)
- moved R41 114.2 mm to (114.4, 182.6)
- moved TP11 113.1 mm to (263.2, 155.4)
- moved D4 112.7 mm to (248.4, 35.1)
- moved U14 110.2 mm to (255.6, 153.9)
- moved TP3 108.9 mm to (51.8, 109.7)
- moved D19 108.3 mm to (258.2, 158.0), turned to 180 degrees
- moved TP21 108.1 mm to (266.2, 131.1)
- moved R76 107.1 mm to (262.2, 151.4), turned to -90 degrees
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Routing:
- net /right_turn: track 0.00 -> 7.28 mm
- net /alarm: track 0.00 -> 7.28 mm
- net /ignition: track 0.00 -> 7.28 mm
- net /coolant: track 0.00 -> 7.28 mm
- net /full_beams: track 0.00 -> 7.28 mm
- net /backlight: track 0.00 -> 7.28 mm
- net /left_turn: track 0.00 -> 7.28 mm
- net R_TURN_ActLO: track 0.00 -> 6.39 mm
- net Net-(R47-Pad1): track 0.00 -> 6.39 mm
- net BRAKE_ActLO: track 0.00 -> 6.39 mm
- net CEL_ActLO: track 0.00 -> 6.39 mm
- net Net-(R74-Pad1): track 0.00 -> 6.39 mm
- net Net-(R71-Pad1): track 0.00 -> 6.39 mm
- net Net-(R68-Pad1): track 0.00 -> 6.39 mm
- net Net-(R65-Pad1): track 0.00 -> 6.39 mm
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- added copper zone on F.Cu, net /3V3_SMPS/3V3_OUT
- added copper zone on F.Cu, net /3V3_SMPS/3V3_SW
- added copper zone on F.Cu, net /5V_SMPS_1/5V_OUT
- added copper zone on F.Cu, net /5V_SMPS_1/5V_SW

Commit message: Emulator : groupings
Parts:
- moved J1 119.0 mm to (135.1, 114.3), turned to 90 degrees
- moved C1 103.8 mm to (154.8, 180.9)
- moved R10 103.8 mm to (158.8, 180.9)
- moved U1 103.8 mm to (157.0, 186.4)
- moved R18 77.6 mm to (55.1, 142.2)
- moved TP1 76.5 mm to (20.1, 176.2)
- moved TP2 76.5 mm to (20.1, 179.8)
- moved D7 75.1 mm to (59.2, 142.2), turned to 180 degrees
- moved U2 64.7 mm to (25.4, 131.1), turned to 0 degrees
- moved SW1 63.9 mm to (53.4, 138.6)
- moved R19 59.8 mm to (63.2, 137.6), turned to -90 degrees
- moved TP28 58.6 mm to (102.6, 164.6)
- moved R61 58.6 mm to (117.3, 150.9)
- moved R62 58.6 mm to (104.1, 150.9)
- moved TP27 58.6 mm to (117.9, 164.6)
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Routing:
- net /5V_SMPS_1/5V_OUT: track 0.00 -> 32.2 mm, vias 0 -> 2
- net /3V3_SMPS/3V3_OUT: track 0.00 -> 32.2 mm, vias 0 -> 2
- net Net-(D32-A): track 0.00 -> 9.71 mm, vias 0 -> 2
- net /ign_EN: track 0.00 -> 9.38 mm
- net Net-(R17-Pad1): track 0.00 -> 6.89 mm
- net /3V3_SMPS/3V3_FB: track 0.00 -> 5.91 mm
- net /5V_SMPS_1/5V_FB: track 0.00 -> 5.91 mm
- net /3V3_SMPS/3V3_EN: track 0.00 -> 5.66 mm
- net Net-(IC1-EN): track 0.00 -> 5.66 mm
- net /ledc_chan_3: track 0.00 -> 5.56 mm
- net /ledc_chan_4: track 0.00 -> 5.52 mm
- net Net-(U2-5V): track 0.00 -> 4.94 mm
- net /3V3_SMPS/3V3_SW: track 0.00 -> 3.74 mm
- net /5V_SMPS_1/5V_SW: track 0.00 -> 3.69 mm
- net Net-(Q10-D): track 0.00 -> 3.33 mm
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- added copper zone on F.Cu, net /POWER INPUT/Power_Fused
- added copper zone on F.Cu, net /POWER INPUT/Power_Mid
- added copper zone on F.Cu, net /POWER INPUT/Power_Pre-Filter
- added copper zone on F.Cu, net BATT12V+
- added copper zone on F.Cu, net Net-(D31-K)
- added copper zone on F.Cu, net Net-(D32-A)
- added copper zone on F.Cu, net Protected_12V
Other:
- board size 115 x 95 mm -> 245.1 x 163.1 mm
- board text added: "12V"
- board text added: "3V3 ON"
- board text added: "5V ON"
- board text added: "BATT ON"
- board text added: "BATT+ ----- GRND"
- board text added: "FUEL R"
- board text added: "PRTCT"
- board text added: "START IGN"

Commit message: Emulator board : layout update
- Moved to Open Drain style Mosfets instead of Optoisolators
- Added manual push button for BUTTON
- Did groups in the PCB layout
Parts:
- removed D10, D11, D12, D13, D14, D15, D16, D17, D18, D19, D20, D21, D22, D23, D24, D9: HL State, LED_SMD:LED_0603_1608Metric_Pad1.05x0.95mm_HandSolder
- removed R46, R49, R52, R55, R58, R61, R64, R67, R70, R73, R76, R79, R82, R85, R88, R95: 33k, Resistor_SMD:R_0805_2012Metric_Pad1.20x1.40mm_HandSolder
- removed R47, R50, R53, R56, R59, R62, R65, R68, R71, R74, R77, R80, R83, R86, R89, R96: 2k, Resistor_SMD:R_0805_2012Metric_Pad1.20x1.40mm_HandSolder
- removed R48, R51, R54, R57, R60, R63, R66, R69, R72, R75, R78, R81, R84, R87, R90, R97: 270, Resistor_SMD:R_0603_1608Metric_Pad0.98x0.95mm_HandSolder
- removed TP10, TP12, TP14, TP16, TP18, TP20, TP22, TP24, TP26, TP28, TP30, TP32, TP34, TP36, TP38, TP40: TP_LL, TestPoint:TestPoint_Pad_D2.0mm
- removed TP11, TP13, TP15, TP17, TP19, TP21, TP9: TP_HL, TestPoint:TestPoint_Pad_D2.0mm
- removed TP23, TP25, TP27, TP29, TP31, TP33, TP35, TP37, TP39: ~{TP_HL}, TestPoint:TestPoint_Pad_D2.0mm
- removed U10, U11, U12, U13, U14, U15, U16, U17, U18, U19, U4, U5, U6, U7, U8, U9: ~, Package_DIP:SMDIP-4_W7.62mm
- added D43: Out Lo, LED_SMD:LED_0603_1608Metric_Pad1.05x0.95mm_HandSolder, F.Cu at (151.8, 94.9)
- added D44: Out Hi, LED_SMD:LED_0603_1608Metric_Pad1.05x0.95mm_HandSolder, F.Cu at (158.8, 95.0)
- added D45: Out Hi, LED_SMD:LED_0603_1608Metric_Pad1.05x0.95mm_HandSolder, F.Cu at (184.2, 95.4)
- added D46: Out Lo, LED_SMD:LED_0603_1608Metric_Pad1.05x0.95mm_HandSolder, F.Cu at (177.2, 95.2)
- added D47: Out Hi, LED_SMD:LED_0603_1608Metric_Pad1.05x0.95mm_HandSolder, F.Cu at (189.5, 80.1)
- added D48: Out Lo, LED_SMD:LED_0603_1608Metric_Pad1.05x0.95mm_HandSolder, F.Cu at (182.5, 80.0)
- added D49: Out Hi, LED_SMD:LED_0603_1608Metric_Pad1.05x0.95mm_HandSolder, F.Cu at (115.6, 130.9)
- added D50: Out Lo, LED_SMD:LED_0603_1608Metric_Pad1.05x0.95mm_HandSolder, F.Cu at (108.6, 130.8)
- added D51: Out Hi, LED_SMD:LED_0603_1608Metric_Pad1.05x0.95mm_HandSolder, F.Cu at (127.6, 131.4)
- added D52: Out Lo, LED_SMD:LED_0603_1608Metric_Pad1.05x0.95mm_HandSolder, F.Cu at (120.7, 131.3)
- added D53: Out Hi, LED_SMD:LED_0603_1608Metric_Pad1.05x0.95mm_HandSolder, F.Cu at (217.2, 133.5)
- added D54: Out Lo, LED_SMD:LED_0603_1608Metric_Pad1.05x0.95mm_HandSolder, F.Cu at (210.2, 133.3)
- added D55: Out Hi, LED_SMD:LED_0603_1608Metric_Pad1.05x0.95mm_HandSolder, F.Cu at (224.8, 148.7)
- added D56: Out Lo, LED_SMD:LED_0603_1608Metric_Pad1.05x0.95mm_HandSolder, F.Cu at (217.8, 148.6)
- added D57: Out Hi, LED_SMD:LED_0603_1608Metric_Pad1.05x0.95mm_HandSolder, F.Cu at (229.9, 133.5)
- added D58: Out Lo, LED_SMD:LED_0603_1608Metric_Pad1.05x0.95mm_HandSolder, F.Cu at (222.9, 133.3)
- added D59: Out Hi, LED_SMD:LED_0603_1608Metric_Pad1.05x0.95mm_HandSolder, F.Cu at (201.9, 80.1)
- added D60: Out Lo, LED_SMD:LED_0603_1608Metric_Pad1.05x0.95mm_HandSolder, F.Cu at (194.9, 80.0)
- added D61: Out Hi, LED_SMD:LED_0603_1608Metric_Pad1.05x0.95mm_HandSolder, F.Cu at (196.8, 95.4)
- added D62: Out Lo, LED_SMD:LED_0603_1608Metric_Pad1.05x0.95mm_HandSolder, F.Cu at (189.9, 95.2)
- added D63: Out Hi, LED_SMD:LED_0603_1608Metric_Pad1.05x0.95mm_HandSolder, F.Cu at (268.0, 133.5)
- added D64: Out Lo, LED_SMD:LED_0603_1608Metric_Pad1.05x0.95mm_HandSolder, F.Cu at (261.0, 133.3)
- added D65: Out Hi, LED_SMD:LED_0603_1608Metric_Pad1.05x0.95mm_HandSolder, F.Cu at (262.9, 148.7)
- added D66: Out Lo, LED_SMD:LED_0603_1608Metric_Pad1.05x0.95mm_HandSolder, F.Cu at (255.9, 148.6)
- added D67: Out Hi, LED_SMD:LED_0603_1608Metric_Pad1.05x0.95mm_HandSolder, F.Cu at (255.3, 133.5)
- added D68: Out Lo, LED_SMD:LED_0603_1608Metric_Pad1.05x0.95mm_HandSolder, F.Cu at (248.3, 133.3)
- added D69: Out Hi, LED_SMD:LED_0603_1608Metric_Pad1.05x0.95mm_HandSolder, F.Cu at (250.2, 148.7)
- added D70: Out Lo, LED_SMD:LED_0603_1608Metric_Pad1.05x0.95mm_HandSolder, F.Cu at (243.2, 148.6)
- added D71: Out Hi, LED_SMD:LED_0603_1608Metric_Pad1.05x0.95mm_HandSolder, F.Cu at (242.6, 133.5)
- added D72: Out Lo, LED_SMD:LED_0603_1608Metric_Pad1.05x0.95mm_HandSolder, F.Cu at (235.6, 133.3)
- added D73: Out Hi, LED_SMD:LED_0603_1608Metric_Pad1.05x0.95mm_HandSolder, F.Cu at (237.5, 148.7)
- added D74: Out Lo, LED_SMD:LED_0603_1608Metric_Pad1.05x0.95mm_HandSolder, F.Cu at (230.5, 148.6)
- added J10: Manual backup, Connector_PinHeader_2.54mm:PinHeader_1x03_P2.54mm_Vertical, F.Cu at (109.2, 134.6)
- added J11: Manual backup, Connector_PinHeader_2.54mm:PinHeader_1x03_P2.54mm_Vertical, F.Cu at (121.3, 135.1)
- added J12: Manual backup, Connector_PinHeader_2.54mm:PinHeader_1x03_P2.54mm_Vertical, F.Cu at (210.8, 137.2)
- added J13: Manual backup, Connector_PinHeader_2.54mm:PinHeader_1x03_P2.54mm_Vertical, F.Cu at (218.4, 152.4)
- added J14: Manual backup, Connector_PinHeader_2.54mm:PinHeader_1x03_P2.54mm_Vertical, F.Cu at (223.5, 137.2)
- added J15: Manual backup, Connector_PinHeader_2.54mm:PinHeader_1x03_P2.54mm_Vertical, F.Cu at (195.6, 83.8)
- added J16: Manual backup, Connector_PinHeader_2.54mm:PinHeader_1x03_P2.54mm_Vertical, F.Cu at (190.5, 99.1)
- added J17: Manual backup, Connector_PinHeader_2.54mm:PinHeader_1x03_P2.54mm_Vertical, F.Cu at (261.6, 137.2)
- added J18: Manual backup, Connector_PinHeader_2.54mm:PinHeader_1x03_P2.54mm_Vertical, F.Cu at (256.5, 152.4)
- added J19: Manual backup, Connector_PinHeader_2.54mm:PinHeader_1x03_P2.54mm_Vertical, F.Cu at (248.9, 137.2)
- added J20: Manual backup, Connector_PinHeader_2.54mm:PinHeader_1x03_P2.54mm_Vertical, F.Cu at (243.8, 152.4)
- added J21: Manual backup, Connector_PinHeader_2.54mm:PinHeader_1x03_P2.54mm_Vertical, F.Cu at (236.2, 137.2)
- added J22: Manual backup, Connector_PinHeader_2.54mm:PinHeader_1x03_P2.54mm_Vertical, F.Cu at (231.1, 152.4)
- added J23: Manual backup, Connector_PinHeader_2.54mm:PinHeader_1x03_P2.54mm_Vertical, F.Cu at (152.4, 98.7)
- added J8: Manual backup, Connector_PinHeader_2.54mm:PinHeader_1x03_P2.54mm_Vertical, F.Cu at (177.8, 99.1)
- added J9: Manual backup, Connector_PinHeader_2.54mm:PinHeader_1x03_P2.54mm_Vertical, F.Cu at (183.1, 83.8)
- added JP1: Bypass JP, Jumper:SolderJumper-2_P1.3mm_Bridged_RoundedPad1.0x1.5mm, F.Cu at (181.5, 101.0)
- added JP10: Bypass JP, Jumper:SolderJumper-2_P1.3mm_Bridged_RoundedPad1.0x1.5mm, F.Cu at (265.3, 139.1)
- added JP11: Bypass JP, Jumper:SolderJumper-2_P1.3mm_Bridged_RoundedPad1.0x1.5mm, F.Cu at (260.2, 154.3)
- added JP12: Bypass JP, Jumper:SolderJumper-2_P1.3mm_Bridged_RoundedPad1.0x1.5mm, F.Cu at (252.6, 139.1)
- added JP13: Bypass JP, Jumper:SolderJumper-2_P1.3mm_Bridged_RoundedPad1.0x1.5mm, F.Cu at (247.5, 154.3)
- added JP14: Bypass JP, Jumper:SolderJumper-2_P1.3mm_Bridged_RoundedPad1.0x1.5mm, F.Cu at (239.9, 139.1)
- added JP15: Bypass JP, Jumper:SolderJumper-2_P1.3mm_Bridged_RoundedPad1.0x1.5mm, F.Cu at (234.8, 154.3)
- added JP16: Bypass JP, Jumper:SolderJumper-2_P1.3mm_Bridged_RoundedPad1.0x1.5mm, F.Cu at (156.1, 100.6)
- added JP2: Bypass JP, Jumper:SolderJumper-2_P1.3mm_Bridged_RoundedPad1.0x1.5mm, F.Cu at (186.8, 85.7)
- added JP3: Bypass JP, Jumper:SolderJumper-2_P1.3mm_Bridged_RoundedPad1.0x1.5mm, F.Cu at (112.9, 136.5)
- added JP4: Bypass JP, Jumper:SolderJumper-2_P1.3mm_Bridged_RoundedPad1.0x1.5mm, F.Cu at (125.0, 137.0)
- added JP5: Bypass JP, Jumper:SolderJumper-2_P1.3mm_Bridged_RoundedPad1.0x1.5mm, F.Cu at (214.5, 139.1)
- added JP6: Bypass JP, Jumper:SolderJumper-2_P1.3mm_Bridged_RoundedPad1.0x1.5mm, F.Cu at (222.1, 154.3)
- added JP7: Bypass JP, Jumper:SolderJumper-2_P1.3mm_Bridged_RoundedPad1.0x1.5mm, F.Cu at (227.2, 139.1)
- added JP8: Bypass JP, Jumper:SolderJumper-2_P1.3mm_Bridged_RoundedPad1.0x1.5mm, F.Cu at (199.3, 85.7)
- added JP9: Bypass JP, Jumper:SolderJumper-2_P1.3mm_Bridged_RoundedPad1.0x1.5mm, F.Cu at (194.2, 101.0)
- added Q23: 2N7002, Package_TO_SOT_SMD:SOT-23, F.Cu at (156.1, 96.8)
- added Q24: 2N7002, Package_TO_SOT_SMD:SOT-23, F.Cu at (181.5, 97.2)
- added Q25: 2N7002, Package_TO_SOT_SMD:SOT-23, F.Cu at (186.8, 81.9)
- added Q26: 2N7002, Package_TO_SOT_SMD:SOT-23, F.Cu at (112.9, 132.7)
- added Q27: 2N7002, Package_TO_SOT_SMD:SOT-23, F.Cu at (125.0, 133.2)
- added Q28: 2N7002, Package_TO_SOT_SMD:SOT-23, F.Cu at (214.5, 135.3)
- added Q29: 2N7002, Package_TO_SOT_SMD:SOT-23, F.Cu at (222.1, 150.5)
- added Q30: 2N7002, Package_TO_SOT_SMD:SOT-23, F.Cu at (227.2, 135.3)
- added Q31: 2N7002, Package_TO_SOT_SMD:SOT-23, F.Cu at (199.3, 81.9)
- added Q32: 2N7002, Package_TO_SOT_SMD:SOT-23, F.Cu at (194.2, 97.2)
- added Q33: 2N7002, Package_TO_SOT_SMD:SOT-23, F.Cu at (265.3, 135.3)
- added Q34: 2N7002, Package_TO_SOT_SMD:SOT-23, F.Cu at (260.2, 150.5)
- added Q35: 2N7002, Package_TO_SOT_SMD:SOT-23, F.Cu at (252.6, 135.3)
- added Q36: 2N7002, Package_TO_SOT_SMD:SOT-23, F.Cu at (247.5, 150.5)
- added Q37: 2N7002, Package_TO_SOT_SMD:SOT-23, F.Cu at (239.9, 135.3)
- added Q38: 2N7002, Package_TO_SOT_SMD:SOT-23, F.Cu at (234.8, 150.5)
- added R135: 270, Resistor_SMD:R_0603_1608Metric_Pad0.98x0.95mm_HandSolder, F.Cu at (153.4, 94.9)
- added R136: 270, Resistor_SMD:R_0603_1608Metric_Pad0.98x0.95mm_HandSolder, F.Cu at (160.4, 95.0)
- added R137: 1k, Resistor_SMD:R_0603_1608Metric_Pad0.98x0.95mm_HandSolder, F.Cu at (156.1, 93.8)
- added R138: 270, Resistor_SMD:R_0603_1608Metric_Pad0.98x0.95mm_HandSolder, F.Cu at (185.8, 95.4)
- added R139: 1k, Resistor_SMD:R_0805_2012Metric_Pad1.20x1.40mm_HandSolder, F.Cu at (159.8, 104.0)
- added R140: 1k, Resistor_SMD:R_0805_2012Metric_Pad1.20x1.40mm_HandSolder, F.Cu at (157.6, 104.0)
- added R141: 1k, Resistor_SMD:R_0805_2012Metric_Pad1.20x1.40mm_HandSolder, F.Cu at (155.4, 104.0)
- added R142: 270, Resistor_SMD:R_0603_1608Metric_Pad0.98x0.95mm_HandSolder, F.Cu at (178.8, 95.2)
- added R143: 1k, Resistor_SMD:R_0603_1608Metric_Pad0.98x0.95mm_HandSolder, F.Cu at (181.5, 94.2)
- added R144: 1k, Resistor_SMD:R_0805_2012Metric_Pad1.20x1.40mm_HandSolder, F.Cu at (183.0, 104.4)
- added R145: 1k, Resistor_SMD:R_0805_2012Metric_Pad1.20x1.40mm_HandSolder, F.Cu at (185.2, 104.4)
- added R146: 1k, Resistor_SMD:R_0805_2012Metric_Pad1.20x1.40mm_HandSolder, F.Cu at (180.8, 104.4)
- added R147: 270, Resistor_SMD:R_0603_1608Metric_Pad0.98x0.95mm_HandSolder, F.Cu at (191.1, 80.1)
- added R148: 270, Resistor_SMD:R_0603_1608Metric_Pad0.98x0.95mm_HandSolder, F.Cu at (184.2, 80.0)
- added R149: 1k, Resistor_SMD:R_0603_1608Metric_Pad0.98x0.95mm_HandSolder, F.Cu at (186.8, 79.0)
- added R150: 1k, Resistor_SMD:R_0805_2012Metric_Pad1.20x1.40mm_HandSolder, F.Cu at (188.3, 89.2)
- added R151: 1k, Resistor_SMD:R_0805_2012Metric_Pad1.20x1.40mm_HandSolder, F.Cu at (190.5, 89.2)
- added R152: 1k, Resistor_SMD:R_0805_2012Metric_Pad1.20x1.40mm_HandSolder, F.Cu at (186.2, 89.2)
- added R153: 270, Resistor_SMD:R_0603_1608Metric_Pad0.98x0.95mm_HandSolder, F.Cu at (117.2, 130.9)
- added R154: 270, Resistor_SMD:R_0603_1608Metric_Pad0.98x0.95mm_HandSolder, F.Cu at (110.2, 130.8)
- added R155: 1k, Resistor_SMD:R_0603_1608Metric_Pad0.98x0.95mm_HandSolder, F.Cu at (112.9, 129.8)
- added R156: 1k, Resistor_SMD:R_0805_2012Metric_Pad1.20x1.40mm_HandSolder, F.Cu at (114.4, 140.0)
- added R157: 1k, Resistor_SMD:R_0805_2012Metric_Pad1.20x1.40mm_HandSolder, F.Cu at (116.6, 140.0)
- added R158: 1k, Resistor_SMD:R_0805_2012Metric_Pad1.20x1.40mm_HandSolder, F.Cu at (112.3, 140.0)
- added R159: 270, Resistor_SMD:R_0603_1608Metric_Pad0.98x0.95mm_HandSolder, F.Cu at (129.3, 131.4)
- added R160: 270, Resistor_SMD:R_0603_1608Metric_Pad0.98x0.95mm_HandSolder, F.Cu at (122.3, 131.3)
- added R161: 1k, Resistor_SMD:R_0603_1608Metric_Pad0.98x0.95mm_HandSolder, F.Cu at (125.0, 130.3)
- added R162: 1k, Resistor_SMD:R_0805_2012Metric_Pad1.20x1.40mm_HandSolder, F.Cu at (126.5, 140.4)
- added R163: 1k, Resistor_SMD:R_0805_2012Metric_Pad1.20x1.40mm_HandSolder, F.Cu at (128.7, 140.4)
- added R164: 1k, Resistor_SMD:R_0805_2012Metric_Pad1.20x1.40mm_HandSolder, F.Cu at (124.3, 140.4)
- added R165: 270, Resistor_SMD:R_0603_1608Metric_Pad0.98x0.95mm_HandSolder, F.Cu at (218.8, 133.5)
- added R166: 270, Resistor_SMD:R_0603_1608Metric_Pad0.98x0.95mm_HandSolder, F.Cu at (211.8, 133.3)
- added R167: 1k, Resistor_SMD:R_0603_1608Metric_Pad0.98x0.95mm_HandSolder, F.Cu at (214.5, 132.3)
- added R168: 1k, Resistor_SMD:R_0805_2012Metric_Pad1.20x1.40mm_HandSolder, F.Cu at (216.0, 142.5)
- added R169: 1k, Resistor_SMD:R_0805_2012Metric_Pad1.20x1.40mm_HandSolder, F.Cu at (218.2, 142.5)
- added R170: 1k, Resistor_SMD:R_0805_2012Metric_Pad1.20x1.40mm_HandSolder, F.Cu at (213.9, 142.5)
- added R171: 270, Resistor_SMD:R_0603_1608Metric_Pad0.98x0.95mm_HandSolder, F.Cu at (226.4, 148.7)
- added R172: 270, Resistor_SMD:R_0603_1608Metric_Pad0.98x0.95mm_HandSolder, F.Cu at (219.5, 148.6)
- added R173: 1k, Resistor_SMD:R_0603_1608Metric_Pad0.98x0.95mm_HandSolder, F.Cu at (222.1, 147.6)
- added R174: 1k, Resistor_SMD:R_0805_2012Metric_Pad1.20x1.40mm_HandSolder, F.Cu at (223.6, 157.7)
- added R175: 1k, Resistor_SMD:R_0805_2012Metric_Pad1.20x1.40mm_HandSolder, F.Cu at (225.8, 157.7)
- added R176: 1k, Resistor_SMD:R_0805_2012Metric_Pad1.20x1.40mm_HandSolder, F.Cu at (221.5, 157.7)
- added R177: 270, Resistor_SMD:R_0603_1608Metric_Pad0.98x0.95mm_HandSolder, F.Cu at (231.5, 133.5)
- added R178: 270, Resistor_SMD:R_0603_1608Metric_Pad0.98x0.95mm_HandSolder, F.Cu at (224.5, 133.3)
- added R179: 1k, Resistor_SMD:R_0603_1608Metric_Pad0.98x0.95mm_HandSolder, F.Cu at (227.2, 132.3)
- added R180: 1k, Resistor_SMD:R_0805_2012Metric_Pad1.20x1.40mm_HandSolder, F.Cu at (228.7, 142.5)
- added R181: 1k, Resistor_SMD:R_0805_2012Metric_Pad1.20x1.40mm_HandSolder, F.Cu at (230.9, 142.5)
- added R182: 1k, Resistor_SMD:R_0805_2012Metric_Pad1.20x1.40mm_HandSolder, F.Cu at (226.6, 142.5)
- added R183: 270, Resistor_SMD:R_0603_1608Metric_Pad0.98x0.95mm_HandSolder, F.Cu at (203.6, 80.1)
- added R184: 270, Resistor_SMD:R_0603_1608Metric_Pad0.98x0.95mm_HandSolder, F.Cu at (196.6, 80.0)
- added R185: 1k, Resistor_SMD:R_0603_1608Metric_Pad0.98x0.95mm_HandSolder, F.Cu at (199.3, 79.0)
- added R186: 1k, Resistor_SMD:R_0805_2012Metric_Pad1.20x1.40mm_HandSolder, F.Cu at (200.8, 89.2)
- added R187: 1k, Resistor_SMD:R_0805_2012Metric_Pad1.20x1.40mm_HandSolder, F.Cu at (202.9, 89.2)
- added R188: 1k, Resistor_SMD:R_0805_2012Metric_Pad1.20x1.40mm_HandSolder, F.Cu at (198.6, 89.2)
- added R189: 270, Resistor_SMD:R_0603_1608Metric_Pad0.98x0.95mm_HandSolder, F.Cu at (198.5, 95.4)
- added R190: 270, Resistor_SMD:R_0603_1608Metric_Pad0.98x0.95mm_HandSolder, F.Cu at (191.5, 95.2)
- added R191: 1k, Resistor_SMD:R_0603_1608Metric_Pad0.98x0.95mm_HandSolder, F.Cu at (194.2, 94.2)
- added R192: 1k, Resistor_SMD:R_0805_2012Metric_Pad1.20x1.40mm_HandSolder, F.Cu at (195.7, 104.4)
- added R193: 1k, Resistor_SMD:R_0805_2012Metric_Pad1.20x1.40mm_HandSolder, F.Cu at (197.9, 104.4)
- added R194: 1k, Resistor_SMD:R_0805_2012Metric_Pad1.20x1.40mm_HandSolder, F.Cu at (193.5, 104.4)
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Routing:
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- added copper zone on F.Cu, net Net-(JP1-A)
- added copper zone on F.Cu, net Net-(JP10-A)
- added copper zone on F.Cu, net Net-(JP11-A)
- added copper zone on F.Cu, net Net-(JP12-A)
- added copper zone on F.Cu, net Net-(JP13-A)
- added copper zone on F.Cu, net Net-(JP14-A)
- added copper zone on F.Cu, net Net-(JP15-A)
- added copper zone on F.Cu, net Net-(JP16-A)
- added copper zone on F.Cu, net Net-(JP2-A)
- added copper zone on F.Cu, net Net-(JP3-A)
- added copper zone on F.Cu, net Net-(JP4-A)
- added copper zone on F.Cu, net Net-(JP5-A)
- added copper zone on F.Cu, net Net-(JP6-A)
- added copper zone on F.Cu, net Net-(JP7-A)
- added copper zone on F.Cu, net Net-(JP8-A)
- added copper zone on F.Cu, net Net-(JP9-A)
Other:
- board text added: "5V"
- board text added: "V+"

Commit message: Emulator - block layout complete
Parts:
- moved C2 173.9 mm to (210.3, 60.8)
- moved D28 173.9 mm to (195.6, 65.0)
- moved D34 173.9 mm to (195.6, 79.2)
- moved D35 173.9 mm to (230.1, 74.7)
- moved D37 173.9 mm to (230.1, 67.5)
- moved D41 173.9 mm to (230.1, 60.4)
- moved D42 173.9 mm to (230.1, 53.3)
- moved Q13 173.9 mm to (202.7, 76.7)
- moved Q14 173.9 mm to (197.6, 76.7)
- moved Q15 173.9 mm to (228.1, 77.2)
- moved Q16 173.9 mm to (223.0, 77.2)
- moved Q17 173.9 mm to (228.1, 70.1)
- moved Q18 173.9 mm to (223.0, 70.1)
- moved Q19 173.9 mm to (223.0, 55.9)
- moved Q20 173.9 mm to (223.0, 63.0)
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Connections:
- U1 pad 10: /airbag -> /alarm
- U1 pad 11: /cel -> /button
- U1 pad 13: /right_turn -> /coolant
- U1 pad 14: /left_turn -> /door
- U1 pad 16: /door -> /right_turn
- U1 pad 17: /coolant -> /left_turn
- U1 pad 18: /button -> /alternator
- U1 pad 19: /alarm -> /full_beams
- U1 pad 20: /backlight -> /ignition
- U1 pad 4: /ignition -> /brakes
- U1 pad 5: /full_beams -> /parking
- U1 pad 6: /alternator -> /oil
- U1 pad 7: /brakes -> /airbag
- U1 pad 8: /parking -> /cel
- U1 pad 9: /oil -> /backlight
