File: KiCad PCB Files/VXDash_Emulator/VXDash_Emulator.kicad_pcb (KiCad board)
At the start: 2 copper layers, 245.1 x 163.1 mm, 359 parts, among them IC1 AP62200, IC2 AP62200, J1 Car 24P Connector, J10 Manual backup, J11 Manual backup, J12 Manual backup, J13 Manual backup, J14 Manual backup, J15 Manual backup, J16 Manual backup, J17 Manual backup, J18 Manual backup, J19 Manual backup, J2 Level_Select, J20 Manual backup, J21 Manual backup, J22 Manual backup, J23 Manual backup, J3 Level_Select, J4 Board supply, J5 Level_Select, J6 I²C debug, J7 R bypass, J8 Manual backup, J9 Manual backup, Q1 2N7002, Q10 2N7002, Q11 PJA3441, Q12 PJA3441, Q13 2N7002, Q14 2N7002, Q15 2N7002, Q16 2N7002, Q17 2N7002, Q18 2N7002, Q19 2N7002, Q2 2N7002, Q20 2N7002, Q21 2N7002, Q22 2N7002, Q23 2N7002, Q24 2N7002, Q25 2N7002, Q26 2N7002, Q27 2N7002, Q28 2N7002, Q29 2N7002, Q3 2N7002, Q30 2N7002, Q31 2N7002, Q32 2N7002, Q33 2N7002, Q34 2N7002, Q35 2N7002, Q36 2N7002, Q37 2N7002, Q38 2N7002, Q4 2N7002, Q5 2N7002, Q6 2N7002, Q7 2N7002, Q8 2N7002, Q9 2N7002, SW1 Enable, SW2 Button Manual, U1 TCA9555PWR, U2 ESP32-S3-DevKitC, U3 TCA9555PWR

Commit message: Emulator board basic routing done
Parts:
- moved J6 161.7 mm to (246.1, 57.7), turned to 180 degrees
- moved TP7 124.2 mm to (143.5, 64.8)
- moved TP8 120.6 mm to (143.5, 72.4)
- moved R41 120.4 mm to (143.5, 69.8)
- moved R40 120.4 mm to (143.5, 67.3)
- moved R134 33.5 mm to (143.5, 120.7), turned to 180 degrees
- moved TP1 33.3 mm to (144.8, 101.6)
- moved TP2 33.3 mm to (144.8, 105.4)
- moved R17 8.26 mm to (116.8, 54.6), turned to 90 degrees
- moved C3 4.45 mm to (158.9, 112.5)
- moved C7 4.45 mm to (160.4, 109.0)
- moved C8 4.45 mm to (155.8, 108.5)
- moved IC1 4.45 mm to (166.5, 111.0)
- moved R42 4.45 mm to (173.6, 112.5)
- moved R43 4.45 mm to (172.1, 112.5)
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Connections:
- U2 pad 16: /ledc_chan_0 -> /ledc_chan_2
- U2 pad 18: /ledc_chan_2 -> /ledc_chan_0
Routing:
- net +3V3: track 9.56 -> 394.1 mm, vias 0 -> 30
- net BATT12V+: track 0.00 -> 269.7 mm, vias 0 -> 6
- net /SDA: track 0.00 -> 181.0 mm, vias 0 -> 3
- net /SCL: track 0.00 -> 180.8 mm, vias 0 -> 3
- net /ignition: track 6.87 -> 113.8 mm, vias 0 -> 2
- net /5v_enable: track 0.00 -> 95.9 mm
- net IGNITION_ActHI: track 3.30 -> 94.6 mm, vias 0 -> 1
- net +5V_1: track 2.07 -> 89.6 mm, vias 0 -> 5
- net /ledc_chan_2: track 1.52 -> 87.9 mm
- net /brakes: track 3.06 -> 83.0 mm, vias 0 -> 2
- net /parking: track 3.06 -> 82.8 mm, vias 0 -> 2
- net /ledc_chan_0: track 1.52 -> 74.6 mm, vias 0 -> 1
- net /oil: track 3.06 -> 71.0 mm, vias 0 -> 2
- net /airbag: track 3.06 -> 70.3 mm, vias 0 -> 2
- net /ledc_chan_1: track 1.52 -> 67.6 mm
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- added copper zone on F.Cu, net +3V3
- added copper zone on In2.Cu, net +3V3
- added copper zone on F.Cu, net +5V_1
- added copper zone on In2.Cu, net BATT12V+
- added copper zone on B.Cu, net GND
- added copper zone on F.Cu, net GND
- added copper zone on In1.Cu, net GND
- added copper zone on In2.Cu, net GND
- added copper zone on B.Cu, net Protected_12V
Other:
- board size 245.1 x 163.1 mm -> 149.9 x 72.4 mm
- copper layers 2 -> 4
- board text added: "BTN"
- board text added: "CH3"
- board text added: "CH4"
