File: KiCad PCB Files/VXDash_Emulator/VXDash_Emulator.kicad_sch (KiCad schematic)
At the start: 9 parts, among them J1 Conn_02x12_Odd_Even, J2 Conn_01x02, J3 Passthrough, J4 I²C debug, U17 ESP32-S3-DevKitC, U18 TCA9555PWR, U5 TCA9555PWR

Commit message: Emulator board refinements
- Is there stupid with the Active Hi Optos so that the logic is not inverted ?
- Added N-Mosfet activatable resistors. Stupidly simple ? Better MOSFET recommendation ?
Parts:
- removed J2: Conn_01x02, symbol Connector_Generic:Conn_01x02
- removed J3: Passthrough, Connector_PinHeader_2.54mm:PinHeader_2x15_P2.54mm_Vertical, symbol Connector_Generic:Conn_02x15_Odd_Even
- added J2: Conn_02x02_Odd_Even, symbol Connector_Generic:Conn_02x02_Odd_Even
- added Q24, Q25, Q26: 2N7002, Package_TO_SOT_SMD:SOT-23, symbol Transistor_FET:Q_NMOS_GSD
- added R1, R2: 4k7, Resistor_SMD:R_0603_1608Metric_Pad0.98x0.95mm_HandSolder, symbol VXDash_passives:Res
- added R10: 30, Resistor_SMD:R_0603_1608Metric_Pad0.98x0.95mm_HandSolder, symbol VXDash_passives:Res
- added R11: 51, Resistor_SMD:R_0603_1608Metric_Pad0.98x0.95mm_HandSolder, symbol VXDash_passives:Res
- added R12: 91, Resistor_SMD:R_0603_1608Metric_Pad0.98x0.95mm_HandSolder, symbol VXDash_passives:Res
- added R13: 130, Resistor_SMD:R_0603_1608Metric_Pad0.98x0.95mm_HandSolder, symbol VXDash_passives:Res
- added R14: 180, Resistor_SMD:R_0603_1608Metric_Pad0.98x0.95mm_HandSolder, symbol VXDash_passives:Res
- added R15: 270, Resistor_SMD:R_0603_1608Metric_Pad0.98x0.95mm_HandSolder, symbol VXDash_passives:Res
- added R16: 470, Resistor_SMD:R_0603_1608Metric_Pad0.98x0.95mm_HandSolder, symbol VXDash_passives:Res
- added R17: 750, Resistor_SMD:R_0603_1608Metric_Pad0.98x0.95mm_HandSolder, symbol VXDash_passives:Res
- added R18: 1k1, Resistor_SMD:R_0603_1608Metric_Pad0.98x0.95mm_HandSolder, symbol VXDash_passives:Res
- added R19: 1k6, Resistor_SMD:R_0603_1608Metric_Pad0.98x0.95mm_HandSolder, symbol VXDash_passives:Res
- added R20: 2k, Resistor_SMD:R_0603_1608Metric_Pad0.98x0.95mm_HandSolder, symbol VXDash_passives:Res
- added R21: 2k4, Resistor_SMD:R_0603_1608Metric_Pad0.98x0.95mm_HandSolder, symbol VXDash_passives:Res
- added R22: 3k, Resistor_SMD:R_0603_1608Metric_Pad0.98x0.95mm_HandSolder, symbol VXDash_passives:Res
- added R7: 0, Resistor_SMD:R_0603_1608Metric_Pad0.98x0.95mm_HandSolder, symbol VXDash_passives:Res
- added R8: 10, Resistor_SMD:R_0603_1608Metric_Pad0.98x0.95mm_HandSolder, symbol VXDash_passives:Res
- added R9: 20, Resistor_SMD:R_0603_1608Metric_Pad0.98x0.95mm_HandSolder, symbol VXDash_passives:Res
- added R92, R93, R94, R95, R96, R97, R98: 1k, Resistor_SMD:R_0603_1608Metric_Pad0.98x0.95mm_HandSolder, symbol VXDash_passives:Res
- added SW2: Enable, symbol Switch:SW_SPST
- J1: value Conn_02x12_Odd_Even -> Car 24P Connector
Connections:
- net +3V3: now also U17.1 (3V3), U17.2 (3V3), R1.2, R2.2, R98.1
- net ABS_ActLO: now also J1.24 (Pin_24)
- net AIRBAG_ActLO: now also J1.8 (Pin_8)
- net ALARM_ActHI: now also J1.14 (Pin_14)
- net ALTERN_ActLO: now also J1.19 (Pin_19)
- net BATT12V+: now also J1.1 (Pin_1), R93.2, R95.2, R97.2
- net BRAKE_ActLO: now also J1.2 (Pin_2)
- net BTN_ActLO: now also J1.18 (Pin_18)
- net CEL_ActLO: now also J1.10 (Pin_10)
- net COOLANT_ActHI: now also J1.20 (Pin_20)
- net DOOR_ActLO: now also J1.22 (Pin_22)
- net FUEL_LVL_Rsense: now also J1.13 (Pin_13), R10.1, R11.1, R12.1, R13.1, R14.1, R15.1, R16.1, R17.1, R18.1, R19.1, R20.1, R21.1, R22.1, R7.1, R8.1, R9.1
- net GND: now also J1.3 (Pin_3), U17.22 (GND), U17.23 (GND), U17.24 (GND), U17.44 (GND), Q24.2 (S), Q25.2 (S), Q26.2 (S)
- net H_BEAM_ActHI: now also J1.17 (Pin_17)
- net IGNITION_ActHI: now also J1.5 (Pin_5)
- net L_BEAM_ActHI: now also J1.12 (Pin_12)
- net L_TURN_ActHI: now also J1.21 (Pin_21)
- net OIL_ALRM_ActLO: now also J1.6 (Pin_6)
- net PARK_ActLO: now also J1.4 (Pin_4)
- net RPM_HALL: now also J1.7 (Pin_7), Q25.3 (D), R95.1
- net R_TURN_ActLO: now also J1.23 (Pin_23)
- net SCL: now also U17.6 (GPIO6/ADC1_CH5), R2.1; no longer U17.7 (GPIO7/ADC1_CH6)
- net SDA: now also U17.5 (GPIO5/ADC1_CH4), R1.1; no longer U17.6 (GPIO6/ADC1_CH5)
- net SPEED_HALL: now also J1.9 (Pin_9), Q26.3 (D), R97.1
- net WATER_T_PWM: now also J1.11 (Pin_11), Q24.3 (D), R93.1
- net Switchable Resistor3/Res_ON: now reaches U18.10 (P06)
- net Switchable Resistor3/Res_ON: now reaches U18.11 (P07)
- net Switchable Resistor4/Res_ON: now reaches U18.13 (P10)
- net Switchable Resistor4/Res_ON: now reaches U18.14 (P11)
- net Switchable Resistor4/Res_ON: now reaches U18.15 (P12)
- net Switchable Resistor4/Res_ON: now reaches U18.16 (P13)
- net Switchable Resistor4/Res_ON: now reaches U18.17 (P14)
- net Switchable Resistor4/Res_ON: now reaches U18.18 (P15)
- net Switchable Resistor4/Res_ON: now reaches U18.19 (P16)
- net Switchable Resistor4/Res_ON: now reaches U18.20 (P17)
- net Switchable Resistor/Res_ON: now reaches U18.4 (P00)
- net Switchable Resistor1/Res_ON: now reaches U18.5 (P01)
- net Switchable Resistor2/Res_ON: now reaches U18.6 (P02)
- net Switchable Resistor2/Res_ON: now reaches U18.7 (P03)
- net Switchable Resistor3/Res_ON: now reaches U18.8 (P04)
- net Switchable Resistor3/Res_ON: now reaches U18.9 (P05)
- net ledc_chan_0: now reaches U17.16 (GPIO10/ADC1_CH9)
- net ledc_chan_0: now also R92.1
- net ledc_chan_1: now reaches U17.17 (GPIO11/ADC2_CH0)
- net ledc_chan_1: now also R94.1
- net ledc_chan_2: now reaches U17.18 (GPIO12/ADC2_CH1)
- net ledc_chan_2: now also R96.1
- net ledc_chan_3: now reaches U17.19 (GPIO13/ADC2_CH2)
- net ledc_chan_4: now reaches U17.20 (GPIO14/ADC2_CH3)
- net at U17.41 (GPIO1/ADC1_CH0): now also SW2.1 (A)
- new net: Q25.1 (G), R94.2
- new net: Q24.1 (G), R92.2
- new net: Q26.1 (G), R96.2
- new net: R98.2, SW2.2 (B)
- new net Switchable Resistor/Res_GND: R7.2
- new net Switchable Resistor1/Res_GND: R8.2
- new net Switchable Resistor2/Res_GND: R10.2
- new net Switchable Resistor2/Res_GND: R9.2
- new net Switchable Resistor3/Res_GND: R14.2
- new net Switchable Resistor3/Res_GND: R12.2
- new net Switchable Resistor3/Res_GND: R11.2
- new net Switchable Resistor3/Res_GND: R13.2
- new net Switchable Resistor4/Res_GND: R18.2
- new net Switchable Resistor4/Res_GND: R16.2
- new net Switchable Resistor4/Res_GND: R21.2
- new net Switchable Resistor4/Res_GND: R17.2
- new net Switchable Resistor4/Res_GND: R22.2
- new net Switchable Resistor4/Res_GND: R19.2
- new net Switchable Resistor4/Res_GND: R15.2
- new net Switchable Resistor4/Res_GND: R20.2
- no-connect marks 3 -> 4
Other:
- removed sheet Opto_ActHi4
- removed sheet Opto_ActHi5
- removed sheet Opto_ActHi6
- removed sheet Opto_ActHi7
- removed sheet Opto_ActLo1
- removed sheet Opto_ActLo2
- removed sheet Opto_ActLo3
- removed sheet Opto_ActLo4
- removed sheet Opto_ActLo6
- removed sheet Opto_ActLo7
- removed sheet Opto_ActLo8
- removed sheet Opto_ActLo9
- added sheet Opto_ActHi11 (Opto_ActHi.kicad_sch)
- added sheet Opto_ActHi12 (Opto_ActHi.kicad_sch)
- added sheet Opto_ActHi13 (Opto_ActHi.kicad_sch)
- added sheet Opto_ActHi14 (Opto_ActHi.kicad_sch)
- added sheet Opto_ActLo11 (Opto_ActLo.kicad_sch)
- added sheet Opto_ActLo12 (Opto_ActLo.kicad_sch)
- added sheet Opto_ActLo13 (Opto_ActLo.kicad_sch)
- added sheet Opto_ActLo14 (Opto_ActLo.kicad_sch)
- added sheet Opto_ActLo15 (Opto_ActLo.kicad_sch)
- added sheet Opto_ActLo16 (Opto_ActLo.kicad_sch)
- added sheet Opto_ActLo17 (Opto_ActLo.kicad_sch)
- added sheet Opto_ActLo18 (Opto_ActLo.kicad_sch)
- added sheet Switchable Resistor (Switchable_Res.kicad_sch)
- added sheet Switchable Resistor1 (Switchable_Res.kicad_sch)
- added sheet Switchable Resistor2 (Switchable_Res.kicad_sch)
- added sheet Switchable Resistor3 (Switchable_Res.kicad_sch)
- added sheet Switchable Resistor4 (Switchable_Res.kicad_sch)
- sheet Opto_ActHi10 ports: added HL_output, LL_input; removed HL_Input, ~{LL_output}
- sheet Opto_ActHi8 ports: added HL_output, LL_input; removed HL_Input, ~{LL_output}
- sheet Opto_ActHi9 ports: added HL_output, LL_input; removed HL_Input, ~{LL_output}
- sheet Opto_ActLo10 ports: added LL_input, ~{HL_output}; removed ~{HL_Input}, ~{LL_Output}
- note added: "Outputs have pull up enabled by default"
- moved on the sheet: C22, J1, J4, U17, U18

Commit message: ERC corrections, idiot lights
- VXDash : added idiot lights (also to emulator board)
- VXDash : corrected some ERC violations
Parts:
- added D1: ledc_chan_0_ON, LED_SMD:LED_0603_1608Metric_Pad1.05x0.95mm_HandSolder, symbol VXDash_diodes:LED_Small
- added D2: ledc_chan_1_ON, LED_SMD:LED_0603_1608Metric_Pad1.05x0.95mm_HandSolder, symbol VXDash_diodes:LED_Small
- added D3: ledc_chan_2_ON, LED_SMD:LED_0603_1608Metric_Pad1.05x0.95mm_HandSolder, symbol VXDash_diodes:LED_Small
- added D38: BATT_ON, LED_SMD:LED_0603_1608Metric_Pad1.05x0.95mm_HandSolder, symbol VXDash_diodes:LED_Small
- added D39: PROT12V ON, LED_SMD:LED_0603_1608Metric_Pad1.05x0.95mm_HandSolder, symbol VXDash_diodes:LED_Small
- added D40: 3V3_ON, LED_SMD:LED_0603_1608Metric_Pad1.05x0.95mm_HandSolder, symbol VXDash_diodes:LED_Small
- added D41: 5V_ON, LED_SMD:LED_0603_1608Metric_Pad1.05x0.95mm_HandSolder, symbol VXDash_diodes:LED_Small
- added D42: IGN_ON, LED_SMD:LED_0603_1608Metric_Pad1.05x0.95mm_HandSolder, symbol VXDash_diodes:LED_Small
- added R100, R101, R136, R138, R99: 270, Resistor_SMD:R_0603_1608Metric_Pad0.98x0.95mm_HandSolder, symbol VXDash_passives:Res
- added R134, R135: 3k, Resistor_SMD:R_0603_1608Metric_Pad0.98x0.95mm_HandSolder, symbol VXDash_passives:Res
- added R137: 620, Resistor_SMD:R_0603_1608Metric_Pad0.98x0.95mm_HandSolder, symbol VXDash_passives:Res
- added R139, R140, R141, R142, R143, R144, R145, R146: 0R, Resistor_SMD:R_0805_2012Metric_Pad1.20x1.40mm_HandSolder, symbol VXDash_passives:Res
- added TP1: TP12VP, TestPoint:TestPoint_Pad_D2.0mm, symbol Connector:TestPoint_Small
- added TP2: TP5V, TestPoint:TestPoint_Pad_D2.0mm, symbol Connector:TestPoint_Small
- added TP3: TP3V3, TestPoint:TestPoint_Pad_D2.0mm, symbol Connector:TestPoint_Small
- added TP4: TP_FUEL, TestPoint:TestPoint_Pad_D2.0mm, symbol Connector:TestPoint_Small
- added TP5: TPSDA, TestPoint:TestPoint_Pad_D2.0mm, symbol Connector:TestPoint_Small
- added TP6: TPSCL, TestPoint:TestPoint_Pad_D2.0mm, symbol Connector:TestPoint_Small
- added TP7: TP_LEDC3, TestPoint:TestPoint_Pad_D2.0mm, symbol Connector:TestPoint_Small
- added TP8: TP_LEDC4, TestPoint:TestPoint_Pad_D2.0mm, symbol Connector:TestPoint_Small
- J2: value Conn_02x02_Odd_Even -> Board supply
Connections:
- net Switchable Resistor2/Res_GND is gone; now on net Switchable Resistor2/Res_GND: R9.2
- net Switchable Resistor2/Res_ON is gone; now on net Switchable Resistor2/Res_ON: U18.7 (P03)
- net Switchable Resistor3/Res_GND is gone; now on net Switchable Resistor3/Res_GND: R13.2
- net Switchable Resistor3/Res_ON is gone; now on net Switchable Resistor3/Res_ON: U18.9 (P05)
- net Switchable Resistor4/Res_GND is gone; now on net Switchable Resistor4/Res_GND: R20.2
- net Switchable Resistor4/Res_ON is gone; now on net Switchable Resistor4/Res_ON: U18.20 (P17)
- net +3V3: now also R136.1, R139.2, R140.2, R141.2, R145.1; no longer U17.1 (3V3), U17.2 (3V3), U18.24 (VCC), U5.24 (VCC)
- net +5V_1: now also R137.1, R146.1
- net BATT12V+: now also J2.1 (Pin_1), J2.3 (Pin_3), R134.1, R142.2, R143.2, R144.2; no longer R93.2, R95.2, R97.2
- net FUEL_LVL_Rsense: now also TP4.1
- net GND: now also J2.2 (Pin_2), J2.4 (Pin_4), D1.1 (K), D2.1 (K), D3.1 (K), D38.1 (K), D39.1 (K), D40.1 (K), D41.1 (K), D42.1 (K)
- net Protected_12V: now also R135.1, TP1.1
- net SCL: now also TP6.1
- net SDA: now also TP5.1
- net Switchable Resistor2/Res_GND: no longer R10.2
- net Switchable Resistor2/Res_ON: no longer U18.6 (P02)
- net Switchable Resistor3/Res_GND: no longer R14.2
- net Switchable Resistor3/Res_ON: no longer U18.10 (P06)
- net Switchable Resistor4/Res_GND: no longer R18.2
- net Switchable Resistor4/Res_ON: no longer U18.13 (P10)
- net ledc_chan_0: now also R99.1
- net ledc_chan_1: now also R100.1
- net ledc_chan_2: now also R101.1
- net ledc_chan_3: now also TP7.1
- net ledc_chan_4: now also TP8.1
- net 5v_enable: now reaches U17.12 (GPIO8/ADC1_CH7)
- net ign_EN: now reaches SW2.1 (A), U17.41 (GPIO1/ADC1_CH0)
- net ign_EN: now also R138.1
- new net: D42.2 (A), R138.2
- new net: R144.1, R97.2
- new net: D2.2 (A), R100.2
- new net: R141.1, U18.24 (VCC)
- new net: D3.2 (A), R101.2
- new net: D40.2 (A), R136.2
- new net: R142.1, R93.2
- new net: D41.2 (A), R137.2
- new net: D38.2 (A), R134.2
- new net: R140.1, U17.1 (3V3), U17.2 (3V3)
- new net: D1.2 (A), R99.2
- new net: R143.1, R95.2
- new net: D39.2 (A), R135.2
- new net: R139.1, U5.24 (VCC)
- new net 3V3_SMPS/3V3_OUT: R145.2, TP3.1
- new net 5V_SMPS_1/5V_OUT: R146.2, TP2.1
- new net Switchable Resistor2/Res_GND: R10.2
- new net Switchable Resistor2/Res_ON: U18.6 (P02)
- new net Switchable Resistor3/Res_GND: R14.2
- new net Switchable Resistor3/Res_ON: U18.10 (P06)
- new net Switchable Resistor4/Res_GND: R18.2
- new net Switchable Resistor4/Res_ON: U18.13 (P10)
Other:
- sheet 3V3_SMPS ports: added 3V3_OUT, V_IN; removed 12V_in, 3V3_out
- sheet 5V_SMPS_1 ports: added 5V_EN, 5V_OUT, V_IN; removed 12V_in, 5V_en, 5V_out
- moved on the sheet: R1, R2, R98, SW2

Commit message: Emulator : ERC and footprints
Also moving some 0402 capacitors to 0603...
Parts:
- added J2, J3, J5: Level_Select, Connector_PinHeader_2.54mm:PinHeader_1x03_P2.54mm_Vertical, symbol Connector_Generic:Conn_01x03
- added R134: 0R, Resistor_SMD:R_0805_2012Metric_Pad1.20x1.40mm_HandSolder, symbol VXDash_passives:Res
- C1: renamed from C21; footprint (none) -> Capacitor_SMD:C_0603_1608Metric_Pad1.08x0.95mm_HandSolder
- C2: renamed from C22; footprint (none) -> Capacitor_SMD:C_0603_1608Metric_Pad1.08x0.95mm_HandSolder
- J4: renamed from J2; footprint (none) -> Connector_PinHeader_2.54mm:PinHeader_2x02_P2.54mm_Vertical
- J6: renamed from J4; footprint (none) -> Connector_PinHeader_2.54mm:PinHeader_1x02_P2.54mm_Vertical
- SW1: renamed from SW2; footprint (none) -> Button_Switch_THT:SW_DIP_SPSTx01_Slide_9.78x4.72mm_W7.62mm_P2.54mm
- U1: renamed from U5; MFT (none) -> Texas Instrument; MFT_PN (none) -> TCA9555PWR
- U3: renamed from U18; MFT (none) -> Texas Instrument; MFT_PN (none) -> TCA9555PWR
- renumbered D3 to D1, D38 to D3, D1 to D4, D41 to D5, D40 to D6, D42 to D7, D39 to D8, Q26 to Q1, Q25 to Q2, Q24 to Q3, R96 to R1, R139 to R10, R92 to R11, R99 to R12, R142 to R13, R93 to R14, R137 to R15, R136 to R16, R140 to R17, R138 to R18, R98 to R19, R101 to R2, R135 to R20, R7 to R21, R8 to R22, R9 to R23, R10 to R24, R11 to R25, R12 to R26, R13 to R27, R14 to R28, R15 to R29, R144 to R3, R16 to R30, R17 to R31, R18 to R32, R19 to R33, R20 to R34, R21 to R35, R22 to R36, R146 to R37, R145 to R38, R141 to R39, R97 to R4, R1 to R40, R2 to R41, R94 to R5, R100 to R6, R143 to R7, R95 to R8, R134 to R9, TP7 to TP1, TP8 to TP2, TP4 to TP3, TP1 to TP4, TP2 to TP5, TP3 to TP6, TP5 to TP7, TP6 to TP8, U17 to U2
Connections:
- net Switchable Resistor 3/Res_ON is gone; now on net Switchable Resistor 3/Res_ON: U3.7 (P03)
- net Switchable Resistor 5/Res_GND is gone; now on net Switchable Resistor 5/Res_GND: R26.2
- net Switchable Resistor 5/Res_ON is gone; now on net Switchable Resistor 5/Res_ON: U3.9 (P05)
- net Switchable Resistor 14/Res_GND is gone; now on net Switchable Resistor 14/Res_GND: R33.2
- net Switchable Resistor 14/Res_ON is gone; now on net Switchable Resistor 14/Res_ON: U3.17 (P14)
- net +5V_1: now also J2.3 (Pin_3), J3.3 (Pin_3), J5.3 (Pin_3), R134.1
- net BATT12V+: now also J2.1 (Pin_1), J3.1 (Pin_1), J5.1 (Pin_1); no longer R13.2, R3.2, R7.2
- net Switchable Resistor 3/Res_ON: no longer U3.6 (P02)
- net Switchable Resistor 5/Res_GND: no longer R28.2
- net Switchable Resistor 5/Res_ON: no longer U3.10 (P06)
- net Switchable Resistor 14/Res_GND: no longer R32.2
- net Switchable Resistor 14/Res_ON: no longer U3.13 (P10)
- net at U2.21 (5V): now also R134.2
- net Switchable Resistor 3/Res_GND renamed Switchable Resistor 2/Res_GND
- net Switchable Resistor 5/Res_GND renamed Switchable Resistor 4/Res_GND
- net Switchable Resistor 5/Res_GND renamed Switchable Resistor 6/Res_GND
- net Switchable Resistor 5/Res_ON renamed Switchable Resistor 7/Res_ON
- net Switchable Resistor 5/Res_ON renamed Switchable Resistor 4/Res_ON
- net Switchable Resistor 14/Res_GND renamed Switchable Resistor11/Res_GND
- net Switchable Resistor 14/Res_GND renamed Switchable Resistor 16/Res_GND
- net Switchable Resistor 14/Res_GND renamed Switchable Resistor 12/Res_GND
- net Switchable Resistor 14/Res_GND renamed Switchable Resistor 17/Res_GND
- net Switchable Resistor 14/Res_GND renamed Switchable Resistor 10/Res_GND
- net Switchable Resistor 14/Res_GND renamed Switchable Resistor 15/Res_GND
- net Switchable Resistor 14/Res_ON renamed Switchable Resistor11/Res_ON
- net Switchable Resistor 14/Res_ON renamed Switchable Resistor 12/Res_ON
- net Switchable Resistor 14/Res_ON renamed Switchable Resistor 13/Res_ON
- net Switchable Resistor 14/Res_ON renamed Switchable Resistor 15/Res_ON
- net Switchable Resistor 14/Res_ON renamed Switchable Resistor 16/Res_ON
- net Switchable Resistor 14/Res_ON renamed Switchable Resistor 17/Res_ON
- new net: J5.2 (Pin_2), R13.2
- new net: J3.2 (Pin_2), R7.2
- new net: J2.2 (Pin_2), R3.2
- new net Switchable Resistor 10/Res_ON: U3.13 (P10)
- new net Switchable Resistor 13/Res_GND: R32.2
- new net Switchable Resistor 2/Res_ON: U3.6 (P02)
- new net Switchable Resistor 6/Res_ON: U3.10 (P06)
- new net Switchable Resistor 7/Res_GND: R28.2
- no-connect marks 4 -> 32
Other:
- sheet Switchable Resistor renamed Switchable Resistor 0
- sheet Switchable Resistor1 renamed Switchable Resistor 1
- sheet Switchable Resistor2 renamed Switchable Resistor 3
- sheet Switchable Resistor3 renamed Switchable Resistor 5
- sheet Switchable Resistor4 renamed Switchable Resistor 14
- added sheet Switchable Resistor 10 (Switchable_Res.kicad_sch)
- added sheet Switchable Resistor 12 (Switchable_Res.kicad_sch)
- added sheet Switchable Resistor 13 (Switchable_Res.kicad_sch)
- added sheet Switchable Resistor 15 (Switchable_Res.kicad_sch)
- added sheet Switchable Resistor 16 (Switchable_Res.kicad_sch)
- added sheet Switchable Resistor 17 (Switchable_Res.kicad_sch)
- added sheet Switchable Resistor 2 (Switchable_Res.kicad_sch)
- added sheet Switchable Resistor 4 (Switchable_Res.kicad_sch)
- added sheet Switchable Resistor 6 (Switchable_Res.kicad_sch)
- added sheet Switchable Resistor 7 (Switchable_Res.kicad_sch)
- added sheet Switchable Resistor11 (Switchable_Res.kicad_sch)
- note added: "Address is 0x21 Max 160mA"
- note added: "Max consumption 500mA"
- note added: "Outputs have pull up enabled by default Expected consumption below 30mA"
- note removed: "Address is 0x21"
- note removed: "Outputs have pull up enabled by default"
- moved on the sheet: R17

Commit message: Emulator : resistance banks layout
Parts:
- added J7: R bypass, Connector_PinSocket_2.54mm:PinSocket_1x02_P2.54mm_Vertical, symbol Connector_Generic:Conn_01x02
- R21: value 0 -> 270
- R22: value 10 -> 270
- R23: value 20 -> 270
- R24: value 30 -> 270
- R25: value 51 -> 270
- R26: value 91 -> 270
- R27: value 130 -> 270
- R28: value 180 -> 270
- R29: value 270 -> 2k
- R30: value 470 -> 2k
- R31: value 750 -> 2k
- R32: value 1k1 -> 2k
- R33: value 1k6 -> 2k
- R35: value 2k4 -> 2k
- R36: value 3k -> 2k
Connections:
- net FUEL_LVL_Rsense: now also J7.1 (Pin_1)
- net GND: now also J7.2 (Pin_2)

Commit message: Emulator board : layout update
- Moved to Open Drain style Mosfets instead of Optoisolators
- Added manual push button for BUTTON
- Did groups in the PCB layout
Parts:
- added SW2: Button Manual, Button_Switch_THT:SW_PUSH_1P1T_6x3.5mm_H5.0_APEM_MJTP1250, symbol Switch:SW_Push
Connections:
- net GND: now also SW2.1
- net button: now also SW2.2
Other:
- removed sheet Opto_ActHi10
- removed sheet Opto_ActHi11
- removed sheet Opto_ActHi12
- removed sheet Opto_ActHi13
- removed sheet Opto_ActHi14
- removed sheet Opto_ActHi8
- removed sheet Opto_ActHi9
- removed sheet Opto_ActLo10
- removed sheet Opto_ActLo11
- removed sheet Opto_ActLo12
- removed sheet Opto_ActLo13
- removed sheet Opto_ActLo14
- removed sheet Opto_ActLo15
- removed sheet Opto_ActLo16
- removed sheet Opto_ActLo17
- removed sheet Opto_ActLo18
- added sheet NMOSFET Shifter (FET_Active_Hi.kicad_sch)
- added sheet NMOSFET Shifter1 (FET_Active_Hi.kicad_sch)
- added sheet NMOSFET Shifter10 (FET_Active_Hi.kicad_sch)
- added sheet NMOSFET Shifter11 (FET_Active_Hi.kicad_sch)
- added sheet NMOSFET Shifter12 (FET_Active_Hi.kicad_sch)
- added sheet NMOSFET Shifter13 (FET_Active_Hi.kicad_sch)
- added sheet NMOSFET Shifter14 (FET_Active_Hi.kicad_sch)
- added sheet NMOSFET Shifter15 (FET_Active_Hi.kicad_sch)
- added sheet NMOSFET Shifter2 (FET_Active_Hi.kicad_sch)
- added sheet NMOSFET Shifter3 (FET_Active_Hi.kicad_sch)
- added sheet NMOSFET Shifter4 (FET_Active_Hi.kicad_sch)
- added sheet NMOSFET Shifter5 (FET_Active_Hi.kicad_sch)
- added sheet NMOSFET Shifter6 (FET_Active_Hi.kicad_sch)
- added sheet NMOSFET Shifter7 (FET_Active_Hi.kicad_sch)
- added sheet NMOSFET Shifter8 (FET_Active_Hi.kicad_sch)
- added sheet NMOSFET Shifter9 (FET_Active_Hi.kicad_sch)

Commit message: Emulator - block layout complete
Connections:
- net airbag: now also U1.7 (P03); no longer U1.10 (P06)
- net alarm: now also U1.10 (P06); no longer U1.19 (P16)
- net alternator: now also U1.18 (P15); no longer U1.6 (P02)
- net backlight: now also U1.9 (P05); no longer U1.20 (P17)
- net brakes: now also U1.4 (P00); no longer U1.7 (P03)
- net button: now also U1.11 (P07); no longer U1.18 (P15)
- net cel: now also U1.8 (P04); no longer U1.11 (P07)
- net coolant: now also U1.13 (P10); no longer U1.17 (P14)
- net door: now also U1.14 (P11); no longer U1.16 (P13)
- net full_beams: now also U1.19 (P16); no longer U1.5 (P01)
- net ignition: now also U1.20 (P17); no longer U1.4 (P00)
- net left_turn: now also U1.17 (P14); no longer U1.14 (P11)
- net oil: now also U1.6 (P02); no longer U1.9 (P05)
- net parking: now also U1.5 (P01); no longer U1.8 (P04)
- net right_turn: now also U1.16 (P13); no longer U1.13 (P10)

Commit message: Emulator board basic routing done
Connections:
- net ledc_chan_0: now also U2.18 (GPIO12/ADC2_CH1); no longer U2.16 (GPIO10/ADC1_CH9)
- net ledc_chan_2: now also U2.16 (GPIO10/ADC1_CH9); no longer U2.18 (GPIO12/ADC2_CH1)

Commit message: Emulator board : DRC pass, review
Parts:
- J1: now not fitted
Changed lines of the file:
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@@
 		(in_bom yes)
 		(on_board yes)
-		(dnp no)
+		(dnp yes)
 		(fields_autoplaced yes)
 		(property "Reference" "J1"
