File: KiCad PCB Files/VXDash_Emulator/3V3_SMPS.kicad_sch (KiCad schematic)
At the start: 13 parts, among them IC4 AP62200

Commit message: More changes (Primarily Remote ECU)
- Emulator board project to a functional skeleton
- Connectors board with ignition routing on CAN pin 4 to have switched signal available in the harness.
- Remote ECU : added 12V reduced protection circuit (to be reviewed)
- Remote ECU : Removed integrated CAN termination (should be on harness)
- Remote ECU : added CAN passthrough
- Remote ECU : added MCPWM channels
- Remote ECU : Added some opto inputs
- Remote ECU : Added internal USB C (overkill ?)
Connections:
- net V_IN renamed 12V_in
Other:
- company: (none) -> Alex Miller & Martin Roger
- title: VXDash RemoteECU -> Main architecture
Changed lines of the file:
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@@
 	(paper "A4")
 	(title_block
-		(title "VXDash RemoteECU")
-		(date "2025-08-08")
-		(rev "Proto A")
+		(title "Main architecture")
+		(date "2025-08-10")
+		(rev "0.0")
+		(company "Alex Miller & Martin Roger")
 		(comment 1 "https://github.com/martinroger/VXDash")
 		(comment 2 "https://cadlab.io/projects/vxdash")
@@
 		)
 	)
-	(hierarchical_label "V_IN"
+	(hierarchical_label "12V_in"
 		(shape input)
 		(at 76.2 55.88 180)
@@
 		(instances
 			(project ""
-				(path "/f2858fc4-50de-4ff0-a01c-5b985ee14aef/dc9f18a6-856d-4175-9fbd-d6bbcc89eb0a"
+				(path "/f2858fc4-50de-4ff0-a01c-5b985ee14aef/21f2fd69-aa93-4550-8877-dde4aa3e5582"
 					(reference "#PWR033")
 					(unit 1)
@@
 		(instances
 			(project ""
-				(path "/f2858fc4-50de-4ff0-a01c-5b985ee14aef/dc9f18a6-856d-4175-9fbd-d6bbcc89eb0a"
+				(path "/f2858fc4-50de-4ff0-a01c-5b985ee14aef/21f2fd69-aa93-4550-8877-dde4aa3e5582"
 					(reference "IC4")
 					(unit 1)
@@
 		(instances
 			(project ""
-				(path "/f2858fc4-50de-4ff0-a01c-5b985ee14aef/dc9f18a6-856d-4175-9fbd-d6bbcc89eb0a"
+				(path "/f2858fc4-50de-4ff0-a01c-5b985ee14aef/21f2fd69-aa93-4550-8877-dde4aa3e5582"
 					(reference "C17")
 					(unit 1)
@@
 		(instances
 			(project "VXDash"
-				(path "/f2858fc4-50de-4ff0-a01c-5b985ee14aef/dc9f18a6-856d-4175-9fbd-d6bbcc89eb0a"
+				(path "/f2858fc4-50de-4ff0-a01c-5b985ee14aef/21f2fd69-aa93-4550-8877-dde4aa3e5582"
 					(reference "R40")
 					(unit 1)
@@
 		(instances
 			(project "VXDash"
-				(path "/f2858fc4-50de-4ff0-a01c-5b985ee14aef/dc9f18a6-856d-4175-9fbd-d6bbcc89eb0a"
+				(path "/f2858fc4-50de-4ff0-a01c-5b985ee14aef/21f2fd69-aa93-4550-8877-dde4aa3e5582"
 					(reference "C14")
 					(unit 1)
@@
 		(instances
 			(project ""
-				(path "/f2858fc4-50de-4ff0-a01c-5b985ee14aef/dc9f18a6-856d-4175-9fbd-d6bbcc89eb0a"
+				(path "/f2858fc4-50de-4ff0-a01c-5b985ee14aef/21f2fd69-aa93-4550-8877-dde4aa3e5582"
 					(reference "R39")
 					(unit 1)
@@
 		(instances
 			(project "VXDash"
-				(path "/f2858fc4-50de-4ff0-a01c-5b985ee14aef/dc9f18a6-856d-4175-9fbd-d6bbcc89eb0a"
+				(path "/f2858fc4-50de-4ff0-a01c-5b985ee14aef/21f2fd69-aa93-4550-8877-dde4aa3e5582"
 					(reference "R37")
 					(unit 1)
@@
 		(instances
 			(project "VXDash"
-				(path "/f2858fc4-50de-4ff0-a01c-5b985ee14aef/dc9f18a6-856d-4175-9fbd-d6bbcc89eb0a"
+				(path "/f2858fc4-50de-4ff0-a01c-5b985ee14aef/21f2fd69-aa93-4550-8877-dde4aa3e5582"
 					(reference "C20")
 					(unit 1)
@@
 		(instances
 			(project ""
-				(path "/f2858fc4-50de-4ff0-a01c-5b985ee14aef/dc9f18a6-856d-4175-9fbd-d6bbcc89eb0a"
+				(path "/f2858fc4-50de-4ff0-a01c-5b985ee14aef/21f2fd69-aa93-4550-8877-dde4aa3e5582"
 					(reference "C19")
 					(unit 1)
@@
 		(instances
 			(project ""
-				(path "/f2858fc4-50de-4ff0-a01c-5b985ee14aef/dc9f18a6-856d-4175-9fbd-d6bbcc89eb0a"
+				(path "/f2858fc4-50de-4ff0-a01c-5b985ee14aef/21f2fd69-aa93-4550-8877-dde4aa3e5582"
 					(reference "L2")
 					(unit 1)
@@
 		(instances
 			(project "VXDash"
-				(path "/f2858fc4-50de-4ff0-a01c-5b985ee14aef/dc9f18a6-856d-4175-9fbd-d6bbcc89eb0a"
+				(path "/f2858fc4-50de-4ff0-a01c-5b985ee14aef/21f2fd69-aa93-4550-8877-dde4aa3e5582"
 					(reference "R38")
 					(unit 1)
@@
 		(instances
 			(project "VXDash"
-				(path "/f2858fc4-50de-4ff0-a01c-5b985ee14aef/dc9f18a6-856d-4175-9fbd-d6bbcc89eb0a"
+				(path "/f2858fc4-50de-4ff0-a01c-5b985ee14aef/21f2fd69-aa93-4550-8877-dde4aa3e5582"
 					(reference "C15")
 					(unit 1)
@@
 		(instances
 			(project "VXDash"
-				(path "/f2858fc4-50de-4ff0-a01c-5b985ee14aef/dc9f18a6-856d-4175-9fbd-d6bbcc89eb0a"
+				(path "/f2858fc4-50de-4ff0-a01c-5b985ee14aef/21f2fd69-aa93-4550-8877-dde4aa3e5582"
 					(reference "C16")
 					(unit 1)
@@
 		(instances
 			(project "VXDash"
-				(path "/f2858fc4-50de-4ff0-a01c-5b985ee14aef/dc9f18a6-856d-4175-9fbd-d6bbcc89eb0a"
+				(path "/f2858fc4-50de-4ff0-a01c-5b985ee14aef/21f2fd69-aa93-4550-8877-dde4aa3e5582"
 					(reference "C18")
 					(unit 1)

Commit message: ERC corrections, idiot lights
- VXDash : added idiot lights (also to emulator board)
- VXDash : corrected some ERC violations
Parts:
- C21: renamed from C15; footprint (none) -> Capacitor_SMD:C_0603_1608Metric_Pad1.08x0.95mm_HandSolder
- C22: renamed from C16; footprint (none) -> Capacitor_SMD:C_0603_1608Metric_Pad1.08x0.95mm_HandSolder
- C24: renamed from C18; footprint (none) -> Capacitor_SMD:C_0603_1608Metric_Pad1.08x0.95mm_HandSolder
- renumbered C14 to C20, C17 to C23, C19 to C25, C20 to C26, IC4 to IC3, R37 to R41, R38 to R42, R39 to R43, R40 to R44
Connections:
- net 3V3_SW: now reaches C22.1, IC3.2 (SW), L2.1
- net 3V3_FB: now reaches C23.2, IC3.4 (FB), R43.2, R44.1
- net 3V3_EN: now reaches IC3.5 (EN), R41.2, R42.1
- net 12V_in renamed V_IN
- net 3V3_out renamed 3V3_OUT
Changed lines of the file:
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@@
 		(title "Main architecture")
 		(date "2025-08-10")
-		(rev "0.0")
+		(rev "1.4")
 		(company "Alex Miller & Martin Roger")
 		(comment 1 "https://github.com/martinroger/VXDash")
@@
 		)
 	)
-	(hierarchical_label "3V3_out"
+	(label "3V3_EN"
+		(at 102.87 71.12 0)
+		(effects
+			(font
+				(size 1.27 1.27)
+			)
+			(justify left bottom)
+		)
+	)
+	(label "3V3_SW"
+		(at 140.97 60.96 0)
+		(effects
+			(font
+				(size 1.27 1.27)
+			)
+			(justify left bottom)
+		)
+	)
+	(label "3V3_FB"
+		(at 144.78 71.12 0)
+		(effects
+			(font
+				(size 1.27 1.27)
+			)
+			(justify left bottom)
+		)
+	)
+	(hierarchical_label "3V3_OUT"
 		(shape output)
 		(at 207.01 60.96 0)
@@
 		)
 	)
-	(hierarchical_label "12V_in"
+	(hierarchical_label "V_IN"
 		(shape input)
 		(at 76.2 55.88 180)
@@
 		(dnp no)
 		(fields_autoplaced yes)
-		(property "Reference" "#PWR033"
+		(property "Reference" "#PWR044"
 			(at 124.46 93.98 0)
 			(effects
@@
 			(project ""
 				(path "/f2858fc4-50de-4ff0-a01c-5b985ee14aef/21f2fd69-aa93-4550-8877-dde4aa3e5582"
-					(reference "#PWR033")
+					(reference "#PWR044")
 					(unit 1)
 				)
@@
 		(dnp no)
 		(fields_autoplaced yes)
-		(property "Reference" "IC4"
+		(property "Reference" "IC3"
 			(at 124.46 48.26 0)
 			(effects
@@
 		(property "MFT_PN" "AP62200WU-7"
 			(at 124.46 38.1 0)
+			(effects
+				(font
+					(size 1.27 1.27)
+				)
+				(hide yes)
+			)
+		)
+		(property "Tolerance" ""
+			(at 124.46 53.34 0)
 			(effects
 				(font
@@
 			(project ""
 				(path "/f2858fc4-50de-4ff0-a01c-5b985ee14aef/21f2fd69-aa93-4550-8877-dde4aa3e5582"
-					(reference "IC4")
+					(reference "IC3")
 					(unit 1)
 				)
@@
 		(dnp yes)
 		(fields_autoplaced yes)
-		(property "Reference" "C17"
+		(property "Reference" "C23"
 			(at 172.72 63.4999 0)
 			(effects
@@
 		)
 		(property "MFT_PN" ""
+			(at 168.91 66.04 0)
+			(effects
+				(font
+					(size 1.27 1.27)
+				)
+				(hide yes)
+			)
+		)
+		(property "Tolerance" ""
 			(at 168.91 66.04 0)
 			(effects
@@
 			(project ""
 				(path "/f2858fc4-50de-4ff0-a01c-5b985ee14aef/21f2fd69-aa93-4550-8877-dde4aa3e5582"
-					(reference "C17")
+					(reference "C23")
 					(unit 1)
 				)
@@
 		(dnp no)
 		(fields_autoplaced yes)
-		(property "Reference" "R40"
+		(property "Reference" "R44"
 			(at 162.56 76.1999 0)
 			(effects
@@
 		)
 		(property "MFT_PN" ""
+			(at 160.02 77.47 0)
+			(effects
+				(font
+					(size 1.27 1.27)
+				)
+				(hide yes)
+			)
+		)
+		(property "Tolerance" ""
 			(at 160.02 77.47 0)
 			(effects
@@
 			(project "VXDash"
 				(path "/f2858fc4-50de-4ff0-a01c-5b985ee14aef/21f2fd69-aa93-4550-8877-dde4aa3e5582"
-					(reference "R40")
+					(reference "R44")
 					(unit 1)
 				)
@@
 		(on_board yes)
 		(dnp no)
-		(property "Reference" "C14"
+		(property "Reference" "C20"
 			(at 97.79 48.26 0)
 			(effects
@@
 				)
 				(justify left)
+			)
+		)
+		(property "Tolerance" ""
+			(at 99.06 62.23 0)
+			(effects
+				(font
+					(size 1.27 1.27)
+				)
+				(hide yes)
 			)
 		)
@@
 			(project "VXDash"
 				(path "/f2858fc4-50de-4ff0-a01c-5b985ee14aef/21f2fd69-aa93-4550-8877-dde4aa3e5582"
-					(reference "C14")
+					(reference "C20")
 					(unit 1)
 				)
@@
 		(dnp no)
 		(fields_autoplaced yes)
-		(property "Reference" "R39"
+		(property "Reference" "R43"
 			(at 162.56 64.7699 0)
 			(effects
@@
 		)
 		(property "MFT_PN" ""
+			(at 160.02 66.04 0)
+			(effects
+				(font
+					(size 1.27 1.27)
+				)
+				(hide yes)
+			)
+		)
+		(property "Tolerance" ""
 			(at 160.02 66.04 0)
 			(effects
@@
 			(project ""
 				(path "/f2858fc4-50de-4ff0-a01c-5b985ee14aef/21f2fd69-aa93-4550-8877-dde4aa3e5582"
-					(reference "R39")
+					(reference "R43")
 					(unit 1)
 				)
@@
 		(dnp no)
 		(fields_autoplaced yes)
-		(property "Reference" "R37"
+		(property "Reference" "R41"
 			(at 91.44 62.2299 0)
 			(effects
@@
 		)
 		(property "MFT_PN" ""
+			(at 88.9 63.5 0)
+			(effects
+				(font
+					(size 1.27 1.27)
+				)
+				(hide yes)
+			)
+		)
+		(property "Tolerance" ""
 			(at 88.9 63.5 0)
 			(effects
@@
 			(project "VXDash"
 				(path "/f2858fc4-50de-4ff0-a01c-5b985ee14aef/21f2fd69-aa93-4550-8877-dde4aa3e5582"
-					(reference "R37")
+					(reference "R41")
 					(unit 1)
 				)
@@
 		(on_board yes)
 		(dnp no)
-		(property "Reference" "C20"
+		(property "Reference" "C26"
 			(at 199.39 53.34 0)
 			(effects
@@
 		)
 		(property "MFT_PN" ""
+			(at 200.66 66.04 0)
+			(effects
+				(font
+					(size 1.27 1.27)
+				)
+				(hide yes)
+			)
+		)
+		(property "Tolerance" ""
 			(at 200.66 66.04 0)
 			(effects
@@
 			(project "VXDash"
 				(path "/f2858fc4-50de-4ff0-a01c-5b985ee14aef/21f2fd69-aa93-4550-8877-dde4aa3e5582"
-					(reference "C20")
+					(reference "C26")
 					(unit 1)
 				)
@@
 		(on_board yes)
 		(dnp no)
-		(property "Reference" "C19"
+		(property "Reference" "C25"
 			(at 191.77 53.34 0)
 			(effects
@@
 		)
 		(property "MFT_PN" ""
+			(at 193.04 66.04 0)
+			(effects
+				(font
+					(size 1.27 1.27)
+				)
+				(hide yes)
+			)
+		)
+		(property "Tolerance" ""
 			(at 193.04 66.04 0)
 			(effects
@@
 			(project ""
 				(path "/f2858fc4-50de-4ff0-a01c-5b985ee14aef/21f2fd69-aa93-4550-8877-dde4aa3e5582"
-					(reference "C19")
+					(reference "C25")
 					(unit 1)
 				)
@@
 			)
 		)
+		(property "Tolerance" ""
+			(at 153.67 60.96 0)
+			(effects
+				(font
+					(size 1.27 1.27)
+				)
+				(hide yes)
+			)
+		)
 		(pin "2"
 		)
@@
 		(dnp no)
 		(fields_autoplaced yes)
-		(property "Reference" "R38"
+		(property "Reference" "R42"
 			(at 91.44 74.9299 0)
 			(effects
@@
 		)
 		(property "MFT_PN" ""
+			(at 88.9 76.2 0)
+			(effects
+				(font
+					(size 1.27 1.27)
+				)
+				(hide yes)
+			)
+		)
+		(property "Tolerance" ""
 			(at 88.9 76.2 0)
 			(effects
@@
 			(project "VXDash"
 				(path "/f2858fc4-50de-4ff0-a01c-5b985ee14aef/21f2fd69-aa93-4550-8877-dde4aa3e5582"
-					(reference "R38")
+					(reference "R42")
 					(unit 1)
 				)
@@
 		(on_board yes)
 		(dnp no)
-		(property "Reference" "C15"
+		(property "Reference" "C21"
 			(at 105.41 48.26 0)
 			(effects
@@
 			)
 		)
-		(property "Footprint" ""
+		(property "Footprint" "Capacitor_SMD:C_0603_1608Metric_Pad1.08x0.95mm_HandSolder"
 			(at 107.6452 58.42 0)
 			(effects
@@
 				)
 				(justify left)
+			)
+		)
+		(property "Tolerance" ""
+			(at 106.68 62.23 0)
+			(effects
+				(font
+					(size 1.27 1.27)
+				)
+				(hide yes)
 			)
 		)
@@
 			(project "VXDash"
 				(path "/f2858fc4-50de-4ff0-a01c-5b985ee14aef/21f2fd69-aa93-4550-8877-dde4aa3e5582"
-					(reference "C15")
+					(reference "C21")
 					(unit 1)
 				)
@@
 		(dnp no)
 		(fields_autoplaced yes)
-		(property "Reference" "C16"
+		(property "Reference" "C22"
 			(at 140.97 45.72 90)
 			(effects
@@
 			)
 		)
-		(property "Footprint" ""
+		(property "Footprint" "Capacitor_SMD:C_0603_1608Metric_Pad1.08x0.95mm_HandSolder"
 			(at 137.16 54.9148 0)
 			(effects
@@
 					(size 1.27 1.27)
 				)
+			)
+		)
+		(property "Tolerance" ""
+			(at 140.97 55.88 90)
+			(effects
+				(font
+					(size 1.27 1.27)
+				)
+				(hide yes)
 			)
 		)
@@
 			(project "VXDash"
 				(path "/f2858fc4-50de-4ff0-a01c-5b985ee14aef/21f2fd69-aa93-4550-8877-dde4aa3e5582"
-					(reference "C16")
+					(reference "C22")
 					(unit 1)
 				)
@@
 		(on_board yes)
 		(dnp no)
-		(property "Reference" "C18"
+		(property "Reference" "C24"
 			(at 184.15 53.34 0)
 			(effects
@@
 			)
 		)
-		(property "Footprint" ""
+		(property "Footprint" "Capacitor_SMD:C_0603_1608Metric_Pad1.08x0.95mm_HandSolder"
 			(at 186.3852 62.23 0)
 			(effects
@@
 				)
 				(justify left)
+			)
+		)
+		(property "Tolerance" ""
+			(at 185.42 66.04 0)
+			(effects
+				(font
+					(size 1.27 1.27)
+				)
+				(hide yes)
 			)
 		)
@@
 			(project "VXDash"
 				(path "/f2858fc4-50de-4ff0-a01c-5b985ee14aef/21f2fd69-aa93-4550-8877-dde4aa3e5582"
-					(reference "C18")
+					(reference "C24")
 					(unit 1)
 				)

Commit message: Emulator : ERC and footprints
Also moving some 0402 capacitors to 0603...
Parts:
- C13: renamed from C23; footprint Capacitor_SMD:C_0402_1005Metric_Pad0.74x0.62mm_HandSolder -> Capacitor_SMD:C_0603_1608Metric_Pad1.08x0.95mm_HandSolder
- renumbered C20 to C10, C21 to C11, C22 to C12, C24 to C14, C25 to C15, C26 to C16, IC3 to IC2, R41 to R91, R42 to R92, R43 to R93, R44 to R94
Changed lines of the file:
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@@
 		(dnp no)
 		(fields_autoplaced yes)
-		(property "Reference" "#PWR044"
+		(property "Reference" "#PWR050"
 			(at 124.46 93.98 0)
 			(effects
@@
 			(project ""
 				(path "/f2858fc4-50de-4ff0-a01c-5b985ee14aef/21f2fd69-aa93-4550-8877-dde4aa3e5582"
-					(reference "#PWR044")
+					(reference "#PWR050")
 					(unit 1)
 				)
@@
 		(dnp no)
 		(fields_autoplaced yes)
-		(property "Reference" "IC3"
+		(property "Reference" "IC2"
 			(at 124.46 48.26 0)
 			(effects
@@
 			(project ""
 				(path "/f2858fc4-50de-4ff0-a01c-5b985ee14aef/21f2fd69-aa93-4550-8877-dde4aa3e5582"
-					(reference "IC3")
+					(reference "IC2")
 					(unit 1)
 				)
@@
 		(dnp yes)
 		(fields_autoplaced yes)
-		(property "Reference" "C23"
+		(property "Reference" "C13"
 			(at 172.72 63.4999 0)
 			(effects
@@
 			)
 		)
-		(property "Footprint" "Capacitor_SMD:C_0402_1005Metric_Pad0.74x0.62mm_HandSolder"
+		(property "Footprint" "Capacitor_SMD:C_0603_1608Metric_Pad1.08x0.95mm_HandSolder"
 			(at 169.8752 69.85 0)
 			(effects
@@
 			(project ""
 				(path "/f2858fc4-50de-4ff0-a01c-5b985ee14aef/21f2fd69-aa93-4550-8877-dde4aa3e5582"
-					(reference "C23")
+					(reference "C13")
 					(unit 1)
 				)
@@
 		(dnp no)
 		(fields_autoplaced yes)
-		(property "Reference" "R44"
+		(property "Reference" "R94"
 			(at 162.56 76.1999 0)
 			(effects
@@
 			(project "VXDash"
 				(path "/f2858fc4-50de-4ff0-a01c-5b985ee14aef/21f2fd69-aa93-4550-8877-dde4aa3e5582"
-					(reference "R44")
+					(reference "R94")
 					(unit 1)
 				)
@@
 		(on_board yes)
 		(dnp no)
-		(property "Reference" "C20"
+		(property "Reference" "C10"
 			(at 97.79 48.26 0)
 			(effects
@@
 			(project "VXDash"
 				(path "/f2858fc4-50de-4ff0-a01c-5b985ee14aef/21f2fd69-aa93-4550-8877-dde4aa3e5582"
-					(reference "C20")
+					(reference "C10")
 					(unit 1)
 				)
@@
 		(dnp no)
 		(fields_autoplaced yes)
-		(property "Reference" "R43"
+		(property "Reference" "R93"
 			(at 162.56 64.7699 0)
 			(effects
@@
 			(project ""
 				(path "/f2858fc4-50de-4ff0-a01c-5b985ee14aef/21f2fd69-aa93-4550-8877-dde4aa3e5582"
-					(reference "R43")
+					(reference "R93")
 					(unit 1)
 				)
@@
 		(dnp no)
 		(fields_autoplaced yes)
-		(property "Reference" "R41"
+		(property "Reference" "R91"
 			(at 91.44 62.2299 0)
 			(effects
@@
 			(project "VXDash"
 				(path "/f2858fc4-50de-4ff0-a01c-5b985ee14aef/21f2fd69-aa93-4550-8877-dde4aa3e5582"
-					(reference "R41")
+					(reference "R91")
 					(unit 1)
 				)
@@
 		(on_board yes)
 		(dnp no)
-		(property "Reference" "C26"
+		(property "Reference" "C16"
 			(at 199.39 53.34 0)
 			(effects
@@
 			(project "VXDash"
 				(path "/f2858fc4-50de-4ff0-a01c-5b985ee14aef/21f2fd69-aa93-4550-8877-dde4aa3e5582"
-					(reference "C26")
+					(reference "C16")
 					(unit 1)
 				)
@@
 		(on_board yes)
 		(dnp no)
-		(property "Reference" "C25"
+		(property "Reference" "C15"
 			(at 191.77 53.34 0)
 			(effects
@@
 			(project ""
 				(path "/f2858fc4-50de-4ff0-a01c-5b985ee14aef/21f2fd69-aa93-4550-8877-dde4aa3e5582"
-					(reference "C25")
+					(reference "C15")
 					(unit 1)
 				)
@@
 		(dnp no)
 		(fields_autoplaced yes)
-		(property "Reference" "R42"
+		(property "Reference" "R92"
 			(at 91.44 74.9299 0)
 			(effects
@@
 			(project "VXDash"
 				(path "/f2858fc4-50de-4ff0-a01c-5b985ee14aef/21f2fd69-aa93-4550-8877-dde4aa3e5582"
-					(reference "R42")
+					(reference "R92")
 					(unit 1)
 				)
@@
 		(on_board yes)
 		(dnp no)
-		(property "Reference" "C21"
+		(property "Reference" "C11"
 			(at 105.41 48.26 0)
 			(effects
@@
 			(project "VXDash"
 				(path "/f2858fc4-50de-4ff0-a01c-5b985ee14aef/21f2fd69-aa93-4550-8877-dde4aa3e5582"
-					(reference "C21")
+					(reference "C11")
 					(unit 1)
 				)
@@
 		(dnp no)
 		(fields_autoplaced yes)
-		(property "Reference" "C22"
+		(property "Reference" "C12"
 			(at 140.97 45.72 90)
 			(effects
@@
 			(project "VXDash"
 				(path "/f2858fc4-50de-4ff0-a01c-5b985ee14aef/21f2fd69-aa93-4550-8877-dde4aa3e5582"
-					(reference "C22")
+					(reference "C12")
 					(unit 1)
 				)
@@
 		(on_board yes)
 		(dnp no)
-		(property "Reference" "C24"
+		(property "Reference" "C14"
 			(at 184.15 53.34 0)
 			(effects
@@
 			(project "VXDash"
 				(path "/f2858fc4-50de-4ff0-a01c-5b985ee14aef/21f2fd69-aa93-4550-8877-dde4aa3e5582"
-					(reference "C24")
+					(reference "C14")
 					(unit 1)
 				)

Commit message: Emulator board : BOM and fab prep
Parts:
- C10: MFT (none) -> Samsung Electro-Mechanics; MFT_PN (none) -> CL31B106KAHNNNE
- C11, C12, C14: MFT (none) -> Samsung Electro-Mechanics; MFT_PN (none) -> CL10B104KB8NNWC
- C13: MFT (none) -> Kyocera AVX; MFT_PN (none) -> 06035C220JAT2A
- C15, C16: MFT (none) -> Samsung Electro-Mechanics; MFT_PN (none) -> CL31B226KPHNNNE
- R91: MFT (none) -> StackPole Electronics; MFT_PN (none) -> RMCF0603FT820K
- R92: MFT (none) -> StackPole Electronics; MFT_PN (none) -> RMCF0603FT120K
- R93: MFT (none) -> StackPole Electronics; MFT_PN (none) -> RMCF0603FT75K0
- R94: MFT (none) -> Yageo; MFT_PN (none) -> RC0603FR-1324KL
Changed lines of the file:
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@@
 			)
 		)
-		(property "Description" ""
+		(property "Description" "CAP CER 22PF 50V X7R 0603"
 			(at 168.91 66.04 0)
 			(effects
@@
 			)
 		)
-		(property "MFT" ""
+		(property "MFT" "Kyocera AVX"
 			(at 168.91 66.04 0)
 			(effects
@@
 			)
 		)
-		(property "MFT_PN" ""
+		(property "MFT_PN" "06035C220JAT2A"
 			(at 168.91 66.04 0)
 			(effects
@@
 			)
 		)
-		(property "Description" ""
+		(property "Description" "RES 24K OHM 1% 1/10W 0603"
 			(at 160.02 77.47 0)
 			(effects
@@
 			)
 		)
-		(property "MFT" ""
+		(property "MFT" "Yageo"
 			(at 160.02 77.47 0)
 			(effects
@@
 			)
 		)
-		(property "MFT_PN" ""
+		(property "MFT_PN" "RC0603FR-1324KL"
 			(at 160.02 77.47 0)
 			(effects
@@
 			)
 		)
-		(property "Description" ""
+		(property "Description" "CAP CER 10UF 25V X7R 1206"
 			(at 99.06 62.23 0)
 			(effects
@@
 			)
 		)
-		(property "MFT" ""
+		(property "MFT" "Samsung Electro-Mechanics"
 			(at 99.06 62.23 0)
 			(effects
@@
 			)
 		)
-		(property "MFT_PN" ""
+		(property "MFT_PN" "CL31B106KAHNNNE"
 			(at 99.06 62.23 0)
 			(effects
@@
 			)
 		)
-		(property "Description" ""
+		(property "Description" "RES 75K OHM 1% 1/10W 0603"
 			(at 160.02 66.04 0)
 			(effects
@@
 			)
 		)
-		(property "MFT" ""
+		(property "MFT" "StackPole Electronics"
 			(at 160.02 66.04 0)
 			(effects
@@
 			)
 		)
-		(property "MFT_PN" ""
+		(property "MFT_PN" "RMCF0603FT75K0"
 			(at 160.02 66.04 0)
 			(effects
@@
 			)
 		)
-		(property "Description" ""
+		(property "Description" "RES 820K OHM 1% 1/10W 0603"
 			(at 88.9 63.5 0)
 			(effects
@@
 			)
 		)
-		(property "MFT" ""
+		(property "MFT" "StackPole Electronics"
 			(at 88.9 63.5 0)
 			(effects
@@
 			)
 		)
-		(property "MFT_PN" ""
+		(property "MFT_PN" "RMCF0603FT820K"
 			(at 88.9 63.5 0)
 			(effects
@@
 			)
 		)
-		(property "Description" ""
+		(property "Description" "CAP CER 22UF 10V X7R 1206"
 			(at 200.66 66.04 0)
 			(effects
@@
 			)
 		)
-		(property "MFT" ""
+		(property "MFT" "Samsung Electro-Mechanics"
 			(at 200.66 66.04 0)
 			(effects
@@
 			)
 		)
-		(property "MFT_PN" ""
+		(property "MFT_PN" "CL31B226KPHNNNE"
 			(at 200.66 66.04 0)
 			(effects
@@
 			)
 		)
-		(property "Description" ""
+		(property "Description" "CAP CER 22UF 10V X7R 1206"
 			(at 193.04 66.04 0)
 			(effects
@@
 			)
 		)
-		(property "MFT" ""
+		(property "MFT" "Samsung Electro-Mechanics"
 			(at 193.04 66.04 0)
 			(effects
@@
 			)
 		)
-		(property "MFT_PN" ""
+		(property "MFT_PN" "CL31B226KPHNNNE"
 			(at 193.04 66.04 0)
 			(effects
@@
 			)
 		)
-		(property "Description" ""
+		(property "Description" "FIXED IND 3.3UH 3A 30 MOHM SMD"
 			(at 153.67 63.5 0)
 			(effects
@@
 			)
 		)
-		(property "Description" ""
+		(property "Description" "RES 120K OHM 1% 1/10W 0603"
 			(at 88.9 76.2 0)
 			(effects
@@
 			)
 		)
-		(property "MFT" ""
+		(property "MFT" "StackPole Electronics"
 			(at 88.9 76.2 0)
 			(effects
@@
 			)
 		)
-		(property "MFT_PN" ""
+		(property "MFT_PN" "RMCF0603FT120K"
 			(at 88.9 76.2 0)
 			(effects
@@
 			)
 		)
-		(property "Description" ""
+		(property "Description" "CAP CER 0.1UF 50V X7R 0603"
 			(at 106.68 62.23 0)
 			(effects
@@
 			)
 		)
-		(property "MFT" ""
+		(property "MFT" "Samsung Electro-Mechanics"
 			(at 106.68 62.23 0)
 			(effects
@@
 			)
 		)
-		(property "MFT_PN" ""
+		(property "MFT_PN" "CL10B104KB8NNWC"
 			(at 106.68 62.23 0)
 			(effects
@@
 			)
 		)
-		(property "Description" ""
+		(property "Description" "CAP CER 0.1UF 50V X7R 0603"
 			(at 140.97 55.88 0)
 			(effects
@@
 			)
 		)
-		(property "MFT" ""
+		(property "MFT" "Samsung Electro-Mechanics"
 			(at 140.97 55.88 0)
 			(effects
@@
 			)
 		)
-		(property "MFT_PN" ""
+		(property "MFT_PN" "CL10B104KB8NNWC"
 			(at 140.97 55.88 0)
 			(effects
@@
 			)
 		)
-		(property "Description" ""
+		(property "Description" "CAP CER 0.1UF 50V X7R 0603"
 			(at 185.42 66.04 0)
 			(effects
@@
 			)
 		)
-		(property "MFT" ""
+		(property "MFT" "Samsung Electro-Mechanics"
 			(at 185.42 66.04 0)
 			(effects
@@
 			)
 		)
-		(property "MFT_PN" ""
+		(property "MFT_PN" "CL10B104KB8NNWC"
 			(at 185.42 66.04 0)
 			(effects
