File: KiCad PCB Files/VXDash_Emulator/FET_Active_Hi.kicad_sch (KiCad schematic)
At the start: 11 parts, among them J8 Manual backup, Q24 2N7002

Commit message: Emulator board : BOM and fab prep
Parts:
- D45, D46: MFT (none) -> Harvatek Corp; MFT_PN (none) -> B1911PG--20D000514U1930; Voltage (none) -> 2V
- J8: MFT (none) -> Würth Elektronik; MFT_PN (none) -> 61300311121; now not fitted
- R138, R142: MFT (none) -> Yageo; MFT_PN (none) -> RC0603FR-07270RL
- R143: MFT (none) -> Yageo; MFT_PN (none) -> RC0603FR-071KL
- R144, R145, R146: MFT (none) -> StackPole Electronics; MFT_PN (none) -> RNCP0805FTD1K00
Changed lines of the file:
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@@
 		(in_bom yes)
 		(on_board yes)
-		(dnp no)
+		(dnp yes)
 		(property "Reference" "J8"
 			(at 204.47 85.0901 0)
@@
 			)
 		)
-		(property "Description" "Generic connector, single row, 01x03, script generated (kicad-library-utils/schlib/autogen/connector/)"
+		(property "Description" "CONN HEADER VERT 3POS 2.54MM"
 			(at 201.93 83.82 0)
 			(effects
@@
 				)
 				(hide yes)
+			)
+		)
+		(property "MFT" "Würth Elektronik"
+			(at 201.93 83.82 0)
+			(effects
+				(font
+					(size 1.27 1.27)
+				)
+			)
+		)
+		(property "MFT_PN" "61300311121"
+			(at 201.93 83.82 0)
+			(effects
+				(font
+					(size 1.27 1.27)
+				)
 			)
 		)
@@
 			)
 		)
-		(property "Description" ""
+		(property "Description" "RES 1K OHM 1% 1/4W 0805"
 			(at 120.65 57.15 0)
 			(effects
@@
 			)
 		)
-		(property "MFT" ""
+		(property "MFT" "StackPole Electronics"
 			(at 120.65 57.15 0)
 			(effects
@@
 			)
 		)
-		(property "MFT_PN" ""
+		(property "MFT_PN" "RNCP0805FTD1K00"
 			(at 120.65 57.15 0)
 			(effects
@@
 			)
 		)
-		(property "Description" "Light emitting diode, small symbol"
+		(property "Description" "LED GREEN DIFFUSED 0603 SMD"
 			(at 96.52 85.09 0)
 			(effects
@@
 			)
 		)
-		(property "MFT" ""
+		(property "MFT" "Harvatek Corp"
 			(at 96.52 85.09 0)
 			(effects
@@
 			)
 		)
-		(property "MFT_PN" ""
+		(property "MFT_PN" "B1911PG--20D000514U1930"
 			(at 96.52 85.09 0)
 			(effects
@@
 		(property "If" "5mA"
 			(at 100.838 83.82 90)
+			(effects
+				(font
+					(size 1.27 1.27)
+				)
+			)
+		)
+		(property "Voltage" "2V"
+			(at 96.52 85.09 0)
 			(effects
 				(font
@@
 			)
 		)
-		(property "Description" ""
+		(property "Description" "RES 270 OHM 1% 1/10W 0603"
 			(at 96.52 76.2 0)
 			(effects
@@
 			)
 		)
-		(property "MFT" ""
+		(property "MFT" "Yageo"
 			(at 96.52 76.2 0)
 			(effects
@@
 			)
 		)
-		(property "MFT_PN" ""
+		(property "MFT_PN" "RC0603FR-07270RL"
 			(at 96.52 76.2 0)
 			(effects
@@
 			)
 		)
-		(property "Description" ""
+		(property "Description" "RES 1K OHM 1% 1/10W 0603"
 			(at 107.95 69.85 0)
 			(effects
@@
 			)
 		)
-		(property "MFT" ""
+		(property "MFT" "Yageo"
 			(at 107.95 69.85 0)
 			(effects
@@
 			)
 		)
-		(property "MFT_PN" ""
+		(property "MFT_PN" "RC0603FR-071KL"
 			(at 107.95 69.85 0)
 			(effects
@@
 			)
 		)
-		(property "Description" ""
+		(property "Description" "RES 270 OHM 1% 1/10W 0603"
 			(at 96.52 52.07 0)
 			(effects
@@
 			)
 		)
-		(property "MFT" ""
+		(property "MFT" "Yageo"
 			(at 96.52 52.07 0)
 			(effects
@@
 			)
 		)
-		(property "MFT_PN" ""
+		(property "MFT_PN" "RC0603FR-07270RL"
 			(at 96.52 52.07 0)
 			(effects
@@
 			)
 		)
-		(property "Description" "Light emitting diode, small symbol"
+		(property "Description" "LED GREEN DIFFUSED 0603 SMD"
 			(at 96.52 60.96 0)
 			(effects
@@
 			)
 		)
-		(property "MFT" ""
+		(property "MFT" "Harvatek Corp"
 			(at 96.52 60.96 0)
 			(effects
@@
 			)
 		)
-		(property "MFT_PN" ""
+		(property "MFT_PN" "B1911PG--20D000514U1930"
 			(at 96.52 60.96 0)
 			(effects
@@
 		(property "If" "5mA"
 			(at 100.838 59.69 90)
+			(effects
+				(font
+					(size 1.27 1.27)
+				)
+			)
+		)
+		(property "Voltage" "2V"
+			(at 96.52 60.96 0)
 			(effects
 				(font
@@
 			)
 		)
-		(property "Description" ""
+		(property "Description" "RES 1K OHM 1% 1/4W 0805"
 			(at 133.35 57.15 0)
 			(effects
@@
 			)
 		)
-		(property "MFT" ""
+		(property "MFT" "StackPole Electronics"
 			(at 133.35 57.15 0)
 			(effects
@@
 			)
 		)
-		(property "MFT_PN" ""
+		(property "MFT_PN" "RNCP0805FTD1K00"
 			(at 133.35 57.15 0)
 			(effects
@@
 			)
 		)
-		(property "Description" ""
+		(property "Description" "RES 1K OHM 1% 1/4W 0805"
 			(at 143.51 57.15 0)
 			(effects
@@
 			)
 		)
-		(property "MFT" ""
+		(property "MFT" "StackPole Electronics"
 			(at 143.51 57.15 0)
 			(effects
@@
 			)
 		)
-		(property "MFT_PN" ""
+		(property "MFT_PN" "RNCP0805FTD1K00"
 			(at 143.51 57.15 0)
 			(effects

Commit message: Emulator : LCSC part numbers and production files
Parts:
- D45, D46: LCSC (none) -> C5556934
- J8: LCSC (none) -> C2915006
- Q24: LCSC (none) -> C78712
- R138, R142: LCSC (none) -> C137754
- R143: LCSC (none) -> C22548
- R144, R145, R146: LCSC (none) -> C2441430
Changed lines of the file:
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@@
+			)
+		)
+		(property "LCSC" "C2915006"
+			(at 201.93 83.82 0)
+			(effects
+				(font
+					(size 1.27 1.27)
+				)
 			)
 		)
@@
 			)
 		)
+		(property "LCSC" "C2441430"
+			(at 120.65 57.15 0)
+			(effects
+				(font
+					(size 1.27 1.27)
+				)
+			)
+		)
 		(pin "1"
 		)
@@
 			)
 		)
+		(property "LCSC" "C78712"
+			(at 118.11 69.85 0)
+			(effects
+				(font
+					(size 1.27 1.27)
+				)
+			)
+		)
 		(pin "1"
 		)
@@
 		)
 		(property "Voltage" "2V"
+			(at 96.52 85.09 0)
+			(effects
+				(font
+					(size 1.27 1.27)
+				)
+			)
+		)
+		(property "LCSC" "C5556934"
 			(at 96.52 85.09 0)
 			(effects
@@
 			)
 		)
+		(property "LCSC" "C137754"
+			(at 96.52 76.2 0)
+			(effects
+				(font
+					(size 1.27 1.27)
+				)
+			)
+		)
 		(pin "1"
 		)
@@
 			)
 		)
+		(property "LCSC" "C22548"
+			(at 107.95 69.85 0)
+			(effects
+				(font
+					(size 1.27 1.27)
+				)
+			)
+		)
 		(pin "1"
 		)
@@
 			)
 		)
+		(property "LCSC" "C137754"
+			(at 96.52 52.07 0)
+			(effects
+				(font
+					(size 1.27 1.27)
+				)
+			)
+		)
 		(pin "1"
 		)
@@
 		)
 		(property "Voltage" "2V"
+			(at 96.52 60.96 0)
+			(effects
+				(font
+					(size 1.27 1.27)
+				)
+			)
+		)
+		(property "LCSC" "C5556934"
 			(at 96.52 60.96 0)
 			(effects
@@
 			)
 		)
+		(property "LCSC" "C2441430"
+			(at 133.35 57.15 0)
+			(effects
+				(font
+					(size 1.27 1.27)
+				)
+			)
+		)
 		(pin "1"
 		)
@@
 			)
 		)
+		(property "LCSC" "C2441430"
+			(at 143.51 57.15 0)
+			(effects
+				(font
+					(size 1.27 1.27)
+				)
+			)
+		)
 		(pin "1"
 		)
@@
 			)
 		)
+		(property "LCSC" ""
+			(at 161.29 63.5 0)
+			(effects
+				(font
+					(size 1.27 1.27)
+				)
+			)
+		)

Commit message: Emulator : Updating BOM with LCSC alts
Parts:
- D45, D46: LCSC alt (none) -> C284909
- J8: LCSC alt (none) -> C2937625
- Q24: LCSC alt (none) -> C78712
- R138, R142: LCSC alt (none) -> C137754
- R143: LCSC alt (none) -> C22548
- R144, R145, R146: LCSC alt (none) -> C727989
Changed lines of the file:
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@@
+			)
+		)
+		(property "LCSC alt" "C2937625"
+			(at 201.93 83.82 0)
+			(effects
+				(font
+					(size 1.27 1.27)
+				)
 			)
 		)
@@
 			)
 		)
+		(property "LCSC alt" "C727989"
+			(at 120.65 57.15 0)
+			(effects
+				(font
+					(size 1.27 1.27)
+				)
+			)
+		)
 		(pin "1"
 		)
@@
 			)
 		)
+		(property "LCSC alt" "C78712"
+			(at 118.11 69.85 0)
+			(effects
+				(font
+					(size 1.27 1.27)
+				)
+			)
+		)
 		(pin "1"
 		)
@@
 		)
 		(property "LCSC" "C5556934"
+			(at 96.52 85.09 0)
+			(effects
+				(font
+					(size 1.27 1.27)
+				)
+			)
+		)
+		(property "LCSC alt" "C284909"
 			(at 96.52 85.09 0)
 			(effects
@@
 			)
 		)
+		(property "LCSC alt" "C137754"
+			(at 96.52 76.2 0)
+			(effects
+				(font
+					(size 1.27 1.27)
+				)
+			)
+		)
 		(pin "1"
 		)
@@
 			)
 		)
+		(property "LCSC alt" "C22548"
+			(at 107.95 69.85 0)
+			(effects
+				(font
+					(size 1.27 1.27)
+				)
+			)
+		)
 		(pin "1"
 		)
@@
 			)
 		)
+		(property "LCSC alt" "C137754"
+			(at 96.52 52.07 0)
+			(effects
+				(font
+					(size 1.27 1.27)
+				)
+			)
+		)
 		(pin "1"
 		)
@@
 		)
 		(property "LCSC" "C5556934"
+			(at 96.52 60.96 0)
+			(effects
+				(font
+					(size 1.27 1.27)
+				)
+			)
+		)
+		(property "LCSC alt" "C284909"
 			(at 96.52 60.96 0)
 			(effects
@@
 			)
 		)
+		(property "LCSC alt" "C727989"
+			(at 133.35 57.15 0)
+			(effects
+				(font
+					(size 1.27 1.27)
+				)
+			)
+		)
 		(pin "1"
 		)
@@
 			)
 		)
+		(property "LCSC alt" "C727989"
+			(at 143.51 57.15 0)
+			(effects
+				(font
+					(size 1.27 1.27)
+				)
+			)
+		)
 		(pin "1"
 		)
@@
 			(at 161.29 63.5 0)
 			(effects
+				(font
+					(size 1.27 1.27)
+				)
+			)
+		)
+		(property "LCSC alt" ""
+			(at 161.29 63.5 0)
+			(effects
