File: KiCad PCB Files/ESP32P4_display_adapter_board/BacklightPSU.kicad_sch (KiCad schematic)
At the start: 15 parts, among them U1 AP3032KTR-G1

Commit message: BOM updates
Parts:
- C3, C4: value 1u -> 1uF
- C5, C6: value 10u -> 10uF
- C7: value 0.1u -> 100nF
- D1: Arrow Part Number 1N5819HW-7-F -> (none); Arrow Price/Stock https://www.arrow.com/en/products/1n5819hw-7-f/diodes-incor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 -> (none); Mouser Part Number 621-1N5819HW-F -> (none); Mouser Price/Stock https://www.mouser.co.uk/ProductDetail/Diodes-Incorporated/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 -> (none)

Commit message: CTP connector spec
Parts:
- renumbered C7 to C3, C6 to C4, C3 to C5, C5 to C6, C4 to C7, R7 to R3, R6 to R4, R3 to R5, R5 to R6, R4 to R7, R2 to R8, R1 to R9
Changed lines of the file:
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@@
 		(dnp no)
 		(fields_autoplaced yes)
-		(property "Reference" "R2"
+		(property "Reference" "R8"
 			(at 193.04 86.3599 0)
 			(effects
@@
 			(project "ESP32P4_display_adapter_board"
 				(path "/ab7fe2a8-21c6-4fbd-85af-cbc3a22ae1d9/3b913174-38a9-4126-84b3-80f845d68af5"
-					(reference "R2")
+					(reference "R8")
 					(unit 1)
 				)
@@
 		(dnp no)
 		(fields_autoplaced yes)
-		(property "Reference" "R5"
+		(property "Reference" "R6"
 			(at 119.38 124.4599 0)
 			(effects
@@
 			(project "ESP32P4_display_adapter_board"
 				(path "/ab7fe2a8-21c6-4fbd-85af-cbc3a22ae1d9/3b913174-38a9-4126-84b3-80f845d68af5"
-					(reference "R5")
+					(reference "R6")
 					(unit 1)
 				)
@@
 		(dnp no)
 		(fields_autoplaced yes)
-		(property "Reference" "R4"
+		(property "Reference" "R7"
 			(at 119.38 134.6199 0)
 			(effects
@@
 			(project "ESP32P4_display_adapter_board"
 				(path "/ab7fe2a8-21c6-4fbd-85af-cbc3a22ae1d9/3b913174-38a9-4126-84b3-80f845d68af5"
-					(reference "R4")
+					(reference "R7")
 					(unit 1)
 				)
@@
 		(dnp no)
 		(fields_autoplaced yes)
-		(property "Reference" "C3"
+		(property "Reference" "C5"
 			(at 198.12 119.3799 0)
 			(effects
@@
 			(project ""
 				(path "/ab7fe2a8-21c6-4fbd-85af-cbc3a22ae1d9/3b913174-38a9-4126-84b3-80f845d68af5"
-					(reference "C3")
+					(reference "C5")
 					(unit 1)
 				)
@@
 		(dnp no)
 		(fields_autoplaced yes)
-		(property "Reference" "#PWR07"
+		(property "Reference" "#PWR028"
 			(at 194.31 132.08 0)
 			(effects
@@
 			(project ""
 				(path "/ab7fe2a8-21c6-4fbd-85af-cbc3a22ae1d9/3b913174-38a9-4126-84b3-80f845d68af5"
-					(reference "#PWR07")
+					(reference "#PWR028")
 					(unit 1)
 				)
@@
 		(dnp no)
 		(fields_autoplaced yes)
-		(property "Reference" "#PWR010"
+		(property "Reference" "#PWR027"
 			(at 116.84 149.86 0)
 			(effects
@@
 			(project "ESP32P4_display_adapter_board"
 				(path "/ab7fe2a8-21c6-4fbd-85af-cbc3a22ae1d9/3b913174-38a9-4126-84b3-80f845d68af5"
-					(reference "#PWR010")
+					(reference "#PWR027")
 					(unit 1)
 				)
@@
 		(dnp no)
 		(fields_autoplaced yes)
-		(property "Reference" "R3"
+		(property "Reference" "R5"
 			(at 109.22 134.6199 0)
 			(effects
@@
 			(project "ESP32P4_display_adapter_board"
 				(path "/ab7fe2a8-21c6-4fbd-85af-cbc3a22ae1d9/3b913174-38a9-4126-84b3-80f845d68af5"
-					(reference "R3")
+					(reference "R5")
 					(unit 1)
 				)
@@
 		(dnp no)
 		(fields_autoplaced yes)
-		(property "Reference" "R7"
+		(property "Reference" "R3"
 			(at 81.28 115.57 90)
 			(effects
@@
 			(project "ESP32P4_display_adapter_board"
 				(path "/ab7fe2a8-21c6-4fbd-85af-cbc3a22ae1d9/3b913174-38a9-4126-84b3-80f845d68af5"
-					(reference "R7")
+					(reference "R3")
 					(unit 1)
 				)
@@
 		(dnp no)
 		(fields_autoplaced yes)
-		(property "Reference" "R6"
+		(property "Reference" "R4"
 			(at 101.6 115.57 90)
 			(effects
@@
 			(project "ESP32P4_display_adapter_board"
 				(path "/ab7fe2a8-21c6-4fbd-85af-cbc3a22ae1d9/3b913174-38a9-4126-84b3-80f845d68af5"
-					(reference "R6")
+					(reference "R4")
 					(unit 1)
 				)
@@
 		(dnp no)
 		(fields_autoplaced yes)
-		(property "Reference" "C6"
+		(property "Reference" "C4"
 			(at 107.95 87.6299 0)
 			(effects
@@
 			(project "ESP32P4_display_adapter_board"
 				(path "/ab7fe2a8-21c6-4fbd-85af-cbc3a22ae1d9/3b913174-38a9-4126-84b3-80f845d68af5"
-					(reference "C6")
+					(reference "C4")
 					(unit 1)
 				)
@@
 		(dnp no)
 		(fields_autoplaced yes)
-		(property "Reference" "C4"
+		(property "Reference" "C7"
 			(at 223.52 85.0899 0)
 			(effects
@@
 			(project "ESP32P4_display_adapter_board"
 				(path "/ab7fe2a8-21c6-4fbd-85af-cbc3a22ae1d9/3b913174-38a9-4126-84b3-80f845d68af5"
-					(reference "C4")
+					(reference "C7")
 					(unit 1)
 				)
@@
 		(dnp no)
 		(fields_autoplaced yes)
-		(property "Reference" "C7"
+		(property "Reference" "C3"
 			(at 95.25 133.3499 0)
 			(effects
@@
 			(project "ESP32P4_display_adapter_board"
 				(path "/ab7fe2a8-21c6-4fbd-85af-cbc3a22ae1d9/3b913174-38a9-4126-84b3-80f845d68af5"
-					(reference "C7")
+					(reference "C3")
 					(unit 1)
 				)
@@
 		(dnp no)
 		(fields_autoplaced yes)
-		(property "Reference" "R1"
+		(property "Reference" "R9"
 			(at 196.85 113.0299 0)
 			(effects
@@
 			(project ""
 				(path "/ab7fe2a8-21c6-4fbd-85af-cbc3a22ae1d9/3b913174-38a9-4126-84b3-80f845d68af5"
-					(reference "R1")
+					(reference "R9")
 					(unit 1)
 				)
@@
 		(dnp no)
 		(fields_autoplaced yes)
-		(property "Reference" "#PWR09"
+		(property "Reference" "#PWR026"
 			(at 104.14 105.41 0)
 			(effects
@@
 			(project "ESP32P4_display_adapter_board"
 				(path "/ab7fe2a8-21c6-4fbd-85af-cbc3a22ae1d9/3b913174-38a9-4126-84b3-80f845d68af5"
-					(reference "#PWR09")
+					(reference "#PWR026")
 					(unit 1)
 				)
@@
 		(dnp no)
 		(fields_autoplaced yes)
-		(property "Reference" "#PWR08"
+		(property "Reference" "#PWR029"
 			(at 219.71 105.41 0)
 			(effects
@@
 			(project "ESP32P4_display_adapter_board"
 				(path "/ab7fe2a8-21c6-4fbd-85af-cbc3a22ae1d9/3b913174-38a9-4126-84b3-80f845d68af5"
-					(reference "#PWR08")
+					(reference "#PWR029")
 					(unit 1)
 				)
@@
 		(dnp no)
 		(fields_autoplaced yes)
-		(property "Reference" "#PWR011"
+		(property "Reference" "#PWR025"
 			(at 91.44 149.86 0)
 			(effects
@@
 			(project "ESP32P4_display_adapter_board"
 				(path "/ab7fe2a8-21c6-4fbd-85af-cbc3a22ae1d9/3b913174-38a9-4126-84b3-80f845d68af5"
-					(reference "#PWR011")
+					(reference "#PWR025")
 					(unit 1)
 				)
@@
 		(dnp no)
 		(fields_autoplaced yes)
-		(property "Reference" "C5"
+		(property "Reference" "C6"
 			(at 209.55 85.0899 0)
 			(effects
@@
 			(project "ESP32P4_display_adapter_board"
 				(path "/ab7fe2a8-21c6-4fbd-85af-cbc3a22ae1d9/3b913174-38a9-4126-84b3-80f845d68af5"
-					(reference "C5")
+					(reference "C6")
 					(unit 1)
 				)

Commit message: BOM and Pre-routing
Connections:
- net VCC_5V: now also L1.2, U1.6 (VIN); no longer L1.1, U1.1 (SW)
- net VLED+: now also R8.2; no longer R8.1
- net at U1.5 (OV): now also R8.1; no longer R8.2
- new net: D1.2, L1.1, U1.1 (SW)
Other:
- moved on the sheet: C4, C6, C7, D1, R8
