File: KiCad PCB Files/ESP32P4_display_adapter_board/ESP32P4_display_adapter_board.kicad_pcb (KiCad board)
At the start: 2 copper layers, 0 parts

Commit message: BOM and Pre-routing
Parts:
- added C1: 100nF, Capacitor_SMD:C_0603_1608Metric_Pad1.08x0.95mm_HandSolder, F.Cu at (101.1, 108.9)
- added C10: 10uF, Capacitor_SMD:C_0805_2012Metric, F.Cu at (131.7, 136.8)
- added C11: 10uF, Capacitor_SMD:C_0805_2012Metric, F.Cu at (123.6, 135.9)
- added C2: 10uF, Capacitor_SMD:C_0603_1608Metric_Pad1.08x0.95mm_HandSolder, F.Cu at (101.1, 114.0)
- added C3: 100nF, Capacitor_SMD:C_0603_1608Metric_Pad1.08x0.95mm_HandSolder, F.Cu at (83.9, 149.5)
- added C4: 10uF, Capacitor_SMD:C_0603_1608Metric_Pad1.08x0.95mm_HandSolder, F.Cu at (89.8, 141.9)
- added C5: 1uF, Capacitor_SMD:C_0603_1608Metric_Pad1.08x0.95mm_HandSolder, F.Cu at (88.5, 146.7)
- added C6: 10uF, Capacitor_SMD:C_0603_1608Metric_Pad1.08x0.95mm_HandSolder, F.Cu at (80.4, 145.0)
- added C7: 1uF, Capacitor_SMD:C_0603_1608Metric_Pad1.08x0.95mm_HandSolder, F.Cu at (80.4, 146.7)
- added C8: 10uF, Capacitor_SMD:C_0805_2012Metric, F.Cu at (127.4, 131.8)
- added C9: 100nF, Capacitor_SMD:C_0805_2012Metric, F.Cu at (130.2, 132.0)
- added D1: 1N5819HW-7-F, Diode_SMD:D_SOD-123, F.Cu at (78.6, 141.4)
- added J1: Sel_VCC, Connector_PinHeader_2.54mm:PinHeader_1x03_P2.54mm_Vertical, F.Cu at (119.2, 131.6)
- added J2: MIPI DSI, VXDash_connectors:TE_1-1734248-5, F.Cu at (136.7, 61.5)
- added J4: S1, Connector_PinSocket_2.54mm:PinSocket_2x13_P2.54mm_Vertical, B.Cu at (122.5, 71.8)
- added J5: S2, Connector_PinSocket_2.54mm:PinSocket_2x13_P2.54mm_Vertical, B.Cu at (167.6, 71.8)
- added J6: 39Pin FPC, Connector_FFC-FPC:Hirose_FH26-39S-0.3SHW_2Rows-39Pins-1MP_P0.60mm_Horizontal, F.Cu at (149.9, 53.0)
- added J7: WS_30P_rev, Connector_FFC-FPC:Hirose_FH12-30S-0.5SH_1x30-1MP_P0.50mm_Horizontal, F.Cu at (132.1, 37.5)
- added J8: WS_30P, Connector_FFC-FPC:Hirose_FH12-30S-0.5SH_1x30-1MP_P0.50mm_Horizontal, F.Cu at (125.3, 37.5)
- added JP1: SDA_P-UP, Jumper:SolderJumper-2_P1.3mm_Bridged_RoundedPad1.0x1.5mm, F.Cu at (104.1, 109.8)
- added JP2: SCL_P-UP, Jumper:SolderJumper-2_P1.3mm_Bridged_RoundedPad1.0x1.5mm, F.Cu at (104.1, 113.1)
- added L1: 15uH, Inductor_SMD:L_Taiyo-Yuden_NR-60xx_HandSoldering, F.Cu at (84.4, 140.6)
- added L2: 4.7uH, Inductor_SMD:L_1008_2520Metric, F.Cu at (123.8, 132.9)
- added L3: 4.7uH, Inductor_SMD:L_1008_2520Metric, F.Cu at (132.7, 133.8)
- added R1: 4k7, Resistor_SMD:R_0603_1608Metric, F.Cu at (101.1, 110.5)
- added R2: 4k7, Resistor_SMD:R_0603_1608Metric, F.Cu at (101.1, 112.3)
- added R3: 10k, Resistor_SMD:R_0603_1608Metric_Pad0.98x0.95mm_HandSolder, F.Cu at (85.7, 149.5)
- added R4: 30k, Resistor_SMD:R_0603_1608Metric_Pad0.98x0.95mm_HandSolder, F.Cu at (82.2, 149.5)
- added R5: 10, Resistor_SMD:R_0603_1608Metric_Pad0.98x0.95mm_HandSolder, F.Cu at (76.8, 149.5)
- added R6: 3k3, Resistor_SMD:R_0603_1608Metric_Pad0.98x0.95mm_HandSolder, F.Cu at (80.4, 149.5)
- added R7: 10, Resistor_SMD:R_0603_1608Metric_Pad0.98x0.95mm_HandSolder, F.Cu at (78.6, 149.5)
- added R8: 0, Resistor_SMD:R_0603_1608Metric_Pad0.98x0.95mm_HandSolder, F.Cu at (88.5, 145.0)
- added R9: 100k, Resistor_SMD:R_0603_1608Metric_Pad0.98x0.95mm_HandSolder, F.Cu at (88.5, 148.5)
- added U1: AP3032KTR-G1, Package_TO_SOT_SMD:SOT-23-6, F.Cu at (84.4, 145.7)
- added U2: TPS65133DPDR, Package_SON:WSON-12-1EP_3x3mm_P0.5mm_EP1.5x2.5mm_ThermalVias, F.Cu at (127.6, 135.6)
Routing:
- net /39-40Pin Bias Controller/Vin: track 0.00 -> 2.80 mm
- net /BIAS_EN: track 0.00 -> 2.18 mm
- added copper zone on F.Cu, net /39-40Pin Bias Controller/Vin
- added copper zone on F.Cu, net /VDD(+5V)
- added copper zone on F.Cu, net /VDD(-5V)
- added copper zone on F.Cu, net Net-(U2-SWN)
- added copper zone on F.Cu, net Net-(U2-SWP)
Other:
- board outline added: 50 x 50 mm

Commit message: DP routing sucks
Parts:
- moved R5 113.8 mm to (148.4, 61.1), turned to 0 degrees
- moved R7 111.3 mm to (148.4, 62.9), turned to 0 degrees
- moved D1 110.6 mm to (156.6, 62.9), turned to 0 degrees
- moved R6 108.8 mm to (148.4, 64.7), turned to 180 degrees
- moved C7 108.4 mm to (151.2, 64.7), turned to -90 degrees
- moved C6 108.3 mm to (153.0, 64.7), turned to -90 degrees
- moved R4 106.3 mm to (148.4, 66.5), turned to 0 degrees
- moved C3 103.8 mm to (148.4, 68.2), turned to 0 degrees
- moved U1 102.6 mm to (152.2, 68.7), turned to -90 degrees
- moved L1 102.4 mm to (157.3, 68.7), turned to -90 degrees
- moved R3 101.3 mm to (148.4, 70.0), turned to 0 degrees
- moved C10 97.8 mm to (117.2, 40.2), turned to 90 degrees
- moved R9 97.2 mm to (149.5, 72.8), turned to 90 degrees
- moved C5 97.0 mm to (151.2, 72.8), turned to -90 degrees
- moved R8 96.8 mm to (153.0, 72.8), turned to -90 degrees
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Routing:
- net /LEDA: track 0.00 -> 32.0 mm, vias 0 -> 2
- net Net-(U1-FB): track 0.00 -> 4.69 mm
- net Net-(C3-Pad1): track 0.00 -> 4.31 mm
- net Net-(U1-CTRL): track 0.00 -> 3.89 mm
- net /SDA: track 0.00 -> 3.75 mm
- net /SCL: track 0.00 -> 3.75 mm
- net Net-(U1-OV): track 0.00 -> 2.33 mm
- added copper zone on F.Cu, net +5V
- added copper zone on F.Cu, net /LEDA
- added copper zone on F.Cu, net /LEDK
- added copper zone on F.Cu, net Net-(U1-SW)
Other:
- board size 50 x 50 mm -> 50 x 74 mm

Commit message: Struggles with extended routing
Parts:
- J7: moved to B.Cu
- moved J8 39.7 mm to (164.6, 37.4), turned to 90 degrees
- moved J6 6.48 mm to (143.5, 37.3), turned to 0 degrees
- moved J7 0.56 mm to (164.6, 37.4), turned to -90 degrees
Routing:
- net /DSI_D0_P: track 0.00 -> 21.0 mm
- net /DSI_D0_N: track 0.13 -> 21.0 mm
- net /DSI_D1_N: track 0.00 -> 20.2 mm, vias 0 -> 2
- net /DSI_D1_P: track 0.00 -> 20.2 mm, vias 0 -> 2
- net /DSI_CLK_N: track 0.00 -> 19.1 mm, vias 0 -> 2
- net /DSI_CLK_P: track 0.00 -> 19.1 mm, vias 0 -> 2

Commit message: Moving to single 39P
Parts:
- removed J7: WS_30P_rev, Connector_FFC-FPC:Hirose_FH12-30S-0.5SH_1x30-1MP_P0.50mm_Horizontal
- removed J8: WS_30P, Connector_FFC-FPC:Hirose_FH12-30S-0.5SH_1x30-1MP_P0.50mm_Horizontal
- added J9: TP passthru, Connector_PinHeader_2.54mm:PinHeader_1x07_P2.54mm_Vertical, F.Cu at (132.6, 75.9)
- moved C1 55.7 mm to (109.0, 53.7)
- moved JP2 55.7 mm to (112.0, 57.9)
- moved R2 55.7 mm to (109.0, 57.2)
- moved C2 55.7 mm to (109.0, 58.8)
- moved JP1 55.7 mm to (112.0, 54.6)
- moved R1 55.7 mm to (109.0, 55.4)
- moved J1 53.7 mm to (167.2, 49.8)
- moved L2 41.3 mm to (154.3, 44.4), turned to -90 degrees
- moved C11 38.9 mm to (154.6, 41.3), turned to 0 degrees
- moved C8 38.7 mm to (150.8, 45.5), turned to 0 degrees
- moved C9 35.8 mm to (148.0, 45.2), turned to -90 degrees
- moved U2 34.7 mm to (150.5, 41.7), turned to 180 degrees
- moved L3 31.6 mm to (145.5, 43.5), turned to 90 degrees
- moved C10 29.3 mm to (146.5, 40.4), turned to 180 degrees
- moved R9 19.3 mm to (150.4, 53.5), turned to 0 degrees
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Routing:
- net /SCL: track 3.75 -> 36.4 mm
- net /SDA: track 3.75 -> 33.3 mm
- net /TP_INT: track 0.00 -> 26.0 mm
- net /DSI_CLK_N: track 19.1 -> 44.8 mm, vias 2 -> 0
- net /DSI_CLK_P: track 19.1 -> 44.8 mm, vias 2 -> 0
- net /DSI_D1_N: track 20.2 -> 45.0 mm, vias 2 -> 0
- net /DSI_D1_P: track 20.2 -> 45.0 mm, vias 2 -> 0
- net /TP_RESET: track 0.00 -> 21.2 mm
- net /DSI_D0_N: track 21.0 -> 41.8 mm, vias 0 -> 2
- net /DSI_D0_P: track 21.0 -> 41.8 mm, vias 0 -> 2
