File: KiCad PCB Files/VXDash_Connectors/VXDash_Connectors.kicad_pcb (KiCad board)
At the start: 2 copper layers, 27.5 x 110 mm, 4 parts, among them J1 Header_VX220_RightAngle, J2 CANbus, J3 Conn_02x16_Odd_Even

Commit message: Added smaller DT connector to connector board
Parts:
- removed J2: CANbus, VXDash_connectors:DT13-4P_TE_Deutsch
- added H1: M4 Thread mount, VXDash_mech:KEYSTONE_7765, F.Cu at (117.8, 52.3)
- added J4: CANbus, VXDash_connectors:TE_DTF13-4P, F.Cu at (126.5, 73.2)
- J3: value Conn_02x16_Odd_Even -> Passthrough
Connections:
- J3 pad 25: /5V_EXT -> unconnected-(J3-Pin_25-Pad25)
Other:
- board size 27.5 x 110 mm -> 27.5 x 112.5 mm

Commit message: New main dash PCB - WIP inc. CAD
Parts:
- J3: footprint Connector_PinHeader_2.54mm:PinHeader_2x15_P2.54mm_Vertical -> Connector_IDC:IDC-Header_2x15_P2.54mm_Vertical
- moved J3 0.96 mm to (141.5, 125.0)
- renumbered H1 to H2
Connections:
- H1 pad MP: (no net) -> GND
