File: KiCad PCB Files/VXDash_MinBuild/VXDash_MinBuild.kicad_sch (KiCad schematic)
At the start: 87 parts, among them IC1 CD74HC4050M96, J1 Header_VX220_RightAngle, J10 CANbus, J11 LD connector, J12 RD connector, J2 FASCIA PASSTHRU, J5 CAN debug, SW1 RESET, SW2 BOOT, U1 TCA9555PWR, U2 ESP32-S3-WROOM-1

Commit message: Manual Mini Build BOM
Parts:
- C53, C54, C55: value 100n -> 22p; LCSC C16194176 -> C22409299; MFT Samsung Electro-Mechanics -> KEMET; MFT_PN CL10B104KB8NNWC -> C0603C220K5RACTU
- C56, C61, C62, D13, D14, D15, D16, D17, D18, D19, R100, R101, R102, R103, R104, R105, R89: now not fitted; now left out of the parts list
- J5: now left out of the parts list
Other:
- note removed: "Add 2P JST PH for the 3v3 and 5V internal reconnections ?"
