File: KiCad PCB Files/VXDash_RemoteECU/5V_SMPS.kicad_sch (KiCad schematic)
At the start: 13 parts, among them IC4 AP62200

Commit message: More changes (Primarily Remote ECU)
- Emulator board project to a functional skeleton
- Connectors board with ignition routing on CAN pin 4 to have switched signal available in the harness.
- Remote ECU : added 12V reduced protection circuit (to be reviewed)
- Remote ECU : Removed integrated CAN termination (should be on harness)
- Remote ECU : added CAN passthrough
- Remote ECU : added MCPWM channels
- Remote ECU : Added some opto inputs
- Remote ECU : Added internal USB C (overkill ?)
Parts:
- removed C14: 10u, Capacitor_SMD:C_1206_3216Metric_Pad1.33x1.80mm_HandSolder, symbol VXDash_passives:Cap_MLCC
- removed C15, C16, C18: 100n, symbol VXDash_passives:Cap_MLCC
- removed C17: 22p, Capacitor_SMD:C_0402_1005Metric_Pad0.74x0.62mm_HandSolder, symbol VXDash_passives:Cap_MLCC
- removed C19, C20: 22u, Capacitor_SMD:C_1206_3216Metric_Pad1.33x1.80mm_HandSolder, symbol VXDash_passives:Cap_MLCC
- removed IC4: AP62200, Package_TO_SOT_SMD:TSOT-23-6_HandSoldering, symbol VXDash_regulators:AP62200
- removed L2: 3u3, Inductor_SMD:L_Taiyo-Yuden_NR-50xx_HandSoldering, symbol VXDash_passives:Ind
- removed R37: 820k, Resistor_SMD:R_0603_1608Metric_Pad0.98x0.95mm_HandSolder, symbol VXDash_passives:Res
- removed R38: 120k, Resistor_SMD:R_0603_1608Metric_Pad0.98x0.95mm_HandSolder, symbol VXDash_passives:Res
- removed R39: 75k, Resistor_SMD:R_0603_1608Metric_Pad0.98x0.95mm_HandSolder, symbol VXDash_passives:Res
- removed R40: 24k, Resistor_SMD:R_0603_1608Metric_Pad0.98x0.95mm_HandSolder, symbol VXDash_passives:Res
- added C48: 10u, Capacitor_SMD:C_1206_3216Metric_Pad1.33x1.80mm_HandSolder, symbol VXDash_passives:Cap_MLCC
- added C49, C50, C52: 100n, symbol VXDash_passives:Cap_MLCC
- added C51: 22p, Capacitor_SMD:C_0402_1005Metric_Pad0.74x0.62mm_HandSolder, symbol VXDash_passives:Cap_MLCC
- added C53, C54: 22u, Capacitor_SMD:C_1206_3216Metric_Pad1.33x1.80mm_HandSolder, symbol VXDash_passives:Cap_MLCC
- added IC8: AP62200, Package_TO_SOT_SMD:TSOT-23-6_HandSoldering, symbol VXDash_regulators:AP62200
- added L3: 4u7, VXDash_inductors:Ind_5050, symbol VXDash_passives:Ind
- added R114: 1k8, Resistor_SMD:R_0603_1608Metric_Pad0.98x0.95mm_HandSolder, symbol VXDash_passives:Res
- added R115: 1k5, Resistor_SMD:R_0603_1608Metric_Pad0.98x0.95mm_HandSolder, symbol VXDash_passives:Res
- added R96: 1k, Resistor_SMD:R_0603_1608Metric_Pad0.98x0.95mm_HandSolder, symbol VXDash_passives:Res
- added R97: 100k, Resistor_SMD:R_0603_1608Metric_Pad0.98x0.95mm_HandSolder, symbol VXDash_passives:Res
- added R98: 43k, Resistor_SMD:R_0603_1608Metric_Pad0.98x0.95mm_HandSolder, symbol VXDash_passives:Res
- added R99: 8k2, Resistor_SMD:R_0603_1608Metric_Pad0.98x0.95mm_HandSolder, symbol VXDash_passives:Res
Connections:
- net GND: now also C48.1, C49.1, C52.1, C53.2, C54.2, IC8.1 (GND), R115.1, R97.2, R99.2
- new net: C51.2, IC8.4 (FB), R98.2, R99.1
- new net: C50.1, IC8.2 (SW), L3.1
- new net: IC8.5 (EN), R96.2, R97.1
- new net: C50.2, IC8.6 (BST)
- new net: R114.1, R115.2, R96.1
- new net 12V_in: C48.2, C49.2, IC8.3 (VIN)
- new net 5V_en: R114.2
- new net 5V_out: C51.1, C52.2, C53.1, C54.1, L3.2, R98.1
Other:
- company: (none) -> Alex Miller & Martin Roger

Commit message: Started work on RemoteECU schematic
Parts:
- removed C49, C52: 100n, symbol VXDash_passives:Cap_MLCC
- removed R115: 1k5, Resistor_SMD:R_0603_1608Metric_Pad0.98x0.95mm_HandSolder, symbol VXDash_passives:Res
- removed R96: 1k, Resistor_SMD:R_0603_1608Metric_Pad0.98x0.95mm_HandSolder, symbol VXDash_passives:Res
- added C7: 10u, Capacitor_SMD:C_1206_3216Metric_Pad1.33x1.80mm_HandSolder, symbol VXDash_passives:Cap_MLCC
- R114: value 1k8 -> 180k
- R97: value 100k -> 150k
Connections:
- net 12V_in: now also C7.2
- net GND: now also C7.1
- net at IC8.5 (EN), R97.1: now also R114.1
Other:
- moved on the sheet: C53, C54, R114

Commit message: Initial work towards remote ECU functions
Parts:
- C12: renamed from C50; footprint (none) -> Capacitor_SMD:C_0603_1608Metric_Pad1.08x0.95mm_HandSolder
- C19: renamed from C51; footprint Capacitor_SMD:C_0402_1005Metric_Pad0.74x0.62mm_HandSolder -> Capacitor_SMD:C_0603_1608Metric_Pad1.08x0.95mm_HandSolder
- R20: renamed from R114; value 180k -> 130k
- R22: renamed from R97; value 150k -> 100k
- renumbered C48 to C13, C7 to C14, C53 to C20, C54 to C21, IC8 to IC3, L3 to L2, R98 to R19, R99 to R23
Changed lines of the file:
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@@
 	(title_block
 		(title "VXDash RemoteECU")
-		(date "2025-08-08")
+		(date "2026-01-25")
 		(rev "Proto A")
 		(company "Alex Miller & Martin Roger")
@@
 		(exclude_from_sim no)
 		(at 133.35 109.22 0)
-		(size 27.94 12.7)
+		(size 44.45 12.7)
 		(margins 0.9525 0.9525 0.9525 0.9525)
 		(stroke
@@
 		)
 	)
-	(text_box "EN locking up at 1.5V when 5V_en at 3V3"
+	(text_box "EN from 3V3 MCU pin. \nQuicker turn off as 3V3 falls.\nRising threshold = 2.76 typ, ~3V max\nFalling threshold = 2.53 typ, ~2.3V min"
 		(exclude_from_sim no)
-		(at 50.8 99.06 0)
-		(size 27.94 12.7)
+		(at 33.02 95.25 0)
+		(size 41.91 12.7)
 		(margins 0.9525 0.9525 0.9525 0.9525)
 		(stroke
@@
 		(dnp no)
 		(fields_autoplaced yes)
-		(property "Reference" "#PWR061"
+		(property "Reference" "#PWR016"
 			(at 113.03 114.3 0)
 			(effects
@@
 			(project "VXDash"
 				(path "/f2858fc4-50de-4ff0-a01c-5b985ee14aef/f28d59c3-3184-4c96-b6c0-966ec9ca6979"
-					(reference "#PWR061")
+					(reference "#PWR016")
 					(unit 1)
 				)
@@
 		(dnp yes)
 		(fields_autoplaced yes)
-		(property "Reference" "C51"
+		(property "Reference" "C19"
 			(at 161.29 83.8199 0)
 			(effects
@@
 			)
 		)
-		(property "Footprint" "Capacitor_SMD:C_0402_1005Metric_Pad0.74x0.62mm_HandSolder"
+		(property "Footprint" "Capacitor_SMD:C_0603_1608Metric_Pad1.08x0.95mm_HandSolder"
 			(at 158.4452 90.17 0)
 			(effects
@@
 			(project "VXDash"
 				(path "/f2858fc4-50de-4ff0-a01c-5b985ee14aef/f28d59c3-3184-4c96-b6c0-966ec9ca6979"
-					(reference "C51")
+					(reference "C19")
 					(unit 1)
 				)
@@
 		(on_board yes)
 		(dnp no)
-		(property "Reference" "C54"
+		(property "Reference" "C21"
 			(at 175.26 73.66 0)
 			(effects
@@
 			(project "VXDash"
 				(path "/f2858fc4-50de-4ff0-a01c-5b985ee14aef/f28d59c3-3184-4c96-b6c0-966ec9ca6979"
-					(reference "C54")
+					(reference "C21")
 					(unit 1)
 				)
@@
 		(on_board yes)
 		(dnp no)
-		(property "Reference" "C53"
+		(property "Reference" "C20"
 			(at 167.64 73.66 0)
 			(effects
@@
 			(project "VXDash"
 				(path "/f2858fc4-50de-4ff0-a01c-5b985ee14aef/f28d59c3-3184-4c96-b6c0-966ec9ca6979"
-					(reference "C53")
+					(reference "C20")
 					(unit 1)
 				)
@@
 		(on_board yes)
 		(dnp no)
-		(property "Reference" "C7"
+		(property "Reference" "C14"
 			(at 87.63 68.58 0)
 			(effects
@@
 			(project "VXDash_RemoteECU"
 				(path "/f2858fc4-50de-4ff0-a01c-5b985ee14aef/f28d59c3-3184-4c96-b6c0-966ec9ca6979"
-					(reference "C7")
+					(reference "C14")
 					(unit 1)
 				)
@@
 		(dnp no)
 		(fields_autoplaced yes)
-		(property "Reference" "IC8"
+		(property "Reference" "IC3"
 			(at 113.03 68.58 0)
 			(effects
@@
 			(project "VXDash"
 				(path "/f2858fc4-50de-4ff0-a01c-5b985ee14aef/f28d59c3-3184-4c96-b6c0-966ec9ca6979"
-					(reference "IC8")
+					(reference "IC3")
 					(unit 1)
 				)
@@
 		(dnp no)
 		(fields_autoplaced yes)
-		(property "Reference" "L3"
+		(property "Reference" "L2"
 			(at 142.24 76.2 0)
 			(effects
@@
 			(project "VXDash"
 				(path "/f2858fc4-50de-4ff0-a01c-5b985ee14aef/f28d59c3-3184-4c96-b6c0-966ec9ca6979"
-					(reference "L3")
+					(reference "L2")
 					(unit 1)
 				)
@@
 		(dnp no)
 		(fields_autoplaced yes)
-		(property "Reference" "C50"
+		(property "Reference" "C12"
 			(at 129.54 66.04 90)
 			(effects
@@
 			)
 		)
-		(property "Footprint" ""
+		(property "Footprint" "Capacitor_SMD:C_0603_1608Metric_Pad1.08x0.95mm_HandSolder"
 			(at 125.73 75.2348 0)
 			(effects
@@
 			(project "VXDash"
 				(path "/f2858fc4-50de-4ff0-a01c-5b985ee14aef/f28d59c3-3184-4c96-b6c0-966ec9ca6979"
-					(reference "C50")
+					(reference "C12")
 					(unit 1)
 				)
@@
 		(dnp no)
 		(fields_autoplaced yes)
-		(property "Reference" "R114"
+		(property "Reference" "R20"
 			(at 72.39 85.09 90)
 			(effects
@@
 			)
 		)
-		(property "Value" "180k"
+		(property "Value" "130k"
 			(at 72.39 87.63 90)
 			(effects
@@
 			(project "VXDash_RemoteECU"
 				(path "/f2858fc4-50de-4ff0-a01c-5b985ee14aef/f28d59c3-3184-4c96-b6c0-966ec9ca6979"
-					(reference "R114")
+					(reference "R20")
 					(unit 1)
 				)
@@
 		(dnp no)
 		(fields_autoplaced yes)
-		(property "Reference" "R99"
+		(property "Reference" "R23"
 			(at 151.13 96.5199 0)
 			(effects
@@
 			(project "VXDash"
 				(path "/f2858fc4-50de-4ff0-a01c-5b985ee14aef/f28d59c3-3184-4c96-b6c0-966ec9ca6979"
-					(reference "R99")
+					(reference "R23")
 					(unit 1)
 				)
@@
 		(on_board yes)
 		(dnp no)
-		(property "Reference" "C48"
+		(property "Reference" "C13"
 			(at 81.28 68.58 0)
 			(effects
@@
 			(project "VXDash"
 				(path "/f2858fc4-50de-4ff0-a01c-5b985ee14aef/f28d59c3-3184-4c96-b6c0-966ec9ca6979"
-					(reference "C48")
+					(reference "C13")
 					(unit 1)
 				)
@@
 		(on_board yes)
 		(dnp no)
-		(property "Reference" "R97"
+		(property "Reference" "R22"
 			(at 97.79 95.2499 0)
 			(effects
@@
 			)
 		)
-		(property "Value" "150k"
+		(property "Value" "100k"
 			(at 97.79 97.7899 0)
 			(effects
@@
 			(project "VXDash"
 				(path "/f2858fc4-50de-4ff0-a01c-5b985ee14aef/f28d59c3-3184-4c96-b6c0-966ec9ca6979"
-					(reference "R97")
+					(reference "R22")
 					(unit 1)
 				)
@@
 		(dnp no)
 		(fields_autoplaced yes)
-		(property "Reference" "R98"
+		(property "Reference" "R19"
 			(at 151.13 85.0899 0)
 			(effects
@@
 			(project "VXDash"
 				(path "/f2858fc4-50de-4ff0-a01c-5b985ee14aef/f28d59c3-3184-4c96-b6c0-966ec9ca6979"
-					(reference "R98")
+					(reference "R19")
 					(unit 1)
 				)
