File: KiCad PCB Files/VXDash_RemoteECU/AnalogV_Divider.kicad_sch (KiCad schematic)
At the start: 7 parts

Commit message: Started work on RemoteECU schematic
Parts:
- removed D1: 5.5V, Diode_SMD:D_SOD-323_HandSoldering, symbol VXDash_diodes:TVS_Uni
- removed R43: 100k, Resistor_SMD:R_0805_2012Metric_Pad1.20x1.40mm_HandSolder, symbol VXDash_passives:Res
- removed R44: 150k, Resistor_SMD:R_0805_2012Metric_Pad1.20x1.40mm_HandSolder, symbol VXDash_passives:Res
- added D1: BAV199, Package_TO_SOT_SMD:SOT-23-3, symbol Device:D_Schottky_Dual_Series_AKC_Split
Connections:
- net GND: now also D1.1 (A)
- net at R45.1: now also C22.2, R42.2, D1.3 (K), D1.3 (K)
- new net V_SUPPLY: D1.2 (K)
Other:
- moved on the sheet: C22, C23, R42, R45

Commit message: Initial work towards remote ECU functions
Parts:
- C24: renamed from C22; footprint (none) -> Capacitor_SMD:C_0603_1608Metric_Pad1.08x0.95mm_HandSolder
- C25: renamed from C23; footprint (none) -> Capacitor_SMD:C_0603_1608Metric_Pad1.08x0.95mm_HandSolder
- R44: renamed from R45; footprint Resistor_SMD:R_0805_2012Metric_Pad1.20x1.40mm_HandSolder -> Resistor_SMD:R_0603_1608Metric_Pad0.98x0.95mm_HandSolder
- renumbered D1 to D3, R42 to R43
Connections:
- net V_SUPPLY: now also D3.3 (K); no longer D3.2 (K)
- net at C24.2, D3.3 (K), R43.2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: now also D3.2 (K); no longer D3.3 (K)
Other:
- moved on the sheet: D3B
