File: KiCad PCB Files/VXDash_RemoteECU/Opto_4xactivelow.kicad_sch (KiCad schematic)
At the start: 9 parts, among them U1 LTV-847S

Commit message: Initial work towards remote ECU functions
Parts:
- R25: renamed from R?; footprint Resistor_SMD:R_0805_2012Metric_Pad1.20x1.40mm_HandSolder -> Resistor_SMD:R_0603_1608Metric_Pad0.98x0.95mm_HandSolder
- R27: renamed from R9; footprint Resistor_SMD:R_0805_2012Metric_Pad1.20x1.40mm_HandSolder -> Resistor_SMD:R_0603_1608Metric_Pad0.98x0.95mm_HandSolder
- R28: renamed from R11; footprint Resistor_SMD:R_0805_2012Metric_Pad1.20x1.40mm_HandSolder -> Resistor_SMD:R_0603_1608Metric_Pad0.98x0.95mm_HandSolder
- R29: renamed from R10; footprint Resistor_SMD:R_0603_1608Metric_Pad0.98x0.95mm_HandSolder -> Resistor_SMD:R_0805_2012Metric_Pad1.20x1.40mm_HandSolder
- R30: renamed from R13; footprint Resistor_SMD:R_0805_2012Metric_Pad1.20x1.40mm_HandSolder -> Resistor_SMD:R_0603_1608Metric_Pad0.98x0.95mm_HandSolder
- R31: renamed from R12; footprint Resistor_SMD:R_0603_1608Metric_Pad0.98x0.95mm_HandSolder -> Resistor_SMD:R_0805_2012Metric_Pad1.20x1.40mm_HandSolder
- gave numbers to parts that had none: 1
- renumbered R8 to R26, U1 to U2
Connections:
- net HL_Input1 is gone; now on net Protected_12V: R24.1
- net HL_Input2 is gone; now on net Protected_12V: R26.1
- net GND: no longer U2.2, U2.4
- net +3V3 renamed 3V3
- new net ~{HL_Input1}: U2.2
- new net ~{HL_Input2}: U2.4
