File: KiCad PCB Files/VXDash_RemoteECU/Power_Input.kicad_sch (KiCad schematic)
At the start: 9 parts

Commit message: Started work on RemoteECU schematic
Parts:
- removed C42, C43: 10u, Capacitor_SMD:C_1206_3216Metric_Pad1.33x1.80mm_HandSolder, symbol VXDash_passives:Cap_MLCC
- removed C44, C6: 100n, symbol VXDash_passives:Cap_MLCC
- removed D11: 18V, Diode_SMD:D_SOD-123, symbol Device:D_Zener
- removed FB1: 120R@100MHz, Inductor_SMD:L_0805_2012Metric, symbol Device:FerriteBead
- added C10, C8, C9: 1u, Capacitor_SMD:C_0805_2012Metric, symbol VXDash_passives:Cap_MLCC
- added R3, R4: 0R, Resistor_SMD:R_0805_2012Metric, symbol Device:R
- C6: value 10u -> 1u; footprint Capacitor_SMD:C_1206_3216Metric_Pad1.33x1.80mm_HandSolder -> Capacitor_SMD:C_0805_2012Metric; Voltage 25V -> 50V
Connections:
- net GND: now also C10.1, R4.1; no longer C6.2, F2.2, RV1.2
- net Power_Protected: now also C8.2, C9.2, R3.2
- new net: C8.1, C9.1, R4.2
- new net Power_Fused: C10.2, C6.2, F2.2, R3.1, RV1.2
Other:
- moved on the sheet: C6

Commit message: Initial work towards remote ECU functions
Parts:
- C15: renamed from C10; footprint Capacitor_SMD:C_0805_2012Metric -> Capacitor_SMD:C_0805_2012Metric_Pad1.18x1.45mm_HandSolder
- C16: renamed from C6; footprint Capacitor_SMD:C_0805_2012Metric -> Capacitor_SMD:C_0805_2012Metric_Pad1.18x1.45mm_HandSolder
- C17: renamed from C8; footprint Capacitor_SMD:C_0805_2012Metric -> Capacitor_SMD:C_0805_2012Metric_Pad1.18x1.45mm_HandSolder
- C18: renamed from C9; footprint Capacitor_SMD:C_0805_2012Metric -> Capacitor_SMD:C_0805_2012Metric_Pad1.18x1.45mm_HandSolder
- renumbered F2 to F1, R3 to R18, R4 to R21
Connections:
- net GND: now also C17.1, C18.1, R21.2; no longer C15.1, C16.1, R21.1, RV1.1
- new net Power_0V: C15.1, C16.1, R21.1, RV1.1
Changed lines of the file:
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@@
 	(title_block
 		(title "VXDash RemoteECU")
-		(date "2025-08-08")
+		(date "2026-01-25")
 		(rev "Proto A")
 		(company "Alex Miller & Martin Roger")
@@
 	(text "Voltage spike protection.\nAutomotive 12V supply can \nsee spikes >60V due to \nload-dump, etc.\n\nVaristor\n18V max working,\n24V max clamping \n250A."
 		(exclude_from_sim no)
-		(at 63.5 100.33 0)
+		(at 50.8 92.71 0)
 		(effects
 			(font
@@
 	)
 	(junction
-		(at 107.95 92.71)
+		(at 161.29 92.71)
 		(diameter 0)
 		(color 0 0 0 0)
@@
 	)
 	(junction
+		(at 107.95 92.71)
+		(diameter 0)
+		(color 0 0 0 0)
+	)
+	(junction
 		(at 132.08 92.71)
 		(diameter 0)
@@
 	(wire
 		(pts
-			(xy 107.95 92.71) (xy 107.95 93.98)
-		)
-		(stroke
-			(width 0)
-			(type default)
-		)
-	)
-	(wire
-		(pts
 			(xy 119.38 74.93) (xy 119.38 80.01)
 		)
@@
 	(wire
 		(pts
+			(xy 92.71 92.71) (xy 107.95 92.71)
+		)
+		(stroke
+			(width 0)
+			(type default)
+		)
+	)
+	(wire
+		(pts
 			(xy 161.29 87.63) (xy 161.29 92.71)
 		)
@@
 		(pts
 			(xy 119.38 87.63) (xy 119.38 92.71)
+		)
+		(stroke
+			(width 0)
+			(type default)
+		)
+	)
+	(wire
+		(pts
+			(xy 161.29 92.71) (xy 161.29 93.98)
 		)
 		(stroke
@@
 			)
 			(justify left bottom)
+		)
+	)
+	(hierarchical_label "Power_0V"
+		(shape input)
+		(at 92.71 92.71 180)
+		(effects
+			(font
+				(size 1.27 1.27)
+			)
+			(justify right)
 		)
 	)
@@
 		(dnp no)
 		(fields_autoplaced yes)
-		(property "Reference" "C10"
+		(property "Reference" "C15"
 			(at 115.57 81.2799 0)
 			(effects
@@
 			)
 		)
-		(property "Footprint" "Capacitor_SMD:C_0805_2012Metric"
+		(property "Footprint" "Capacitor_SMD:C_0805_2012Metric_Pad1.18x1.45mm_HandSolder"
 			(at 120.3452 80.01 0)
 			(effects
@@
 			(project "VXDash_RemoteECU"
 				(path "/f2858fc4-50de-4ff0-a01c-5b985ee14aef/c2d4aa4f-5950-4a72-b3dc-55b93ec0e74f"
-					(reference "C10")
+					(reference "C15")
 					(unit 1)
 				)
@@
 		(dnp no)
 		(fields_autoplaced yes)
-		(property "Reference" "C9"
+		(property "Reference" "C18"
 			(at 157.48 81.2799 0)
 			(effects
@@
 			)
 		)
-		(property "Footprint" "Capacitor_SMD:C_0805_2012Metric"
+		(property "Footprint" "Capacitor_SMD:C_0805_2012Metric_Pad1.18x1.45mm_HandSolder"
 			(at 162.2552 80.01 0)
 			(effects
@@
 			(project "VXDash_RemoteECU"
 				(path "/f2858fc4-50de-4ff0-a01c-5b985ee14aef/c2d4aa4f-5950-4a72-b3dc-55b93ec0e74f"
-					(reference "C9")
+					(reference "C18")
 					(unit 1)
 				)
@@
 	(symbol
 		(lib_id "power:GND")
-		(at 107.95 93.98 0)
+		(at 161.29 93.98 0)
 		(unit 1)
 		(exclude_from_sim no)
@@
 		(on_board yes)
 		(dnp no)
-		(property "Reference" "#PWR06"
-			(at 107.95 100.33 0)
+		(property "Reference" "#PWR015"
+			(at 161.29 100.33 0)
 			(effects
 				(font
@@
 		)
 		(property "Value" "GND"
-			(at 106.68 97.79 0)
+			(at 160.02 97.79 0)
 			(effects
 				(font
@@
 		)
 		(property "Footprint" ""
-			(at 107.95 93.98 0)
+			(at 161.29 93.98 0)
 			(effects
 				(font
@@
 		)
 		(property "Datasheet" ""
-			(at 107.95 93.98 0)
+			(at 161.29 93.98 0)
 			(effects
 				(font
@@
 		)
 		(property "Description" "Power symbol creates a global label with name \"GND\" , ground"
-			(at 107.95 93.98 0)
+			(at 161.29 93.98 0)
 			(effects
 				(font
@@
 			(project "DashSpy"
 				(path "/f2858fc4-50de-4ff0-a01c-5b985ee14aef/c2d4aa4f-5950-4a72-b3dc-55b93ec0e74f"
-					(reference "#PWR06")
+					(reference "#PWR015")
 					(unit 1)
 				)
@@
 		(dnp no)
 		(fields_autoplaced yes)
-		(property "Reference" "R3"
+		(property "Reference" "R18"
 			(at 138.43 68.58 90)
 			(effects
@@
 			(project ""
 				(path "/f2858fc4-50de-4ff0-a01c-5b985ee14aef/c2d4aa4f-5950-4a72-b3dc-55b93ec0e74f"
-					(reference "R3")
+					(reference "R18")
 					(unit 1)
 				)
@@
 		(dnp no)
 		(fields_autoplaced yes)
-		(property "Reference" "C8"
+		(property "Reference" "C17"
 			(at 146.05 81.2799 0)
 			(effects
@@
 			)
 		)
-		(property "Footprint" "Capacitor_SMD:C_0805_2012Metric"
+		(property "Footprint" "Capacitor_SMD:C_0805_2012Metric_Pad1.18x1.45mm_HandSolder"
 			(at 150.8252 80.01 0)
 			(effects
@@
 			(project "VXDash_RemoteECU"
 				(path "/f2858fc4-50de-4ff0-a01c-5b985ee14aef/c2d4aa4f-5950-4a72-b3dc-55b93ec0e74f"
-					(reference "C8")
+					(reference "C17")
 					(unit 1)
 				)
@@
 		(dnp no)
 		(fields_autoplaced yes)
-		(property "Reference" "R4"
+		(property "Reference" "R21"
 			(at 138.43 86.36 90)
 			(effects
@@
 			(project "VXDash_RemoteECU"
 				(path "/f2858fc4-50de-4ff0-a01c-5b985ee14aef/c2d4aa4f-5950-4a72-b3dc-55b93ec0e74f"
-					(reference "R4")
+					(reference "R21")
 					(unit 1)
 				)
@@
 		(dnp no)
 		(fields_autoplaced yes)
-		(property "Reference" "F2"
+		(property "Reference" "F1"
 			(at 99.06 69.85 90)
 			(effects
@@
 			(project "VXDash"
 				(path "/f2858fc4-50de-4ff0-a01c-5b985ee14aef/c2d4aa4f-5950-4a72-b3dc-55b93ec0e74f"
-					(reference "F2")
+					(reference "F1")
 					(unit 1)
 				)
@@
 		(dnp no)
 		(fields_autoplaced yes)
-		(property "Reference" "C6"
+		(property "Reference" "C16"
 			(at 128.27 81.2799 0)
 			(effects
@@
 			)
 		)
-		(property "Footprint" "Capacitor_SMD:C_0805_2012Metric"
+		(property "Footprint" "Capacitor_SMD:C_0805_2012Metric_Pad1.18x1.45mm_HandSolder"
 			(at 133.0452 80.01 0)
 			(effects
@@
 			(project "DashSpy"
 				(path "/f2858fc4-50de-4ff0-a01c-5b985ee14aef/c2d4aa4f-5950-4a72-b3dc-55b93ec0e74f"
-					(reference "C6")
+					(reference "C16")
 					(unit 1)
 				)
