File: KiCad PCB Files/VXDash_RemoteECU/USBC.kicad_sch (KiCad schematic)
At the start: 7 parts, among them J5 USB4105-GF-A

Commit message: Initial work towards remote ECU functions
Parts:
- removed C12: 10u, Capacitor_SMD:C_0603_1608Metric, symbol VXDash_passives:Cap_MLCC
- removed D10: 1N5819HW-7-F, Diode_SMD:D_SOD-123, symbol VXDash_diodes:1N5819HW-7-F
- removed R71: 0, symbol VXDash_passives:Res
- J12: renamed from J5; footprint DIY:GCT_USB4105-GF-A -> VXDash_connectors:GCT_USB4105-GF-A; MANUFACTURER GCT -> (none); MAXIMUM_PACKAGE_HEIGHT 3.31 mm -> (none); Manufacturer_Name GCT -> (none); Manufacturer_Part_Number USB4105-GF-A -> (none); PARTREV B4 -> (none); STANDARD Manufacturer Recommendations -> (none); Type SMD -> (none)
- R40: renamed from R72; footprint (none) -> Resistor_SMD:R_0603_1608Metric_Pad0.98x0.95mm_HandSolder
- R41: renamed from R73; footprint (none) -> Resistor_SMD:R_0603_1608Metric_Pad0.98x0.95mm_HandSolder
- renumbered D7 to D2
Connections:
- net GND: now also J12.SH1 (SHELL_GND), J12.SH2 (SHELL_GND__1), J12.SH3 (SHELL_GND__2), J12.SH4 (SHELL_GND__3)
Other:
- company: Martin Roger -> (none)
- title: A1S Mini Board -> (none)
- moved on the sheet: D2, J12, R40, R41
