File: KiCad PCB Files/VXDash_RemoteECU/VXDash_RemoteECU.kicad_pcb (KiCad board)
At the start: 2 copper layers, 115 x 95 mm, 370 parts, among them IC1 CD74HC4050M96, IC10 ATA6561, IC2 74HC4067BQ-Q100J, IC2 SP721ABG, IC3 AP62200, IC4 AP62200, IC4 MP2322GQH-Z, IC5 AD8542ARMZ-REEL, IC5 AS2333_OpAmp, IC6 AD8542ARMZ-REEL, IC6 AS2333_OpAmp, IC7 AD8542ARMZ-REEL, IC7 AS2333_OpAmp, IC8 AP62200, IC9 AS2333_OpAmp, J1 Conn_02x10_Odd_Even, J1 MX34036UF2, J2 Conn_01x04_Socket, J2 Expansion, Q1 DMP3099L, Q10 DMP3099L, Q11 DMP3099L, Q12 DMP3099L, Q13 DMP3099L, Q14 DMP3099L, Q15 DMP3099L, Q2 DMP3099L, Q3 DMG2301L, Q3 DMP3099L, Q4 DMG2301L, Q4 DMP3099L, Q5 2N7002, Q5 DMG2301L, Q6 DMG2301L, Q6 PJA3441, Q7 DMG2301L, Q7 PJA3441, Q8 DMG2301L, Q8 DMP3099L, Q9 DMP3099L, U10 SFH617A-2X009T, U11 SFH617A-2X009T, U12 SFH617A-2X009T, U13 SFH617A-2X009T, U15 SFH617A-2X009T, U16 ESP32-DevKitC, U16 ESP32-S3-WROOM-1, U17 ADS1115IDGS, U18 ADS1115IDGS, U19 ADS1115IDGS, U2 SFH617A-2X009T, U3 SFH617A-2X009T, U4 SFH617A-2X009T, U5 SFH617A-2X009T, U6 SFH617A-2X009T, U7 SFH617A-2X009T, U8 SFH617A-2X009T, U9 SFH617A-2X009T

Commit message: Initial work towards remote ECU functions
Parts:
- removed the C10 at (59.4, 50.3)
- removed the C10 at (201.8, 65.8)
- removed the C12 at (53.9, 58.9)
- removed the C12 at (192.8, 66.0)
- removed the C13 at (153.9, 75.9)
- removed the C13 at (53.9, 62.2)
- removed the C14 at (167.4, 75.9)
- removed the C14 at (-4.33, 118.9)
- removed the C17 at (4.64, 118.2)
- removed the C17 at (201.2, 52.1)
- removed the C19 at (-4.33, 122.3)
- removed the C19 at (192.0, 54.4)
- removed the C20 at (-4.33, 125.6)
- removed the C20 at (199.6, 50.5)
- removed C22: 22pF, Capacitor_SMD:C_0402_1005Metric
- removed the C31 at (140.5, 80.4)
- removed the C31 at (6.54, 98.1)
- removed the C36 at (200.7, 80.4)
- removed the C36 at (37.7, 50.5)
- removed C38, C46, C47, C56, C57: 33n, Capacitor_SMD:C_0603_1608Metric_Pad1.08x0.95mm_HandSolder
- removed the C40 at (162.6, 80.8)
- removed the C40 at (209.5, 97.7)
- removed the C41 at (200.7, 87.8)
- removed the C41 at (149.1, 80.8)
- removed the C42 at (181.1, 75.9)
- removed the C42 at (53.6, 124.3)
- removed the C43 at (53.6, 127.6)
- removed the C43 at (139.2, 65.3)
- removed C45, C55: 100n, Capacitor_SMD:C_0603_1608Metric_Pad1.08x0.95mm_HandSolder
- removed C45, C46, C47, C48, C49, C50, C51, C52: 0.1uF 50V, Capacitor_SMD:C_0603_1608Metric
- removed C48: 10u, Capacitor_SMD:C_1206_3216Metric_Pad1.33x1.80mm_HandSolder
- removed the C5 at (197.4, 66.0)
- removed the C5 at (118.9, 89.9)
- removed C51: 22p, Capacitor_SMD:C_0402_1005Metric_Pad0.74x0.62mm_HandSolder
- removed C53, C54, C60: 22u, Capacitor_SMD:C_1206_3216Metric_Pad1.33x1.80mm_HandSolder
- removed the C6 at (122.2, 88.9)
- removed the C6 at (204.6, 74.0)
- removed the C7 at (195.1, 66.0)
- removed the C7 at (53.9, 55.5)
- removed D1: 5.5V, Diode_SMD:D_SOD-323_HandSoldering
- removed D15, D16, D17, D18, D19: BAT54, Diode_SMD:D_SOD-123
- removed the D2 at (143.4, 88.1)
- removed the D2 at (57.9, 95.0)
- removed the D3 at (2.54, 95.2)
- removed the D3 at (157.0, 88.1)
- removed the D4 at (57.9, 109.5)
- removed the D4 at (167.2, 88.1)
- removed the D5 at (57.9, 138.6)
- removed the D5 at (170.4, 88.1)
- removed the D6 at (32.6, 51.0)
- removed the D6 at (180.6, 88.1)
- removed the D9 at (153.6, 88.1)
- removed the D9 at (32.6, 61.0)
- removed FB1: 120R@100MHz, Inductor_SMD:L_0805_2012Metric
- removed IC10: ATA6561, Package_SO:SOIC-8_3.9x4.9mm_P1.27mm
- removed the IC2 at (152.1, 128.4)
- removed the IC2 at (119.5, 76.7)
- removed the IC4 at (199.0, 52.9)
- removed the IC4 at (4.70, 113.0)
- removed IC5: AD8542ARMZ-REEL, DIY:SOP65P490X110-8N
- removed IC5, IC9: AS2333_OpAmp, Package_SO:MSOP-8_3x3mm_P0.65mm
- removed the IC6 at (39.2, 68.8)
- removed the IC6 at (162.1, 77.0)
- removed the IC7 at (-13.0, 108.4)
- removed the IC7 at (175.5, 77.0)
- removed IC8: AP62200, Package_TO_SOT_SMD:TSOT-23-6_HandSoldering
- removed the J1 at (15.6, 95.9)
- removed the J1 at (170.1, 97.4)
- removed the J2 at (115.6, 55.3)
- removed the J2 at (18.0, 51.6)
- removed the L2 at (196.8, 55.9)
- removed the L2 at (-3.06, 114.0)
- removed MTH1, MTH2, MTH3, MTH4, MTH5, MTH6: MountingHole_3.5mm_Pad_Via, MountingHole:MountingHole_3.5mm_Pad_Via
- removed PS1: AP63200WU-7, DIY:SOT95P280X100-6N
- removed Q10, Q11, Q12, Q13, Q14, Q15, Q9: DMP3099L, Package_TO_SOT_SMD:SOT-23
- removed the Q3 at (157.7, 81.3)
- removed the Q3 at (27.3, 60.9)
- removed the Q4 at (166.4, 81.3)
- removed the Q4 at (27.3, 65.6)
- removed the Q5 at (205.0, 97.5)
- removed the Q5 at (171.2, 81.3)
- removed the Q6 at (59.1, 125.0)
- removed the Q6 at (179.8, 81.3)
- removed the Q7 at (144.3, 81.3)
- removed the Q7 at (202.9, 90.4)
- removed the Q8 at (152.9, 81.3)
- removed the Q8 at (-30.9, 95.9)
- removed the R1 at (20.0, 94.8)
- removed the R1 at (207.9, 67.1)
- removed the R10 at (39.8, 148.2)
- removed the R10 at (152.5, 106.0)
- removed R100, R101, R107, R108, R89, R90, R96: 1k, Resistor_SMD:R_0603_1608Metric_Pad0.98x0.95mm_HandSolder
- removed R102, R109, R91: 18R, Resistor_SMD:R_0603_1608Metric_Pad0.98x0.95mm_HandSolder
- removed R103, R110, R92: 0R, Resistor_SMD:R_0603_1608Metric_Pad0.98x0.95mm_HandSolder
- removed R104, R111, R86, R93: 1k, Resistor_SMD:R_1206_3216Metric_Pad1.30x1.75mm_HandSolder
- removed R105, R112, R87, R94: 160R, Resistor_SMD:R_0603_1608Metric_Pad0.98x0.95mm_HandSolder
- removed R106, R113, R88, R95: 6R8, Resistor_SMD:R_0603_1608Metric_Pad0.98x0.95mm_HandSolder
- removed the R11 at (26.6, 101.6)
- removed the R11 at (152.5, 121.2)
- removed R114, R115: 60R, Resistor_SMD:R_0805_2012Metric_Pad1.20x1.40mm_HandSolder
- removed the R12 at (146.2, 106.0)
- removed the R12 at (26.6, 104.6)
- removed the R13 at (146.2, 121.2)
- removed the R13 at (39.8, 130.7)
- removed the R14 at (39.8, 133.7)
- removed the R14 at (139.8, 106.0)
- removed the R15 at (26.6, 130.7)
- removed the R15 at (139.8, 121.2)
- removed the R16 at (133.5, 106.0)
- removed the R16 at (26.6, 133.7)
- removed the R17 at (13.1, 131.1)
- removed the R17 at (133.5, 121.2)
- removed the R18 at (127.1, 106.0)
- removed the R18 at (13.1, 134.0)
- removed the R19 at (127.1, 121.2)
- removed the R19 at (26.6, 116.2)
- removed the R2 at (20.0, 97.3)
- removed the R2 at (207.4, 68.7)
- removed the R20 at (26.6, 119.1)
- removed the R20 at (120.8, 106.0)
- removed the R21 at (120.8, 121.2)
- removed the R21 at (40.4, 81.1)
- removed the R22 at (114.4, 106.0)
- removed the R22 at (40.4, 84.1)
- removed the R23 at (114.4, 121.2)
- removed the R23 at (39.8, 101.6)
- removed the R24 at (39.8, 104.6)
- removed the R24 at (108.1, 106.0)
- removed the R25 at (108.1, 121.2)
- removed the R25 at (27.2, 81.1)
- removed the R26 at (27.2, 84.1)
- removed the R26 at (197.0, 105.8)
- removed the R27 at (197.0, 121.4)
- removed the R27 at (26.6, 145.2)
- removed the R28 at (184.3, 105.8)
- removed the R28 at (26.6, 148.2)
- removed the R29 at (184.3, 121.4)
- removed the R29 at (-4.96, 137.4)
- removed the R3 at (59.0, 55.1)
- removed the R3 at (201.8, 68.3)
- removed the R30 at (-4.96, 140.3)
- removed the R30 at (177.9, 105.8)
- removed the R31 at (39.8, 116.2)
- removed the R31 at (177.9, 121.4)
- removed the R34 at (190.6, 105.8)
- removed the R34 at (171.6, 121.4)
- removed the R35 at (-31.0, 144.0)
- removed the R35 at (190.6, 121.4)
- removed the R37 at (0.85, 118.5)
- removed the R37 at (198.1, 50.5)
- removed the R38 at (195.8, 51.1)
- removed the R38 at (0.85, 121.0)
- removed the R39 at (190.0, 55.4)
- removed the R39 at (0.85, 123.5)
- removed the R4 at (200.8, 68.3)
- removed the R4 at (59.0, 57.6)
- removed the R40 at (0.85, 126.0)
- removed the R40 at (127.1, 77.3)
- removed the R41 at (17.8, 72.9)
- removed the R41 at (127.1, 74.0)
- removed R42: 1K, Resistor_SMD:R_0805_2012Metric
- removed R42: 10R, Resistor_SMD:R_0805_2012Metric_Pad1.20x1.40mm_HandSolder
- removed the R43 at (131.6, 74.0)
- removed the R43 at (13.1, 141.9)
- removed the R44 at (13.1, 144.9)
- removed the R44 at (136.0, 77.3)
- removed the R45 at (136.0, 74.0)
- removed the R45 at (13.1, 147.8)
- removed the R46 at (140.5, 77.3)
- removed the R46 at (53.0, 95.0)
- removed the R47 at (53.0, 98.0)
- removed the R47 at (140.5, 74.0)
- removed the R48 at (53.0, 100.9)
- removed the R48 at (162.6, 73.2)
- removed the R49 at (147.6, 73.2)
- removed the R49 at (53.0, 103.9)
- removed the R5 at (59.0, 60.1)
- removed the R5 at (191.8, 62.9)
- removed the R50 at (150.6, 73.2)
- removed the R50 at (1.99, 98.4)
- removed the R51 at (1.99, 101.3)
- removed the R51 at (158.5, 84.6)
- removed the R52 at (1.99, 104.3)
- removed the R52 at (161.0, 73.2)
- removed the R53 at (165.6, 84.6)
- removed the R53 at (1.99, 107.2)
- removed the R54 at (159.3, 87.4)
- removed the R54 at (6.54, 100.7)
- removed the R55 at (164.9, 87.4)
- removed the R55 at (6.54, 103.2)
- removed the R56 at (53.0, 109.5)
- removed the R56 at (176.0, 73.2)
- removed the R57 at (161.0, 80.8)
- removed the R57 at (53.0, 112.5)
- removed the R58 at (53.0, 115.4)
- removed the R58 at (147.6, 80.8)
- removed the R59 at (53.0, 118.4)
- removed the R59 at (174.5, 80.8)
- removed the R60 at (53.0, 138.6)
- removed the R60 at (164.1, 73.1)
- removed the R61 at (172.0, 84.6)
- removed the R61 at (53.0, 141.6)
- removed the R66 at (179.1, 84.6)
- removed the R66 at (42.0, 50.5)
- removed the R67 at (172.7, 87.4)
- removed the R67 at (42.0, 53.1)
- removed the R68 at (45.9, 63.5)
- removed the R68 at (178.3, 87.4)
- removed the R69 at (42.0, 55.6)
- removed the R69 at (174.5, 73.2)
- removed the R70 at (42.0, 58.1)
- removed the R70 at (177.5, 73.2)
- removed the R72 at (149.1, 73.2)
- removed the R72 at (46.4, 50.5)
- removed the R73 at (144.8, 84.6)
- removed the R73 at (46.4, 53.1)
- removed the R74 at (145.7, 87.4)
- removed the R74 at (46.4, 55.6)
- removed the R75 at (45.9, 66.8)
- removed the R75 at (152.1, 84.6)
- removed the R76 at (151.4, 87.4)
- removed the R76 at (46.4, 58.1)
- removed the R8 at (158.9, 106.0)
- removed the R8 at (165.2, 121.2)
- removed the R9 at (158.9, 121.2)
- removed the R9 at (39.8, 145.2)
- removed R97: 100k, Resistor_SMD:R_0603_1608Metric_Pad0.98x0.95mm_HandSolder
- removed R98: 43k, Resistor_SMD:R_0603_1608Metric_Pad0.98x0.95mm_HandSolder
- removed R99: 8k2, Resistor_SMD:R_0603_1608Metric_Pad0.98x0.95mm_HandSolder
- removed U10, U11, U12, U13, U14, U15, U7, U8, U9: ~, Package_DIP:SMDIP-4_W7.62mm
- removed U10, U11, U12, U13, U15, U7, U8, U9: SFH617A-2X009T, Package_DIP:SMDIP-4_W7.62mm
- removed U16: ESP32-S3-WROOM-1, RF_Module:ESP32-S3-WROOM-1
- removed U16: ESP32-DevKitC, PCM_Espressif:ESP32-DevKitC
- removed U17, U18, U19: ADS1115IDGS, Package_SO:TSSOP-10_3x3mm_P0.5mm
- removed the U2 at (43.0, 140.4)
- removed the U2 at (157.6, 113.6)
- removed the U3 at (151.3, 113.6)
- removed the U3 at (29.8, 96.9)
- removed the U4 at (144.9, 113.6)
- removed the U4 at (43.0, 125.9)
- removed the U5 at (29.8, 125.9)
- removed the U5 at (138.6, 113.6)
- removed the U6 at (16.3, 126.3)
- removed the U6 at (132.2, 113.6)
- added C10: 22u, Capacitor_SMD:C_1206_3216Metric_Pad1.33x1.80mm_HandSolder, B.Cu at (170.8, 85.5)
- added C12: 100n, Capacitor_SMD:C_0603_1608Metric_Pad1.08x0.95mm_HandSolder, B.Cu at (143.6, 86.0)
- added C13: 10u, Capacitor_SMD:C_1206_3216Metric_Pad1.33x1.80mm_HandSolder, B.Cu at (153.4, 92.3)
- added C14: 10u, Capacitor_SMD:C_1206_3216Metric_Pad1.33x1.80mm_HandSolder, B.Cu at (153.4, 89.8)
- added C17: 1u, Capacitor_SMD:C_0805_2012Metric_Pad1.18x1.45mm_HandSolder, F.Cu at (137.6, 97.0)
- added C19: 22p, Capacitor_SMD:C_0603_1608Metric_Pad1.08x0.95mm_HandSolder, B.Cu at (146.4, 92.3)
- added C20: 22u, Capacitor_SMD:C_1206_3216Metric_Pad1.33x1.80mm_HandSolder, B.Cu at (156.6, 85.5)
- added C31: 100n, Capacitor_SMD:C_0603_1608Metric_Pad1.08x0.95mm_HandSolder, B.Cu at (169.5, 44.8)
- added C33: 100n, Capacitor_SMD:C_0603_1608Metric_Pad1.08x0.95mm_HandSolder, B.Cu at (174.5, 44.8)
- added C34: 10n, Capacitor_SMD:C_0603_1608Metric_Pad1.08x0.95mm_HandSolder, B.Cu at (173.0, 55.8)
- added C36: 33n, Capacitor_SMD:C_0603_1608Metric_Pad1.08x0.95mm_HandSolder, B.Cu at (207.0, 59.0)
- added C40: 33n, Capacitor_SMD:C_0603_1608Metric_Pad1.08x0.95mm_HandSolder, B.Cu at (206.5, 49.0)
- added C41: 1u, Capacitor_SMD:C_0603_1608Metric_Pad1.08x0.95mm_HandSolder, B.Cu at (149.7, 102.0)
- added C42: 1u, Capacitor_SMD:C_0603_1608Metric_Pad1.08x0.95mm_HandSolder, B.Cu at (159.8, 98.8)
- added C43: 1u, Capacitor_SMD:C_0603_1608Metric_Pad1.08x0.95mm_HandSolder, B.Cu at (161.2, 98.8)
- added C5: 100n, Capacitor_SMD:C_0603_1608Metric_Pad1.08x0.95mm_HandSolder, B.Cu at (160.8, 86.0)
- added C6: 10u, Capacitor_SMD:C_1206_3216Metric_Pad1.33x1.80mm_HandSolder, B.Cu at (170.6, 89.8)
- added C7: 10u, Capacitor_SMD:C_1206_3216Metric_Pad1.33x1.80mm_HandSolder, B.Cu at (170.6, 92.2)
- added D2: SP0503BAHTG, Package_TO_SOT_SMD:SOT-143, F.Cu at (206.6, 121.8)
- added D3: BAV199, Package_TO_SOT_SMD:SOT-23-3, B.Cu at (160.2, 47.8)
- added D4: BAV199, Package_TO_SOT_SMD:SOT-23-3, B.Cu at (165.2, 47.8)
- added D5: BAV199, Package_TO_SOT_SMD:SOT-23-3, B.Cu at (170.2, 47.8)
- added D6: BAV199, Package_TO_SOT_SMD:SOT-23-3, B.Cu at (175.2, 47.8)
- added D9: BAT54, Diode_SMD:D_SOD-123, B.Cu at (188.0, 42.5)
- added F3: Mini blade 1A, Fuse:Fuseholder_Blade_Mini_Keystone_3568, F.Cu at (192.8, 116.0)
- added F4: Mini blade 1A, Fuse:Fuseholder_Blade_Mini_Keystone_3568, F.Cu at (185.6, 116.0)
- added F5: Mini blade 1A, Fuse:Fuseholder_Blade_Mini_Keystone_3568, F.Cu at (178.3, 116.0)
- added IC2: AP62200, Package_TO_SOT_SMD:TSOT-23-6_HandSoldering, B.Cu at (164.8, 88.2)
- added IC4: AS2333_OpAmp, Package_SO:MSOP-8_3x3mm_P0.65mm, B.Cu at (185.0, 67.6)
- added IC6: AS2333_OpAmp, Package_SO:MSOP-8_3x3mm_P0.65mm, B.Cu at (197.2, 67.5)
- added IC7: ATA6561, Package_SO:SOIC-8_3.9x4.9mm_P1.27mm, B.Cu at (151.2, 98.2)
- added J1: UART0 debug, Connector_PinHeader_2.54mm:PinHeader_1x04_P2.54mm_Vertical, F.Cu at (208.2, 64.2)
- added J10: Analogue_R, VXDash_connectors:QT04ASFxxH, F.Cu at (190.8, 39.2)
- added J11: PWM inputs, VXDash_connectors:QT04ASFxxH, F.Cu at (168.5, 129.2)
- added J12: USB4105-GF-A, VXDash_connectors:GCT_USB4105-GF-A, F.Cu at (214.8, 121.8)
- added J2: CANbus IN, VXDash_connectors:DT13-4P_TE_Deutsch, F.Cu at (122.5, 84.2)
- added J3: I²C debug, Connector_PinHeader_2.54mm:PinHeader_1x03_P2.54mm_Vertical, F.Cu at (208.5, 108.0)
- added J4: Outputs, VXDash_connectors:QT04ASFxxH, F.Cu at (191.0, 129.2)
- added J5: Digital ActiveLows, VXDash_connectors:QT04ASFxxH, F.Cu at (123.5, 129.2)
- added J6: Digital ActiveHighs, VXDash_connectors:QT04ASFxxH, F.Cu at (146.0, 129.2)
- added J7: Sensor 5V, VXDash_connectors:QT04ASFxxH, F.Cu at (145.8, 39.2)
- added J8: Sensor 0V, VXDash_connectors:QT04ASFxxH, F.Cu at (123.2, 39.2)
- added J9: Analogue_V, VXDash_connectors:QT04ASFxxH, F.Cu at (168.2, 39.2)
- added L2: 4u7, VXDash_inductors:Ind_5050, B.Cu at (148.6, 83.3)
- added Q3: DMP3099L, Package_TO_SOT_SMD:SOT-23, B.Cu at (182.0, 47.0)
- added Q4: DMP3099L, Package_TO_SOT_SMD:SOT-23, B.Cu at (188.0, 47.0)
- added Q5: DMP3099L, Package_TO_SOT_SMD:SOT-23, B.Cu at (194.8, 59.5)
- added Q6: DMP3099L, Package_TO_SOT_SMD:SOT-23, B.Cu at (200.8, 59.5)
- added Q7: DMP3099L, Package_TO_SOT_SMD:SOT-23, B.Cu at (194.0, 47.0)
- added Q8: DMP3099L, Package_TO_SOT_SMD:SOT-23, B.Cu at (200.0, 47.0)
- added R1: 10k, Resistor_SMD:R_0603_1608Metric_Pad0.98x0.95mm_HandSolder, B.Cu at (123.2, 56.0)
- added R10: R, Resistor_SMD:R_0603_1608Metric, B.Cu at (152.8, 42.3)
- added R11: 100R, Resistor_SMD:R_0603_1608Metric_Pad0.98x0.95mm_HandSolder, B.Cu at (168.2, 111.0)
- added R12: 100R, Resistor_SMD:R_0603_1608Metric_Pad0.98x0.95mm_HandSolder, B.Cu at (168.2, 113.5)
- added R13: 100R, Resistor_SMD:R_0603_1608Metric_Pad0.98x0.95mm_HandSolder, B.Cu at (168.2, 116.0)
- added R14: 820k, Resistor_SMD:R_0603_1608Metric_Pad0.98x0.95mm_HandSolder, B.Cu at (160.8, 89.5)
- added R15: 75k, Resistor_SMD:R_0603_1608Metric_Pad0.98x0.95mm_HandSolder, B.Cu at (163.6, 93.8)
- added R16: 120k, Resistor_SMD:R_0603_1608Metric_Pad0.98x0.95mm_HandSolder, B.Cu at (159.3, 89.5)
- added R17: 24k, Resistor_SMD:R_0603_1608Metric_Pad0.98x0.95mm_HandSolder, B.Cu at (163.6, 90.8)
- added R18: 0R, Resistor_SMD:R_0805_2012Metric, F.Cu at (138.8, 94.0)
- added R19: 43k, Resistor_SMD:R_0603_1608Metric_Pad0.98x0.95mm_HandSolder, B.Cu at (146.4, 93.8)
- added R2: 1k, Resistor_SMD:R_0603_1608Metric_Pad0.98x0.95mm_HandSolder, B.Cu at (123.2, 104.8)
- added R20: 130k, Resistor_SMD:R_0603_1608Metric_Pad0.98x0.95mm_HandSolder, B.Cu at (142.1, 89.5)
- added R21: 0R, Resistor_SMD:R_0805_2012Metric, F.Cu at (136.3, 94.0)
- added R22: 100k, Resistor_SMD:R_0603_1608Metric_Pad0.98x0.95mm_HandSolder, B.Cu at (143.6, 89.5)
- added R23: 8k2, Resistor_SMD:R_0603_1608Metric_Pad0.98x0.95mm_HandSolder, B.Cu at (146.4, 90.8)
- added R24: 8k2, Resistor_SMD:R_0805_2012Metric_Pad1.20x1.40mm_HandSolder, F.Cu at (132.8, 117.2)
- added R25: 10k, Resistor_SMD:R_0603_1608Metric_Pad0.98x0.95mm_HandSolder, B.Cu at (202.8, 98.8)
- added R26: 8k2, Resistor_SMD:R_0805_2012Metric_Pad1.20x1.40mm_HandSolder, F.Cu at (127.8, 117.2)
- added R27: 10k, Resistor_SMD:R_0603_1608Metric_Pad0.98x0.95mm_HandSolder, B.Cu at (201.2, 98.8)
- added R28: 10k, Resistor_SMD:R_0603_1608Metric_Pad0.98x0.95mm_HandSolder, B.Cu at (199.8, 98.8)
- added R29: 8k2, Resistor_SMD:R_0805_2012Metric_Pad1.20x1.40mm_HandSolder, F.Cu at (122.5, 117.2)
- added R3: 1k, Resistor_SMD:R_0603_1608Metric_Pad0.98x0.95mm_HandSolder, B.Cu at (205.4, 99.5)
- added R30: 10k, Resistor_SMD:R_0603_1608Metric_Pad0.98x0.95mm_HandSolder, B.Cu at (198.2, 98.8)
- added R31: 8k2, Resistor_SMD:R_0805_2012Metric_Pad1.20x1.40mm_HandSolder, F.Cu at (117.8, 117.2)
- added R34: 8k2, Resistor_SMD:R_0805_2012Metric_Pad1.20x1.40mm_HandSolder, B.Cu at (149.0, 126.2)
- added R35: 10k, Resistor_SMD:R_0603_1608Metric_Pad0.98x0.95mm_HandSolder, B.Cu at (200.8, 74.0)
- added R37: 10k, Resistor_SMD:R_0603_1608Metric_Pad0.98x0.95mm_HandSolder, B.Cu at (202.2, 74.0)
- added R38: 8k2, Resistor_SMD:R_0805_2012Metric_Pad1.20x1.40mm_HandSolder, B.Cu at (139.0, 126.2)
- added R39: 10k, Resistor_SMD:R_0603_1608Metric_Pad0.98x0.95mm_HandSolder, B.Cu at (203.8, 74.0)
- added R4: 0R, Resistor_SMD:R_0805_2012Metric_Pad1.20x1.40mm_HandSolder, B.Cu at (208.1, 97.8)
- added R40: 5.1K, Resistor_SMD:R_0603_1608Metric_Pad0.98x0.95mm_HandSolder, B.Cu at (213.6, 123.1)
- added R41: 5.1K, Resistor_SMD:R_0603_1608Metric_Pad0.98x0.95mm_HandSolder, B.Cu at (213.6, 120.1)
- added R43: 10R, Resistor_SMD:R_0805_2012Metric_Pad1.20x1.40mm_HandSolder, B.Cu at (160.2, 42.0)
- added R44: 1K, Resistor_SMD:R_0603_1608Metric_Pad0.98x0.95mm_HandSolder, B.Cu at (163.0, 53.8)
- added R45: 10R, Resistor_SMD:R_0805_2012Metric_Pad1.20x1.40mm_HandSolder, B.Cu at (165.2, 42.0)
- added R46: 1K, Resistor_SMD:R_0603_1608Metric_Pad0.98x0.95mm_HandSolder, B.Cu at (165.2, 51.8)
- added R47: 39k, Resistor_SMD:R_0603_1608Metric_Pad0.98x0.95mm_HandSolder, B.Cu at (176.5, 67.8)
- added R48: 820k, Resistor_SMD:R_0603_1608Metric_Pad0.98x0.95mm_HandSolder, B.Cu at (180.5, 67.0)
- added R49: 10R, Resistor_SMD:R_0805_2012Metric_Pad1.20x1.40mm_HandSolder, B.Cu at (170.2, 42.0)
- added R5: 4k7, Resistor_SMD:R_0603_1608Metric_Pad0.98x0.95mm_HandSolder, F.Cu at (204.2, 92.2)
- added R50: 1K, Resistor_SMD:R_0603_1608Metric_Pad0.98x0.95mm_HandSolder, B.Cu at (170.2, 51.8)
- added R51: 10R, Resistor_SMD:R_0805_2012Metric_Pad1.20x1.40mm_HandSolder, B.Cu at (175.2, 42.0)
- added R52: 1K, Resistor_SMD:R_0603_1608Metric_Pad0.98x0.95mm_HandSolder, B.Cu at (173.0, 54.0)
- added R53: 18R, Resistor_SMD:R_0603_1608Metric_Pad0.98x0.95mm_HandSolder, B.Cu at (180.8, 62.2)
- added R54: 160R, Resistor_SMD:R_0603_1608Metric_Pad0.98x0.95mm_HandSolder, B.Cu at (179.8, 59.5)
- added R55: 18R, Resistor_SMD:R_0603_1608Metric_Pad0.98x0.95mm_HandSolder, B.Cu at (186.8, 62.2)
- added R56: 160R, Resistor_SMD:R_0603_1608Metric_Pad0.98x0.95mm_HandSolder, B.Cu at (185.8, 59.5)
- added R57: 6R8, Resistor_SMD:R_0603_1608Metric_Pad0.98x0.95mm_HandSolder, B.Cu at (186.8, 56.8)
- added R58: 1k, Resistor_SMD:R_0603_1608Metric_Pad0.98x0.95mm_HandSolder, B.Cu at (183.2, 63.2)
- added R59: 6R8, Resistor_SMD:R_0603_1608Metric_Pad0.98x0.95mm_HandSolder, B.Cu at (180.8, 56.8)
- added R60: 1k, Resistor_SMD:R_0603_1608Metric_Pad0.98x0.95mm_HandSolder, B.Cu at (189.3, 63.2)
- added R61: 0R, Resistor_SMD:R_0603_1608Metric_Pad0.98x0.95mm_HandSolder, B.Cu at (181.0, 50.8)
- added R66: 1k, Resistor_SMD:R_1206_3216Metric_Pad1.30x1.75mm_HandSolder, B.Cu at (185.0, 49.0)
- added R67: 18R, Resistor_SMD:R_0603_1608Metric_Pad0.98x0.95mm_HandSolder, B.Cu at (193.0, 62.2)
- added R68: 160R, Resistor_SMD:R_0603_1608Metric_Pad0.98x0.95mm_HandSolder, B.Cu at (192.0, 59.5)
- added R69: 18R, Resistor_SMD:R_0603_1608Metric_Pad0.98x0.95mm_HandSolder, B.Cu at (199.0, 62.2)
- added R70: 160R, Resistor_SMD:R_0603_1608Metric_Pad0.98x0.95mm_HandSolder, B.Cu at (198.0, 59.5)
- added R72: 1k, Resistor_SMD:R_0603_1608Metric_Pad0.98x0.95mm_HandSolder, B.Cu at (195.5, 63.2)
- added R73: 6R8, Resistor_SMD:R_0603_1608Metric_Pad0.98x0.95mm_HandSolder, B.Cu at (193.0, 56.8)
- added R74: 1k, Resistor_SMD:R_0603_1608Metric_Pad0.98x0.95mm_HandSolder, B.Cu at (201.5, 63.2)
- added R75: 0R, Resistor_SMD:R_0603_1608Metric_Pad0.98x0.95mm_HandSolder, B.Cu at (193.0, 51.0)
- added R76: 0R, Resistor_SMD:R_0603_1608Metric_Pad0.98x0.95mm_HandSolder, B.Cu at (199.0, 51.0)
- added R8: R, Resistor_SMD:R_0603_1608Metric, B.Cu at (142.2, 42.3)
- added R9: R, Resistor_SMD:R_0603_1608Metric, B.Cu at (147.8, 42.3)
- added SW1: RESET, Button_Switch_THT:SW_Push_1P1T_NO_LED_E-Switch_TL1250, F.Cu at (115.1, 56.0)
- added SW2: BOOT, Button_Switch_THT:SW_Push_1P1T_NO_LED_E-Switch_TL1250, F.Cu at (115.0, 104.7)
- added U2: LTV-847S, Package_DIP:SMDIP-16_W9.53mm, B.Cu at (124.0, 117.5)
- added U3: LTV-847S, Package_DIP:SMDIP-16_W9.53mm, B.Cu at (146.5, 117.5)
- added U4: TPL7407LAPW, Package_SO:TSSOP-16_4.4x5mm_P0.65mm, F.Cu at (190.8, 96.8)
- added U5: ADS1115IDGS, Package_SO:TSSOP-10_3x3mm_P0.5mm, B.Cu at (167.5, 57.0)
- added U6: ADS1115IDGS, Package_SO:TSSOP-10_3x3mm_P0.5mm, B.Cu at (207.5, 54.0)
- C1, C2, C4: value 100n -> 1u; footprint Capacitor_SMD:C_0603_1608Metric -> Capacitor_SMD:C_0603_1608Metric_Pad1.08x0.95mm_HandSolder; moved to B.Cu
- C11: value 100pF -> 22u; footprint Capacitor_SMD:C_0402_1005Metric -> Capacitor_SMD:C_1206_3216Metric_Pad1.33x1.80mm_HandSolder; moved to B.Cu
- C15: value 0.1uF 50V -> 1u; footprint Capacitor_SMD:C_0603_1608Metric -> Capacitor_SMD:C_0805_2012Metric_Pad1.18x1.45mm_HandSolder
- C16: value 100nF 50V -> 1u; footprint Capacitor_SMD:C_0402_1005Metric -> Capacitor_SMD:C_0805_2012Metric_Pad1.18x1.45mm_HandSolder
- C18: value 22uF 16V -> 1u; footprint Capacitor_SMD:C_0805_2012Metric -> Capacitor_SMD:C_0805_2012Metric_Pad1.18x1.45mm_HandSolder
- C21: value 100nF 50V -> 22u; footprint Capacitor_SMD:C_0402_1005Metric -> Capacitor_SMD:C_1206_3216Metric_Pad1.33x1.80mm_HandSolder; moved to B.Cu
- C23: value 100nF 50V -> 1u; footprint Capacitor_SMD:C_0402_1005Metric -> Capacitor_SMD:C_0603_1608Metric_Pad1.08x0.95mm_HandSolder
- C24, C26, C30: value 0.1uF 50V -> 100n; footprint Capacitor_SMD:C_0603_1608Metric -> Capacitor_SMD:C_0603_1608Metric_Pad1.08x0.95mm_HandSolder; moved to B.Cu
- C25, C27, C32: value 0.1uF 50V -> 10n; footprint Capacitor_SMD:C_0603_1608Metric -> Capacitor_SMD:C_0603_1608Metric_Pad1.08x0.95mm_HandSolder; moved to B.Cu
- C28, C29, C35: value 0.1uF 50V -> 1u; footprint Capacitor_SMD:C_0603_1608Metric -> Capacitor_SMD:C_0603_1608Metric_Pad1.08x0.95mm_HandSolder; moved to B.Cu
- C3: footprint Capacitor_SMD:C_0603_1608Metric -> Capacitor_SMD:C_0603_1608Metric_Pad1.08x0.95mm_HandSolder; moved to B.Cu
- C37, D13, D7, IC3, Q1, Q2, R64: moved to B.Cu
- C39: value 100n -> 33n; footprint Capacitor_SMD:C_0603_1608Metric -> Capacitor_SMD:C_0603_1608Metric_Pad1.08x0.95mm_HandSolder; moved to B.Cu
- C44: value 0.1uF 50V -> 4n7; footprint Capacitor_SMD:C_0603_1608Metric -> Capacitor_SMD:C_0603_1608Metric_Pad1.08x0.95mm_HandSolder; moved to B.Cu
- C8: value 22uF 16V -> 22p; footprint Capacitor_SMD:C_0805_2012Metric -> Capacitor_SMD:C_0603_1608Metric_Pad1.08x0.95mm_HandSolder; moved to B.Cu
- C9: value 100nF 50V -> 1u; footprint Capacitor_SMD:C_0402_1005Metric -> Capacitor_SMD:C_0603_1608Metric_Pad1.08x0.95mm_HandSolder; moved to B.Cu
- D10: value 18V -> BAV199; footprint Diode_SMD:D_SOD-123 -> Package_TO_SOT_SMD:SOT-23-3; moved to B.Cu
- D11: value 18V -> BAT54; moved to B.Cu
- D12, D14, D8: value BAT54 -> BAV199; footprint Diode_SMD:D_SOD-123 -> Package_TO_SOT_SMD:SOT-23-3; moved to B.Cu
- F1: value Polyfuse -> 0ZRB0250FF1E; footprint Fuse:Fuse_1210_3225Metric -> Fuse:Fuse_BelFuse_0ZRE0033FF_L11.4mm_W3.8mm
- F2: value 0ZRB0250FF1E -> Mini blade 1A; footprint Fuse:Fuse_BelFuse_0ZRE0033FF_L11.4mm_W3.8mm -> Fuse:Fuseholder_Blade_Mini_Keystone_3568
- IC1: footprint DIY:SOIC127P600X175-16N -> Package_SO:SOIC-16_3.9x9.9mm_P1.27mm; moved to B.Cu
- L1: value 10uH -> 3u3; footprint Inductor_SMD:L_Bourns-SRN6028 -> Inductor_SMD:L_Taiyo-Yuden_NR-50xx_HandSoldering; moved to B.Cu
- R32, R36: value 10k -> 8k2; moved to B.Cu
- R33: value 8k2 -> 10k; footprint Resistor_SMD:R_0805_2012Metric_Pad1.20x1.40mm_HandSolder -> Resistor_SMD:R_0603_1608Metric_Pad0.98x0.95mm_HandSolder; moved to B.Cu
- R6: value 8k2 -> 4k7
- R62: value 150k -> 0R; footprint Resistor_SMD:R_0805_2012Metric_Pad1.20x1.40mm_HandSolder -> Resistor_SMD:R_0603_1608Metric_Pad0.98x0.95mm_HandSolder; moved to B.Cu
- R63: value 1K -> 1k; footprint Resistor_SMD:R_0805_2012Metric_Pad1.20x1.40mm_HandSolder -> Resistor_SMD:R_0603_1608Metric_Pad0.98x0.95mm_HandSolder; moved to B.Cu
- R65: footprint Resistor_SMD:R_0603_1608Metric_Pad0.98x0.95mm_HandSolder -> Resistor_SMD:R_1206_3216Metric_Pad1.30x1.75mm_HandSolder; moved to B.Cu
- R7: value 8k2 -> R; footprint Resistor_SMD:R_0805_2012Metric_Pad1.20x1.40mm_HandSolder -> Resistor_SMD:R_0603_1608Metric; moved to B.Cu
- R71: value 1k -> 6R8; moved to B.Cu
- R77: value 6R8 -> 1k; moved to B.Cu
- R78: value 30k -> 1k; footprint Resistor_SMD:R_0805_2012Metric_Pad1.20x1.40mm_HandSolder -> Resistor_SMD:R_0603_1608Metric_Pad0.98x0.95mm_HandSolder; moved to B.Cu
- R79: value 10k -> 1k; footprint Resistor_SMD:R_0603_1608Metric_Pad0.98x0.95mm_HandSolder -> Resistor_SMD:R_1206_3216Metric_Pad1.30x1.75mm_HandSolder; moved to B.Cu
- R80: value 10k -> 1k; footprint Resistor_SMD:R_0805_2012Metric_Pad1.20x1.40mm_HandSolder -> Resistor_SMD:R_1206_3216Metric_Pad1.30x1.75mm_HandSolder; moved to B.Cu
- R81: value 100K -> 0R; footprint Resistor_SMD:R_0603_1608Metric_Pad0.98x0.95mm_HandSolder -> Resistor_SMD:R_0805_2012Metric_Pad1.20x1.40mm_HandSolder; moved to B.Cu
- R82, R83: value 1k -> 120R; footprint Resistor_SMD:R_0603_1608Metric_Pad0.98x0.95mm_HandSolder -> Resistor_SMD:R_0603_1608Metric; moved to B.Cu
- R84: value 18R -> 120R; footprint Resistor_SMD:R_0603_1608Metric_Pad0.98x0.95mm_HandSolder -> Resistor_SMD:R_0603_1608Metric; moved to B.Cu
- R85: value 0R -> 120R; footprint Resistor_SMD:R_0603_1608Metric_Pad0.98x0.95mm_HandSolder -> Resistor_SMD:R_0603_1608Metric; moved to B.Cu
- U1: value ~ -> ESP32-S3-WROOM-1; footprint Package_DIP:SMDIP-4_W7.62mm -> RF_Module:ESP32-S3-WROOM-1; moved to B.Cu
- moved D13 232.4 mm to (200.0, 42.5), turned to -90 degrees
- moved D14 227.7 mm to (197.0, 53.8), turned to 90 degrees
- moved D12 220.5 mm to (191.0, 53.8), turned to 90 degrees
- moved R36 176.2 mm to (144.0, 126.2), turned to 90 degrees
- moved C37 167.1 mm to (204.8, 55.8), turned to -90 degrees
- moved R82 166.6 mm to (146.0, 96.8), turned to 90 degrees
- moved R83 165.3 mm to (144.5, 96.8), turned to 90 degrees
- moved R62 163.4 mm to (187.0, 51.0), turned to -90 degrees
- moved R84 162.3 mm to (146.0, 99.8), turned to 90 degrees
- moved R63 162.0 mm to (183.0, 50.8), turned to 90 degrees
- moved Q2 161.3 mm to (188.5, 59.5), turned to 90 degrees
- moved R85 160.7 mm to (144.5, 99.8), turned to 90 degrees
- moved R71 157.0 mm to (199.0, 56.8), turned to 180 degrees
- moved Q1 155.4 mm to (182.5, 59.5), turned to 90 degrees
- moved R64 151.5 mm to (189.0, 51.0), turned to 90 degrees
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Connections:
- C1 pad 1: /rpm -> GND
- C1 pad 2: GND -> 3V3
- C11 pad 1: /12V_to_5V_AP63200WU-7/5V_FB -> 3V3
- C11 pad 2: /12V_to_5V_AP63200WU-7/5V_REG_OUT -> GND
- C15 pad 1: GND -> /Input protection/Power_0V
- C15 pad 2: Net-(IC7-+IN_A) -> /Input protection/Power_Fused
- C16 pad 1: /12V_to_5V_AP63200WU-7/5V_REG_OUT -> /Input protection/Power_0V
- C16 pad 2: GND -> /Input protection/Power_Fused
- C18 pad 1: PROTECTED_12V+ -> GND
- C18 pad 2: GND -> /Protected_12V
- C2 pad 2: RPM_HALL -> 3V3
- C21 pad 1: Net-(IC4-BST) -> 5V_SENSOR
- C21 pad 2: Net-(IC4-SW) -> GND
- C23 pad 2: Net-(C19-Pad1) -> /Protected_12V
- C24 pad 1: fuel_level -> GND
- C24 pad 2: GND -> Net-(D3A-K)
- C25 pad 2: AnalogV_1 -> /Analogue/v_adc_1
- C26 pad 2: AnalogV_1 -> Net-(D4A-K)
- C27 pad 2: AnalogV_2 -> /Analogue/v_adc_2
- C28 pad 2: AnalogV_2 -> 5V_SENSOR
- C29 pad 2: AnalogV_3 -> 5V_SENSOR
- C3 pad 1: WATER_T_PWM -> GND
- C3 pad 2: GND -> /esp32_enable
- C30 pad 2: AnalogV_3 -> /Analogue/v_ref
- C32 pad 2: AnalogV_4 -> /Analogue/v_adc_3
- C35 pad 2: PROTECTED_12V+ -> 5V_SENSOR
- C37 pad 2: /ANALOGUE/r_adc_1 -> /Analogue/r_adc_2
- C39 pad 2: /POWER INPUT/Power_Fused -> /Analogue/r_adc_3
- C4 pad 1: /speed -> GND
- C4 pad 2: GND -> 3V3
- C44 pad 1: sensor_V_1 -> GND
- C44 pad 2: GND -> Net-(C44-Pad2)
- C8 pad 1: PROTECTED_12V+ -> 3V3
- C8 pad 2: GND -> Net-(IC2-FB)
- C9 pad 1: PROTECTED_12V+ -> GND
- C9 pad 2: GND -> 5V_SENSOR
- D10 pad 1: Net-(D10-K) -> GND
- D10 pad 2: GND -> 5V_SENSOR
- D11 pad 1: Net-(D11-K) -> /AnaR_3
- D12 pad 1: AnalogR_3 -> GND
- D12 pad 2: Net-(D12-A) -> 5V_SENSOR
- D13 pad 1: +3V3 -> /AnaR_4
- D13 pad 2: /ANALOGUE/r_adc_3 -> Net-(D13-A)
- D14 pad 1: AnalogR_4 -> GND
- D14 pad 2: Net-(D14-A) -> 5V_SENSOR
- D7 pad 1: +3V3 -> /AnaR_1
- D7 pad 2: /ANALOGUE/r_adc_1 -> Net-(D7-A)
- D8 pad 1: AnalogR_2 -> GND
- D8 pad 2: Net-(D8-A) -> 5V_SENSOR
- F1 pad 1: +5V_1 -> /Switched_12V
- F1 pad 2: 5V_SENSOR -> /Input protection/Power_Fused
- F2 pad 1: BATT12V+ -> /Low-side Outputs/Output1
- F2 pad 2: /POWER INPUT/Power_Fused -> Net-(U4-OUT1)
- IC1 pad 1: +3V3 -> 3V3
- IC1 pad 10: /water_T -> unconnected-(IC1-4Y-Pad10)
- IC1 pad 14: SPEED_HALL -> GND
- IC1 pad 15: /speed -> unconnected-(IC1-6Y-Pad15)
- IC1 pad 2: /rpm -> Net-(IC1-1Y)
- IC1 pad 3: RPM_HALL -> /PWM_cap_0
- IC1 pad 4: unconnected-(IC1-2Y-Pad4) -> Net-(IC1-2Y)
- IC1 pad 5: GND -> /PWM_cap_1
- IC1 pad 6: unconnected-(IC1-3Y-Pad6) -> Net-(IC1-3Y)
- IC1 pad 7: GND -> /PWM_cap_2
- IC1 pad 9: WATER_T_PWM -> GND
- IC3 pad 3: Protected_12V -> /Protected_12V
- L1 pad 1: /12V_to_5V_AP63200WU-7/5V_SW -> Net-(IC2-SW)
- L1 pad 2: /12V_to_5V_AP63200WU-7/5V_REG_OUT -> 3V3
- Q2 pad 3: Net-(D6-A) -> Net-(Q2-D)
- R32 pad 1: +3V3 -> /Opto 4xActiveHigh/HL_Input1
- R32 pad 2: /backlight -> Net-(R32-Pad2)
- R33 pad 1: R_TURN_ActLO -> 3V3
- R33 pad 2: Net-(R33-Pad2) -> /~{ActiHigh1}
- R36 pad 1: +3V3 -> /Opto 4xActiveHigh/HL_Input3
- R36 pad 2: /ignition -> Net-(R36-Pad2)
- R6 pad 1: Net-(IC3-FB) -> /SCL
- R6 pad 2: GND -> 3V3
- R62 pad 1: GND -> Net-(IC4B-+)
- R62 pad 2: Net-(R61-Pad2) -> Net-(Q2-D)
- R63 pad 1: Net-(R61-Pad2) -> Net-(IC4-Pad1)
- R63 pad 2: /ANALOGUE/v_adc_4 -> Net-(Q3-G)
- R64 pad 2: Net-(Q2-G) -> Net-(Q4-G)
- R65 pad 1: /ANALOGUE/R_RANGE_1 -> /AnaR_1
- R65 pad 2: Net-(Q1-G) -> /Analogue/r_adc_1
- R7 pad 1: PROTECTED_12V+ -> 5V_SENSOR
- R7 pad 2: Net-(R7-Pad2) -> Net-(J7-Pin_1)
- R78 pad 1: IGNITION_ActHI -> Net-(IC6-Pad7)
- R78 pad 2: Net-(D10-K) -> Net-(Q8-G)
- R79 pad 1: Net-(D10-K) -> /AnaR_3
- R79 pad 2: GND -> /Analogue/r_adc_3
- R80 pad 1: Net-(Q5-D) -> /AnaR_4
- R80 pad 2: Net-(D11-A) -> /Analogue/r_adc_4
- R81 pad 1: Net-(D11-K) -> Net-(IC7-VCC)
- R81 pad 2: Net-(D11-A) -> 5V_SENSOR
- R82 pad 1: Net-(IC7-Pad1) -> Net-(C44-Pad2)
- R82 pad 2: Net-(Q9-G) -> CAN_H
- R83 pad 1: /ANALOGUE/R_RANGE_3 -> Net-(C44-Pad2)
- R83 pad 2: Net-(Q8-G) -> CAN_H
- R84 pad 1: Net-(Q8-S) -> CAN_L
- R84 pad 2: +3V3 -> Net-(C44-Pad2)
- R85 pad 1: Net-(IC7A-+) -> CAN_L
- R85 pad 2: Net-(Q8-D) -> Net-(C44-Pad2)
- RV1 pad 1: GND -> /Input protection/Power_0V
- RV1 pad 2: /POWER INPUT/Power_Fused -> /Input protection/Power_Fused
- U1 pad 1: Net-(R7-Pad2) -> GND
- U1 pad 2: OIL_ALRM_ActLO -> Net-(U1-3V3)
- U1 pad 3: GND -> /esp32_enable
- U1 pad 4: /oil -> /SCL
Routing:
- net REG_3.3V+: track 388.2 -> 0.00 mm, vias 4 -> 0
- net PROTECTED_12V+: track 192.9 -> 0.00 mm, vias 9 -> 0
- net CONV_5V+: track 184.9 -> 0.00 mm, vias 5 -> 0
- net button: track 148.3 -> 0.00 mm, vias 1 -> 0
- net COM: track 134.9 -> 0.00 mm, vias 2 -> 0
- net right_turn: track 133.8 -> 0.00 mm, vias 3 -> 0
- net left_turn: track 131.8 -> 0.00 mm, vias 3 -> 0
- net S1: track 122.2 -> 0.00 mm, vias 2 -> 0
- net S3: track 120.4 -> 0.00 mm, vias 2 -> 0
- net S2: track 116.6 -> 0.00 mm, vias 2 -> 0
- net S0: track 104.7 -> 0.00 mm, vias 3 -> 0
- net rpm: track 65.8 -> 0.00 mm, vias 2 -> 0
- net water_T: track 65.6 -> 0.00 mm, vias 1 -> 0
- net speed: track 57.1 -> 0.00 mm, vias 2 -> 0
- net fuel_level: track 53.4 -> 0.00 mm, vias 1 -> 0
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- added copper zone on F.Cu, net /Low-side Outputs/Output1
- added copper zone on F.Cu, net /Low-side Outputs/Output2
- added copper zone on F.Cu, net /Low-side Outputs/Output3
- added copper zone on F.Cu, net /Low-side Outputs/Output4
- added copper zone on B.Cu, net /Protected_12V
- added copper zone on B.Cu, net 3V3
- added copper zone on B.Cu, net 5V_SENSOR
- added copper zone on B.Cu, net Net-(IC2-SW)
- added copper zone on B.Cu, net Net-(IC3-SW)
- added copper zone on F.Cu, net Net-(U4-OUT1)
- added copper zone on F.Cu, net Net-(U4-OUT3)
- added copper zone on F.Cu, net Net-(U4-OUT5)
- added copper zone on F.Cu, net Net-(U4-OUT7)
- removed copper zone on F.Cu, net /12V_to_5V_AP63200WU-7/5V_REG_OUT
- removed copper zone on F.Cu, net /12V_to_5V_AP63200WU-7/5V_SW
- removed copper zone on F.Cu, net /POWER INPUT/Power_Pre-Filter
- removed copper zone on F.Cu, net /right_turn
- removed copper zone on B.Cu, net GND
- removed copper zone on F.Cu, net GND
- removed copper zone on F.Cu, net Net-(C19-Pad1)
- removed copper zone on F.Cu, net Net-(D11-K)
- removed copper zone on F.Cu, net Net-(IC4-SW)
- removed copper zone on F.Cu, net PROTECTED_12V+
Other:
- board size 115 x 95 mm -> 110.5 x 108.5 mm
- copper layers 2 -> 4
- rule pad_to_mask_clearance: 0.02504 -> 0
- board text removed: "+5V"
- board text removed: "0,1524 mm / 0,0000 mm"
- board text removed: "0,3000 mm"
- board text removed: "1,6000 mm"
- board text removed: "105,0000 mm x 95,0000 mm"
- board text removed: "2"
- board text removed: "BOARD CHARACTERISTICS"
- board text removed: "Board Thickness:"
- board text removed: "Board overall dimensions:"
- board text removed: "Castellated pads:"
- board text removed: "Copper Finish:"
- board text removed: "Copper Layer Count:"
- board text removed: "Edge card connectors:"
- board text removed: "GND"
- board text removed: "Impedance Control:"
- board text removed: "Min hole diameter:"
- board text removed: "Min track/spacing:"
- board text removed: "No"
- board text removed: "None"
- board text removed: "Plated Board Edge:"
- board text removed: "RX"
- board text removed: "TX"
